File: hardware/uart.sch (KiCad schematic (older format))
At the start: 13 parts

Commit message: update,
Parts:
- gave numbers to parts that had none: 9
Changed lines of the file:
@@
 EESchema Schematic File Version 4
 LIBS:eval_board-cache
-LIBS:bb-ch340t-cache
 EELAYER 29 0
 EELAYER END
 $Descr A4 11693 8268
 encoding utf-8
-Sheet 6 20
+Sheet 6 22
 Title ""
 Date ""
@@
 	8450 3950 8600 3950
 $Comp
-L taobao-components:CH340H_T U?
+L taobao-components:CH340H_T U3
 U 1 1 5CE56F9B
 P 5750 4300
-F 0 "U?" H 5750 5300 60  0000 C CNN
+F 0 "U3" H 5750 5300 60  0000 C CNN
 F 1 "CH340H_T" H 5750 5150 60  0000 C CNN
 F 2 "Package_SO:SSOP-20_5.3x7.2mm_P0.65mm" H 5750 5050 60  0000 C CNN
@@
 $EndComp
 $Comp
-L taobao-osc:O_12M,3225 Y?
+L taobao-osc:O_12M,3225 Y2
 U 1 1 5CE59F8A
 P 4550 5300
-F 0 "Y?" H 4550 5550 50  0000 C CNN
+F 0 "Y2" H 4550 5550 50  0000 C CNN
 F 1 "O_12M,3225" H 4550 5450 50  0000 C CNN
 F 2 "footprint-lib:OSC_3225" H 4550 5300 50  0001 C CNN
@@
 	4650 5750 4900 5750
 $Comp
-L taobao-osc:O_12M Y?
+L taobao-osc:O_12M Y1
 U 1 1 5CE5F79C
 P 4550 4850
-F 0 "Y?" H 4550 4650 50  0000 C CNN
+F 0 "Y1" H 4550 4650 50  0000 C CNN
 F 1 "O_12M/OPTIONAL" H 4550 4750 50  0000 C CNN
 F 2 "Crystal:Crystal_HC49-4H_Vertical" H 4550 4850 50  0001 C CNN
@@
 	4900 4850 5100 4850
 $Comp
-L taobao-c:C225,0603 C?
+L taobao-c:C225,0603 C1
 U 1 1 5CE7979B
 P 3800 4000
-F 0 "C?" H 3900 4050 50  0000 L CNN
+F 0 "C1" H 3900 4050 50  0000 L CNN
 F 1 "C225,0603" H 3900 4000 50  0000 L CNN
 F 2 "Capacitor_SMD:C_0603_1608Metric_Pad1.05x0.95mm_HandSolder" H 3800 4000 50  0001 C CNN
@@
 	3800 4100 3800 4150
 $Comp
-L taobao-c:C225,0603 C?
+L taobao-c:C225,0603 C2
 U 1 1 5CE7CBB6
 P 4250 4000
-F 0 "C?" H 4350 4050 50  0000 L CNN
+F 0 "C2" H 4350 4050 50  0000 L CNN
 F 1 "C225,0603" H 4350 4000 50  0000 L CNN
 F 2 "Capacitor_SMD:C_0603_1608Metric_Pad1.05x0.95mm_HandSolder" H 4250 4000 50  0001 C CNN
@@
 	3800 3750 4250 3750
 $Comp
-L taobao-c:C103,0603 C?
+L taobao-c:C103,0603 C3
 U 1 1 5CE8154D
 P 4900 4000
-F 0 "C?" H 5000 4050 50  0000 L CNN
+F 0 "C3" H 5000 4050 50  0000 L CNN
 F 1 "C103,0603" H 5000 4000 50  0000 L CNN
 F 2 "Capacitor_SMD:C_0603_1608Metric_Pad1.05x0.95mm_HandSolder" H 4900 4000 50  0001 C CNN
@@
 	4900 4150 5100 4150
 $Comp
-L taobao-c:C22pf,0603 C?
+L taobao-c:C22pf,0603 C4
 U 1 1 5CE8611F
 P 4150 5550
-F 0 "C?" H 4250 5600 50  0000 L CNN
+F 0 "C4" H 4250 5600 50  0000 L CNN
 F 1 "C22pf,0603" H 4250 5550 50  0000 L CNN
 F 2 "Capacitor_SMD:C_0603_1608Metric_Pad1.05x0.95mm_HandSolder" H 4150 5550 50  0001 C CNN
@@
 $EndComp
 $Comp
-L taobao-c:C22pf,0603 C?
+L taobao-c:C22pf,0603 C5
 U 1 1 5CE863C8
 P 4900 5550
-F 0 "C?" H 5000 5600 50  0000 L CNN
+F 0 "C5" H 5000 5600 50  0000 L CNN
 F 1 "C22pf,0603" H 5000 5550 50  0000 L CNN
 F 2 "Capacitor_SMD:C_0603_1608Metric_Pad1.05x0.95mm_HandSolder" H 4900 5550 50  0001 C CNN
@@
 	4900 5650 4900 5750
 $Comp
-L taobao-r:R103,0603 R?
+L taobao-r:R103,0603 R1
 U 1 1 5CE8F8C3
 P 6800 3650
-F 0 "R?" V 6550 3650 50  0000 C CNN
+F 0 "R1" V 6550 3650 50  0000 C CNN
 F 1 "R103,0603" V 6650 3650 50  0000 C CNN
 F 2 "Resistor_SMD:R_0603_1608Metric_Pad1.05x0.95mm_HandSolder" H 6800 3650 50  0001 C CNN
