File: hardware/CH340T.sch (KiCad schematic (older format))
At the start: 13 parts, among them U3 CH340H_T, Y1 O_12M/OPTIONAL, Y2 O_12M,3225

Commit message: update fixing library,
Parts:
- removed USB?: USB-MINI-B, kicad_wrk:USB_Mini-B, symbol bb-ch340t-rescue:USB-MINI-B
- added J?: USB_B_Mini_1, footprint-lib:USB_Micro-B_Molex-105017-0001, symbol taobao-components:USB_B_Mini_1
- D?: symbol bb-ch340t-rescue:D_Schottky_Small -> taobao-sd:SD_1N5822_SS34
Connections:
- net labels added: USBD+, USBD-
- wire segments 67 -> 61
Changed lines of the file:
@@
 L power:GND #PWR?
 U 1 1 55069BDF
-P 3450 4700
-F 0 "#PWR?" H 3450 4450 60  0001 C CNN
-F 1 "GND" H 3450 4550 60  0000 C CNN
-F 2 "" H 3450 4700 60  0000 C CNN
-F 3 "" H 3450 4700 60  0000 C CNN
-	1    3450 4700
+P 2450 4900
+F 0 "#PWR?" H 2450 4650 60  0001 C CNN
+F 1 "GND" H 2450 4750 60  0000 C CNN
+F 2 "" H 2450 4900 60  0000 C CNN
+F 3 "" H 2450 4900 60  0000 C CNN
+	1    2450 4900
 	1    0    0    -1
 $EndComp
 Wire Wire Line
 	5100 3750 4250 3750
-Wire Wire Line
-	3350 4250 3550 4250
 Connection ~ 3550 3750
 Wire Wire Line
@@
 P 4550 5800
 F 0 "#PWR?" H 4550 5550 60  0001 C CNN
-F 1 "GND" H 4550 5650 60  0000 C CNN
+F 1 "GND" H 4600 5600 60  0000 C CNN
 F 2 "" H 4550 5800 60  0000 C CNN
 F 3 "" H 4550 5800 60  0000 C CNN
@@
 Wire Wire Line
 	3550 3150 7400 3150
-Wire Wire Line
-	3550 4250 3550 3750
-$Comp
-L bb-ch340t-rescue:USB-MINI-B USB?
-U 1 1 5506AA9A
-P 2850 4450
-F 0 "USB?" H 2550 4800 50  0000 C CNN
-F 1 "USB-MINI-B" H 2700 4100 50  0000 C CNN
-F 2 "kicad_wrk:USB_Mini-B" H 2850 4350 50  0001 C CNN
-F 3 "" H 2850 4350 50  0000 C CNN
-	1    2850 4450
-	-1   0    0    -1
-$EndComp
-Wire Wire Line
-	3350 4650 3450 4650
-Wire Wire Line
-	3450 4650 3450 4700
-Wire Wire Line
-	2350 4250 2200 4250
 $Comp
 L power:GND #PWR?
 U 1 1 5506ADD0
-P 2200 4700
-F 0 "#PWR?" H 2200 4450 60  0001 C CNN
-F 1 "GND" H 2200 4550 60  0000 C CNN
-F 2 "" H 2200 4700 60  0000 C CNN
-F 3 "" H 2200 4700 60  0000 C CNN
-	1    2200 4700
-	1    0    0    -1
-$EndComp
-Wire Wire Line
-	2200 4250 2200 4350
-Wire Wire Line
-	2350 4650 2200 4650
-Connection ~ 2200 4650
-Wire Wire Line
-	2350 4550 2200 4550
-Connection ~ 2200 4550
-Wire Wire Line
-	2350 4350 2200 4350
-Connection ~ 2200 4350
+P 2350 4900
+F 0 "#PWR?" H 2350 4650 60  0001 C CNN
+F 1 "GND" H 2350 4750 60  0000 C CNN
+F 2 "" H 2350 4900 60  0000 C CNN
+F 3 "" H 2350 4900 60  0000 C CNN
+	1    2350 4900
+	1    0    0    -1
+$EndComp
 $Comp
 L power:GND #PWR?
@@
 	7400 3350 7200 3350
 $Comp
-L bb-ch340t-rescue:D_Schottky_Small D?
+L taobao-sd:SD_1N5822_SS34 D?
 U 1 1 55937694
 P 6500 3750
@@
 Wire Wire Line
 	4550 5750 4650 5750
-Wire Wire Line
-	2200 4650 2200 4700
-Wire Wire Line
-	2200 4550 2200 4650
-Wire Wire Line
-	2200 4350 2200 4550
 Wire Wire Line
 	6950 3650 7250 3650
@@
 U 1 1 5CE56F9B
 P 5750 4300
-F 0 "U3" H 5750 5300 60  0000 C CNN
-F 1 "CH340H_T" H 5750 5150 60  0000 C CNN
-F 2 "Package_SO:SSOP-20_5.3x7.2mm_P0.65mm" H 5750 5050 60  0000 C CNN
+F 0 "U3" H 5750 5150 60  0000 C CNN
+F 1 "CH340H_T" H 5750 5050 60  0000 C CNN
+F 2 "Package_SO:SSOP-20_5.3x7.2mm_P0.65mm" H 5750 5050 60  0001 C CNN
 F 3 "" H 5750 4300 60  0000 C CNN
 	1    5750 4300
@@
 U 1 1 5CE8611F
 P 4150 5550
-F 0 "C4" H 4250 5600 50  0000 L CNN
-F 1 "C22pf,0603" H 4250 5550 50  0000 L CNN
+F 0 "C4" H 4050 5600 50  0000 R CNN
+F 1 "C22pf,0603" H 4050 5550 50  0000 R CNN
 F 2 "Capacitor_SMD:C_0603_1608Metric_Pad1.05x0.95mm_HandSolder" H 4150 5550 50  0001 C CNN
 F 3 "~" H 4150 5550 50  0001 C CNN
@@
 U 1 1 5507CA9B
 P 6950 3350
-F 0 "3.3/5V?" H 6800 3500 50  0000 L CNN
-F 1 "closed / opened" H 6950 3200 50  0000 C BNN
+F 0 "3.3/5V?" H 6950 3550 50  0000 C CNN
+F 1 "closed / opened" H 6950 3450 50  0000 C CNN
 F 2 "kicad_wrk:JUMP3" H 6950 3350 60  0001 C CNN
 F 3 "" H 6950 3350 60  0000 C CNN
@@
 	1    0    0    -1
 $EndComp
+$Comp
+L taobao-components:USB_B_Mini_1 J?
+U 1 1 5CEA5B6D
+P 2450 4350
+F 0 "J?" H 2550 4850 50  0000 C CNN
+F 1 "USB_B_Mini_1" H 2550 4750 50  0000 C CNN
+F 2 "footprint-lib:USB_Micro-B_Molex-105017-0001" H 2450 3350 50  0001 C CNN
+F 3 "~" H 2600 4300 50  0001 C CNN
+	1    2450 4350
+	1    0    0    -1
+$EndComp
+Wire Wire Line
+	2350 4750 2350 4900
+Wire Wire Line
+	2450 4750 2450 4900
+Wire Wire Line
+	2750 4150 3550 4150
+Wire Wire Line
+	3550 3750 3550 4150
+Text Label 3000 4350 2    50   ~ 0
+USBD+
+Wire Wire Line
+	3000 4350 2750 4350
+Text Label 3350 4450 0    50   ~ 0
+USBD+
+Text Label 3000 4450 2    50   ~ 0
+USBD-
+Wire Wire Line
+	3000 4450 2750 4450
+Text Label 3350 4350 0    50   ~ 0
+USBD-
 $EndSCHEMATC

Commit message: update,
Parts:
- gave numbers to parts that had none: 4
Changed lines of the file:
@@
 	3350 4450 5100 4450
 $Comp
-L power:GND #PWR?
+L power:GND #PWR0209
 U 1 1 55069BDF
 P 2450 4900
-F 0 "#PWR?" H 2450 4650 60  0001 C CNN
+F 0 "#PWR0209" H 2450 4650 60  0001 C CNN
 F 1 "GND" H 2450 4750 60  0000 C CNN
 F 2 "" H 2450 4900 60  0000 C CNN
@@
 Connection ~ 4550 5750
 $Comp
-L power:GND #PWR?
+L power:GND #PWR0210
 U 1 1 55069F3B
 P 4550 5800
-F 0 "#PWR?" H 4550 5550 60  0001 C CNN
+F 0 "#PWR0210" H 4550 5550 60  0001 C CNN
 F 1 "GND" H 4600 5600 60  0000 C CNN
 F 2 "" H 4550 5800 60  0000 C CNN
@@
 	7100 3950 7250 3950
 $Comp
-L power:GND #PWR?
+L power:GND #PWR0211
 U 1 1 5506A094
 P 7100 4050
-F 0 "#PWR?" H 7100 3800 60  0001 C CNN
+F 0 "#PWR0211" H 7100 3800 60  0001 C CNN
 F 1 "GND" H 7100 3900 60  0000 C CNN
 F 2 "" H 7100 4050 60  0000 C CNN
@@
 	3550 3150 7400 3150
 $Comp
-L power:GND #PWR?
+L power:GND #PWR0212
 U 1 1 5506ADD0
 P 2350 4900
-F 0 "#PWR?" H 2350 4650 60  0001 C CNN
+F 0 "#PWR0212" H 2350 4650 60  0001 C CNN
 F 1 "GND" H 2350 4750 60  0000 C CNN
 F 2 "" H 2350 4900 60  0000 C CNN
@@
 $EndComp
 $Comp
-L power:GND #PWR?
+L power:GND #PWR0213
 U 1 1 5506B73B
 P 4100 4150
-F 0 "#PWR?" H 4100 3900 60  0001 C CNN
+F 0 "#PWR0213" H 4100 3900 60  0001 C CNN
 F 1 "GND" H 4100 4000 60  0000 C CNN
 F 2 "" H 4100 4150 60  0000 C CNN
@@
 	7400 3350 7200 3350
 $Comp
-L taobao-sd:SD_1N5822_SS34 D?
+L taobao-sd:SD_1N5822_SS34 D6
 U 1 1 55937694
 P 6500 3750
-F 0 "D?" H 6450 3830 50  0000 L CNN
+F 0 "D6" H 6450 3830 50  0000 L CNN
 F 1 "1N5819/S4" H 6450 3450 50  0000 L CNN
 F 2 "" V 6500 3750 60  0000 C CNN
@@
 	3800 4150 4250 4150
 $Comp
-L taobao-components:TTL_TERMINAL J?
+L taobao-components:TTL_TERMINAL J18
 U 1 1 5CE9678A
 P 8500 3850
-F 0 "J?" H 8450 3750 50  0000 R CNN
+F 0 "J18" H 8450 3750 50  0000 R CNN
 F 1 "TTL_TERMINAL" H 8450 3850 50  0000 R CNN
 F 2 "footprint-lib:TTL_TERMINAL_2.54mm" H 8550 3600 50  0001 C CNN
@@
 $EndComp
 $Comp
-L Jumper:Jumper_3_Bridged12 3.3/5V?
+L Jumper:Jumper_3_Bridged12 3.3/5V1
 U 1 1 5507CA9B
 P 6950 3350
-F 0 "3.3/5V?" H 6950 3550 50  0000 C CNN
+F 0 "3.3/5V1" H 6950 3550 50  0000 C CNN
 F 1 "closed / opened" H 6950 3450 50  0000 C CNN
 F 2 "kicad_wrk:JUMP3" H 6950 3350 60  0001 C CNN
@@
 $EndComp
 $Comp
-L taobao-components:USB_B_Mini_1 J?
+L taobao-components:USB_B_Mini_1 J19
 U 1 1 5CEA5B6D
 P 2450 4350
-F 0 "J?" H 2550 4850 50  0000 C CNN
+F 0 "J19" H 2550 4850 50  0000 C CNN
 F 1 "USB_B_Mini_1" H 2550 4750 50  0000 C CNN
 F 2 "footprint-lib:USB_Micro-B_Molex-105017-0001" H 2450 3350 50  0001 C CNN
