File: hardware/CH340T.sch (KiCad schematic (older format))
At the start: 13 parts, among them J18 TTL_TERMINAL, J19 USB_B_Mini_1, U3 CH340H_T, Y1 O_12M/OPTIONAL, Y2 O_12M,3225

Commit message: update,
Parts:
- J18: symbol taobao-components:TTL_TERMINAL -> taobao-board:TTL_TERMINAL
- J19: symbol taobao-components:USB_B_Mini_1 -> taobao-connector:USB_B_Mini_1
Connections:
- net GND: now also J18.1 (GND); no longer J18.GND
- net RXD: now also J18.3 (RXD); no longer J18.RX
- net TXD: now also J18.2 (TXD); no longer J18.TX
Changed lines of the file:
@@
 $Descr A4 11693 8268
 encoding utf-8
-Sheet 5 27
+Sheet 10 27
 Title ""
 Date ""
@@
 	3800 4150 4250 4150
 $Comp
-L taobao-components:TTL_TERMINAL J18
+L taobao-board:TTL_TERMINAL J18
 U 1 1 5CE9678A
 P 8500 3850
-F 0 "J18" H 8450 3750 50  0000 R CNN
-F 1 "TTL_TERMINAL" H 8450 3850 50  0000 R CNN
+F 0 "J18" H 8550 3450 50  0000 C CNN
+F 1 "TTL_TERMINAL" H 8550 3550 50  0000 C CNN
 F 2 "footprint-lib:TTL_TERMINAL_2.54mm" H 8550 3600 50  0001 C CNN
 F 3 "~" H 8500 3850 50  0001 C CNN
 	1    8500 3850
-	1    0    0    1
+	-1   0    0    1
 $EndComp
 $Comp
@@
 $EndComp
 $Comp
-L taobao-components:USB_B_Mini_1 J19
+L taobao-connector:USB_B_Mini_1 J19
 U 1 1 5CEA5B6D
 P 2450 4350

Commit message: update,
Connections:
- net GND: now also C1.2, C2.2, C3.2, U3.8 (GND)
- net VDD: now also 3.3/5V1.2 (C)
Other:
- moved on the sheet: 3.3/5V1, C1, C2, C3, C4, C5, D6, J18, J19, R1, U3, Y1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
