File: hardware/i2c.sch (KiCad schematic (older format))
At the start: 0 parts

Commit message: update,
Other:
- note added: "LM75"

Commit message: update,
Parts:
- added JP? (x3): SolderJumper_3_Open, symbol Jumper:SolderJumper_3_Open
- added RN?: R_Pack04, symbol Device:R_Pack04
- added U?: LM75, Package_SO:SOP-8_3.76x4.96mm_P1.27mm, symbol taobao-components:LM75
Connections:
- new net: RN?.2 (R2.1), U?.3 (OS)
- new net: JP?.2 (C), U?.5 (A2)
- new net: JP?.2 (C), U?.6 (A1)
- new net: JP?.2 (C), U?.7 (A0)
- new net +3V3: JP?.1 (A), JP?.1 (A), JP?.1 (A), RN?.5 (R4.2), RN?.6 (R3.2), RN?.7 (R2.2), RN?.8 (R1.2), U?.8 (VCC)
- new net GND: JP?.3 (B), JP?.3 (B), JP?.3 (B), U?.4 (GND)
- new net LM75_SCL: RN?.3 (R3.1), U?.2 (SCL)
- new net LM75_SDA: RN?.4 (R4.1), U?.1 (SDA)

Commit message: update,
Parts:
- gave numbers to parts that had none: 5
Changed lines of the file:
@@
 $EndBitmap
 $Comp
-L taobao-components:LM75 U?
+L taobao-components:LM75 U8
 U 1 1 5CF9DF41
 P 4800 5100
-F 0 "U?" H 4800 5550 50  0000 C CNN
+F 0 "U8" H 4800 5550 50  0000 C CNN
 F 1 "LM75" H 4800 5450 50  0000 C CNN
 F 2 "Package_SO:SOP-8_3.76x4.96mm_P1.27mm" H 4800 5100 50  0001 C CNN
@@
 $EndComp
 $Comp
-L Device:R_Pack04 RN?
+L Device:R_Pack04 RN3
 U 1 1 5CF9E2EF
 P 3800 4650
-F 0 "RN?" H 4000 4700 50  0000 L CNN
+F 0 "RN3" H 4000 4700 50  0000 L CNN
 F 1 "R_Pack04" H 4000 4650 50  0000 L CNN
 F 2 "" V 4075 4650 50  0001 C CNN
@@
 $EndBitmap
 $Comp
-L power:+3V3 #PWR?
+L power:+3V3 #PWR0214
 U 1 1 5CFA024B
 P 5350 4800
-F 0 "#PWR?" H 5350 4650 50  0001 C CNN
+F 0 "#PWR0214" H 5350 4650 50  0001 C CNN
 F 1 "+3V3" H 5400 5000 50  0000 C CNN
 F 2 "" H 5350 4800 50  0001 C CNN
@@
 $EndComp
 $Comp
-L power:GND #PWR?
+L power:GND #PWR0215
 U 1 1 5CFA0A82
 P 4250 5500
-F 0 "#PWR?" H 4250 5250 50  0001 C CNN
+F 0 "#PWR0215" H 4250 5250 50  0001 C CNN
 F 1 "GND" H 4300 5300 50  0000 C CNN
 F 2 "" H 4250 5500 50  0001 C CNN
@@
 	5350 4950 5200 4950
 $Comp
-L power:GND #PWR?
+L power:GND #PWR0216
 U 1 1 5CFA112C
 P 6000 5650
-F 0 "#PWR?" H 6000 5400 50  0001 C CNN
+F 0 "#PWR0216" H 6000 5400 50  0001 C CNN
 F 1 "GND" H 6050 5450 50  0000 C CNN
 F 2 "" H 6000 5650 50  0001 C CNN
@@
 $EndComp
 $Comp
-L power:+3V3 #PWR?
+L power:+3V3 #PWR0217
 U 1 1 5CFA13EE
 P 6000 4700
-F 0 "#PWR?" H 6000 4550 50  0001 C CNN
+F 0 "#PWR0217" H 6000 4550 50  0001 C CNN
 F 1 "+3V3" H 6050 4900 50  0000 C CNN
 F 2 "" H 6000 4700 50  0001 C CNN
@@
 $EndComp
 $Comp
-L Jumper:SolderJumper_3_Open JP?
+L Jumper:SolderJumper_3_Open JP4
 U 1 1 5CFA2233
 P 6300 5050
-F 0 "JP?" V 6250 5150 50  0000 L CNN
+F 0 "JP4" V 6250 5150 50  0000 L CNN
 F 1 "SolderJumper_3_Open" V 6300 5150 50  0000 L CNN
 F 2 "" H 6300 5050 50  0001 C CNN
@@
 $EndComp
 $Comp
-L Jumper:SolderJumper_3_Open JP?
+L Jumper:SolderJumper_3_Open JP5
 U 1 1 5CFA349A
 P 6000 5150
-F 0 "JP?" V 5950 5250 50  0000 L CNN
+F 0 "JP5" V 5950 5250 50  0000 L CNN
 F 1 "SolderJumper_3_Open" V 6000 5250 50  0000 L CNN
 F 2 "" H 6000 5150 50  0001 C CNN
@@
 	6000 4800 6000 4950
 $Comp
-L Jumper:SolderJumper_3_Open JP?
+L Jumper:SolderJumper_3_Open JP6
 U 1 1 5CFA3939
 P 5800 5250
-F 0 "JP?" V 5750 5350 50  0000 L CNN
+F 0 "JP6" V 5750 5350 50  0000 L CNN
 F 1 "SolderJumper_3_Open" V 5800 5350 50  0000 L CNN
 F 2 "" H 5800 5250 50  0001 C CNN
@@
 	6000 5550 6000 5600
 $Comp
-L power:+3V3 #PWR?
+L power:+3V3 #PWR0218
 U 1 1 5CFA5F7E
 P 3650 4300
-F 0 "#PWR?" H 3650 4150 50  0001 C CNN
+F 0 "#PWR0218" H 3650 4150 50  0001 C CNN
 F 1 "+3V3" H 3700 4500 50  0000 C CNN
 F 2 "" H 3650 4300 50  0001 C CNN
