File: hardware/i2c.sch (KiCad schematic (older format))
At the start: 5 parts, among them U8 LM75

Commit message: update,
Other:
- note removed: "LM75"
Changed lines of the file:
@@
 EndData
 $EndBitmap
-Text Notes 650  950  0    50   ~ 0
-LM75
 $Bitmap
 Pos -1150 4300

Commit message: update,
Parts:
- renumbered JP4 to JP1, JP5 to JP2, JP6 to JP3, U8 to U3
Connections:
- net LM75_SCL renamed SCL
- net LM75_SDA renamed SDA
Other:
- moved on the sheet: JP1, JP2, JP3, RN3, U3
