File: hardware/oled.sch (KiCad schematic (older format))
At the start: 0 parts

Commit message: update,
Parts:
- added J?: SSD1306-OLED-SPI, footprint-lib:CONN_SPI_SSD1306, symbol taobao-components:SSD1306-OLED-SPI
- added U?: SSD1306-OLED-I2C, footprint-lib:CONN_I2C_SSD1306, symbol taobao-components:SSD1306-OLED-I2C

Commit message: update,
Parts:
- gave numbers to parts that had none: 2
Changed lines of the file:
@@
 EESchema Schematic File Version 4
 LIBS:eval_board-cache
-LIBS:bb-ch340t-cache
 EELAYER 29 0
 EELAYER END
 $Descr A4 11693 8268
 encoding utf-8
-Sheet 5 20
+Sheet 5 22
 Title ""
 Date ""
@@
 Data
 89 50 4E 47 0D 0A 1A 0A 00 00 00 0D 49 48 44 52 00 00 01 94 00 00 02 10 08 02 00 00 00 29 6E 0F
-A4 00 00 00 03 73 42 49 54 08 08 08 DB E1 4F E0 00 00 00 09 70 48 59 73 00 00 0F 61 00 00 0F 61
-01 A8 3F A7 69 00 00 20 00 49 44 41 54 78 9C EC BD 77 BC 24 55 99 FF FF 3E A1 AA 3A DC 30 39 91
+A4 00 00 00 03 73 42 49 54 08 08 08 DB E1 4F E0 00 00 00 09 70 48 59 73 00 00 0F 3C 00 00 0F 3C
+01 17 3A 9F 59 00 00 20 00 49 44 41 54 78 9C EC BD 77 BC 24 55 99 FF FF 3E A1 AA 3A DC 30 39 91
 67 90 CC 90 41 18 11 50 09 66 91 AF AE CB EA AE AE BB 8A 6E D2 FD B9 D1 5D 75 F7 B7 BA EA 8A 62
 76 15 D1 AF 19 D1 55 44 C2 80 20 48 06 19 82 64 06 86 61 18 26 CF 4D 1D 2A 9C F0 FB A3 AA BA FB
@@
 $EndBitmap
 $Comp
-L taobao-components:SSD1306-OLED-SPI J?
+L taobao-components:SSD1306-OLED-SPI J1
 U 1 1 5CE3BBF1
 P 3550 2900
-F 0 "J?" V 3550 2500 50  0000 R CNN
+F 0 "J1" V 3550 2500 50  0000 R CNN
 F 1 "SSD1306-OLED-SPI" V 3450 2500 50  0000 R CNN
 F 2 "footprint-lib:CONN_SPI_SSD1306" H 3550 2900 50  0001 C CNN
@@
 $EndComp
 $Comp
-L taobao-components:SSD1306-OLED-I2C U?
+L taobao-components:SSD1306-OLED-I2C U2
 U 1 1 5CE41586
 P 3300 5400
-F 0 "U?" H 3650 5700 50  0000 L CNN
+F 0 "U2" H 3650 5700 50  0000 L CNN
 F 1 "SSD1306-OLED-I2C" H 3650 5600 50  0000 L CNN
 F 2 "footprint-lib:CONN_I2C_SSD1306" H 3300 4800 50  0001 C CNN

Commit message: update,
Connections:
- net +5V: now reaches J1.5V
- net +5V: now also U2.1 (VCC)
- net OLED_SPI_CS: now reaches J1.CS
- net OLED_SPI_DC: now reaches J1.DC
- net GND: now reaches J1.GND
- net GND: now also U2.2 (GND)
- net OLED_SPI_RST: now reaches J1.RST
- net OLED_SPI_SCK: now reaches J1.SCK
- net OLED_SPI_SDA: now reaches J1.SDA
- net OLED_SPI_SDA: now also U2.4 (SDA)
- net OLED_I2C_SCL: now reaches U2.3 (SCL)
Other:
- moved on the sheet: J1, U2

Commit message: update,
Parts:
- added RN? (x2): R_Pack04, Resistor_SMD:R_Array_Concave_4x0603, symbol Device:R_Pack04
Connections:
- net OLED_I2C_SCL: now also RN?.2 (R2.1)
- net OLED_SPI_CS: now also RN?.1 (R1.1)
- net OLED_SPI_DC: now also RN?.3 (R3.1)
- net OLED_SPI_SCK: now also RN?.2 (R2.1)
- net OLED_SPI_SDA: now also RN?.1 (R1.1), RN?.4 (R4.1)
- net +5V renamed +3V3
- net +3V3: now also RN?.5 (R4.2), RN?.5 (R4.2), RN?.6 (R3.2), RN?.6 (R3.2), RN?.7 (R2.2), RN?.7 (R2.2), RN?.8 (R1.2), RN?.8 (R1.2)
Other:
- moved on the sheet: J1, U2
Changed lines of the file:
@@
 L taobao-components:SSD1306-OLED-SPI J1
 U 1 1 5CE3BBF1
-P 4850 2500
-F 0 "J1" V 4850 2100 50  0000 R CNN
-F 1 "SSD1306-OLED-SPI" V 4750 2100 50  0000 R CNN
-F 2 "footprint-lib:CONN_SPI_SSD1306" H 4850 2500 50  0001 C CNN
-F 3 "~" H 4850 2500 50  0001 C CNN
-	1    4850 2500
+P 5650 2500
+F 0 "J1" V 5650 2100 50  0000 R CNN
+F 1 "SSD1306-OLED-SPI" V 5550 2100 50  0000 R CNN
+F 2 "footprint-lib:CONN_SPI_SSD1306" H 5650 2500 50  0001 C CNN
+F 3 "~" H 5650 2500 50  0001 C CNN
+	1    5650 2500
 	1    0    0    -1
 $EndComp
@@
 L taobao-components:SSD1306-OLED-I2C U2
 U 1 1 5CE41586
-P 4800 5200
-F 0 "U2" H 5150 5500 50  0000 L CNN
-F 1 "SSD1306-OLED-I2C" H 5150 5400 50  0000 L CNN
-F 2 "footprint-lib:CONN_I2C_SSD1306" H 4800 4600 50  0001 C CNN
-F 3 "" H 4800 4600 50  0001 C CNN
-	1    4800 5200
+P 6050 5200
+F 0 "U2" H 6400 5500 50  0000 L CNN
+F 1 "SSD1306-OLED-I2C" H 6400 5400 50  0000 L CNN
+F 2 "footprint-lib:CONN_I2C_SSD1306" H 6050 4600 50  0001 C CNN
+F 3 "" H 6050 4600 50  0001 C CNN
+	1    6050 5200
 	0    1    1    0
 $EndComp
@@
 $EndComp
 Wire Wire Line
-	4650 2200 3800 2200
+	5450 2200 3800 2200
 Wire Wire Line
 	3800 2200 3800 2350
-$Comp
-L power:+5V #PWR?
-U 1 1 5CF7A062
-P 4500 2000
-F 0 "#PWR?" H 4500 1850 50  0001 C CNN
-F 1 "+5V" H 4550 2200 50  0000 C CNN
-F 2 "" H 4500 2000 50  0001 C CNN
-F 3 "" H 4500 2000 50  0001 C CNN
-	1    4500 2000
-	1    0    0    -1
-$EndComp
-Wire Wire Line
-	4500 2000 4500 2300
-Wire Wire Line
-	4500 2300 4650 2300
+Wire Wire Line
+	5350 1550 5350 2300
+Wire Wire Line
+	5350 2300 5450 2300
 Text Label 4050 2400 0    50   ~ 0
 OLED_SPI_SCK
@@
 OLED_SPI_CS
 Wire Wire Line
-	4050 2400 4650 2400
-Wire Wire Line
-	4050 2500 4650 2500
-Wire Wire Line
-	4050 2600 4650 2600
-Wire Wire Line
-	4050 2700 4650 2700
-Wire Wire Line
-	4050 2800 4650 2800
-$Comp
-L power:+5V #PWR?
-U 1 1 5CF7B0E0
-P 4600 4750
-F 0 "#PWR?" H 4600 4600 50  0001 C CNN
-F 1 "+5V" H 4650 4950 50  0000 C CNN
-F 2 "" H 4600 4750 50  0001 C CNN
-F 3 "" H 4600 4750 50  0001 C CNN
-	1    4600 4750
-	1    0    0    -1
-$EndComp
-Wire Wire Line
-	4600 4750 4600 5050
-Wire Wire Line
-	4700 5050 4600 5050
+	4050 2400 4900 2400
+Wire Wire Line
+	4050 2600 5450 2600
+Wire Wire Line
+	4050 2700 5000 2700
+Wire Wire Line
+	4050 2800 4800 2800
+Wire Wire Line
+	5750 4750 5750 5050
+Wire Wire Line
+	5950 5050 5750 5050
 $Comp
 L power:GND #PWR?
@@
 	3950 5300 3950 5150
 Wire Wire Line
-	3950 5150 4700 5150
+	3950 5150 5950 5150
 Text Label 4150 5250 0    50   ~ 0
 OLED_I2C_SCL
@@
 OLED_SPI_SDA
 Wire Wire Line
-	4150 5250 4700 5250
-Wire Wire Line
-	4150 5350 4700 5350
+	4150 5250 5050 5250
+Wire Wire Line
+	4150 5350 4950 5350
+$Comp
+L Device:R_Pack04 RN?
+U 1 1 5CF7E36C
+P 5000 1850
+AR Path="/5CDAB83A/5CF7E36C" Ref="RN?"  Part="1"
+AR Path="/5CDAB790/5CF7E36C" Ref="RN?"  Part="1"
+F 0 "RN?" H 4700 1900 50  0000 R CNN
+F 1 "R_Pack04" H 4700 1850 50  0000 R CNN
+F 2 "Resistor_SMD:R_Array_Concave_4x0603" V 5275 1850 50  0001 C CNN
+F 3 "~" H 5000 1850 50  0001 C CNN
+	1    5000 1850
+	1    0    0    -1
+$EndComp
+Wire Wire Line
+	5050 1450 5050 1550
+Wire Wire Line
+	5050 1550 5000 1550
+Wire Wire Line
+	4800 1550 4800 1650
+Wire Wire Line
+	4900 1650 4900 1550
+Connection ~ 4900 1550
+Wire Wire Line
+	4900 1550 4800 1550
+Wire Wire Line
+	5000 1550 5000 1650
+Connection ~ 5000 1550
+Wire Wire Line
+	5000 1550 4900 1550
+Wire Wire Line
+	5100 1650 5100 1550
+Wire Wire Line
+	5100 1550 5050 1550
+Connection ~ 5050 1550
+Wire Wire Line
+	4800 2050 4800 2800
+Connection ~ 4800 2800
+Wire Wire Line
+	4800 2800 5450 2800
+Wire Wire Line
+	4900 2050 4900 2400
+Connection ~ 4900 2400
+Wire Wire Line
+	4900 2400 5450 2400
+Wire Wire Line
+	4050 2500 5100 2500
+Wire Wire Line
+	5000 2050 5000 2700
+Connection ~ 5000 2700
+Wire Wire Line
+	5000 2700 5450 2700
+Wire Wire Line
+	5100 2050 5100 2500
+Connection ~ 5100 2500
+Wire Wire Line
+	5100 2500 5450 2500
+$Comp
+L Device:R_Pack04 RN?
+U 1 1 5CF83F57
+P 5150 4800
+AR Path="/5CDAB83A/5CF83F57" Ref="RN?"  Part="1"
+AR Path="/5CDAB790/5CF83F57" Ref="RN?"  Part="1"
+F 0 "RN?" H 4850 4850 50  0000 R CNN
+F 1 "R_Pack04" H 4850 4800 50  0000 R CNN
+F 2 "Resistor_SMD:R_Array_Concave_4x0603" V 5425 4800 50  0001 C CNN
+F 3 "~" H 5150 4800 50  0001 C CNN
+	1    5150 4800
+	1    0    0    -1
+$EndComp
+Wire Wire Line
+	5200 4400 5200 4500
+Wire Wire Line
+	5200 4500 5150 4500
+Wire Wire Line
+	4950 4500 4950 4600
+Wire Wire Line
+	5050 4600 5050 4500
+Connection ~ 5050 4500
+Wire Wire Line
+	5050 4500 4950 4500
+Wire Wire Line
+	5150 4500 5150 4600
+Connection ~ 5150 4500
+Wire Wire Line
+	5150 4500 5050 4500
+Wire Wire Line
+	5250 4600 5250 4500
+Wire Wire Line
+	5250 4500 5200 4500
+Connection ~ 5200 4500
+Wire Wire Line
+	4950 5000 4950 5350
+Connection ~ 4950 5350
+Wire Wire Line
+	4950 5350 5950 5350
+Wire Wire Line
+	5050 5000 5050 5250
+Connection ~ 5050 5250
+Wire Wire Line
+	5050 5250 5950 5250
+$Comp
+L power:+3V3 #PWR?
+U 1 1 5CF89EF6
+P 5050 1450
+F 0 "#PWR?" H 5050 1300 50  0001 C CNN
+F 1 "+3V3" H 5100 1650 50  0000 C CNN
+F 2 "" H 5050 1450 50  0001 C CNN
+F 3 "" H 5050 1450 50  0001 C CNN
+	1    5050 1450
+	1    0    0    -1
+$EndComp
+$Comp
+L power:+3V3 #PWR?
+U 1 1 5CF8A20A
+P 5350 1550
+F 0 "#PWR?" H 5350 1400 50  0001 C CNN
+F 1 "+3V3" H 5400 1750 50  0000 C CNN
+F 2 "" H 5350 1550 50  0001 C CNN
+F 3 "" H 5350 1550 50  0001 C CNN
+	1    5350 1550
+	1    0    0    -1
+$EndComp
+$Comp
+L power:+3V3 #PWR?
+U 1 1 5CF8A4BE
+P 5200 4400
+F 0 "#PWR?" H 5200 4250 50  0001 C CNN
+F 1 "+3V3" H 5250 4600 50  0000 C CNN
+F 2 "" H 5200 4400 50  0001 C CNN
+F 3 "" H 5200 4400 50  0001 C CNN
+	1    5200 4400
+	1    0    0    -1
+$EndComp
+$Comp
+L power:+3V3 #PWR?
+U 1 1 5CF8B0B2
+P 5750 4750
+F 0 "#PWR?" H 5750 4600 50  0001 C CNN
+F 1 "+3V3" H 5800 4950 50  0000 C CNN
+F 2 "" H 5750 4750 50  0001 C CNN
+F 3 "" H 5750 4750 50  0001 C CNN
+	1    5750 4750
+	1    0    0    -1
+$EndComp
 $EndSCHEMATC

Commit message: update,
Parts:
- added C? (x2): C106,0805, Capacitor_SMD:C_0805_2012Metric_Pad1.15x1.40mm_HandSolder, symbol taobao-c:C106,0805
Connections:
- net +3V3: now also C?.2, C?.2
- net GND: now also C?.1, C?.1
Changed lines of the file:
@@
 	1    0    0    -1
 $EndComp
+$Comp
+L power:+3V3 #PWR?
+U 1 1 5CF8B64A
+P 6150 4700
+F 0 "#PWR?" H 6150 4550 50  0001 C CNN
+F 1 "+3V3" V 6200 4850 50  0000 L CNN
+F 2 "" H 6150 4700 50  0001 C CNN
+F 3 "" H 6150 4700 50  0001 C CNN
+	1    6150 4700
+	0    -1   -1   0
+$EndComp
+$Comp
+L power:GND #PWR?
+U 1 1 5CF8B9DE
+P 6650 4700
+F 0 "#PWR?" H 6650 4450 50  0001 C CNN
+F 1 "GND" V 6700 4550 50  0000 R CNN
+F 2 "" H 6650 4700 50  0001 C CNN
+F 3 "" H 6650 4700 50  0001 C CNN
+	1    6650 4700
+	0    -1   -1   0
+$EndComp
+$Comp
+L taobao-c:C106,0805 C?
+U 1 1 5CF8C0FD
+P 6400 4700
+F 0 "C?" V 6150 4700 50  0000 C CNN
+F 1 "C106,0805" V 6250 4700 50  0000 C CNN
+F 2 "Capacitor_SMD:C_0805_2012Metric_Pad1.15x1.40mm_HandSolder" H 6400 4700 50  0001 C CNN
+F 3 "~" H 6400 4700 50  0001 C CNN
+	1    6400 4700
+	0    1    1    0
+$EndComp
+Wire Wire Line
+	6150 4700 6300 4700
+Wire Wire Line
+	6500 4700 6650 4700
+$Comp
+L power:+3V3 #PWR?
+U 1 1 5CF8ED07
+P 5750 1900
+F 0 "#PWR?" H 5750 1750 50  0001 C CNN
+F 1 "+3V3" V 5800 2050 50  0000 L CNN
+F 2 "" H 5750 1900 50  0001 C CNN
+F 3 "" H 5750 1900 50  0001 C CNN
+	1    5750 1900
+	0    -1   -1   0
+$EndComp
+$Comp
+L power:GND #PWR?
+U 1 1 5CF8ED11
+P 6250 1900
+F 0 "#PWR?" H 6250 1650 50  0001 C CNN
+F 1 "GND" V 6300 1750 50  0000 R CNN
+F 2 "" H 6250 1900 50  0001 C CNN
+F 3 "" H 6250 1900 50  0001 C CNN
+	1    6250 1900
+	0    -1   -1   0
+$EndComp
+$Comp
+L taobao-c:C106,0805 C?
+U 1 1 5CF8ED1B
+P 6000 1900
+F 0 "C?" V 5750 1900 50  0000 C CNN
+F 1 "C106,0805" V 5850 1900 50  0000 C CNN
+F 2 "Capacitor_SMD:C_0805_2012Metric_Pad1.15x1.40mm_HandSolder" H 6000 1900 50  0001 C CNN
+F 3 "~" H 6000 1900 50  0001 C CNN
+	1    6000 1900
+	0    1    1    0
+$EndComp
+Wire Wire Line
+	5750 1900 5900 1900
+Wire Wire Line
+	6100 1900 6250 1900
 $EndSCHEMATC

Commit message: update,
Parts:
- gave numbers to parts that had none: 4
Changed lines of the file:
@@
 $EndBitmap
 $Comp
-L power:GND #PWR?
+L power:GND #PWR0131
 U 1 1 5CF79C13
 P 3800 2350
-F 0 "#PWR?" H 3800 2100 50  0001 C CNN
+F 0 "#PWR0131" H 3800 2100 50  0001 C CNN
 F 1 "GND" H 3850 2150 50  0000 C CNN
 F 2 "" H 3800 2350 50  0001 C CNN
@@
 	5950 5050 5750 5050
 $Comp
-L power:GND #PWR?
+L power:GND #PWR0151
 U 1 1 5CF7B7D3
 P 3950 5300
-F 0 "#PWR?" H 3950 5050 50  0001 C CNN
+F 0 "#PWR0151" H 3950 5050 50  0001 C CNN
 F 1 "GND" H 4000 5100 50  0000 C CNN
 F 2 "" H 3950 5300 50  0001 C CNN
@@
 P 5000 1850
 AR Path="/5CDAB83A/5CF7E36C" Ref="RN?"  Part="1"
-AR Path="/5CDAB790/5CF7E36C" Ref="RN?"  Part="1"
-F 0 "RN?" H 4700 1900 50  0000 R CNN
+AR Path="/5CDAB790/5CF7E36C" Ref="RN1"  Part="1"
+F 0 "RN1" H 4700 1900 50  0000 R CNN
 F 1 "R_Pack04" H 4700 1850 50  0000 R CNN
 F 2 "Resistor_SMD:R_Array_Concave_4x0603" V 5275 1850 50  0001 C CNN
@@
 P 5150 4800
 AR Path="/5CDAB83A/5CF83F57" Ref="RN?"  Part="1"
-AR Path="/5CDAB790/5CF83F57" Ref="RN?"  Part="1"
-F 0 "RN?" H 4850 4850 50  0000 R CNN
+AR Path="/5CDAB790/5CF83F57" Ref="RN2"  Part="1"
+F 0 "RN2" H 4850 4850 50  0000 R CNN
 F 1 "R_Pack04" H 4850 4800 50  0000 R CNN
 F 2 "Resistor_SMD:R_Array_Concave_4x0603" V 5425 4800 50  0001 C CNN
@@
 	5050 5250 5950 5250
 $Comp
-L power:+3V3 #PWR?
+L power:+3V3 #PWR0201
 U 1 1 5CF89EF6
 P 5050 1450
-F 0 "#PWR?" H 5050 1300 50  0001 C CNN
+F 0 "#PWR0201" H 5050 1300 50  0001 C CNN
 F 1 "+3V3" H 5100 1650 50  0000 C CNN
 F 2 "" H 5050 1450 50  0001 C CNN
@@
 $EndComp
 $Comp
-L power:+3V3 #PWR?
+L power:+3V3 #PWR0202
 U 1 1 5CF8A20A
 P 5350 1550
-F 0 "#PWR?" H 5350 1400 50  0001 C CNN
+F 0 "#PWR0202" H 5350 1400 50  0001 C CNN
 F 1 "+3V3" H 5400 1750 50  0000 C CNN
 F 2 "" H 5350 1550 50  0001 C CNN
@@
 $EndComp
 $Comp
-L power:+3V3 #PWR?
+L power:+3V3 #PWR0203
 U 1 1 5CF8A4BE
 P 5200 4400
-F 0 "#PWR?" H 5200 4250 50  0001 C CNN
+F 0 "#PWR0203" H 5200 4250 50  0001 C CNN
 F 1 "+3V3" H 5250 4600 50  0000 C CNN
 F 2 "" H 5200 4400 50  0001 C CNN
@@
 $EndComp
 $Comp
-L power:+3V3 #PWR?
+L power:+3V3 #PWR0204
 U 1 1 5CF8B0B2
 P 5750 4750
-F 0 "#PWR?" H 5750 4600 50  0001 C CNN
+F 0 "#PWR0204" H 5750 4600 50  0001 C CNN
 F 1 "+3V3" H 5800 4950 50  0000 C CNN
 F 2 "" H 5750 4750 50  0001 C CNN
@@
 $EndComp
 $Comp
-L power:+3V3 #PWR?
+L power:+3V3 #PWR0205
 U 1 1 5CF8B64A
 P 6150 4700
-F 0 "#PWR?" H 6150 4550 50  0001 C CNN
+F 0 "#PWR0205" H 6150 4550 50  0001 C CNN
 F 1 "+3V3" V 6200 4850 50  0000 L CNN
 F 2 "" H 6150 4700 50  0001 C CNN
@@
 $EndComp
 $Comp
-L power:GND #PWR?
+L power:GND #PWR0206
 U 1 1 5CF8B9DE
 P 6650 4700
-F 0 "#PWR?" H 6650 4450 50  0001 C CNN
+F 0 "#PWR0206" H 6650 4450 50  0001 C CNN
 F 1 "GND" V 6700 4550 50  0000 R CNN
 F 2 "" H 6650 4700 50  0001 C CNN
@@
 $EndComp
 $Comp
-L taobao-c:C106,0805 C?
+L taobao-c:C106,0805 C33
 U 1 1 5CF8C0FD
 P 6400 4700
-F 0 "C?" V 6150 4700 50  0000 C CNN
+F 0 "C33" V 6150 4700 50  0000 C CNN
 F 1 "C106,0805" V 6250 4700 50  0000 C CNN
 F 2 "Capacitor_SMD:C_0805_2012Metric_Pad1.15x1.40mm_HandSolder" H 6400 4700 50  0001 C CNN
@@
 	6500 4700 6650 4700
 $Comp
-L power:+3V3 #PWR?
+L power:+3V3 #PWR0207
 U 1 1 5CF8ED07
 P 5750 1900
-F 0 "#PWR?" H 5750 1750 50  0001 C CNN
+F 0 "#PWR0207" H 5750 1750 50  0001 C CNN
 F 1 "+3V3" V 5800 2050 50  0000 L CNN
 F 2 "" H 5750 1900 50  0001 C CNN
@@
 $EndComp
 $Comp
-L power:GND #PWR?
+L power:GND #PWR0208
 U 1 1 5CF8ED11
 P 6250 1900
-F 0 "#PWR?" H 6250 1650 50  0001 C CNN
+F 0 "#PWR0208" H 6250 1650 50  0001 C CNN
 F 1 "GND" V 6300 1750 50  0000 R CNN
 F 2 "" H 6250 1900 50  0001 C CNN
@@
 $EndComp
 $Comp
-L taobao-c:C106,0805 C?
+L taobao-c:C106,0805 C32
 U 1 1 5CF8ED1B
 P 6000 1900
-F 0 "C?" V 5750 1900 50  0000 C CNN
+F 0 "C32" V 5750 1900 50  0000 C CNN
 F 1 "C106,0805" V 5850 1900 50  0000 C CNN
 F 2 "Capacitor_SMD:C_0805_2012Metric_Pad1.15x1.40mm_HandSolder" H 6000 1900 50  0001 C CNN
