File: hardware/_autosave-bluepill.sch (KiCad schematic (older format))
At the start: 3 parts, among them J22 STM32_2_DEBUG1, J23 STM32_2_DEBUG2, U13 bluepill-stm32f103c8t6

Commit message: update,
Connections:
- net A_IN1: now also J22.6 (Pin_6); no longer J22.5 (Pin_5)
- removed net A_IN2: J22.6 (Pin_6), U13.~ (VBAT)
- new net A_IN0: J22.5 (Pin_5), U13.~ (VBAT)
Changed lines of the file:
@@
 $Descr A4 11693 8268
 encoding utf-8
-Sheet 20 20
+Sheet 19 20
 Title ""
 Date ""
@@
 	1050 1950 1400 1950
 Text HLabel 1050 2300 0    50   Input ~ 0
-A_IN1
+A_IN0
 Text HLabel 1050 2400 0    50   Input ~ 0
-A_IN2
+A_IN1
 Text HLabel 1400 2300 2    50   Input ~ 0
 STM32_1_PA0
