File: hardware/_autosave-eval_board.sch (KiCad schematic (older format))
At the start: 0 parts

Commit message: update,
Changed lines of the file:
@@
 $EndSheet
 $Sheet
-S 1050 2250 600  800
+S 2300 3700 600  800
 U 5CE535D6
 F0 "arduino_nano" 50
 F1 "arduino_nano.sch" 50
-F2 "SCL" I R 1650 2400 50
-F3 "SDA" I R 1650 2500 50
-F4 "TXD" I R 1650 2800 50
-F5 "RXD" I R 1650 2900 50
+F2 "SCL" I R 2900 3850 50
+F3 "SDA" I R 2900 3950 50
+F4 "TXD" I R 2900 4250 50
+F5 "RXD" I R 2900 4350 50
 $EndSheet
 $Sheet
@@
 checklist:\n\ndebug terminal
 $Sheet
-S 1050 3300 612  400
+S 2300 1200 600  2300
 U 5CECA6C5
 F0 "nodemcu" 50
 F1 "nodemcu.sch" 50
-F2 "SDA" I R 1662 3550 50
-F3 "SCL" I R 1662 3450 50
+F2 "SDA" I R 2900 1450 50
+F3 "SCL" I R 2900 1350 50
+F4 "SDD0" I R 2900 1700 50
+F5 "SDD1" I R 2900 1800 50
+F6 "SDD2" I R 2900 1900 50
+F7 "SDD3" I R 2900 2000 50
+F8 "SDDCMD" I R 2900 2100 50
+F9 "SDDCLK" I R 2900 2200 50
+F10 "TX" I R 2900 2400 50
+F11 "RX" I R 2900 2500 50
+F12 "HSCLK" I R 2900 2700 50
+F13 "HMISO" I R 2900 2800 50
+F14 "HMOSI" I R 2900 2900 50
+F15 "HCS" I R 2900 3000 50
+F16 "PWM" I R 2900 3200 50
+F17 "A_IN_0" I R 2900 3300 50
 $EndSheet
 Entry Wire Line
@@
 	9050 11100 9150 11000
 $Sheet
-S 1000 800  650  1200
+S 1050 1200 600  1850
 U 5CDAB6B1
 F0 "bluepill" 50
 F1 "bluepill.sch" 50
-F2 "SDA" I R 1650 1050 50
-F3 "SCL" I R 1650 950 50
-F4 "SCK" I R 1650 1450 50
-F5 "MOSI" I R 1650 1350 50
-F6 "MISO" I R 1650 1250 50
-F7 "SS" I R 1650 1550 50
-F8 "TX" I R 1650 1750 50
-F9 "RX" I R 1650 1850 50
+F2 "SDA" I R 1650 1450 50
+F3 "SCL" I R 1650 1350 50
+F4 "SCK" I R 1650 1850 50
+F5 "MOSI" I R 1650 1750 50
+F6 "MISO" I R 1650 1650 50
+F7 "SS" I R 1650 1950 50
+F8 "TX" I R 1650 2150 50
+F9 "RX" I R 1650 2250 50
+F10 "A_IN0" I R 1650 2500 50
+F11 "A_IN1" I R 1650 2600 50
+F12 "PWM" I R 1650 2800 50
 $EndSheet
 $Sheet
