File: hardware/esp8266.sch (KiCad schematic (older format))
At the start: 1 part, among them U1 ESP12

Commit message: update,
Parts:
- removed U1: ESP12, footprint-lib:ESP-12, symbol taobao-components:ESP12
- added U?: ESP-12E, footprint-lib:ESP-12E, symbol taobao-components:ESP-12E

Commit message: update,
Parts:
- removed U?: ESP-12E, footprint-lib:ESP-12E, symbol taobao-components:ESP-12E
