File: hardware/stm32f103c8t6.sch (KiCad schematic (older format))
At the start: 31 parts, among them J11 Conn_01x12, J12 Conn_01x14, J13 Conn_01x12, SW1 SW_Push, U4 STM32F103C8T6, U5 AMS1117-3.3, Y4 O8M, Y5 O32.768K

Commit message: update,
Parts:
- U4: footprint Package_QFP:LQFP-48_7x7mm_P0.5mm -> footprint-lib:STM32F103C8T6
Changed lines of the file:
@@
 $Descr A3 16535 11693
 encoding utf-8
-Sheet 19 27
+Sheet 27 27
 Title ""
 Date ""
@@
 Comment4 ""
 $EndDescr
-$Comp
-L taobao-components:STM32F103C8T6 U4
-U 1 1 5BCB9005
-P 8550 4300
-F 0 "U4" H 8600 5428 50  0000 C CNN
-F 1 "STM32F103C8T6" H 8600 5337 50  0000 C CNN
-F 2 "Package_QFP:LQFP-48_7x7mm_P0.5mm" H 8550 4300 50  0001 C CNN
-F 3 "" H 8550 4300 50  0001 C CNN
-	1    8550 4300
-	1    0    0    -1
-$EndComp
-Text Label 7050 3800 0    50   ~ 0
+Text Label 6900 3750 0    50   ~ 0
 VBAT
 Wire Wire Line
-	7050 3800 7600 3800
-Text Label 7050 3900 0    50   ~ 0
+	6900 3750 7450 3750
+Text Label 6900 3850 0    50   ~ 0
 PC13
 Wire Wire Line
-	7050 3900 7600 3900
-Text Label 7050 4000 0    50   ~ 0
+	6900 3850 7450 3850
+Text Label 6900 3950 0    50   ~ 0
 PC14
 Wire Wire Line
-	7050 4000 7600 4000
-Text Label 7050 4100 0    50   ~ 0
+	6900 3950 7450 3950
+Text Label 6900 4050 0    50   ~ 0
 PC15
 Wire Wire Line
-	7050 4100 7600 4100
-Text Label 7050 4200 0    50   ~ 0
+	6900 4050 7450 4050
+Text Label 6900 4150 0    50   ~ 0
 OSCIN
 Wire Wire Line
-	7050 4200 7600 4200
-Text Label 7050 4300 0    50   ~ 0
+	6900 4150 7450 4150
+Text Label 6900 4250 0    50   ~ 0
 OSCOUT
 Wire Wire Line
-	7050 4300 7600 4300
-Text Label 7050 4400 0    50   ~ 0
+	6900 4250 7450 4250
+Text Label 6900 4350 0    50   ~ 0
 RESET
 Wire Wire Line
-	7050 4400 7600 4400
-Text Label 7050 4500 0    50   ~ 0
+	6900 4350 7450 4350
+Text Label 6900 4450 0    50   ~ 0
 GND
 Wire Wire Line
-	7050 4500 7600 4500
-Text Label 7050 4600 0    50   ~ 0
+	6900 4450 7450 4450
+Text Label 6900 4550 0    50   ~ 0
 VCC3V3
 Wire Wire Line
-	7050 4600 7600 4600
-Text Label 7050 4700 0    50   ~ 0
+	6900 4550 7450 4550
+Text Label 6900 4650 0    50   ~ 0
 PA0
 Wire Wire Line
-	7050 4700 7600 4700
-Text Label 7050 4800 0    50   ~ 0
+	6900 4650 7450 4650
+Text Label 6900 4750 0    50   ~ 0
 PA1
 Wire Wire Line
-	7050 4800 7600 4800
-Text Label 7050 4900 0    50   ~ 0
+	6900 4750 7450 4750
+Text Label 6900 4850 0    50   ~ 0
 PA2
 Wire Wire Line
-	7050 4900 7600 4900
-Text Label 8050 5900 1    50   ~ 0
+	6900 4850 7450 4850
+Text Label 8000 5950 1    50   ~ 0
 PA3
 Wire Wire Line
-	8050 5900 8050 5350
-Text Label 8150 5900 1    50   ~ 0
+	8000 5950 8000 5400
+Text Label 8100 5950 1    50   ~ 0
 PA4
 Wire Wire Line
-	8150 5900 8150 5350
-Text Label 8250 5900 1    50   ~ 0
+	8100 5950 8100 5400
+Text Label 8200 5950 1    50   ~ 0
 PA5
 Wire Wire Line
-	8250 5900 8250 5350
-Text Label 8350 5900 1    50   ~ 0
+	8200 5950 8200 5400
+Text Label 8300 5950 1    50   ~ 0
 PA6
 Wire Wire Line
-	8350 5900 8350 5350
-Text Label 8450 5900 1    50   ~ 0
+	8300 5950 8300 5400
+Text Label 8400 5950 1    50   ~ 0
 PA7
 Wire Wire Line
-	8450 5900 8450 5350
-Text Label 8550 5900 1    50   ~ 0
+	8400 5950 8400 5400
+Text Label 8500 5950 1    50   ~ 0
 PB0
 Wire Wire Line
-	8550 5900 8550 5350
-Text Label 8650 5900 1    50   ~ 0
+	8500 5950 8500 5400
+Text Label 8600 5950 1    50   ~ 0
 PB1
 Wire Wire Line
-	8650 5900 8650 5350
-Text Label 8750 5900 1    50   ~ 0
+	8600 5950 8600 5400
+Text Label 8700 5950 1    50   ~ 0
 BOOT1
 Wire Wire Line
-	8750 5900 8750 5350
-Text Label 8850 5900 1    50   ~ 0
+	8700 5950 8700 5400
+Text Label 8800 5950 1    50   ~ 0
 PB10
 Wire Wire Line
-	8850 5900 8850 5350
-Text Label 8950 5900 1    50   ~ 0
+	8800 5950 8800 5400
+Text Label 8900 5950 1    50   ~ 0
 PB11
 Wire Wire Line
-	8950 5900 8950 5350
-Text Label 9050 5900 1    50   ~ 0
+	8900 5950 8900 5400
+Text Label 9000 5950 1    50   ~ 0
 VSS_1
 Wire Wire Line
-	9050 5900 9050 5350
-Text Label 9150 5900 1    50   ~ 0
+	9000 5950 9000 5400
+Text Label 9100 5950 1    50   ~ 0
 VDD_1
 Wire Wire Line
-	9150 5900 9150 5350
-Text Label 10150 4900 2    50   ~ 0
+	9100 5950 9100 5400
+Text Label 10200 4850 2    50   ~ 0
 PB12
 Wire Wire Line
-	10150 4900 9600 4900
-Text Label 10150 4800 2    50   ~ 0
+	10200 4850 9650 4850
+Text Label 10200 4750 2    50   ~ 0
 PB13
 Wire Wire Line
-	10150 4800 9600 4800
-Text Label 10150 4700 2    50   ~ 0
+	10200 4750 9650 4750
+Text Label 10200 4650 2    50   ~ 0
 PB14
 Wire Wire Line
-	10150 4700 9600 4700
-Text Label 10150 4600 2    50   ~ 0
+	10200 4650 9650 4650
+Text Label 10200 4550 2    50   ~ 0
 PB15
 Wire Wire Line
-	10150 4600 9600 4600
-Text Label 10150 4500 2    50   ~ 0
+	10200 4550 9650 4550
+Text Label 10200 4450 2    50   ~ 0
 PA8
 Wire Wire Line
-	10150 4500 9600 4500
-Text Label 10150 4400 2    50   ~ 0
+	10200 4450 9650 4450
+Text Label 10200 4350 2    50   ~ 0
 PA9
 Wire Wire Line
-	10150 4400 9600 4400
-Text Label 10150 4300 2    50   ~ 0
+	10200 4350 9650 4350
+Text Label 10200 4250 2    50   ~ 0
 PA10
 Wire Wire Line
-	10150 4300 9600 4300
-Text Label 10150 4200 2    50   ~ 0
+	10200 4250 9650 4250
+Text Label 10200 4150 2    50   ~ 0
 PA11
 Wire Wire Line
-	10150 4200 9600 4200
-Text Label 10150 4100 2    50   ~ 0
+	10200 4150 9650 4150
+Text Label 10200 4050 2    50   ~ 0
 PA12
 Wire Wire Line
-	10150 4100 9600 4100
-Text Label 10150 4000 2    50   ~ 0
+	10200 4050 9650 4050
+Text Label 10200 3950 2    50   ~ 0
 SWIO
 Wire Wire Line
-	10150 4000 9600 4000
-Text Label 10150 3900 2    50   ~ 0
+	10200 3950 9650 3950
+Text Label 10200 3850 2    50   ~ 0
 VSS_2
 Wire Wire Line
-	10150 3900 9600 3900
-Text Label 10150 3800 2    50   ~ 0
+	10200 3850 9650 3850
+Text Label 10200 3750 2    50   ~ 0
 VDD_2
 Wire Wire Line
-	10150 3800 9600 3800
-Text Label 9150 2800 3    50   ~ 0
+	10200 3750 9650 3750
+Text Label 9100 2650 3    50   ~ 0
 SWCLK
 Wire Wire Line
-	9150 2800 9150 3350
-Text Label 9050 2800 3    50   ~ 0
+	9100 2650 9100 3200
+Text Label 9000 2650 3    50   ~ 0
 PA15
 Wire Wire Line
-	9050 2800 9050 3350
-Text Label 8950 2800 3    50   ~ 0
+	9000 2650 9000 3200
+Text Label 8900 2650 3    50   ~ 0
 PB3
 Wire Wire Line
-	8950 2800 8950 3350
-Text Label 8850 2800 3    50   ~ 0
+	8900 2650 8900 3200
+Text Label 8800 2650 3    50   ~ 0
 PB4
 Wire Wire Line
-	8850 2800 8850 3350
-Text Label 8750 2800 3    50   ~ 0
+	8800 2650 8800 3200
+Text Label 8700 2650 3    50   ~ 0
 PB5
 Wire Wire Line
-	8750 2800 8750 3350
-Text Label 8650 2800 3    50   ~ 0
+	8700 2650 8700 3200
+Text Label 8600 2650 3    50   ~ 0
 PB6
 Wire Wire Line
-	8650 2800 8650 3350
-Text Label 8550 2800 3    50   ~ 0
+	8600 2650 8600 3200
+Text Label 8500 2650 3    50   ~ 0
 PB7
 Wire Wire Line
-	8550 2800 8550 3350
-Text Label 8450 2800 3    50   ~ 0
+	8500 2650 8500 3200
+Text Label 8400 2650 3    50   ~ 0
 BOOT0
 Wire Wire Line
-	8450 2800 8450 3350
-Text Label 8350 2800 3    50   ~ 0
+	8400 2650 8400 3200
+Text Label 8300 2650 3    50   ~ 0
 PB8
 Wire Wire Line
-	8350 2800 8350 3350
-Text Label 8250 2800 3    50   ~ 0
+	8300 2650 8300 3200
+Text Label 8200 2650 3    50   ~ 0
 PB9
 Wire Wire Line
-	8250 2800 8250 3350
-Text Label 8150 2800 3    50   ~ 0
+	8200 2650 8200 3200
+Text Label 8100 2650 3    50   ~ 0
 GND
 Wire Wire Line
-	8150 2800 8150 3350
-Text Label 8050 2800 3    50   ~ 0
+	8100 2650 8100 3200
+Text Label 8000 2650 3    50   ~ 0
 VCC3V3
 Wire Wire Line
-	8050 2800 8050 3350
+	8000 2650 8000 3200
 $Comp
 L taobao-c:C104 C11
@@
 Wire Wire Line
 	14500 7700 14550 7700
+$Comp
+L taobao-components:STM32F103C8T6 U4
+U 1 1 5CF34EE1
+P 8550 4300
+F 0 "U4" H 9300 3350 50  0000 L CNN
+F 1 "STM32F103C8T6" H 9300 3200 50  0000 L CNN
+F 2 "footprint-lib:STM32F103C8T6" H 8550 4300 50  0001 C CNN
+F 3 "" H 8550 4300 50  0001 C CNN
+	1    8550 4300
+	1    0    0    -1
+$EndComp
 $EndSCHEMATC

Commit message: update,
Parts:
- renumbered C6 to C26, C7 to C27, C8 to C28, C9 to C29, C10 to C30, C11 to C31, C12 to C32, C13 to C33, C14 to C34, C15 to C35, C16 to C36, C17 to C37, C18 to C38, D4 to D11, D5 to D12, J11 to J19, J12 to J20, J13 to J21, JP1 to JP6, R4 to R29, R5 to R30, R6 to R31, R7 to R32, R8 to R33, SW1 to SW4, U4 to U10, U5 to U11, Y4 to Y2, Y5 to Y3

Commit message: update,
Parts:
- renumbered J19 to J22, J20 to J23, J21 to J24
Changed lines of the file:
@@
 	8000 6800 8000 6900
 $Comp
-L power:GND #PWR0138
+L power:GND #PWR0139
 U 1 1 5BCBCE91
 P 8000 7200
-F 0 "#PWR0138" H 8000 6950 50  0001 C CNN
+F 0 "#PWR0139" H 8000 6950 50  0001 C CNN
 F 1 "GND" H 8005 7027 50  0000 C CNN
 F 2 "" H 8000 7200 50  0001 C CNN
@@
 	8450 6800 8450 6900
 $Comp
-L power:GND #PWR0139
+L power:GND #PWR0140
 U 1 1 5BCBD867
 P 8450 7200
-F 0 "#PWR0139" H 8450 6950 50  0001 C CNN
+F 0 "#PWR0140" H 8450 6950 50  0001 C CNN
 F 1 "GND" H 8455 7027 50  0000 C CNN
 F 2 "" H 8450 7200 50  0001 C CNN
@@
 	8850 6800 8850 6900
 $Comp
-L power:GND #PWR0140
+L power:GND #PWR0141
 U 1 1 5BCBE2F9
 P 8850 7200
-F 0 "#PWR0140" H 8850 6950 50  0001 C CNN
+F 0 "#PWR0141" H 8850 6950 50  0001 C CNN
 F 1 "GND" H 8855 7027 50  0000 C CNN
 F 2 "" H 8850 7200 50  0001 C CNN
@@
 	9300 6800 9300 6900
 $Comp
-L power:GND #PWR0141
+L power:GND #PWR0142
 U 1 1 5BCBE30D
 P 9300 7200
-F 0 "#PWR0141" H 9300 6950 50  0001 C CNN
+F 0 "#PWR0142" H 9300 6950 50  0001 C CNN
 F 1 "GND" H 9305 7027 50  0000 C CNN
 F 2 "" H 9300 7200 50  0001 C CNN
@@
 	14850 8450 14850 8550
 $Comp
-L power:GND #PWR0143
+L power:GND #PWR0144
 U 1 1 5BCC0C02
 P 14300 8750
-F 0 "#PWR0143" H 14300 8500 50  0001 C CNN
+F 0 "#PWR0144" H 14300 8500 50  0001 C CNN
 F 1 "GND" H 14305 8577 50  0000 C CNN
 F 2 "" H 14300 8750 50  0001 C CNN
@@
 	14850 8000 14850 7950
 $Comp
-L power:GND #PWR0142
+L power:GND #PWR0143
 U 1 1 5BCC9128
 P 14300 7900
-F 0 "#PWR0142" H 14300 7650 50  0001 C CNN
+F 0 "#PWR0143" H 14300 7650 50  0001 C CNN
 F 1 "GND" H 14305 7727 50  0000 C CNN
 F 2 "" H 14300 7900 50  0001 C CNN
@@
 $EndComp
 $Comp
-L power:GND #PWR0130
+L power:GND #PWR0131
 U 1 1 5BCD1DA6
 P 14350 6650
-F 0 "#PWR0130" H 14350 6400 50  0001 C CNN
+F 0 "#PWR0131" H 14350 6400 50  0001 C CNN
 F 1 "GND" H 14355 6477 50  0000 C CNN
 F 2 "" H 14350 6650 50  0001 C CNN
@@
 	14650 4000 14650 4050
 $Comp
-L power:GND #PWR0122
+L power:GND #PWR0123
 U 1 1 5BCDDB1E
 P 14650 4550
-F 0 "#PWR0122" H 14650 4300 50  0001 C CNN
+F 0 "#PWR0123" H 14650 4300 50  0001 C CNN
 F 1 "GND" H 14655 4377 50  0000 C CNN
 F 2 "" H 14650 4550 50  0001 C CNN
@@
 	11100 4000 11450 4000
 $Comp
-L power:GND #PWR0120
+L power:GND #PWR0121
 U 1 1 5BD0648A
 P 11950 4400
-F 0 "#PWR0120" H 11950 4150 50  0001 C CNN
+F 0 "#PWR0121" H 11950 4150 50  0001 C CNN
 F 1 "GND" H 11955 4227 50  0000 C CNN
 F 2 "" H 11950 4400 50  0001 C CNN
@@
 	12800 3500 12800 3800
 $Comp
-L power:GND #PWR0121
+L power:GND #PWR0122
 U 1 1 5BD0D994
 P 12800 4400
-F 0 "#PWR0121" H 12800 4150 50  0001 C CNN
+F 0 "#PWR0122" H 12800 4150 50  0001 C CNN
 F 1 "GND" H 12805 4227 50  0000 C CNN
 F 2 "" H 12800 4400 50  0001 C CNN
@@
 	10900 6250 11100 6250
 $Comp
-L power:GND #PWR0135
+L power:GND #PWR0136
 U 1 1 5BD310AF
 P 10900 6800
-F 0 "#PWR0135" H 10900 6550 50  0001 C CNN
+F 0 "#PWR0136" H 10900 6550 50  0001 C CNN
 F 1 "GND" H 10905 6627 50  0000 C CNN
 F 2 "" H 10900 6800 50  0001 C CNN
@@
 	10900 6600 10900 6800
 $Comp
-L power:GND #PWR0136
+L power:GND #PWR0137
 U 1 1 5BD33ECC
 P 11400 6800
-F 0 "#PWR0136" H 11400 6550 50  0001 C CNN
+F 0 "#PWR0137" H 11400 6550 50  0001 C CNN
 F 1 "GND" H 11405 6627 50  0000 C CNN
 F 2 "" H 11400 6800 50  0001 C CNN
@@
 Connection ~ 11850 6250
 $Comp
-L power:GND #PWR0137
+L power:GND #PWR0138
 U 1 1 5BD3D1BA
 P 12050 6800
-F 0 "#PWR0137" H 12050 6550 50  0001 C CNN
+F 0 "#PWR0138" H 12050 6550 50  0001 C CNN
 F 1 "GND" H 12055 6627 50  0000 C CNN
 F 2 "" H 12050 6800 50  0001 C CNN
@@
 Connection ~ 12250 6250
 $Comp
-L power:GND #PWR0124
+L power:GND #PWR0125
 U 1 1 5BD5A437
 P 4000 5900
-F 0 "#PWR0124" H 4000 5650 50  0001 C CNN
+F 0 "#PWR0125" H 4000 5650 50  0001 C CNN
 F 1 "GND" H 4005 5727 50  0000 C CNN
 F 2 "" H 4000 5900 50  0001 C CNN
@@
 	2300 3550 2300 3650
 $Comp
-L power:GND #PWR0119
+L power:GND #PWR0120
 U 1 1 5BD90F7D
 P 2300 4050
-F 0 "#PWR0119" H 2300 3800 50  0001 C CNN
+F 0 "#PWR0120" H 2300 3800 50  0001 C CNN
 F 1 "GND" H 2305 3877 50  0000 C CNN
 F 2 "" H 2300 4050 50  0001 C CNN
@@
 $EndComp
 $Comp
-L power:GND #PWR0113
+L power:GND #PWR0114
 U 1 1 5BD957D4
 P 8850 2500
-F 0 "#PWR0113" H 8850 2250 50  0001 C CNN
+F 0 "#PWR0114" H 8850 2250 50  0001 C CNN
 F 1 "GND" H 8855 2327 50  0000 C CNN
 F 2 "" H 8850 2500 50  0001 C CNN
@@
 SWCLK
 $Comp
-L Connector_Generic:Conn_01x12 J19
+L Connector_Generic:Conn_01x12 J22
 U 1 1 5BDC51B3
 P 3400 2800
-F 0 "J19" V 3617 2746 50  0000 C CNN
+F 0 "J22" V 3617 2746 50  0000 C CNN
 F 1 "Conn_01x12" V 3526 2746 50  0000 C CNN
 F 2 "Connector_PinHeader_1.27mm:PinHeader_1x12_P1.27mm_Vertical" H 3400 2800 50  0001 C CNN
@@
 $EndComp
 $Comp
-L Connector_Generic:Conn_01x14 J20
+L Connector_Generic:Conn_01x14 J23
 U 1 1 5BDC5267
 P 1650 4250
-F 0 "J20" H 1570 4967 50  0000 C CNN
+F 0 "J23" H 1570 4967 50  0000 C CNN
 F 1 "Conn_01x14" H 1570 4876 50  0000 C CNN
 F 2 "Connector_PinHeader_1.27mm:PinHeader_1x14_P1.27mm_Vertical" H 1650 4250 50  0001 C CNN
@@
 $EndComp
 $Comp
-L Connector_Generic:Conn_01x20 J21
+L Connector_Generic:Conn_01x20 J24
 U 1 1 5BDCE49F
 P 5100 5050
-F 0 "J21" H 5019 3825 50  0000 C CNN
+F 0 "J24" H 5019 3825 50  0000 C CNN
 F 1 "Conn_01x12" H 5019 3916 50  0000 C CNN
 F 2 "Connector_PinHeader_1.27mm:PinHeader_1x20_P1.27mm_Vertical" H 5100 5050 50  0001 C CNN
@@
 	2300 4850 2300 4800
 $Comp
-L power:+3V3 #PWR0118
+L power:+3V3 #PWR0119
 U 1 1 5BCAC201
 P 2300 3550
-F 0 "#PWR0118" H 2300 3400 50  0001 C CNN
+F 0 "#PWR0119" H 2300 3400 50  0001 C CNN
 F 1 "+3V3" H 2350 3750 50  0000 C CNN
 F 2 "" H 2300 3550 50  0001 C CNN
@@
 $EndComp
 $Comp
-L power:+3V3 #PWR0123
+L power:+3V3 #PWR0124
 U 1 1 5BCACA2F
 P 4100 5700
-F 0 "#PWR0123" H 4100 5550 50  0001 C CNN
+F 0 "#PWR0124" H 4100 5550 50  0001 C CNN
 F 1 "+3V3" H 4150 5900 50  0000 C CNN
 F 2 "" H 4100 5700 50  0001 C CNN
@@
 $EndComp
 $Comp
-L power:+5V #PWR0128
+L power:+5V #PWR0129
 U 1 1 5BCACB86
 P 4350 6100
-F 0 "#PWR0128" H 4350 5950 50  0001 C CNN
+F 0 "#PWR0129" H 4350 5950 50  0001 C CNN
 F 1 "+5V" H 4350 6300 50  0000 C CNN
 F 2 "" H 4350 6100 50  0001 C CNN
@@
 $EndComp
 $Comp
-L power:+3V3 #PWR0111
+L power:+3V3 #PWR0112
 U 1 1 5BCAD5BF
 P 6100 1850
-F 0 "#PWR0111" H 6100 1700 50  0001 C CNN
+F 0 "#PWR0112" H 6100 1700 50  0001 C CNN
 F 1 "+3V3" H 6150 2050 50  0000 C CNN
 F 2 "" H 6100 1850 50  0001 C CNN
@@
 $EndComp
 $Comp
-L power:+3V3 #PWR0131
+L power:+3V3 #PWR0132
 U 1 1 5BCBE3DE
 P 8000 6800
-F 0 "#PWR0131" H 8000 6650 50  0001 C CNN
+F 0 "#PWR0132" H 8000 6650 50  0001 C CNN
 F 1 "+3V3" H 8050 7000 50  0000 C CNN
 F 2 "" H 8000 6800 50  0001 C CNN
@@
 $EndComp
 $Comp
-L power:+3V3 #PWR0132
+L power:+3V3 #PWR0133
 U 1 1 5BCE7C1D
 P 8450 6800
-F 0 "#PWR0132" H 8450 6650 50  0001 C CNN
+F 0 "#PWR0133" H 8450 6650 50  0001 C CNN
 F 1 "+3V3" H 8500 7000 50  0000 C CNN
 F 2 "" H 8450 6800 50  0001 C CNN
@@
 $EndComp
 $Comp
-L power:+3V3 #PWR0133
+L power:+3V3 #PWR0134
 U 1 1 5BCE7C66
 P 8850 6800
-F 0 "#PWR0133" H 8850 6650 50  0001 C CNN
+F 0 "#PWR0134" H 8850 6650 50  0001 C CNN
 F 1 "+3V3" H 8900 7000 50  0000 C CNN
 F 2 "" H 8850 6800 50  0001 C CNN
@@
 $EndComp
 $Comp
-L power:+3V3 #PWR0134
+L power:+3V3 #PWR0135
 U 1 1 5BCE7CAF
 P 9300 6800
-F 0 "#PWR0134" H 9300 6650 50  0001 C CNN
+F 0 "#PWR0135" H 9300 6650 50  0001 C CNN
 F 1 "+3V3" H 9350 7000 50  0000 C CNN
 F 2 "" H 9300 6800 50  0001 C CNN
@@
 $EndComp
 $Comp
-L power:+3V3 #PWR0127
+L power:+3V3 #PWR0128
 U 1 1 5BCE8262
 P 12350 6050
-F 0 "#PWR0127" H 12350 5900 50  0001 C CNN
+F 0 "#PWR0128" H 12350 5900 50  0001 C CNN
 F 1 "+3V3" H 12400 6250 50  0000 C CNN
 F 2 "" H 12350 6050 50  0001 C CNN
@@
 $EndComp
 $Comp
-L power:+3V3 #PWR0125
+L power:+3V3 #PWR0126
 U 1 1 5BCE8771
 P 14350 5900
-F 0 "#PWR0125" H 14350 5750 50  0001 C CNN
+F 0 "#PWR0126" H 14350 5750 50  0001 C CNN
 F 1 "+3V3" H 14400 6100 50  0000 C CNN
 F 2 "" H 14350 5900 50  0001 C CNN
@@
 $EndComp
 $Comp
-L customized_power:+5V #PWR0126
+L customized_power:+5V #PWR0127
 U 1 1 5BCE8D55
 P 10750 6050
-F 0 "#PWR0126" H 10750 5900 50  0001 C CNN
+F 0 "#PWR0127" H 10750 5900 50  0001 C CNN
 F 1 "+5V" H 10800 6250 50  0000 C CNN
 F 2 "" H 10750 6050 50  0001 C CNN
@@
 $EndComp
 $Comp
-L power:+3V3 #PWR0112
+L power:+3V3 #PWR0113
 U 1 1 5BCF284B
 P 8350 2500
-F 0 "#PWR0112" H 8350 2350 50  0001 C CNN
+F 0 "#PWR0113" H 8350 2350 50  0001 C CNN
 F 1 "+3V3" H 8400 2700 50  0000 C CNN
 F 2 "" H 8350 2500 50  0001 C CNN
@@
 $EndComp
 $Comp
-L power:+3V3 #PWR0115
+L power:+3V3 #PWR0116
 U 1 1 5BCF3126
 P 14650 3350
-F 0 "#PWR0115" H 14650 3200 50  0001 C CNN
+F 0 "#PWR0116" H 14650 3200 50  0001 C CNN
 F 1 "+3V3" H 14700 3550 50  0000 C CNN
 F 2 "" H 14650 3350 50  0001 C CNN
@@
 $EndComp
 $Comp
-L power:+3V3 #PWR0117
+L power:+3V3 #PWR0118
 U 1 1 5BCF394E
 P 12800 3500
-F 0 "#PWR0117" H 12800 3350 50  0001 C CNN
+F 0 "#PWR0118" H 12800 3350 50  0001 C CNN
 F 1 "+3V3" H 12850 3700 50  0000 C CNN
 F 2 "" H 12800 3500 50  0001 C CNN
@@
 $EndComp
 $Comp
-L power:+3V3 #PWR0116
+L power:+3V3 #PWR0117
 U 1 1 5BCF3997
 P 11950 3500
-F 0 "#PWR0116" H 11950 3350 50  0001 C CNN
+F 0 "#PWR0117" H 11950 3350 50  0001 C CNN
 F 1 "+3V3" H 12000 3700 50  0000 C CNN
 F 2 "" H 11950 3500 50  0001 C CNN
@@
 	6100 2150 6100 2250
 $Comp
-L power:GND #PWR0114
+L power:GND #PWR0115
 U 1 1 5BDA790B
 P 6100 2850
-F 0 "#PWR0114" H 6100 2600 50  0001 C CNN
+F 0 "#PWR0115" H 6100 2600 50  0001 C CNN
 F 1 "GND" H 6150 2650 50  0000 C CNN
 F 2 "" H 6100 2850 50  0001 C CNN
@@
 $EndComp
 $Comp
-L power:GND #PWR0129
+L power:GND #PWR0130
 U 1 1 5BDD944B
 P 13700 6650
-F 0 "#PWR0129" H 13700 6400 50  0001 C CNN
+F 0 "#PWR0130" H 13700 6400 50  0001 C CNN
 F 1 "GND" H 13705 6477 50  0000 C CNN
 F 2 "" H 13700 6650 50  0001 C CNN

Commit message: update,
Parts:
- renumbered C26 to C24, C27 to C25, C28 to C26, C29 to C27, C30 to C28, C31 to C29, C32 to C30, C33 to C31, C34 to C32, C35 to C33, C36 to C34, C37 to C35, C38 to C36, J22 to J21, J23 to J22, J24 to J23, R29 to R24, R30 to R25, R31 to R26, R32 to R27, R33 to R28, U11 to U10, U10 to U9
