File: hardware/eval_board.sch (KiCad schematic (older format))
At the start: 0 parts

Commit message: update,
Connections:
- net labels removed: DAT, SCL, SDA
- wire segments 11 -> 0
Changed lines of the file:
@@
 $EndDescr
 $Sheet
-S 8200 7400 400  750
+S 12500 2700 400  750
 U 5CDAB790
 F0 "oled.sch" 50
 F1 "oled.sch" 50
-F2 "SDA" I R 8600 7600 50
-F3 "SCL" I R 8600 7500 50
-F4 "SS" I R 8600 7750 50
-F5 "SCK" I R 8600 7850 50
-F6 "MISO" I R 8600 7950 50
-F7 "MOSI" I R 8600 8050 50
+F2 "SDA" I L 12500 2900 50
+F3 "SCL" I L 12500 2800 50
+F4 "SS" I L 12500 3050 50
+F5 "SCK" I L 12500 3150 50
+F6 "MISO" I L 12500 3250 50
+F7 "MOSI" I L 12500 3350 50
 $EndSheet
 $Sheet
-S 8050 10850 550  400
+S 11200 7200 550  400
 U 5CDAB7F3
 F0 "ws2812" 50
 F1 "ws2812.sch" 50
-F2 "DAT" I R 8600 11100 50
+F2 "DAT" I L 11200 7450 50
 $EndSheet
 $Sheet
-S 7650 3250 550  400
+S 12500 2000 550  400
 U 5CDAB838
 F0 "i2c.sch" 50
 F1 "i2c.sch" 50
-F2 "SDA" I R 8200 3500 50
-F3 "SCL" I R 8200 3400 50
+F2 "SDA" I L 12500 2250 50
+F3 "SCL" I L 12500 2150 50
 $EndSheet
 $Sheet
-S 8050 10050 550  500
+S 12500 5200 550  500
 U 5CDAB83A
 F0 "spi.sch" 50
 F1 "spi.sch" 50
-F2 "SCK" I R 8600 10250 50
-F3 "MISO" I R 8600 10350 50
-F4 "MOSI" I R 8600 10450 50
-F5 "SS" I R 8600 10150 50
+F2 "SCK" I L 12500 5400 50
+F3 "MISO" I L 12500 5500 50
+F4 "MOSI" I L 12500 5600 50
+F5 "SS" I L 12500 5300 50
 $EndSheet
 $Sheet
-S 7500 1350 500  400
+S 11200 2850 500  400
 U 5CDAB850
 F0 "blinky" 50
 F1 "blinky.sch" 50
-F2 "TO_PC13" I R 8000 1500 50
+F2 "TO_PC13" I L 11200 3000 50
 $EndSheet
 $Sheet
@@
 $EndSheet
 $Sheet
-S 7150 5750 800  400
+S 11200 5650 800  400
 U 5CDAB9E4
 F0 "button" 50
 F1 "button.sch" 50
-F2 "BTN_PULL_UP" I R 7950 5900 50
-F3 "BTN_PULL_DN" I R 7950 6000 50
+F2 "BTN_PULL_UP" I L 11200 5800 50
+F3 "BTN_PULL_DN" I L 11200 5900 50
 $EndSheet
 $Sheet
-S 7450 4450 500  400
+S 11200 2000 500  400
 U 5CDB1CFA
 F0 "ADC" 50
 F1 "ADC.sch" 50
-F2 "V_VAR" I R 7950 4600 50
-F3 "V_TEMP" I R 7950 4700 50
+F2 "V_VAR" I L 11200 2150 50
+F3 "V_TEMP" I L 11200 2250 50
 $EndSheet
 $Sheet
-S 7200 1850 800  400
+S 11200 3750 800  400
 U 5CDB1D8D
 F0 "PWM" 50
 F1 "PWM.sch" 50
-F2 "STM32_PWM_OUT" I R 8000 2000 50
-F3 "STM32_PWM_IN" I R 8000 2100 50
+F2 "STM32_PWM_OUT" I L 11200 3900 50
+F3 "STM32_PWM_IN" I L 11200 4000 50
 $EndSheet
 $Sheet
-S 7400 4950 500  400
+S 11200 4700 500  400
 U 5CDB1F8F
 F0 "NEO-6M-0-001" 50
 F1 "NEO-6M-0-001.sch" 50
-F2 "UBLOX_TX" I R 7900 5100 50
-F3 "UBLOX_RX" I R 7900 5200 50
+F2 "UBLOX_TX" I L 11200 4850 50
+F3 "UBLOX_RX" I L 11200 4950 50
 $EndSheet
 $Sheet
-S 8050 9050 550  750
+S 12500 4000 550  750
 U 5CDB211F
 F0 "lora" 50
 F1 "lora.sch" 50
-F2 "MOSI" I R 8600 9700 50
-F3 "MISO" I R 8600 9600 50
-F4 "SCK" I R 8600 9500 50
-F5 "SS" I R 8600 9400 50
-F6 "RESET" I R 8600 9250 50
-F7 "DIO0" I R 8600 9150 50
+F2 "MOSI" I L 12500 4650 50
+F3 "MISO" I L 12500 4550 50
+F4 "SCK" I L 12500 4450 50
+F5 "SS" I L 12500 4350 50
+F6 "RESET" I L 12500 4200 50
+F7 "DIO0" I L 12500 4100 50
 $EndSheet
 $Sheet
@@
 $EndSheet
 $Sheet
-S 8100 8400 500  400
+S 11200 6450 500  400
 U 5CE4AEFB
 F0 "buzzer" 50
 F1 "buzzer.sch" 50
-F2 "BUZZER_IN" I R 8600 8650 50
+F2 "BUZZER_IN" I L 11200 6700 50
 $EndSheet
 $Sheet
-S 1050 2250 600  800
+S 5900 2000 600  1500
 U 5CE535D6
 F0 "arduino_nano" 50
 F1 "arduino_nano.sch" 50
-F2 "SCL" I R 1650 2400 50
-F3 "SDA" I R 1650 2500 50
-F4 "TXD" I R 1650 2800 50
-F5 "RXD" I R 1650 2900 50
+F2 "SCL" I R 6500 2150 50
+F3 "SDA" I R 6500 2250 50
+F4 "TXD" I R 6500 2400 50
+F5 "RXD" I R 6500 2500 50
+F6 "PWM" I R 6500 3100 50
+F7 "SS" I R 6500 2650 50
+F8 "SCK" I R 6500 2750 50
+F9 "MISO" I R 6500 2850 50
+F10 "MOSI" I R 6500 2950 50
+F11 "A_IN0" I R 6500 3250 50
+F12 "A_IN1" I R 6500 3350 50
 $EndSheet
 $Sheet
@@
 checklist:\n\ndebug terminal
 $Sheet
-S 1050 3300 612  400
+S 4400 2000 600  2300
 U 5CECA6C5
 F0 "nodemcu" 50
 F1 "nodemcu.sch" 50
-F2 "SDA" I R 1662 3550 50
-F3 "SCL" I R 1662 3450 50
+F2 "SDA" I R 5000 2250 50
+F3 "SCL" I R 5000 2150 50
+F4 "SDD0" I R 5000 2500 50
+F5 "SDD1" I R 5000 2600 50
+F6 "SDD2" I R 5000 2700 50
+F7 "SDD3" I R 5000 2800 50
+F8 "SDDCMD" I R 5000 2900 50
+F9 "SDDCLK" I R 5000 3000 50
+F10 "TX" I R 5000 3200 50
+F11 "RX" I R 5000 3300 50
+F12 "HSCLK" I R 5000 3500 50
+F13 "HMISO" I R 5000 3600 50
+F14 "HMOSI" I R 5000 3700 50
+F15 "HCS" I R 5000 3800 50
+F16 "PWM" I R 5000 4000 50
+F17 "A_IN_0" I R 5000 4100 50
 $EndSheet
-Entry Wire Line
-	9500 1350 9600 1450
-Entry Wire Line
-	9500 1450 9600 1550
-Entry Wire Line
-	9500 2000 9600 2100
-Entry Wire Line
-	9500 2100 9600 2200
-Entry Wire Line
-	9500 2100 9600 2200
-Wire Wire Line
-	8200 1350 9500 1350
-Wire Wire Line
-	8200 1450 9500 1450
-Wire Wire Line
-	8200 2000 9500 2000
-Wire Wire Line
-	8200 2100 9500 2100
-Text Label 8350 1350 0    50   ~ 0
-SCL
-Text Label 8350 1450 0    50   ~ 0
-SDA
-Text Label 8350 2000 0    50   ~ 0
-SCL
-Text Label 8350 2100 0    50   ~ 0
-SDA
-Entry Wire Line
-	9500 2750 9600 2850
-Entry Wire Line
-	9500 2850 9600 2950
-Entry Wire Line
-	9500 2850 9600 2950
-Wire Wire Line
-	8200 2750 9500 2750
-Wire Wire Line
-	8200 2850 9500 2850
-Text Label 8350 2750 0    50   ~ 0
-SCL
-Text Label 8350 2850 0    50   ~ 0
-SDA
-Entry Wire Line
-	9500 3400 9600 3500
-Entry Wire Line
-	9500 3500 9600 3600
-Entry Wire Line
-	9500 3500 9600 3600
-Wire Wire Line
-	8200 3400 9500 3400
-Wire Wire Line
-	8200 3500 9500 3500
-Text Label 8350 3400 0    50   ~ 0
-SCL
-Text Label 8350 3500 0    50   ~ 0
-SDA
-Entry Wire Line
-	9500 4050 9600 4150
-Entry Wire Line
-	9500 4150 9600 4250
-Entry Wire Line
-	9500 4150 9600 4250
-Wire Wire Line
-	8200 4050 9500 4050
-Wire Wire Line
-	8200 4150 9500 4150
-Text Label 8350 4050 0    50   ~ 0
-SCL
-Text Label 8350 4150 0    50   ~ 0
-SDA
-Wire Wire Line
-	8600 11100 9050 11100
-Text Label 8750 11100 0    50   ~ 0
-DAT
-Entry Wire Line
-	9050 11100 9150 11000
 $Sheet
-S 1000 800  650  1200
+S 2900 2000 600  1850
 U 5CDAB6B1
 F0 "bluepill" 50
 F1 "bluepill.sch" 50
-F2 "SDA" I R 1650 1050 50
-F3 "SCL" I R 1650 950 50
-F4 "SCK" I R 1650 1450 50
-F5 "MOSI" I R 1650 1350 50
-F6 "MISO" I R 1650 1250 50
-F7 "SS" I R 1650 1550 50
-F8 "TX" I R 1650 1750 50
-F9 "RX" I R 1650 1850 50
+F2 "SDA" I R 3500 2250 50
+F3 "SCL" I R 3500 2150 50
+F4 "SCK" I R 3500 2650 50
+F5 "MOSI" I R 3500 2550 50
+F6 "MISO" I R 3500 2450 50
+F7 "SS" I R 3500 2750 50
+F8 "TX" I R 3500 2950 50
+F9 "RX" I R 3500 3050 50
+F10 "A_IN0" I R 3500 3300 50
+F11 "A_IN1" I R 3500 3400 50
+F12 "PWM" I R 3500 3600 50
 $EndSheet
 $Sheet
-S 1050 3950 600  900
+S 14000 2000 600  900
 U 5D08041F
 F0 "sdio" 50
 F1 "sdio.sch" 50
-F2 "D0" I R 1650 4100 50
-F3 "D1" I R 1650 4200 50
-F4 "D2" I R 1650 4300 50
-F5 "D3" I R 1650 4400 50
-F6 "CLK" I R 1650 4600 50
-F7 "CMD" I R 1650 4700 50
+F2 "D0" I L 14000 2150 50
+F3 "D1" I L 14000 2250 50
+F4 "D2" I L 14000 2350 50
+F5 "D3" I L 14000 2450 50
+F6 "CLK" I L 14000 2650 50
+F7 "CMD" I L 14000 2750 50
 $EndSheet
-Wire Bus Line
-	9600 1450 9600 4750
 $EndSCHEMATC

Commit message: update,
Changed lines of the file:
@@
 $EndDescr
 $Sheet
-S 12500 2700 400  750
+S 12500 2700 550  750
 U 5CDAB790
 F0 "oled.sch" 50
@@
 $EndSheet
 $Sheet
-S 11200 7200 550  400
+S 10600 5750 550  400
 U 5CDAB7F3
 F0 "ws2812" 50
 F1 "ws2812.sch" 50
-F2 "DAT" I L 11200 7450 50
+F2 "DAT" I L 10600 6000 50
 $EndSheet
 $Sheet
 S 12500 2000 550  400
 U 5CDAB838
-F0 "i2c.sch" 50
-F1 "i2c.sch" 50
+F0 "LM75_i2c" 50
+F1 "LM75_i2c.sch" 50
 F2 "SDA" I L 12500 2250 50
 F3 "SCL" I L 12500 2150 50
@@
 $EndSheet
 $Sheet
-S 11200 2850 500  400
+S 10600 2850 500  400
 U 5CDAB850
 F0 "blinky" 50
 F1 "blinky.sch" 50
-F2 "TO_PC13" I L 11200 3000 50
+F2 "TO_PC13" I L 10600 3000 50
 $EndSheet
 $Sheet
@@
 $EndSheet
 $Sheet
-S 11200 5650 800  400
+S 10600 4200 800  400
 U 5CDAB9E4
 F0 "button" 50
 F1 "button.sch" 50
-F2 "BTN_PULL_UP" I L 11200 5800 50
-F3 "BTN_PULL_DN" I L 11200 5900 50
-$EndSheet
-$Sheet
-S 11200 2000 500  400
+F2 "BTN_PULL_UP" I L 10600 4350 50
+F3 "BTN_PULL_DN" I L 10600 4450 50
+$EndSheet
+$Sheet
+S 10600 2000 500  400
 U 5CDB1CFA
 F0 "ADC" 50
 F1 "ADC.sch" 50
-F2 "V_VAR" I L 11200 2150 50
-F3 "V_TEMP" I L 11200 2250 50
-$EndSheet
-$Sheet
-S 11200 3750 800  400
+F2 "V_VAR" I L 10600 2150 50
+F3 "V_TEMP" I L 10600 2250 50
+$EndSheet
+$Sheet
+S 10600 6400 800  400
 U 5CDB1D8D
 F0 "PWM" 50
 F1 "PWM.sch" 50
-F2 "STM32_PWM_OUT" I L 11200 3900 50
-F3 "STM32_PWM_IN" I L 11200 4000 50
-$EndSheet
-$Sheet
-S 11200 4700 500  400
+F2 "STM32_PWM_OUT" I L 10600 6550 50
+F3 "STM32_PWM_IN" I L 10600 6650 50
+$EndSheet
+$Sheet
+S 10600 3600 500  400
 U 5CDB1F8F
 F0 "NEO-6M-0-001" 50
 F1 "NEO-6M-0-001.sch" 50
-F2 "UBLOX_TX" I L 11200 4850 50
-F3 "UBLOX_RX" I L 11200 4950 50
+F2 "UBLOX_TX" I L 10600 3750 50
+F3 "UBLOX_RX" I L 10600 3850 50
 $EndSheet
 $Sheet
@@
 $EndSheet
 $Sheet
-S 11200 6450 500  400
+S 10600 5000 500  400
 U 5CE4AEFB
 F0 "buzzer" 50
 F1 "buzzer.sch" 50
-F2 "BUZZER_IN" I L 11200 6700 50
+F2 "BUZZER_IN" I L 10600 5250 50
 $EndSheet
 $Sheet
@@
 Wire Wire Line
 	6250 3350 6850 3350
+Connection ~ 6950 1400
+Wire Bus Line
+	6950 1400 11900 1400
+Text Label 10150 2150 0    50   ~ 0
+A_IN0
+Text Label 10150 2250 0    50   ~ 0
+A_IN1
+Text Label 10150 3000 0    50   ~ 0
+DEBUG_LED
+Text Label 10150 3750 0    50   ~ 0
+TX
+Text Label 10150 3850 0    50   ~ 0
+RX
+Text Label 10000 4350 0    50   ~ 0
+BTN_PULL_UP
+Text Label 10000 4450 0    50   ~ 0
+BTN_PULL_DN
+Text Label 10000 5250 0    50   ~ 0
+BUZZER_OUT
+Text Label 10000 6000 0    50   ~ 0
+WS2812_OUT
+Text Label 12200 2150 0    50   ~ 0
+SCL
+Text Label 12200 2250 0    50   ~ 0
+SDA
+Text Label 12050 2800 0    50   ~ 0
+SCL
+Text Label 12050 2900 0    50   ~ 0
+SDA
+Wire Wire Line
+	12000 2800 12500 2800
+Wire Wire Line
+	12500 2900 12000 2900
+Text Label 12050 3050 0    50   ~ 0
+OLED_SS
+Text Label 12050 3150 0    50   ~ 0
+OLED_SCK
+Text Label 12050 3250 0    50   ~ 0
+OLED_MISO
+Text Label 12050 3350 0    50   ~ 0
+OLED_MOSI
+Wire Wire Line
+	12000 3050 12500 3050
+Wire Wire Line
+	12000 3150 12500 3150
+Wire Wire Line
+	12000 3250 12500 3250
+Wire Wire Line
+	12000 3350 12500 3350
+Text Label 12050 4350 0    50   ~ 0
+LORA_SS
+Text Label 12050 4450 0    50   ~ 0
+SCK
+Text Label 12050 4550 0    50   ~ 0
+MISO
+Text Label 12050 4650 0    50   ~ 0
+MOSI
+Text Label 12050 5300 0    50   ~ 0
+W25_SS
+Text Label 12050 5400 0    50   ~ 0
+SCK
+Text Label 12050 5500 0    50   ~ 0
+MISO
+Text Label 12050 5600 0    50   ~ 0
+MOSI
+Entry Wire Line
+	11900 5200 12000 5300
+Entry Wire Line
+	11900 5300 12000 5400
+Entry Wire Line
+	11900 5400 12000 5500
+Entry Wire Line
+	11900 5500 12000 5600
+Wire Wire Line
+	12000 5300 12500 5300
+Wire Wire Line
+	12000 5400 12500 5400
+Wire Wire Line
+	12000 5500 12500 5500
+Wire Wire Line
+	12000 5600 12500 5600
+Entry Wire Line
+	11900 4250 12000 4350
+Entry Wire Line
+	11900 4350 12000 4450
+Entry Wire Line
+	11900 4450 12000 4550
+Entry Wire Line
+	11900 4550 12000 4650
+Wire Wire Line
+	12000 4350 12500 4350
+Wire Wire Line
+	12000 4450 12500 4450
+Wire Wire Line
+	12000 4550 12500 4550
+Wire Wire Line
+	12000 4650 12500 4650
+Entry Wire Line
+	11900 2950 12000 3050
+Entry Wire Line
+	11900 3050 12000 3150
+Entry Wire Line
+	11900 3150 12000 3250
+Entry Wire Line
+	11900 3250 12000 3350
+Entry Wire Line
+	11900 2700 12000 2800
+Entry Wire Line
+	11900 2800 12000 2900
+Entry Wire Line
+	11900 2050 12000 2150
+Entry Wire Line
+	11900 2150 12000 2250
+Wire Wire Line
+	12000 2150 12500 2150
+Wire Wire Line
+	12000 2250 12500 2250
+Connection ~ 11900 1400
+Wire Bus Line
+	11900 1400 13450 1400
 Wire Bus Line
 	13450 1400 13450 2650
@@
 	6950 1400 6950 3250
 Wire Bus Line
+	11900 1400 11900 5500
+Wire Bus Line
 	5450 1400 5450 4000
-Connection ~ 6950 1400
-Wire Bus Line
-	6950 1400 13450 1400
 $EndSCHEMATC

Commit message: update,
Changed lines of the file:
@@
 F0 "PWM" 50
 F1 "PWM.sch" 50
-F2 "STM32_PWM_OUT" I L 10600 6550 50
-F3 "STM32_PWM_IN" I L 10600 6650 50
+F2 "STM32_PWM_OUT" I R 11400 6650 50
+F3 "STM32_PWM_IN" I L 10600 6550 50
 $EndSheet
 $Sheet
@@
 F15 "HCS" I R 4900 3800 50
 F16 "PWM" I R 4900 4000 50
-F17 "A_IN_0" I R 4900 4100 50
+F17 "A_IN0" I R 4900 4100 50
 $EndSheet
 $Sheet
@@
 MOSI
 Text Label 5300 3800 2    50   ~ 0
-SS_NODE
+SS_ESP
 Text Label 6750 2650 2    50   ~ 0
 SS_ARDUINO
@@
 Connection ~ 6950 1400
 Wire Bus Line
-	6950 1400 11900 1400
+	6950 1400 9850 1400
 Text Label 10150 2150 0    50   ~ 0
 A_IN0
@@
 Wire Bus Line
 	11900 1400 13450 1400
+Text Label 10000 6550 0    50   ~ 0
+PWM_IN
+Entry Wire Line
+	9850 6450 9950 6550
+Wire Wire Line
+	10600 6550 9950 6550
+Connection ~ 9850 1400
+Wire Bus Line
+	9850 1400 11900 1400
+Entry Wire Line
+	9850 5900 9950 6000
+Wire Wire Line
+	9950 6000 10600 6000
+Entry Wire Line
+	9850 5150 9950 5250
+Entry Wire Line
+	9850 4250 9950 4350
+Entry Wire Line
+	9850 4350 9950 4450
+Entry Wire Line
+	9850 3650 9950 3750
+Entry Wire Line
+	9850 3750 9950 3850
+Entry Wire Line
+	9850 2900 9950 3000
+Entry Wire Line
+	9850 2050 9950 2150
+Entry Wire Line
+	9850 2150 9950 2250
+Wire Wire Line
+	9950 2150 10600 2150
+Wire Wire Line
+	9950 2250 10600 2250
+Wire Wire Line
+	9950 3000 10600 3000
+Wire Wire Line
+	9950 3750 10600 3750
+Wire Wire Line
+	9950 3850 10600 3850
+Wire Wire Line
+	10600 4350 9950 4350
+Wire Wire Line
+	9950 4450 10600 4450
+Wire Wire Line
+	9950 5250 10600 5250
 Wire Bus Line
 	13450 1400 13450 2650
@@
 	11900 1400 11900 5500
 Wire Bus Line
+	9850 1400 9850 6450
+Wire Bus Line
 	5450 1400 5450 4000

Commit message: update,
Connections:
- net labels removed: OLED_MOSI, OLED_SCK
Changed lines of the file:
@@
 $EndSheet
 $Sheet
-S 2750 2000 600  2150
+S 2500 2000 718  2150
 U 5CDAB6B1
 F0 "bluepill" 50
 F1 "bluepill.sch" 50
-F2 "SDA" I R 3350 2250 50
-F3 "SCL" I R 3350 2150 50
-F4 "SCK" I R 3350 2650 50
-F5 "MOSI" I R 3350 2550 50
-F6 "MISO" I R 3350 2450 50
-F7 "SS" I R 3350 2750 50
-F8 "TX" I R 3350 2950 50
-F9 "RX" I R 3350 3050 50
-F10 "A_IN0" I R 3350 3300 50
-F11 "A_IN1" I R 3350 3400 50
-F12 "PWM" I R 3350 3600 50
-F13 "WS2812_OUT" I R 3350 3850 50
+F2 "SDA" I R 3218 2250 50
+F3 "SCL" I R 3218 2150 50
+F4 "SCK" I R 3218 2650 50
+F5 "MOSI" I R 3218 2550 50
+F6 "MISO" I R 3218 2450 50
+F7 "SS" I R 3218 2750 50
+F8 "TX" I R 3218 2950 50
+F9 "RX" I R 3218 3050 50
+F10 "A_IN0" I R 3218 3300 50
+F11 "A_IN1" I R 3218 3400 50
+F12 "PWM" I R 3218 3600 50
+F13 "WS2812_OUT" I R 3218 3850 50
 $EndSheet
 $Sheet
@@
 F7 "CMD" I L 14000 2750 50
 $EndSheet
-Text Label 3750 2150 2    50   ~ 0
+Text Label 3600 2150 2    50   ~ 0
 SCL
-Text Label 3750 2250 2    50   ~ 0
+Text Label 3600 2250 2    50   ~ 0
 SDA
 Text Label 5300 2150 2    50   ~ 0
@@
 Text Label 6750 2250 2    50   ~ 0
 SDA
-Text Label 3750 2950 2    50   ~ 0
+Text Label 3600 2950 2    50   ~ 0
 TX
-Text Label 3750 3050 2    50   ~ 0
+Text Label 3600 3050 2    50   ~ 0
 RX
 Text Label 5300 3200 2    50   ~ 0
@@
 Text Label 6750 2500 2    50   ~ 0
 RX
-Text Label 3750 2450 2    50   ~ 0
+Text Label 3600 2450 2    50   ~ 0
 MISO
-Text Label 3750 2550 2    50   ~ 0
+Text Label 3600 2550 2    50   ~ 0
 MOSI
-Text Label 3750 2650 2    50   ~ 0
+Text Label 3600 2650 2    50   ~ 0
 SCK
-Text Label 3750 2750 2    50   ~ 0
+Text Label 3600 2750 2    50   ~ 0
 SS_STM32
 Text Label 5300 3500 2    50   ~ 0
@@
 Text Label 6750 2950 2    50   ~ 0
 MOSI
-Text Label 3750 3600 2    50   ~ 0
+Text Label 3600 3600 2    50   ~ 0
 PWM
 Text Label 5300 4000 2    50   ~ 0
@@
 Text Label 6750 3100 2    50   ~ 0
 PWM
-Text Label 3750 3300 2    50   ~ 0
+Text Label 3600 3300 2    50   ~ 0
 A_IN0
 Text Label 5300 4100 2    50   ~ 0
@@
 Text Label 6750 3250 2    50   ~ 0
 A_IN0
-Text Label 3750 3400 2    50   ~ 0
+Text Label 3600 3400 2    50   ~ 0
 A_IN1
 Text Label 6750 3350 2    50   ~ 0
@@
 	13550 2750 14000 2750
 Entry Wire Line
-	3850 2150 3950 2050
-Entry Wire Line
-	3950 2150 3850 2250
-Entry Wire Line
-	3950 2350 3850 2450
-Entry Wire Line
-	3950 2450 3850 2550
-Entry Wire Line
-	3950 2550 3850 2650
-Entry Wire Line
-	3950 2650 3850 2750
-Entry Wire Line
-	3950 2850 3850 2950
-Entry Wire Line
-	3950 2950 3850 3050
-Entry Wire Line
-	3950 3200 3850 3300
-Entry Wire Line
-	3950 3300 3850 3400
-Entry Wire Line
-	3950 3500 3850 3600
-Wire Wire Line
-	3350 2150 3850 2150
-Wire Wire Line
-	3350 2250 3850 2250
-Wire Wire Line
-	3350 2450 3850 2450
-Wire Wire Line
-	3350 2550 3850 2550
-Wire Wire Line
-	3350 2650 3850 2650
-Wire Wire Line
-	3350 2750 3850 2750
-Wire Wire Line
-	3350 2950 3850 2950
-Wire Wire Line
-	3350 3050 3850 3050
-Wire Wire Line
-	3350 3300 3850 3300
-Wire Wire Line
-	3350 3400 3850 3400
-Wire Wire Line
-	3350 3600 3850 3600
+	3700 2150 3800 2050
+Entry Wire Line
+	3800 2150 3700 2250
+Entry Wire Line
+	3800 2350 3700 2450
+Entry Wire Line
+	3800 2450 3700 2550
+Entry Wire Line
+	3800 2550 3700 2650
+Entry Wire Line
+	3800 2650 3700 2750
+Entry Wire Line
+	3800 2850 3700 2950
+Entry Wire Line
+	3800 2950 3700 3050
+Entry Wire Line
+	3800 3200 3700 3300
+Entry Wire Line
+	3800 3300 3700 3400
+Entry Wire Line
+	3800 3500 3700 3600
+Wire Wire Line
+	3200 2150 3700 2150
+Wire Wire Line
+	3200 2250 3700 2250
+Wire Wire Line
+	3200 2450 3700 2450
+Wire Wire Line
+	3200 2550 3700 2550
+Wire Wire Line
+	3200 2650 3700 2650
+Wire Wire Line
+	3200 2750 3700 2750
+Wire Wire Line
+	3200 2950 3700 2950
+Wire Wire Line
+	3200 3050 3700 3050
+Wire Wire Line
+	3200 3300 3700 3300
+Wire Wire Line
+	3200 3400 3700 3400
+Wire Wire Line
+	3200 3600 3700 3600
 Wire Bus Line
-	3950 1400 5450 1400
+	3800 1400 5450 1400
 Entry Wire Line
 	5350 4100 5450 4000
@@
 Wire Wire Line
 	12500 2900 12000 2900
-Text Label 12050 3050 0    50   ~ 0
-OLED_SS
 Text Label 12050 3150 0    50   ~ 0
-OLED_SCK
+SCK
 Text Label 12050 3250 0    50   ~ 0
-OLED_MOSI
+MOSI
 Wire Wire Line
 	12000 3050 12500 3050
@@
 Wire Wire Line
 	12000 3250 12500 3250
-Text Label 3800 3850 2    50   ~ 0
+Text Label 3650 3850 2    50   ~ 0
 WS2812_OUT
 Entry Wire Line
-	3850 3850 3950 3750
-Wire Wire Line
-	3350 3850 3850 3850
+	3700 3850 3800 3750
+Wire Wire Line
+	3200 3850 3700 3850
+Text Label 12050 3050 0    50   ~ 0
+OLED_SS
 Wire Bus Line
 	13450 1400 13450 2650
 Wire Bus Line
-	3950 1400 3950 3750
+	3800 1400 3800 3750
 Wire Bus Line
 	6950 1400 6950 3250

Commit message: update,
Connections:
- wire segments 72 -> 75
Changed lines of the file:
@@
-$EndSheet
-$Sheet
-S 2500 2000 718  2150
-U 5CDAB6B1
-F0 "bluepill" 50
-F1 "bluepill.sch" 50
-F2 "SDA" I R 3218 2250 50
-F3 "SCL" I R 3218 2150 50
-F4 "SCK" I R 3218 2650 50
-F5 "MOSI" I R 3218 2550 50
-F6 "MISO" I R 3218 2450 50
-F7 "SS" I R 3218 2750 50
-F8 "TX" I R 3218 2950 50
-F9 "RX" I R 3218 3050 50
-F10 "A_IN0" I R 3218 3300 50
-F11 "A_IN1" I R 3218 3400 50
-F12 "PWM" I R 3218 3600 50
-F13 "WS2812_OUT" I R 3218 3850 50
 $EndSheet
 $Sheet
@@
 Text Label 12050 3050 0    50   ~ 0
 OLED_SS
+$Sheet
+S 2500 2000 700  3000
+U 5CDAB6B1
+F0 "bluepill" 50
+F1 "bluepill.sch" 50
+F2 "SDA" I R 3200 2250 50
+F3 "SCL" I R 3200 2150 50
+F4 "SCK" I R 3200 2650 50
+F5 "MOSI" I R 3200 2550 50
+F6 "MISO" I R 3200 2450 50
+F7 "SS" I R 3200 2750 50
+F8 "TX" I R 3200 2950 50
+F9 "RX" I R 3200 3050 50
+F10 "A_IN0" I R 3200 3300 50
+F11 "A_IN1" I R 3200 3400 50
+F12 "PWM" I R 3200 3600 50
+F13 "WS2812_OUT" I R 3200 3850 50
+F14 "OLED_DC" I R 3200 4150 50
+F15 "OLED_RST" I R 3200 4250 50
+F16 "OLED_SS" I R 3200 4350 50
+$EndSheet
+Text Label 3650 4150 2    50   ~ 0
+OLED_DC
+Text Label 3650 4250 2    50   ~ 0
+OLED_RST
+Text Label 3650 4350 2    50   ~ 0
+OLED_SS
+Entry Wire Line
+	3700 4150 3800 4050
+Entry Wire Line
+	3700 4250 3800 4150
+Entry Wire Line
+	3700 4350 3800 4250
+Wire Wire Line
+	3200 4150 3700 4150
+Wire Wire Line
+	3200 4250 3700 4250
+Wire Wire Line
+	3200 4350 3700 4350
 Wire Bus Line
 	13450 1400 13450 2650
-Wire Bus Line
-	3800 1400 3800 3750
 Wire Bus Line
 	6950 1400 6950 3250
@@
 	9850 1400 9850 6450
 Wire Bus Line
+	3800 1400 3800 4250
+Wire Bus Line
 	5450 1400 5450 4000

Commit message: update,
Changed lines of the file:
@@
 F15 "OLED_RST" I R 3200 4250 50
 F16 "OLED_SS" I R 3200 4350 50
+F17 "DEBUG_LED" I R 3200 4550 50
 $EndSheet
 Text Label 3650 4150 2    50   ~ 0
@@
 Wire Wire Line
 	3200 4350 3700 4350
+Text Label 3650 4550 2    50   ~ 0
+DEBUG_LED
+Entry Wire Line
+	3700 4550 3800 4450
+Wire Wire Line
+	3200 4550 3700 4550
 Wire Bus Line
 	13450 1400 13450 2650
@@
 	9850 1400 9850 6450
 Wire Bus Line
-	3800 1400 3800 4250
+	3800 1400 3800 4450
 Wire Bus Line
 	5450 1400 5450 4000
