File: hardware/blinky.sch (KiCad schematic (older format))
At the start: 0 parts

Commit message: update,
Parts:
- added D?: LED_GREEN,0603, footprint-lib:LED_0603_1608Metric, symbol taobao-led:LED_GREEN,0603
- added R?: R471,0603, Resistor_SMD:R_0603_1608Metric_Pad1.05x0.95mm_HandSolder, symbol taobao-r:R471,0603
Connections:
- new net: D?.2 (A), R?.2
- new net +3V3: R?.1
- new net TO_PC13: D?.1 (K)
Other:
- note removed: "debug led\nPC13"
Changed lines of the file:
@@
 EELAYER 29 0
 EELAYER END
-$Descr A4 11693 8268
+$Descr User 8500 5500
 encoding utf-8
-Sheet 13 22
+Sheet 9 22
 Title ""
 Date ""
@@
 Comment4 ""
 $EndDescr
-Text Notes 650  950  0    50   ~ 0
-debug led\nPC13
 $Bitmap
-Pos -800 1150
+Pos -700 2250
 Scale 1.000000
 Data
@@
 EndData
 $EndBitmap
+$Comp
+L power:+3V3 #PWR?
+U 1 1 5CE6E1A4
+P 2550 1750
+F 0 "#PWR?" H 2550 1600 50  0001 C CNN
+F 1 "+3V3" H 2600 1950 50  0000 C CNN
+F 2 "" H 2550 1750 50  0001 C CNN
+F 3 "" H 2550 1750 50  0001 C CNN
+	1    2550 1750
+	1    0    0    -1
+$EndComp
+$Comp
+L taobao-r:R471,0603 R?
+U 1 1 5CE6E5A4
+P 2550 2100
+F 0 "R?" H 2650 2150 50  0000 L CNN
+F 1 "R471,0603" H 2650 2100 50  0000 L CNN
+F 2 "Resistor_SMD:R_0603_1608Metric_Pad1.05x0.95mm_HandSolder" H 2550 2100 50  0001 C CNN
+F 3 "~" H 2550 2100 50  0001 C CNN
+	1    2550 2100
+	1    0    0    -1
+$EndComp
+$Comp
+L taobao-led:LED_GREEN,0603 D?
+U 1 1 5CE6E983
+P 2550 2400
+F 0 "D?" V 2600 2300 50  0000 R CNN
+F 1 "LED_GREEN,0603" V 2550 2300 50  0000 R CNN
+F 2 "footprint-lib:LED_0603_1608Metric" V 2550 2400 50  0001 C CNN
+F 3 "" V 2550 2400 50  0001 C CNN
+	1    2550 2400
+	0    -1   -1   0
+$EndComp
+Text HLabel 2850 2600 2    50   Input ~ 0
+TO_PC13
+Wire Wire Line
+	2550 1750 2550 2000
+Wire Wire Line
+	2550 2200 2550 2300
+Wire Wire Line
+	2550 2500 2550 2600
+Wire Wire Line
+	2550 2600 2850 2600
 $EndSCHEMATC

Commit message: update,
Parts:
- gave numbers to parts that had none: 2
Changed lines of the file:
@@
 $Descr User 8500 5500
 encoding utf-8
-Sheet 9 27
+Sheet 6 20
 Title ""
 Date ""
@@
 $EndBitmap
 $Comp
-L power:+3V3 #PWR?
+L power:+3V3 #PWR035
 U 1 1 5CE6E1A4
 P 2550 1750
-F 0 "#PWR?" H 2550 1600 50  0001 C CNN
+F 0 "#PWR035" H 2550 1600 50  0001 C CNN
 F 1 "+3V3" H 2600 1950 50  0000 C CNN
 F 2 "" H 2550 1750 50  0001 C CNN
@@
 $EndComp
 $Comp
-L taobao-r:R471,0603 R?
+L taobao-r:R471,0603 R7
 U 1 1 5CE6E5A4
 P 2550 2100
-F 0 "R?" H 2650 2150 50  0000 L CNN
+F 0 "R7" H 2650 2150 50  0000 L CNN
 F 1 "R471,0603" H 2650 2100 50  0000 L CNN
 F 2 "Resistor_SMD:R_0603_1608Metric_Pad1.05x0.95mm_HandSolder" H 2550 2100 50  0001 C CNN
@@
 $EndComp
 $Comp
-L taobao-led:LED_GREEN,0603 D?
+L taobao-led:LED_GREEN,0603 D6
 U 1 1 5CE6E983
 P 2550 2400
-F 0 "D?" V 2600 2300 50  0000 R CNN
+F 0 "D6" V 2600 2300 50  0000 R CNN
 F 1 "LED_GREEN,0603" V 2550 2300 50  0000 R CNN
 F 2 "footprint-lib:LED_0603_1608Metric" V 2550 2400 50  0001 C CNN

Commit message: update,
Parts:
- renumbered R7 to R2
Changed lines of the file:
@@
 $Descr User 8500 5500
 encoding utf-8
-Sheet 6 20
+Sheet 5 20
 Title ""
 Date ""
@@
 $EndBitmap
 $Comp
-L power:+3V3 #PWR035
+L power:+3V3 #PWR028
 U 1 1 5CE6E1A4
 P 2550 1750
-F 0 "#PWR035" H 2550 1600 50  0001 C CNN
+F 0 "#PWR028" H 2550 1600 50  0001 C CNN
 F 1 "+3V3" H 2600 1950 50  0000 C CNN
 F 2 "" H 2550 1750 50  0001 C CNN
@@
 $EndComp
 $Comp
-L taobao-r:R471,0603 R7
+L taobao-r:R471,0603 R2
 U 1 1 5CE6E5A4
 P 2550 2100
-F 0 "R7" H 2650 2150 50  0000 L CNN
+F 0 "R2" H 2650 2150 50  0000 L CNN
 F 1 "R471,0603" H 2650 2100 50  0000 L CNN
 F 2 "Resistor_SMD:R_0603_1608Metric_Pad1.05x0.95mm_HandSolder" H 2550 2100 50  0001 C CNN
