File: hardware/sdio.sch (KiCad schematic (older format))
At the start: 0 parts

Commit message: update,
Other:
- note removed: "sdcard"
Changed lines of the file:
@@
 Comment4 ""
 $EndDescr
-Text Notes 650  950  0    50   ~ 0
-sdcard
 $EndSCHEMATC

Commit message: update,
Parts:
- added C?: C475,0805, Capacitor_SMD:C_0603_1608Metric_Pad1.05x0.95mm_HandSolder, symbol taobao-c:C475,0603
- added J?: sdcard_header, footprint-lib:SDCARD_HEADER, symbol Connector:Conn_01x10_Female
- added RN? (x2): R_Pack04, Resistor_SMD:R_Array_Concave_4x0603, symbol Device:R_Pack04
- added SDC?: TF_CARD_SOCKET,SELF_EJECT, footprint-lib:SUNTECH_ST-TF-003A, symbol taobao-components:TF_CARD_SOCKET,SELF_EJECT
Connections:
- new net: J?.9 (Pin_9), SDC?.9 (CARD_DET)
- new net +3V3: C?.1, J?.4 (Pin_4), RN?.5 (R4.2), RN?.5 (R4.2), RN?.6 (R3.2), RN?.6 (R3.2), RN?.7 (R2.2), RN?.7 (R2.2), RN?.8 (R1.2), RN?.8 (R1.2), SDC?.4 (VDD)
- new net CLK: J?.5 (Pin_5), RN?.2 (R2.1), SDC?.5 (CLK)
- new net CMD: J?.3 (Pin_3), RN?.4 (R4.1), SDC?.3 (CMD)
- new net D0: J?.7 (Pin_7), RN?.2 (R2.1), SDC?.7 (DAT0)
- new net D1: J?.8 (Pin_8), RN?.1 (R1.1), SDC?.8 (CAT1)
- new net D2: J?.1 (Pin_1), RN?.4 (R4.1), SDC?.1 (DAT2)
- new net D3: J?.2 (Pin_2), RN?.3 (R3.1), SDC?.2 (CD/DAT3)
- new net GND: C?.2, J?.10 (Pin_10), J?.6 (Pin_6), SDC?.10 (GND), SDC?.6 (VSS)

Commit message: update,
Parts:
- gave numbers to parts that had none: 5
Changed lines of the file:
@@
 AR Path="/5BE65513/5C29852B" Ref="#PWR?"  Part="1"
 AR Path="/5C19BBA6/5C1A1380/5C29852B" Ref="#PWR?"  Part="1"
-AR Path="/5D08041F/5C29852B" Ref="#PWR?"  Part="1"
-F 0 "#PWR?" H 3050 1000 50  0001 C CNN
+AR Path="/5D08041F/5C29852B" Ref="#PWR0160"  Part="1"
+F 0 "#PWR0160" H 3050 1000 50  0001 C CNN
 F 1 "+3V3" H 3065 1323 50  0000 C CNN
 F 2 "" H 3050 1150 50  0001 C CNN
@@
 AR Path="/5BE65513/5C298562" Ref="#PWR?"  Part="1"
 AR Path="/5C19BBA6/5C1A1380/5C298562" Ref="#PWR?"  Part="1"
-AR Path="/5D08041F/5C298562" Ref="#PWR?"  Part="1"
-F 0 "#PWR?" H 5750 2900 50  0001 C CNN
+AR Path="/5D08041F/5C298562" Ref="#PWR0165"  Part="1"
+F 0 "#PWR0165" H 5750 2900 50  0001 C CNN
 F 1 "GND" V 5755 3022 50  0000 R CNN
 F 2 "" H 5750 3150 50  0001 C CNN
@@
 AR Path="/5BE65513/5C29856D" Ref="#PWR?"  Part="1"
 AR Path="/5C19BBA6/5C1A1380/5C29856D" Ref="#PWR?"  Part="1"
-AR Path="/5D08041F/5C29856D" Ref="#PWR?"  Part="1"
-F 0 "#PWR?" H 5600 2900 50  0001 C CNN
+AR Path="/5D08041F/5C29856D" Ref="#PWR0164"  Part="1"
+F 0 "#PWR0164" H 5600 2900 50  0001 C CNN
 F 1 "GND" H 5605 2977 50  0000 C CNN
 F 2 "" H 5600 3150 50  0001 C CNN
@@
 AR Path="/5BE65513/5BEBAC6E" Ref="C?"  Part="1"
 AR Path="/5C19BBA6/5C1A1380/5BEBAC6E" Ref="C?"  Part="1"
-AR Path="/5D08041F/5BEBAC6E" Ref="C?"  Part="1"
-F 0 "C?" H 6292 1846 50  0000 L CNN
+AR Path="/5D08041F/5BEBAC6E" Ref="C39"  Part="1"
+F 0 "C39" H 6292 1846 50  0000 L CNN
 F 1 "C475,0805" H 6292 1755 50  0000 L CNN
 F 2 "Capacitor_SMD:C_0603_1608Metric_Pad1.05x0.95mm_HandSolder" H 6200 1800 50  0001 C CNN
@@
 AR Path="/5BE65513/5BEBAC74" Ref="#PWR?"  Part="1"
 AR Path="/5C19BBA6/5C1A1380/5BEBAC74" Ref="#PWR?"  Part="1"
-AR Path="/5D08041F/5BEBAC74" Ref="#PWR?"  Part="1"
-F 0 "#PWR?" H 6500 1550 50  0001 C CNN
+AR Path="/5D08041F/5BEBAC74" Ref="#PWR0163"  Part="1"
+F 0 "#PWR0163" H 6500 1550 50  0001 C CNN
 F 1 "GND" H 6505 1627 50  0000 C CNN
 F 2 "" H 6500 1800 50  0001 C CNN
@@
 AR Path="/5BE65513/5BEBB902" Ref="#PWR?"  Part="1"
 AR Path="/5C19BBA6/5C1A1380/5BEBB902" Ref="#PWR?"  Part="1"
-AR Path="/5D08041F/5BEBB902" Ref="#PWR?"  Part="1"
-F 0 "#PWR?" H 6000 1650 50  0001 C CNN
+AR Path="/5D08041F/5BEBB902" Ref="#PWR0162"  Part="1"
+F 0 "#PWR0162" H 6000 1650 50  0001 C CNN
 F 1 "+3V3" H 6015 1973 50  0000 C CNN
 F 2 "" H 6000 1800 50  0001 C CNN
@@
 AR Path="/5BE639C4/5BF8FC76" Ref="SDC?"  Part="1"
 AR Path="/5C19BBA6/5C1A1380/5BF8FC76" Ref="SDC?"  Part="1"
-AR Path="/5D08041F/5BF8FC76" Ref="SDC?"  Part="1"
-F 0 "SDC?" H 6750 2550 50  0000 L CNN
+AR Path="/5D08041F/5BF8FC76" Ref="SDC1"  Part="1"
+F 0 "SDC1" H 6750 2550 50  0000 L CNN
 F 1 "TF_CARD_SOCKET,SELF_EJECT" H 6750 2500 50  0000 L CNN
 F 2 "footprint-lib:SUNTECH_ST-TF-003A" H 6000 2500 50  0001 C CNN
@@
 	5300 2150 5800 2150
 $Comp
-L Connector:Conn_01x10_Female J?
+L Connector:Conn_01x10_Female J31
 U 1 1 5D089C8E
 P 5000 3350
-F 0 "J?" V 5100 3300 50  0000 C CNN
+F 0 "J31" V 5100 3300 50  0000 C CNN
 F 1 "sdcard_header" V 5200 3300 50  0000 C CNN
 F 2 "footprint-lib:SDCARD_HEADER" H 5000 3350 50  0001 C CNN
@@
 Connection ~ 5600 2950
 $Comp
-L Device:R_Pack04 RN?
+L Device:R_Pack04 RN4
 U 1 1 5D09497F
 P 3500 1500
-F 0 "RN?" H 3700 1550 50  0000 L CNN
+F 0 "RN4" H 3700 1550 50  0000 L CNN
 F 1 "R_Pack04" H 3700 1500 50  0000 L CNN
 F 2 "Resistor_SMD:R_Array_Concave_4x0603" V 3775 1500 50  0001 C CNN
@@
 	5750 3150 5750 2550
 $Comp
-L Device:R_Pack04 RN?
+L Device:R_Pack04 RN5
 U 1 1 5D09B375
 P 4000 1500
-F 0 "RN?" H 4200 1550 50  0000 L CNN
+F 0 "RN5" H 4200 1550 50  0000 L CNN
 F 1 "R_Pack04" H 4200 1500 50  0000 L CNN
 F 2 "Resistor_SMD:R_Array_Concave_4x0603" V 4275 1500 50  0001 C CNN
@@
 AR Path="/5BE65513/5D0FA3F5" Ref="#PWR?"  Part="1"
 AR Path="/5C19BBA6/5C1A1380/5D0FA3F5" Ref="#PWR?"  Part="1"
-AR Path="/5D08041F/5D0FA3F5" Ref="#PWR?"  Part="1"
-F 0 "#PWR?" H 4650 1000 50  0001 C CNN
+AR Path="/5D08041F/5D0FA3F5" Ref="#PWR0161"  Part="1"
+F 0 "#PWR0161" H 4650 1000 50  0001 C CNN
 F 1 "+3V3" H 4665 1323 50  0000 C CNN
 F 2 "" H 4650 1150 50  0001 C CNN

Commit message: update,
Parts:
- renumbered C39 to C37, J31 to J28, RN4 to RN2, RN5 to RN3
Changed lines of the file:
@@
 AR Path="/5BE65513/5C29852B" Ref="#PWR?"  Part="1"
 AR Path="/5C19BBA6/5C1A1380/5C29852B" Ref="#PWR?"  Part="1"
-AR Path="/5D08041F/5C29852B" Ref="#PWR0160"  Part="1"
-F 0 "#PWR0160" H 3050 1000 50  0001 C CNN
+AR Path="/5D08041F/5C29852B" Ref="#PWR0141"  Part="1"
+F 0 "#PWR0141" H 3050 1000 50  0001 C CNN
 F 1 "+3V3" H 3065 1323 50  0000 C CNN
 F 2 "" H 3050 1150 50  0001 C CNN
@@
 AR Path="/5BE65513/5C298562" Ref="#PWR?"  Part="1"
 AR Path="/5C19BBA6/5C1A1380/5C298562" Ref="#PWR?"  Part="1"
-AR Path="/5D08041F/5C298562" Ref="#PWR0165"  Part="1"
-F 0 "#PWR0165" H 5750 2900 50  0001 C CNN
+AR Path="/5D08041F/5C298562" Ref="#PWR0146"  Part="1"
+F 0 "#PWR0146" H 5750 2900 50  0001 C CNN
 F 1 "GND" V 5755 3022 50  0000 R CNN
 F 2 "" H 5750 3150 50  0001 C CNN
@@
 AR Path="/5BE65513/5C29856D" Ref="#PWR?"  Part="1"
 AR Path="/5C19BBA6/5C1A1380/5C29856D" Ref="#PWR?"  Part="1"
-AR Path="/5D08041F/5C29856D" Ref="#PWR0164"  Part="1"
-F 0 "#PWR0164" H 5600 2900 50  0001 C CNN
+AR Path="/5D08041F/5C29856D" Ref="#PWR0145"  Part="1"
+F 0 "#PWR0145" H 5600 2900 50  0001 C CNN
 F 1 "GND" H 5605 2977 50  0000 C CNN
 F 2 "" H 5600 3150 50  0001 C CNN
@@
 AR Path="/5BE65513/5BEBAC6E" Ref="C?"  Part="1"
 AR Path="/5C19BBA6/5C1A1380/5BEBAC6E" Ref="C?"  Part="1"
-AR Path="/5D08041F/5BEBAC6E" Ref="C39"  Part="1"
-F 0 "C39" H 6292 1846 50  0000 L CNN
+AR Path="/5D08041F/5BEBAC6E" Ref="C37"  Part="1"
+F 0 "C37" H 6292 1846 50  0000 L CNN
 F 1 "C475,0805" H 6292 1755 50  0000 L CNN
 F 2 "Capacitor_SMD:C_0603_1608Metric_Pad1.05x0.95mm_HandSolder" H 6200 1800 50  0001 C CNN
@@
 AR Path="/5BE65513/5BEBAC74" Ref="#PWR?"  Part="1"
 AR Path="/5C19BBA6/5C1A1380/5BEBAC74" Ref="#PWR?"  Part="1"
-AR Path="/5D08041F/5BEBAC74" Ref="#PWR0163"  Part="1"
-F 0 "#PWR0163" H 6500 1550 50  0001 C CNN
+AR Path="/5D08041F/5BEBAC74" Ref="#PWR0144"  Part="1"
+F 0 "#PWR0144" H 6500 1550 50  0001 C CNN
 F 1 "GND" H 6505 1627 50  0000 C CNN
 F 2 "" H 6500 1800 50  0001 C CNN
@@
 AR Path="/5BE65513/5BEBB902" Ref="#PWR?"  Part="1"
 AR Path="/5C19BBA6/5C1A1380/5BEBB902" Ref="#PWR?"  Part="1"
-AR Path="/5D08041F/5BEBB902" Ref="#PWR0162"  Part="1"
-F 0 "#PWR0162" H 6000 1650 50  0001 C CNN
+AR Path="/5D08041F/5BEBB902" Ref="#PWR0143"  Part="1"
+F 0 "#PWR0143" H 6000 1650 50  0001 C CNN
 F 1 "+3V3" H 6015 1973 50  0000 C CNN
 F 2 "" H 6000 1800 50  0001 C CNN
@@
 	5300 2150 5800 2150
 $Comp
-L Connector:Conn_01x10_Female J31
+L Connector:Conn_01x10_Female J28
 U 1 1 5D089C8E
 P 5000 3350
-F 0 "J31" V 5100 3300 50  0000 C CNN
+F 0 "J28" V 5100 3300 50  0000 C CNN
 F 1 "sdcard_header" V 5200 3300 50  0000 C CNN
 F 2 "footprint-lib:SDCARD_HEADER" H 5000 3350 50  0001 C CNN
@@
 Connection ~ 5600 2950
 $Comp
-L Device:R_Pack04 RN4
+L Device:R_Pack04 RN2
 U 1 1 5D09497F
 P 3500 1500
-F 0 "RN4" H 3700 1550 50  0000 L CNN
+F 0 "RN2" H 3700 1550 50  0000 L CNN
 F 1 "R_Pack04" H 3700 1500 50  0000 L CNN
 F 2 "Resistor_SMD:R_Array_Concave_4x0603" V 3775 1500 50  0001 C CNN
@@
 	5750 3150 5750 2550
 $Comp
-L Device:R_Pack04 RN5
+L Device:R_Pack04 RN3
 U 1 1 5D09B375
 P 4000 1500
-F 0 "RN5" H 4200 1550 50  0000 L CNN
+F 0 "RN3" H 4200 1550 50  0000 L CNN
 F 1 "R_Pack04" H 4200 1500 50  0000 L CNN
 F 2 "Resistor_SMD:R_Array_Concave_4x0603" V 4275 1500 50  0001 C CNN
@@
 AR Path="/5BE65513/5D0FA3F5" Ref="#PWR?"  Part="1"
 AR Path="/5C19BBA6/5C1A1380/5D0FA3F5" Ref="#PWR?"  Part="1"
-AR Path="/5D08041F/5D0FA3F5" Ref="#PWR0161"  Part="1"
-F 0 "#PWR0161" H 4650 1000 50  0001 C CNN
+AR Path="/5D08041F/5D0FA3F5" Ref="#PWR0142"  Part="1"
+F 0 "#PWR0142" H 4650 1000 50  0001 C CNN
 F 1 "+3V3" H 4665 1323 50  0000 C CNN
 F 2 "" H 4650 1150 50  0001 C CNN
