File: hardware/bluepill.sch (KiCad schematic (older format))
At the start: 3 parts, among them J22 STM32_2_DEBUG1, J23 STM32_2_DEBUG2, U13 bluepill-stm32f103c8t6

Commit message: update,
Parts:
- renumbered J22 to J29, J23 to J30
Changed lines of the file:
@@
 $EndComp
 $Comp
-L power:+5V #PWR0148
+L power:+5V #PWR0150
 U 1 1 5CDCC5C9
 P 9500 1350
-AR Path="/5CDAB6B1/5CDCC5C9" Ref="#PWR0148"  Part="1"
+AR Path="/5CDAB6B1/5CDCC5C9" Ref="#PWR0150"  Part="1"
 AR Path="/5CE0453C/5CDCC5C9" Ref="#PWR?"  Part="1"
 AR Path="/5CE8F13B/5CDCC5C9" Ref="#PWR?"  Part="1"
 AR Path="/5CF5AEBC/5CDCC5C9" Ref="#PWR?"  Part="1"
-F 0 "#PWR0148" H 9500 1200 50  0001 C CNN
+F 0 "#PWR0150" H 9500 1200 50  0001 C CNN
 F 1 "+5V" V 9500 1500 50  0000 L CNN
 F 2 "" H 9500 1350 50  0001 C CNN
@@
 	9150 1350 9500 1350
 $Comp
-L power:+3V3 #PWR0146
+L power:+3V3 #PWR0148
 U 1 1 5CDCDBFF
 P 9500 1150
-AR Path="/5CDAB6B1/5CDCDBFF" Ref="#PWR0146"  Part="1"
+AR Path="/5CDAB6B1/5CDCDBFF" Ref="#PWR0148"  Part="1"
 AR Path="/5CE0453C/5CDCDBFF" Ref="#PWR?"  Part="1"
 AR Path="/5CE8F13B/5CDCDBFF" Ref="#PWR?"  Part="1"
 AR Path="/5CF5AEBC/5CDCDBFF" Ref="#PWR?"  Part="1"
-F 0 "#PWR0146" H 9500 1000 50  0001 C CNN
+F 0 "#PWR0148" H 9500 1000 50  0001 C CNN
 F 1 "+3V3" V 9500 1300 50  0000 L CNN
 F 2 "" H 9500 1150 50  0001 C CNN
@@
 	9150 1150 9500 1150
 $Comp
-L power:GND #PWR0147
+L power:GND #PWR0149
 U 1 1 5CDCE1E2
 P 9350 1250
-AR Path="/5CDAB6B1/5CDCE1E2" Ref="#PWR0147"  Part="1"
+AR Path="/5CDAB6B1/5CDCE1E2" Ref="#PWR0149"  Part="1"
 AR Path="/5CE0453C/5CDCE1E2" Ref="#PWR?"  Part="1"
 AR Path="/5CE8F13B/5CDCE1E2" Ref="#PWR?"  Part="1"
 AR Path="/5CF5AEBC/5CDCE1E2" Ref="#PWR?"  Part="1"
-F 0 "#PWR0147" H 9350 1000 50  0001 C CNN
+F 0 "#PWR0149" H 9350 1000 50  0001 C CNN
 F 1 "GND" V 9400 1100 50  0000 R CNN
 F 2 "" H 9350 1250 50  0001 C CNN
@@
 	9150 3050 9350 3050
 $Comp
-L power:+3V3 #PWR0149
+L power:+3V3 #PWR0151
 U 1 1 5CE16ACF
 P 7400 2850
-AR Path="/5CDAB6B1/5CE16ACF" Ref="#PWR0149"  Part="1"
+AR Path="/5CDAB6B1/5CE16ACF" Ref="#PWR0151"  Part="1"
 AR Path="/5CE0453C/5CE16ACF" Ref="#PWR?"  Part="1"
 AR Path="/5CE8F13B/5CE16ACF" Ref="#PWR?"  Part="1"
 AR Path="/5CF5AEBC/5CE16ACF" Ref="#PWR?"  Part="1"
-F 0 "#PWR0149" H 7400 2700 50  0001 C CNN
+F 0 "#PWR0151" H 7400 2700 50  0001 C CNN
 F 1 "+3V3" V 7400 3000 50  0000 L CNN
 F 2 "" H 7400 2850 50  0001 C CNN
@@
 	7750 2850 7400 2850
 $Comp
-L power:GND #PWR0150
+L power:GND #PWR0152
 U 1 1 5CE16ADA
 P 7550 2950
-AR Path="/5CDAB6B1/5CE16ADA" Ref="#PWR0150"  Part="1"
+AR Path="/5CDAB6B1/5CE16ADA" Ref="#PWR0152"  Part="1"
 AR Path="/5CE0453C/5CE16ADA" Ref="#PWR?"  Part="1"
 AR Path="/5CE8F13B/5CE16ADA" Ref="#PWR?"  Part="1"
 AR Path="/5CF5AEBC/5CE16ADA" Ref="#PWR?"  Part="1"
-F 0 "#PWR0150" H 7550 2700 50  0001 C CNN
+F 0 "#PWR0152" H 7550 2700 50  0001 C CNN
 F 1 "GND" V 7600 2800 50  0000 R CNN
 F 2 "" H 7550 2950 50  0001 C CNN
@@
 	7550 2950 7750 2950
 $Comp
-L power:GND #PWR0151
+L power:GND #PWR0153
 U 1 1 5CE1CBEC
 P 7550 3050
-AR Path="/5CDAB6B1/5CE1CBEC" Ref="#PWR0151"  Part="1"
+AR Path="/5CDAB6B1/5CE1CBEC" Ref="#PWR0153"  Part="1"
 AR Path="/5CE0453C/5CE1CBEC" Ref="#PWR?"  Part="1"
 AR Path="/5CE8F13B/5CE1CBEC" Ref="#PWR?"  Part="1"
 AR Path="/5CF5AEBC/5CE1CBEC" Ref="#PWR?"  Part="1"
-F 0 "#PWR0151" H 7550 2800 50  0001 C CNN
+F 0 "#PWR0153" H 7550 2800 50  0001 C CNN
 F 1 "GND" V 7600 2900 50  0000 R CNN
 F 2 "" H 7550 3050 50  0001 C CNN
@@
 	7550 3050 7750 3050
 $Comp
-L Connector:Conn_01x20_Male J23
+L Connector:Conn_01x20_Male J30
 U 1 1 5CEDE89A
 P 8700 4700
-AR Path="/5CDAB6B1/5CEDE89A" Ref="J23"  Part="1"
+AR Path="/5CDAB6B1/5CEDE89A" Ref="J30"  Part="1"
 AR Path="/5CF5AEBC/5CEDE89A" Ref="J?"  Part="1"
-F 0 "J23" H 8850 5800 50  0000 C CNN
+F 0 "J30" H 8850 5800 50  0000 C CNN
 F 1 "STM32_2_DEBUG2" H 8850 5700 50  0000 C CNN
 F 2 "Connector_PinHeader_1.00mm:PinHeader_1x20_P1.00mm_Vertical" H 8700 4700 50  0001 C CNN
@@
 $EndComp
 $Comp
-L Connector:Conn_01x20_Male J22
+L Connector:Conn_01x20_Male J29
 U 1 1 5CEDE8A4
 P 8200 4700
-AR Path="/5CDAB6B1/5CEDE8A4" Ref="J22"  Part="1"
+AR Path="/5CDAB6B1/5CEDE8A4" Ref="J29"  Part="1"
 AR Path="/5CF5AEBC/5CEDE8A4" Ref="J?"  Part="1"
-F 0 "J22" H 8300 5800 50  0000 C CNN
+F 0 "J29" H 8300 5800 50  0000 C CNN
 F 1 "STM32_2_DEBUG1" H 8300 5700 50  0000 C CNN
 F 2 "Connector_PinHeader_1.00mm:PinHeader_1x20_P1.00mm_Vertical" H 8200 4700 50  0001 C CNN
@@
 $EndComp
 $Comp
-L power:+5V #PWR0154
+L power:+5V #PWR0156
 U 1 1 5CEF351D
 P 9250 4000
-AR Path="/5CDAB6B1/5CEF351D" Ref="#PWR0154"  Part="1"
+AR Path="/5CDAB6B1/5CEF351D" Ref="#PWR0156"  Part="1"
 AR Path="/5CE0453C/5CEF351D" Ref="#PWR?"  Part="1"
 AR Path="/5CE8F13B/5CEF351D" Ref="#PWR?"  Part="1"
 AR Path="/5CF5AEBC/5CEF351D" Ref="#PWR?"  Part="1"
-F 0 "#PWR0154" H 9250 3850 50  0001 C CNN
+F 0 "#PWR0156" H 9250 3850 50  0001 C CNN
 F 1 "+5V" V 9250 4150 50  0000 L CNN
 F 2 "" H 9250 4000 50  0001 C CNN
@@
 	8900 4000 9250 4000
 $Comp
-L power:+3V3 #PWR0152
+L power:+3V3 #PWR0154
 U 1 1 5CEF3528
 P 9250 3800
-AR Path="/5CDAB6B1/5CEF3528" Ref="#PWR0152"  Part="1"
+AR Path="/5CDAB6B1/5CEF3528" Ref="#PWR0154"  Part="1"
 AR Path="/5CE0453C/5CEF3528" Ref="#PWR?"  Part="1"
 AR Path="/5CE8F13B/5CEF3528" Ref="#PWR?"  Part="1"
 AR Path="/5CF5AEBC/5CEF3528" Ref="#PWR?"  Part="1"
-F 0 "#PWR0152" H 9250 3650 50  0001 C CNN
+F 0 "#PWR0154" H 9250 3650 50  0001 C CNN
 F 1 "+3V3" V 9250 3950 50  0000 L CNN
 F 2 "" H 9250 3800 50  0001 C CNN
@@
 	8900 3800 9250 3800
 $Comp
-L power:GND #PWR0153
+L power:GND #PWR0155
 U 1 1 5CEF3533
 P 9100 3900
-AR Path="/5CDAB6B1/5CEF3533" Ref="#PWR0153"  Part="1"
+AR Path="/5CDAB6B1/5CEF3533" Ref="#PWR0155"  Part="1"
 AR Path="/5CE0453C/5CEF3533" Ref="#PWR?"  Part="1"
 AR Path="/5CE8F13B/5CEF3533" Ref="#PWR?"  Part="1"
 AR Path="/5CF5AEBC/5CEF3533" Ref="#PWR?"  Part="1"
-F 0 "#PWR0153" H 9100 3650 50  0001 C CNN
+F 0 "#PWR0155" H 9100 3650 50  0001 C CNN
 F 1 "GND" V 9150 3750 50  0000 R CNN
 F 2 "" H 9100 3900 50  0001 C CNN
@@
 	7800 5400 8000 5400
 $Comp
-L power:+3V3 #PWR0155
+L power:+3V3 #PWR0157
 U 1 1 5CEFE118
 P 7650 5500
-AR Path="/5CDAB6B1/5CEFE118" Ref="#PWR0155"  Part="1"
+AR Path="/5CDAB6B1/5CEFE118" Ref="#PWR0157"  Part="1"
 AR Path="/5CE0453C/5CEFE118" Ref="#PWR?"  Part="1"
 AR Path="/5CE8F13B/5CEFE118" Ref="#PWR?"  Part="1"
 AR Path="/5CF5AEBC/5CEFE118" Ref="#PWR?"  Part="1"
-F 0 "#PWR0155" H 7650 5350 50  0001 C CNN
+F 0 "#PWR0157" H 7650 5350 50  0001 C CNN
 F 1 "+3V3" V 7650 5650 50  0000 L CNN
 F 2 "" H 7650 5500 50  0001 C CNN
@@
 	8000 5500 7650 5500
 $Comp
-L power:GND #PWR0156
+L power:GND #PWR0158
 U 1 1 5CEFE123
 P 7800 5600
-AR Path="/5CDAB6B1/5CEFE123" Ref="#PWR0156"  Part="1"
+AR Path="/5CDAB6B1/5CEFE123" Ref="#PWR0158"  Part="1"
 AR Path="/5CE0453C/5CEFE123" Ref="#PWR?"  Part="1"
 AR Path="/5CE8F13B/5CEFE123" Ref="#PWR?"  Part="1"
 AR Path="/5CF5AEBC/5CEFE123" Ref="#PWR?"  Part="1"
-F 0 "#PWR0156" H 7800 5350 50  0001 C CNN
+F 0 "#PWR0158" H 7800 5350 50  0001 C CNN
 F 1 "GND" V 7850 5450 50  0000 R CNN
 F 2 "" H 7800 5600 50  0001 C CNN
@@
 	7800 5600 8000 5600
 $Comp
-L power:GND #PWR0157
+L power:GND #PWR0159
 U 1 1 5CEFE12E
 P 7800 5700
-AR Path="/5CDAB6B1/5CEFE12E" Ref="#PWR0157"  Part="1"
+AR Path="/5CDAB6B1/5CEFE12E" Ref="#PWR0159"  Part="1"
 AR Path="/5CE0453C/5CEFE12E" Ref="#PWR?"  Part="1"
 AR Path="/5CE8F13B/5CEFE12E" Ref="#PWR?"  Part="1"
 AR Path="/5CF5AEBC/5CEFE12E" Ref="#PWR?"  Part="1"
-F 0 "#PWR0157" H 7800 5450 50  0001 C CNN
+F 0 "#PWR0159" H 7800 5450 50  0001 C CNN
 F 1 "GND" V 7850 5550 50  0000 R CNN
 F 2 "" H 7800 5700 50  0001 C CNN

Commit message: update,
Changed lines of the file:
@@
 $Descr A4 11693 8268
 encoding utf-8
-Sheet 19 20
+Sheet 18 20
 Title ""
 Date ""
@@
 Wire Wire Line
 	1050 2400 1400 2400
+Text HLabel 1050 2650 0    50   Input ~ 0
+WS2812_OUT
+Text Label 1550 2650 2    50   ~ 0
+PB11
+Wire Wire Line
+	1550 2650 1050 2650
 $EndSCHEMATC

Commit message: update,
Parts:
- added RN?: R_Pack04, symbol Device:R_Pack04
Connections:
- net STM32_1_PB11 is gone; now on net WS2812_OUT: J29.16 (Pin_16), U13.~ (VBAT)
- net +3V3: now also RN?.5 (R4.2), RN?.6 (R3.2), RN?.7 (R2.2), RN?.8 (R1.2)
- net SCL: now also RN?.2 (R2.1)
- net SDA: now also RN?.1 (R1.1)
- net STM32_1_NRST renamed NRST
- net STM32_1_PA11 renamed PA11
- net STM32_1_PA12 renamed PA12
- net STM32_1_PA2 renamed PA2
- net STM32_1_PA3 renamed PA3
- net STM32_1_PA8 renamed PA8
- net STM32_1_PA9 renamed TX
- net STM32_1_PB0 renamed PB0
- net STM32_1_PB1 renamed PB1
- net STM32_1_PB10 renamed PB10
- net STM32_1_PB12 renamed PB12
- net STM32_1_PB13 renamed PB13
- net STM32_1_PB14 renamed PB14
- net STM32_1_PB15 renamed PB15
- net STM32_1_PB3 renamed PB3
- net STM32_1_PB4 renamed PB4
- net STM32_1_PB5 renamed PB5
- net STM32_1_PB8 renamed PB8
- net STM32_1_PB9 renamed PB9
- net STM32_1_PC13 renamed PC13
- net STM32_1_PC14 renamed PC14
- net STM32_1_PC15 renamed PC15

Commit message: update,
Connections:
- net PB1 renamed OLED_DC
- net PB3 renamed OLED_SS
Changed lines of the file:
@@
 $Descr A4 11693 8268
 encoding utf-8
-Sheet 18 20
+Sheet 20 20
 Title ""
 Date ""
@@
 Wire Wire Line
 	7800 5700 8000 5700
-Text HLabel 1150 1350 0    50   Input ~ 0
+Text HLabel 1550 1350 0    50   Input ~ 0
 SDA
-Text HLabel 1150 1450 0    50   Input ~ 0
+Text HLabel 1550 1450 0    50   Input ~ 0
 SCL
-Text HLabel 1150 2450 0    50   Input ~ 0
+Text HLabel 1550 1750 0    50   Input ~ 0
 TX
-Text HLabel 1150 2550 0    50   Input ~ 0
+Text HLabel 1550 1850 0    50   Input ~ 0
 RX
 $Bitmap
@@
 EndData
 $EndBitmap
-Text HLabel 1150 2800 0    50   Input ~ 0
+Text HLabel 1550 2100 0    50   Input ~ 0
 SS
-Text HLabel 1150 2900 0    50   Input ~ 0
+Text HLabel 1550 2200 0    50   Input ~ 0
 SCK
-Text HLabel 1150 3000 0    50   Input ~ 0
+Text HLabel 1550 2300 0    50   Input ~ 0
 MISO
-Text HLabel 1150 3100 0    50   Input ~ 0
+Text HLabel 1550 2400 0    50   Input ~ 0
 MOSI
-Text HLabel 1150 3350 0    50   Input ~ 0
+Text HLabel 1550 2650 0    50   Input ~ 0
 PWM
-Text HLabel 1150 3700 0    50   Input ~ 0
+Text HLabel 1550 3000 0    50   Input ~ 0
 A_IN0
-Text HLabel 1150 3800 0    50   Input ~ 0
+Text HLabel 1550 3100 0    50   Input ~ 0
 A_IN1
-Text HLabel 1150 4050 0    50   Input ~ 0
+Text HLabel 1550 3350 0    50   Input ~ 0
 WS2812_OUT
-Text Label 1650 4050 2    50   ~ 0
+Text Label 2050 3350 2    50   ~ 0
 PB11
 Wire Wire Line
-	1650 4050 1150 4050
+	2050 3350 1550 3350
 Text Label 7150 2650 0    50   ~ 0
 PB11
@@
 PB6
 Wire Wire Line
-	1150 1350 2050 1350
-Text Label 2050 2450 2    50   ~ 0
+	1550 1350 2050 1350
+Text Label 2050 1750 2    50   ~ 0
 PA9
-Text Label 2050 2550 2    50   ~ 0
+Text Label 2050 1850 2    50   ~ 0
 PA10
 Wire Wire Line
-	1150 1450 2050 1450
+	1550 1450 2050 1450
 Wire Wire Line
-	1150 2450 2050 2450
-Text Label 2050 2800 2    50   ~ 0
+	1550 1750 2050 1750
+Text Label 2050 2100 2    50   ~ 0
 PA4
-Text Label 2050 2900 2    50   ~ 0
+Text Label 2050 2200 2    50   ~ 0
 PA5
-Text Label 2050 3000 2    50   ~ 0
+Text Label 2050 2300 2    50   ~ 0
 PA6
-Text Label 2050 3100 2    50   ~ 0
+Text Label 2050 2400 2    50   ~ 0
 PA7
-Text Label 2050 3350 2    50   ~ 0
+Text Label 2050 2650 2    50   ~ 0
 PA15
 Wire Wire Line
-	1150 2550 2050 2550
+	1550 1850 2050 1850
 Wire Wire Line
-	1150 2800 2050 2800
+	1550 2100 2050 2100
 Wire Wire Line
-	1150 2900 2050 2900
+	1550 2200 2050 2200
 Wire Wire Line
-	1150 3000 2050 3000
+	1550 2300 2050 2300
 Wire Wire Line
-	1150 3100 2050 3100
+	1550 2400 2050 2400
 Wire Wire Line
-	1150 3350 2050 3350
-Text Label 2050 3700 2    50   ~ 0
+	1550 2650 2050 2650
+Text Label 2050 3000 2    50   ~ 0
 PA0
-Text Label 2050 3800 2    50   ~ 0
+Text Label 2050 3100 2    50   ~ 0
 PA1
 Wire Wire Line
-	1150 3700 2050 3700
+	1550 3000 2050 3000
 Wire Wire Line
-	1150 3800 2050 3800
+	1550 3100 2050 3100
 $Comp
 L Device:R_Pack04 RN?
@@
 Wire Wire Line
 	3300 1450 3850 1450
+Text HLabel 1550 3900 0    50   Input ~ 0
+OLED_DC
+Text HLabel 1550 4000 0    50   Input ~ 0
+OLED_RST
+Text Label 2050 3900 2    50   ~ 0
+PB1
+Wire Wire Line
+	2050 3900 1550 3900
+Text Label 2050 4000 2    50   ~ 0
+PB2
+Wire Wire Line
+	2050 4000 1550 4000
+Text HLabel 1550 4100 0    50   Input ~ 0
+OLED_SS
+Text Label 2050 4100 2    50   ~ 0
+PB3
+Wire Wire Line
+	2050 4100 1550 4100
 $EndSCHEMATC

Commit message: update,
Parts:
- gave numbers to parts that had none: 1
- renumbered J29 to J30, J30 to J31
Connections:
- net PB4 renamed DEBUG_LED
Changed lines of the file:
@@
 $EndComp
 $Comp
-L power:+5V #PWR0150
+L power:+5V #PWR0160
 U 1 1 5CDCC5C9
 P 9500 1350
-AR Path="/5CDAB6B1/5CDCC5C9" Ref="#PWR0150"  Part="1"
+AR Path="/5CDAB6B1/5CDCC5C9" Ref="#PWR0160"  Part="1"
 AR Path="/5CE0453C/5CDCC5C9" Ref="#PWR?"  Part="1"
 AR Path="/5CE8F13B/5CDCC5C9" Ref="#PWR?"  Part="1"
 AR Path="/5CF5AEBC/5CDCC5C9" Ref="#PWR?"  Part="1"
-F 0 "#PWR0150" H 9500 1200 50  0001 C CNN
+F 0 "#PWR0160" H 9500 1200 50  0001 C CNN
 F 1 "+5V" V 9500 1500 50  0000 L CNN
 F 2 "" H 9500 1350 50  0001 C CNN
@@
 	9150 1350 9500 1350
 $Comp
-L power:+3V3 #PWR0148
+L power:+3V3 #PWR0158
 U 1 1 5CDCDBFF
 P 9500 1150
-AR Path="/5CDAB6B1/5CDCDBFF" Ref="#PWR0148"  Part="1"
+AR Path="/5CDAB6B1/5CDCDBFF" Ref="#PWR0158"  Part="1"
 AR Path="/5CE0453C/5CDCDBFF" Ref="#PWR?"  Part="1"
 AR Path="/5CE8F13B/5CDCDBFF" Ref="#PWR?"  Part="1"
 AR Path="/5CF5AEBC/5CDCDBFF" Ref="#PWR?"  Part="1"
-F 0 "#PWR0148" H 9500 1000 50  0001 C CNN
+F 0 "#PWR0158" H 9500 1000 50  0001 C CNN
 F 1 "+3V3" V 9500 1300 50  0000 L CNN
 F 2 "" H 9500 1150 50  0001 C CNN
@@
 	9150 1150 9500 1150
 $Comp
-L power:GND #PWR0149
+L power:GND #PWR0159
 U 1 1 5CDCE1E2
 P 9350 1250
-AR Path="/5CDAB6B1/5CDCE1E2" Ref="#PWR0149"  Part="1"
+AR Path="/5CDAB6B1/5CDCE1E2" Ref="#PWR0159"  Part="1"
 AR Path="/5CE0453C/5CDCE1E2" Ref="#PWR?"  Part="1"
 AR Path="/5CE8F13B/5CDCE1E2" Ref="#PWR?"  Part="1"
 AR Path="/5CF5AEBC/5CDCE1E2" Ref="#PWR?"  Part="1"
-F 0 "#PWR0149" H 9350 1000 50  0001 C CNN
+F 0 "#PWR0159" H 9350 1000 50  0001 C CNN
 F 1 "GND" V 9400 1100 50  0000 R CNN
 F 2 "" H 9350 1250 50  0001 C CNN
@@
 	7150 2650 7750 2650
 $Comp
-L power:+3V3 #PWR0151
+L power:+3V3 #PWR0161
 U 1 1 5CE16ACF
 P 7400 2850
-AR Path="/5CDAB6B1/5CE16ACF" Ref="#PWR0151"  Part="1"
+AR Path="/5CDAB6B1/5CE16ACF" Ref="#PWR0161"  Part="1"
 AR Path="/5CE0453C/5CE16ACF" Ref="#PWR?"  Part="1"
 AR Path="/5CE8F13B/5CE16ACF" Ref="#PWR?"  Part="1"
 AR Path="/5CF5AEBC/5CE16ACF" Ref="#PWR?"  Part="1"
-F 0 "#PWR0151" H 7400 2700 50  0001 C CNN
+F 0 "#PWR0161" H 7400 2700 50  0001 C CNN
 F 1 "+3V3" V 7400 3000 50  0000 L CNN
 F 2 "" H 7400 2850 50  0001 C CNN
@@
 	7750 2850 7400 2850
 $Comp
-L power:GND #PWR0152
+L power:GND #PWR0162
 U 1 1 5CE16ADA
 P 7550 2950
-AR Path="/5CDAB6B1/5CE16ADA" Ref="#PWR0152"  Part="1"
+AR Path="/5CDAB6B1/5CE16ADA" Ref="#PWR0162"  Part="1"
 AR Path="/5CE0453C/5CE16ADA" Ref="#PWR?"  Part="1"
 AR Path="/5CE8F13B/5CE16ADA" Ref="#PWR?"  Part="1"
 AR Path="/5CF5AEBC/5CE16ADA" Ref="#PWR?"  Part="1"
-F 0 "#PWR0152" H 7550 2700 50  0001 C CNN
+F 0 "#PWR0162" H 7550 2700 50  0001 C CNN
 F 1 "GND" V 7600 2800 50  0000 R CNN
 F 2 "" H 7550 2950 50  0001 C CNN
@@
 	7550 2950 7750 2950
 $Comp
-L power:GND #PWR0153
+L power:GND #PWR0163
 U 1 1 5CE1CBEC
 P 7550 3050
-AR Path="/5CDAB6B1/5CE1CBEC" Ref="#PWR0153"  Part="1"
+AR Path="/5CDAB6B1/5CE1CBEC" Ref="#PWR0163"  Part="1"
 AR Path="/5CE0453C/5CE1CBEC" Ref="#PWR?"  Part="1"
 AR Path="/5CE8F13B/5CE1CBEC" Ref="#PWR?"  Part="1"
 AR Path="/5CF5AEBC/5CE1CBEC" Ref="#PWR?"  Part="1"
-F 0 "#PWR0153" H 7550 2800 50  0001 C CNN
+F 0 "#PWR0163" H 7550 2800 50  0001 C CNN
 F 1 "GND" V 7600 2900 50  0000 R CNN
 F 2 "" H 7550 3050 50  0001 C CNN
@@
 	7550 3050 7750 3050
 $Comp
-L Connector:Conn_01x20_Male J30
+L Connector:Conn_01x20_Male J31
 U 1 1 5CEDE89A
 P 8700 4700
-AR Path="/5CDAB6B1/5CEDE89A" Ref="J30"  Part="1"
+AR Path="/5CDAB6B1/5CEDE89A" Ref="J31"  Part="1"
 AR Path="/5CF5AEBC/5CEDE89A" Ref="J?"  Part="1"
-F 0 "J30" H 8850 5800 50  0000 C CNN
+F 0 "J31" H 8850 5800 50  0000 C CNN
 F 1 "STM32_2_DEBUG2" H 8850 5700 50  0000 C CNN
 F 2 "Connector_PinHeader_1.00mm:PinHeader_1x20_P1.00mm_Vertical" H 8700 4700 50  0001 C CNN
@@
 $EndComp
 $Comp
-L Connector:Conn_01x20_Male J29
+L Connector:Conn_01x20_Male J30
 U 1 1 5CEDE8A4
 P 8200 4700
-AR Path="/5CDAB6B1/5CEDE8A4" Ref="J29"  Part="1"
+AR Path="/5CDAB6B1/5CEDE8A4" Ref="J30"  Part="1"
 AR Path="/5CF5AEBC/5CEDE8A4" Ref="J?"  Part="1"
-F 0 "J29" H 8300 5800 50  0000 C CNN
+F 0 "J30" H 8300 5800 50  0000 C CNN
 F 1 "STM32_2_DEBUG1" H 8300 5700 50  0000 C CNN
 F 2 "Connector_PinHeader_1.00mm:PinHeader_1x20_P1.00mm_Vertical" H 8200 4700 50  0001 C CNN
@@
 $EndComp
 $Comp
-L power:+5V #PWR0156
+L power:+5V #PWR0166
 U 1 1 5CEF351D
 P 9250 4000
-AR Path="/5CDAB6B1/5CEF351D" Ref="#PWR0156"  Part="1"
+AR Path="/5CDAB6B1/5CEF351D" Ref="#PWR0166"  Part="1"
 AR Path="/5CE0453C/5CEF351D" Ref="#PWR?"  Part="1"
 AR Path="/5CE8F13B/5CEF351D" Ref="#PWR?"  Part="1"
 AR Path="/5CF5AEBC/5CEF351D" Ref="#PWR?"  Part="1"
-F 0 "#PWR0156" H 9250 3850 50  0001 C CNN
+F 0 "#PWR0166" H 9250 3850 50  0001 C CNN
 F 1 "+5V" V 9250 4150 50  0000 L CNN
 F 2 "" H 9250 4000 50  0001 C CNN
@@
 	8900 4000 9250 4000
 $Comp
-L power:+3V3 #PWR0154
+L power:+3V3 #PWR0164
 U 1 1 5CEF3528
 P 9250 3800
-AR Path="/5CDAB6B1/5CEF3528" Ref="#PWR0154"  Part="1"
+AR Path="/5CDAB6B1/5CEF3528" Ref="#PWR0164"  Part="1"
 AR Path="/5CE0453C/5CEF3528" Ref="#PWR?"  Part="1"
 AR Path="/5CE8F13B/5CEF3528" Ref="#PWR?"  Part="1"
 AR Path="/5CF5AEBC/5CEF3528" Ref="#PWR?"  Part="1"
-F 0 "#PWR0154" H 9250 3650 50  0001 C CNN
+F 0 "#PWR0164" H 9250 3650 50  0001 C CNN
 F 1 "+3V3" V 9250 3950 50  0000 L CNN
 F 2 "" H 9250 3800 50  0001 C CNN
@@
 	8900 3800 9250 3800
 $Comp
-L power:GND #PWR0155
+L power:GND #PWR0165
 U 1 1 5CEF3533
 P 9100 3900
-AR Path="/5CDAB6B1/5CEF3533" Ref="#PWR0155"  Part="1"
+AR Path="/5CDAB6B1/5CEF3533" Ref="#PWR0165"  Part="1"
 AR Path="/5CE0453C/5CEF3533" Ref="#PWR?"  Part="1"
 AR Path="/5CE8F13B/5CEF3533" Ref="#PWR?"  Part="1"
 AR Path="/5CF5AEBC/5CEF3533" Ref="#PWR?"  Part="1"
-F 0 "#PWR0155" H 9100 3650 50  0001 C CNN
+F 0 "#PWR0165" H 9100 3650 50  0001 C CNN
 F 1 "GND" V 9150 3750 50  0000 R CNN
 F 2 "" H 9100 3900 50  0001 C CNN
@@
 	9100 3900 8900 3900
 $Comp
-L power:+3V3 #PWR0157
+L power:+3V3 #PWR0167
 U 1 1 5CEFE118
 P 7650 5500
-AR Path="/5CDAB6B1/5CEFE118" Ref="#PWR0157"  Part="1"
+AR Path="/5CDAB6B1/5CEFE118" Ref="#PWR0167"  Part="1"
 AR Path="/5CE0453C/5CEFE118" Ref="#PWR?"  Part="1"
 AR Path="/5CE8F13B/5CEFE118" Ref="#PWR?"  Part="1"
 AR Path="/5CF5AEBC/5CEFE118" Ref="#PWR?"  Part="1"
-F 0 "#PWR0157" H 7650 5350 50  0001 C CNN
+F 0 "#PWR0167" H 7650 5350 50  0001 C CNN
 F 1 "+3V3" V 7650 5650 50  0000 L CNN
 F 2 "" H 7650 5500 50  0001 C CNN
@@
 	8000 5500 7650 5500
 $Comp
-L power:GND #PWR0158
+L power:GND #PWR0168
 U 1 1 5CEFE123
 P 7800 5600
-AR Path="/5CDAB6B1/5CEFE123" Ref="#PWR0158"  Part="1"
+AR Path="/5CDAB6B1/5CEFE123" Ref="#PWR0168"  Part="1"
 AR Path="/5CE0453C/5CEFE123" Ref="#PWR?"  Part="1"
 AR Path="/5CE8F13B/5CEFE123" Ref="#PWR?"  Part="1"
 AR Path="/5CF5AEBC/5CEFE123" Ref="#PWR?"  Part="1"
-F 0 "#PWR0158" H 7800 5350 50  0001 C CNN
+F 0 "#PWR0168" H 7800 5350 50  0001 C CNN
 F 1 "GND" V 7850 5450 50  0000 R CNN
 F 2 "" H 7800 5600 50  0001 C CNN
@@
 	7800 5600 8000 5600
 $Comp
-L power:GND #PWR0159
+L power:GND #PWR0169
 U 1 1 5CEFE12E
 P 7800 5700
-AR Path="/5CDAB6B1/5CEFE12E" Ref="#PWR0159"  Part="1"
+AR Path="/5CDAB6B1/5CEFE12E" Ref="#PWR0169"  Part="1"
 AR Path="/5CE0453C/5CEFE12E" Ref="#PWR?"  Part="1"
 AR Path="/5CE8F13B/5CEFE12E" Ref="#PWR?"  Part="1"
 AR Path="/5CF5AEBC/5CEFE12E" Ref="#PWR?"  Part="1"
-F 0 "#PWR0159" H 7800 5450 50  0001 C CNN
+F 0 "#PWR0169" H 7800 5450 50  0001 C CNN
 F 1 "GND" V 7850 5550 50  0000 R CNN
 F 2 "" H 7800 5700 50  0001 C CNN
@@
 P 3400 1100
 AR Path="/5CDAB838/5CFCEDDC" Ref="RN?"  Part="1"
-AR Path="/5CDAB6B1/5CFCEDDC" Ref="RN?"  Part="1"
-F 0 "RN?" H 3600 1150 50  0000 L CNN
+AR Path="/5CDAB6B1/5CFCEDDC" Ref="RN6"  Part="1"
+F 0 "RN6" H 3600 1150 50  0000 L CNN
 F 1 "R_Pack04" H 3600 1100 50  0000 L CNN
 F 2 "" V 3675 1100 50  0001 C CNN
@@
 $EndComp
 $Comp
-L power:+3V3 #PWR?
+L power:+3V3 #PWR0157
 U 1 1 5CFCEDE6
 P 3050 750
-F 0 "#PWR?" H 3050 600 50  0001 C CNN
+F 0 "#PWR0157" H 3050 600 50  0001 C CNN
 F 1 "+3V3" H 3100 950 50  0000 C CNN
 F 2 "" H 3050 750 50  0001 C CNN
@@
 Wire Wire Line
 	2050 4100 1550 4100
+Text HLabel 1550 4300 0    50   Input ~ 0
+DEBUG_LED
+Text Label 2050 4300 2    50   ~ 0
+PB4
+Wire Wire Line
+	2050 4300 1550 4300
 $EndSCHEMATC

Commit message: update,
Connections:
- net PB5 renamed BUZZER
Changed lines of the file:
@@
 $Descr A4 11693 8268
 encoding utf-8
-Sheet 20 20
+Sheet 18 18
 Title ""
 Date ""
@@
 Wire Wire Line
 	2050 4300 1550 4300
+Text HLabel 1550 4450 0    50   Input ~ 0
+BUZZER
+Text Label 2050 4450 2    50   ~ 0
+PB5
+Wire Wire Line
+	2050 4450 1550 4450
 $EndSCHEMATC
