File: hardware/bluepill.sch (KiCad schematic (older format))
At the start: 4 parts, among them J30 STM32_2_DEBUG1, J31 STM32_2_DEBUG2, U13 bluepill-stm32f103c8t6

Commit message: update,
Parts:
- renumbered J30 to J21, J31 to J22, U13 to U9
Connections:
- net PB10 renamed ROT_ENC_SW
- net PB8 renamed ROT_ENC_A
- net PB9 renamed ROT_ENC_B
Changed lines of the file:
@@
 P 8450 2300
 AR Path="/5CDAB6B1/5CDABA4D/5CDCAABB" Ref="U?"  Part="1"
-AR Path="/5CDAB6B1/5CDCAABB" Ref="U13"  Part="1"
+AR Path="/5CDAB6B1/5CDCAABB" Ref="U9"  Part="1"
 AR Path="/5CE0453C/5CDCAABB" Ref="U?"  Part="1"
 AR Path="/5CE8F13B/5CDCAABB" Ref="U?"  Part="1"
 AR Path="/5CF5AEBC/5CDCAABB" Ref="U?"  Part="1"
-F 0 "U13" H 8450 3300 50  0000 C CNN
+F 0 "U9" H 8450 3300 50  0000 C CNN
 F 1 "bluepill-stm32f103c8t6" H 8450 3400 50  0000 C CNN
 F 2 "Package_DIP:DIP-40_W15.24mm_LongPads" H 8450 2400 50  0001 C CNN
@@
 $EndComp
 $Comp
-L power:+5V #PWR0160
+L power:+5V #PWR086
 U 1 1 5CDCC5C9
 P 9500 1350
-AR Path="/5CDAB6B1/5CDCC5C9" Ref="#PWR0160"  Part="1"
+AR Path="/5CDAB6B1/5CDCC5C9" Ref="#PWR086"  Part="1"
 AR Path="/5CE0453C/5CDCC5C9" Ref="#PWR?"  Part="1"
 AR Path="/5CE8F13B/5CDCC5C9" Ref="#PWR?"  Part="1"
 AR Path="/5CF5AEBC/5CDCC5C9" Ref="#PWR?"  Part="1"
-F 0 "#PWR0160" H 9500 1200 50  0001 C CNN
+F 0 "#PWR086" H 9500 1200 50  0001 C CNN
 F 1 "+5V" V 9500 1500 50  0000 L CNN
 F 2 "" H 9500 1350 50  0001 C CNN
@@
 	9150 1350 9500 1350
 $Comp
-L power:+3V3 #PWR0158
+L power:+3V3 #PWR084
 U 1 1 5CDCDBFF
 P 9500 1150
-AR Path="/5CDAB6B1/5CDCDBFF" Ref="#PWR0158"  Part="1"
+AR Path="/5CDAB6B1/5CDCDBFF" Ref="#PWR084"  Part="1"
 AR Path="/5CE0453C/5CDCDBFF" Ref="#PWR?"  Part="1"
 AR Path="/5CE8F13B/5CDCDBFF" Ref="#PWR?"  Part="1"
 AR Path="/5CF5AEBC/5CDCDBFF" Ref="#PWR?"  Part="1"
-F 0 "#PWR0158" H 9500 1000 50  0001 C CNN
+F 0 "#PWR084" H 9500 1000 50  0001 C CNN
 F 1 "+3V3" V 9500 1300 50  0000 L CNN
 F 2 "" H 9500 1150 50  0001 C CNN
@@
 	9150 1150 9500 1150
 $Comp
-L power:GND #PWR0159
+L power:GND #PWR085
 U 1 1 5CDCE1E2
 P 9350 1250
-AR Path="/5CDAB6B1/5CDCE1E2" Ref="#PWR0159"  Part="1"
+AR Path="/5CDAB6B1/5CDCE1E2" Ref="#PWR085"  Part="1"
 AR Path="/5CE0453C/5CDCE1E2" Ref="#PWR?"  Part="1"
 AR Path="/5CE8F13B/5CDCE1E2" Ref="#PWR?"  Part="1"
 AR Path="/5CF5AEBC/5CDCE1E2" Ref="#PWR?"  Part="1"
-F 0 "#PWR0159" H 9350 1000 50  0001 C CNN
+F 0 "#PWR085" H 9350 1000 50  0001 C CNN
 F 1 "GND" V 9400 1100 50  0000 R CNN
 F 2 "" H 9350 1250 50  0001 C CNN
@@
 	7150 2650 7750 2650
 $Comp
-L power:+3V3 #PWR0161
+L power:+3V3 #PWR087
 U 1 1 5CE16ACF
 P 7400 2850
-AR Path="/5CDAB6B1/5CE16ACF" Ref="#PWR0161"  Part="1"
+AR Path="/5CDAB6B1/5CE16ACF" Ref="#PWR087"  Part="1"
 AR Path="/5CE0453C/5CE16ACF" Ref="#PWR?"  Part="1"
 AR Path="/5CE8F13B/5CE16ACF" Ref="#PWR?"  Part="1"
 AR Path="/5CF5AEBC/5CE16ACF" Ref="#PWR?"  Part="1"
-F 0 "#PWR0161" H 7400 2700 50  0001 C CNN
+F 0 "#PWR087" H 7400 2700 50  0001 C CNN
 F 1 "+3V3" V 7400 3000 50  0000 L CNN
 F 2 "" H 7400 2850 50  0001 C CNN
@@
 	7750 2850 7400 2850
 $Comp
-L power:GND #PWR0162
+L power:GND #PWR088
 U 1 1 5CE16ADA
 P 7550 2950
-AR Path="/5CDAB6B1/5CE16ADA" Ref="#PWR0162"  Part="1"
+AR Path="/5CDAB6B1/5CE16ADA" Ref="#PWR088"  Part="1"
 AR Path="/5CE0453C/5CE16ADA" Ref="#PWR?"  Part="1"
 AR Path="/5CE8F13B/5CE16ADA" Ref="#PWR?"  Part="1"
 AR Path="/5CF5AEBC/5CE16ADA" Ref="#PWR?"  Part="1"
-F 0 "#PWR0162" H 7550 2700 50  0001 C CNN
+F 0 "#PWR088" H 7550 2700 50  0001 C CNN
 F 1 "GND" V 7600 2800 50  0000 R CNN
 F 2 "" H 7550 2950 50  0001 C CNN
@@
 	7550 2950 7750 2950
 $Comp
-L power:GND #PWR0163
+L power:GND #PWR089
 U 1 1 5CE1CBEC
 P 7550 3050
-AR Path="/5CDAB6B1/5CE1CBEC" Ref="#PWR0163"  Part="1"
+AR Path="/5CDAB6B1/5CE1CBEC" Ref="#PWR089"  Part="1"
 AR Path="/5CE0453C/5CE1CBEC" Ref="#PWR?"  Part="1"
 AR Path="/5CE8F13B/5CE1CBEC" Ref="#PWR?"  Part="1"
 AR Path="/5CF5AEBC/5CE1CBEC" Ref="#PWR?"  Part="1"
-F 0 "#PWR0163" H 7550 2800 50  0001 C CNN
+F 0 "#PWR089" H 7550 2800 50  0001 C CNN
 F 1 "GND" V 7600 2900 50  0000 R CNN
 F 2 "" H 7550 3050 50  0001 C CNN
@@
 	7550 3050 7750 3050
 $Comp
-L Connector:Conn_01x20_Male J31
+L Connector:Conn_01x20_Male J22
 U 1 1 5CEDE89A
 P 8700 4700
-AR Path="/5CDAB6B1/5CEDE89A" Ref="J31"  Part="1"
+AR Path="/5CDAB6B1/5CEDE89A" Ref="J22"  Part="1"
 AR Path="/5CF5AEBC/5CEDE89A" Ref="J?"  Part="1"
-F 0 "J31" H 8850 5800 50  0000 C CNN
+F 0 "J22" H 8850 5800 50  0000 C CNN
 F 1 "STM32_2_DEBUG2" H 8850 5700 50  0000 C CNN
 F 2 "Connector_PinHeader_1.00mm:PinHeader_1x20_P1.00mm_Vertical" H 8700 4700 50  0001 C CNN
@@
 $EndComp
 $Comp
-L Connector:Conn_01x20_Male J30
+L Connector:Conn_01x20_Male J21
 U 1 1 5CEDE8A4
 P 8200 4700
-AR Path="/5CDAB6B1/5CEDE8A4" Ref="J30"  Part="1"
+AR Path="/5CDAB6B1/5CEDE8A4" Ref="J21"  Part="1"
 AR Path="/5CF5AEBC/5CEDE8A4" Ref="J?"  Part="1"
-F 0 "J30" H 8300 5800 50  0000 C CNN
+F 0 "J21" H 8300 5800 50  0000 C CNN
 F 1 "STM32_2_DEBUG1" H 8300 5700 50  0000 C CNN
 F 2 "Connector_PinHeader_1.00mm:PinHeader_1x20_P1.00mm_Vertical" H 8200 4700 50  0001 C CNN
@@
 $EndComp
 $Comp
-L power:+5V #PWR0166
+L power:+5V #PWR092
 U 1 1 5CEF351D
 P 9250 4000
-AR Path="/5CDAB6B1/5CEF351D" Ref="#PWR0166"  Part="1"
+AR Path="/5CDAB6B1/5CEF351D" Ref="#PWR092"  Part="1"
 AR Path="/5CE0453C/5CEF351D" Ref="#PWR?"  Part="1"
 AR Path="/5CE8F13B/5CEF351D" Ref="#PWR?"  Part="1"
 AR Path="/5CF5AEBC/5CEF351D" Ref="#PWR?"  Part="1"
-F 0 "#PWR0166" H 9250 3850 50  0001 C CNN
+F 0 "#PWR092" H 9250 3850 50  0001 C CNN
 F 1 "+5V" V 9250 4150 50  0000 L CNN
 F 2 "" H 9250 4000 50  0001 C CNN
@@
 	8900 4000 9250 4000
 $Comp
-L power:+3V3 #PWR0164
+L power:+3V3 #PWR090
 U 1 1 5CEF3528
 P 9250 3800
-AR Path="/5CDAB6B1/5CEF3528" Ref="#PWR0164"  Part="1"
+AR Path="/5CDAB6B1/5CEF3528" Ref="#PWR090"  Part="1"
 AR Path="/5CE0453C/5CEF3528" Ref="#PWR?"  Part="1"
 AR Path="/5CE8F13B/5CEF3528" Ref="#PWR?"  Part="1"
 AR Path="/5CF5AEBC/5CEF3528" Ref="#PWR?"  Part="1"
-F 0 "#PWR0164" H 9250 3650 50  0001 C CNN
+F 0 "#PWR090" H 9250 3650 50  0001 C CNN
 F 1 "+3V3" V 9250 3950 50  0000 L CNN
 F 2 "" H 9250 3800 50  0001 C CNN
@@
 	8900 3800 9250 3800
 $Comp
-L power:GND #PWR0165
+L power:GND #PWR091
 U 1 1 5CEF3533
 P 9100 3900
-AR Path="/5CDAB6B1/5CEF3533" Ref="#PWR0165"  Part="1"
+AR Path="/5CDAB6B1/5CEF3533" Ref="#PWR091"  Part="1"
 AR Path="/5CE0453C/5CEF3533" Ref="#PWR?"  Part="1"
 AR Path="/5CE8F13B/5CEF3533" Ref="#PWR?"  Part="1"
 AR Path="/5CF5AEBC/5CEF3533" Ref="#PWR?"  Part="1"
-F 0 "#PWR0165" H 9100 3650 50  0001 C CNN
+F 0 "#PWR091" H 9100 3650 50  0001 C CNN
 F 1 "GND" V 9150 3750 50  0000 R CNN
 F 2 "" H 9100 3900 50  0001 C CNN
@@
 	9100 3900 8900 3900
 $Comp
-L power:+3V3 #PWR0167
+L power:+3V3 #PWR093
 U 1 1 5CEFE118
 P 7650 5500
-AR Path="/5CDAB6B1/5CEFE118" Ref="#PWR0167"  Part="1"
+AR Path="/5CDAB6B1/5CEFE118" Ref="#PWR093"  Part="1"
 AR Path="/5CE0453C/5CEFE118" Ref="#PWR?"  Part="1"
 AR Path="/5CE8F13B/5CEFE118" Ref="#PWR?"  Part="1"
 AR Path="/5CF5AEBC/5CEFE118" Ref="#PWR?"  Part="1"
-F 0 "#PWR0167" H 7650 5350 50  0001 C CNN
+F 0 "#PWR093" H 7650 5350 50  0001 C CNN
 F 1 "+3V3" V 7650 5650 50  0000 L CNN
 F 2 "" H 7650 5500 50  0001 C CNN
@@
 	8000 5500 7650 5500
 $Comp
-L power:GND #PWR0168
+L power:GND #PWR094
 U 1 1 5CEFE123
 P 7800 5600
-AR Path="/5CDAB6B1/5CEFE123" Ref="#PWR0168"  Part="1"
+AR Path="/5CDAB6B1/5CEFE123" Ref="#PWR094"  Part="1"
 AR Path="/5CE0453C/5CEFE123" Ref="#PWR?"  Part="1"
 AR Path="/5CE8F13B/5CEFE123" Ref="#PWR?"  Part="1"
 AR Path="/5CF5AEBC/5CEFE123" Ref="#PWR?"  Part="1"
-F 0 "#PWR0168" H 7800 5350 50  0001 C CNN
+F 0 "#PWR094" H 7800 5350 50  0001 C CNN
 F 1 "GND" V 7850 5450 50  0000 R CNN
 F 2 "" H 7800 5600 50  0001 C CNN
@@
 	7800 5600 8000 5600
 $Comp
-L power:GND #PWR0169
+L power:GND #PWR095
 U 1 1 5CEFE12E
 P 7800 5700
-AR Path="/5CDAB6B1/5CEFE12E" Ref="#PWR0169"  Part="1"
+AR Path="/5CDAB6B1/5CEFE12E" Ref="#PWR095"  Part="1"
 AR Path="/5CE0453C/5CEFE12E" Ref="#PWR?"  Part="1"
 AR Path="/5CE8F13B/5CEFE12E" Ref="#PWR?"  Part="1"
 AR Path="/5CF5AEBC/5CEFE12E" Ref="#PWR?"  Part="1"
-F 0 "#PWR0169" H 7800 5450 50  0001 C CNN
+F 0 "#PWR095" H 7800 5450 50  0001 C CNN
 F 1 "GND" V 7850 5550 50  0000 R CNN
 F 2 "" H 7800 5700 50  0001 C CNN
@@
 $EndComp
 $Comp
-L power:+3V3 #PWR0157
+L power:+3V3 #PWR083
 U 1 1 5CFCEDE6
 P 3050 750
-F 0 "#PWR0157" H 3050 600 50  0001 C CNN
+F 0 "#PWR083" H 3050 600 50  0001 C CNN
 F 1 "+3V3" H 3100 950 50  0000 C CNN
 F 2 "" H 3050 750 50  0001 C CNN
@@
 Wire Wire Line
 	2050 4450 1550 4450
+Text HLabel 1550 4700 0    50   Input ~ 0
+ROT_ENC_A
+Text HLabel 1550 4800 0    50   Input ~ 0
+ROT_ENC_B
+Text Label 2050 4700 2    50   ~ 0
+PB8
+Wire Wire Line
+	2050 4700 1550 4700
+Text Label 2050 4800 2    50   ~ 0
+PB9
+Wire Wire Line
+	2050 4800 1550 4800
+Text HLabel 1550 4900 0    50   Input ~ 0
+ROT_ENC_SW
+Text Label 2050 4900 2    50   ~ 0
+PB10
+Wire Wire Line
+	2050 4900 1550 4900
 $EndSCHEMATC
