File: hardware/buzzer.sch (KiCad schematic (older format))
At the start: 0 parts

Commit message: update,
Parts:
- added BZ?: BUZZER,MLT-8530, footprint-lib:MLT-8530, symbol taobao-components:BUZZER,MLT-8530
- added D?: D_1N4148_T4, Diode_SMD:D_SOD-123, symbol taobao-d:D_1N4148_T4
- added Q?: SS9013_J3, footprint-lib:9013,J3,SOT23, symbol taobao-transistor:SS9013_J3
- added R?: R471,0603, Resistor_SMD:R_0603_1608Metric_Pad1.05x0.95mm_HandSolder, symbol taobao-r:R471,0603
Connections:
- new net: BZ?.N, D?.2 (A), Q?.3 (C)
- new net: Q?.1 (B), R?.1
- new net +3V3: BZ?.P, D?.1 (K)
- new net BUZZER_OUT: R?.2
- new net GND: Q?.2 (E)

Commit message: update,
Changed lines of the file:
@@
 U 1 1 5CECC56E
 P 4450 1950
-F 0 "D?" V 4400 2050 50  0000 L CNN
-F 1 "D_1N4148_T4" V 4450 2050 50  0000 L CNN
+F 0 "D?" V 4400 1850 50  0000 R CNN
+F 1 "D_1N4148_T4" V 4450 1850 50  0000 R CNN
 F 2 "Diode_SMD:D_SOD-123" V 4450 1950 50  0001 C CNN
 F 3 "~" V 4450 1950 50  0001 C CNN

Commit message: update,
Parts:
- gave numbers to parts that had none: 4
Connections:
- net BUZZER_OUT renamed BUZZER_IN
Changed lines of the file:
@@
 $Descr User 8500 5500
 encoding utf-8
-Sheet 20 27
+Sheet 15 20
 Title ""
 Date ""
@@
 $EndBitmap
 $Comp
-L power:+3V3 #PWR?
+L power:+3V3 #PWR0107
 U 1 1 5CEBF99F
 P 4600 1600
-F 0 "#PWR?" H 4600 1450 50  0001 C CNN
+F 0 "#PWR0107" H 4600 1450 50  0001 C CNN
 F 1 "+3V3" H 4650 1800 50  0000 C CNN
 F 2 "" H 4600 1600 50  0001 C CNN
@@
 $EndComp
 $Comp
-L taobao-components:BUZZER,MLT-8530 BZ?
+L taobao-components:BUZZER,MLT-8530 BZ1
 U 1 1 5CEC8447
 P 4750 1950
-F 0 "BZ?" H 4950 2000 50  0000 L CNN
+F 0 "BZ1" H 4950 2000 50  0000 L CNN
 F 1 "BUZZER,MLT-8530" H 4950 1900 50  0000 L CNN
 F 2 "footprint-lib:MLT-8530" V 4725 2050 50  0001 C CNN
@@
 $EndComp
 $Comp
-L taobao-transistor:SS9013_J3 Q?
+L taobao-transistor:SS9013_J3 Q1
 U 1 1 5CEC8A45
 P 4500 2500
-F 0 "Q?" H 4700 2550 50  0000 L CNN
+F 0 "Q1" H 4700 2550 50  0000 L CNN
 F 1 "SS9013_J3" H 4700 2500 50  0000 L CNN
 F 2 "footprint-lib:9013,J3,SOT23" H 4700 2425 50  0001 L CIN
@@
 $EndComp
 $Comp
-L taobao-r:R471,0603 R?
+L taobao-r:R471,0603 R28
 U 1 1 5CEC945D
 P 3850 2500
-F 0 "R?" V 3600 2500 50  0000 C CNN
+F 0 "R28" V 3600 2500 50  0000 C CNN
 F 1 "R471,0603" V 3700 2500 50  0000 C CNN
 F 2 "Resistor_SMD:R_0603_1608Metric_Pad1.05x0.95mm_HandSolder" H 3850 2500 50  0001 C CNN
@@
 	4600 2150 4600 2300
 $Comp
-L taobao-d:D_1N4148_T4 D?
+L taobao-d:D_1N4148_T4 D10
 U 1 1 5CECC56E
 P 4450 1950
-F 0 "D?" V 4400 1850 50  0000 R CNN
+F 0 "D10" V 4400 1850 50  0000 R CNN
 F 1 "D_1N4148_T4" V 4450 1850 50  0000 R CNN
 F 2 "Diode_SMD:D_SOD-123" V 4450 1950 50  0001 C CNN
@@
 $EndComp
 $Comp
-L power:GND #PWR?
+L power:GND #PWR0108
 U 1 1 5CECCC65
 P 4600 3000
-F 0 "#PWR?" H 4600 2750 50  0001 C CNN
+F 0 "#PWR0108" H 4600 2750 50  0001 C CNN
 F 1 "GND" H 4650 2800 50  0000 C CNN
 F 2 "" H 4600 3000 50  0001 C CNN
@@
 Wire Wire Line
 	4600 2700 4600 3000
-Text HLabel 3400 2500 0    50   Input ~ 0
-BUZZER_OUT
-Wire Wire Line
-	3400 2500 3750 2500
+Text HLabel 1050 700  0    50   Input ~ 0
+BUZZER_IN
 Wire Wire Line
 	3950 2500 4300 2500
+Text Label 1550 700  2    50   ~ 0
+TO_BUZZER
+Wire Wire Line
+	1050 700  1550 700
+Text Label 2900 2500 0    50   ~ 0
+TO_BUZZER
+Wire Wire Line
+	2900 2500 3750 2500
 $EndSCHEMATC

Commit message: update,
Parts:
- renumbered R28 to R23
Changed lines of the file:
@@
 $EndBitmap
 $Comp
-L power:+3V3 #PWR0107
+L power:+3V3 #PWR0100
 U 1 1 5CEBF99F
 P 4600 1600
-F 0 "#PWR0107" H 4600 1450 50  0001 C CNN
+F 0 "#PWR0100" H 4600 1450 50  0001 C CNN
 F 1 "+3V3" H 4650 1800 50  0000 C CNN
 F 2 "" H 4600 1600 50  0001 C CNN
@@
 $EndComp
 $Comp
-L taobao-r:R471,0603 R28
+L taobao-r:R471,0603 R23
 U 1 1 5CEC945D
 P 3850 2500
-F 0 "R28" V 3600 2500 50  0000 C CNN
+F 0 "R23" V 3600 2500 50  0000 C CNN
 F 1 "R471,0603" V 3700 2500 50  0000 C CNN
 F 2 "Resistor_SMD:R_0603_1608Metric_Pad1.05x0.95mm_HandSolder" H 3850 2500 50  0001 C CNN
@@
 $EndComp
 $Comp
-L power:GND #PWR0108
+L power:GND #PWR0101
 U 1 1 5CECCC65
 P 4600 3000
-F 0 "#PWR0108" H 4600 2750 50  0001 C CNN
+F 0 "#PWR0101" H 4600 2750 50  0001 C CNN
 F 1 "GND" H 4650 2800 50  0000 C CNN
 F 2 "" H 4600 3000 50  0001 C CNN

Commit message: update,
Parts:
- renumbered D10 to D9, R23 to R12
Changed lines of the file:
@@
 $EndBitmap
 $Comp
-L power:+3V3 #PWR0100
+L power:+3V3 #PWR062
 U 1 1 5CEBF99F
 P 4600 1600
-F 0 "#PWR0100" H 4600 1450 50  0001 C CNN
+F 0 "#PWR062" H 4600 1450 50  0001 C CNN
 F 1 "+3V3" H 4650 1800 50  0000 C CNN
 F 2 "" H 4600 1600 50  0001 C CNN
@@
 $EndComp
 $Comp
-L taobao-r:R471,0603 R23
+L taobao-r:R471,0603 R12
 U 1 1 5CEC945D
 P 3850 2500
-F 0 "R23" V 3600 2500 50  0000 C CNN
+F 0 "R12" V 3600 2500 50  0000 C CNN
 F 1 "R471,0603" V 3700 2500 50  0000 C CNN
 F 2 "Resistor_SMD:R_0603_1608Metric_Pad1.05x0.95mm_HandSolder" H 3850 2500 50  0001 C CNN
@@
 	4600 2150 4600 2300
 $Comp
-L taobao-d:D_1N4148_T4 D10
+L taobao-d:D_1N4148_T4 D9
 U 1 1 5CECC56E
 P 4450 1950
-F 0 "D10" V 4400 1850 50  0000 R CNN
+F 0 "D9" V 4400 1850 50  0000 R CNN
 F 1 "D_1N4148_T4" V 4450 1850 50  0000 R CNN
 F 2 "Diode_SMD:D_SOD-123" V 4450 1950 50  0001 C CNN
@@
 $EndComp
 $Comp
-L power:GND #PWR0101
+L power:GND #PWR063
 U 1 1 5CECCC65
 P 4600 3000
-F 0 "#PWR0101" H 4600 2750 50  0001 C CNN
+F 0 "#PWR063" H 4600 2750 50  0001 C CNN
 F 1 "GND" H 4650 2800 50  0000 C CNN
 F 2 "" H 4600 3000 50  0001 C CNN
