File: hardware/buzzer.sch (KiCad schematic (older format))
At the start: 4 parts, among them Q1 SS9013_J3

Commit message: update,
Parts:
- added J?: Conn_01x02_Female, symbol Connector:Conn_01x02_Female
Connections:
- wire segments 14 -> 17
Changed lines of the file:
@@
 Wire Wire Line
 	2900 2500 3750 2500
+$Comp
+L Connector:Conn_01x02_Female J?
+U 1 1 5CF28177
+P 2350 1750
+F 0 "J?" H 2200 1950 50  0000 C CNN
+F 1 "Conn_01x02_Female" H 2200 1850 50  0000 C CNN
+F 2 "" H 2350 1750 50  0001 C CNN
+F 3 "~" H 2350 1750 50  0001 C CNN
+	1    2350 1750
+	-1   0    0    -1
+$EndComp
+Text Label 3400 1750 2    50   ~ 0
+TO_BUZZER
+Wire Wire Line
+	3400 1750 2550 1750
+$Comp
+L power:GND #PWR?
+U 1 1 5CF28714
+P 2750 2000
+F 0 "#PWR?" H 2750 1750 50  0001 C CNN
+F 1 "GND" H 2800 1800 50  0000 C CNN
+F 2 "" H 2750 2000 50  0001 C CNN
+F 3 "" H 2750 2000 50  0001 C CNN
+	1    2750 2000
+	1    0    0    -1
+$EndComp
+Wire Wire Line
+	2550 1850 2750 1850
+Wire Wire Line
+	2750 1850 2750 2000
 $EndSCHEMATC

Commit message: update,
Parts:
- gave numbers to parts that had none: 1
- renumbered D9 to D12, R12 to R15
Changed lines of the file:
@@
 $EndBitmap
 $Comp
-L power:+3V3 #PWR062
+L power:+3V3 #PWR099
 U 1 1 5CEBF99F
 P 4600 1600
-F 0 "#PWR062" H 4600 1450 50  0001 C CNN
+F 0 "#PWR099" H 4600 1450 50  0001 C CNN
 F 1 "+3V3" H 4650 1800 50  0000 C CNN
 F 2 "" H 4600 1600 50  0001 C CNN
@@
 $EndComp
 $Comp
-L taobao-r:R471,0603 R12
+L taobao-r:R471,0603 R15
 U 1 1 5CEC945D
 P 3850 2500
-F 0 "R12" V 3600 2500 50  0000 C CNN
+F 0 "R15" V 3600 2500 50  0000 C CNN
 F 1 "R471,0603" V 3700 2500 50  0000 C CNN
 F 2 "Resistor_SMD:R_0603_1608Metric_Pad1.05x0.95mm_HandSolder" H 3850 2500 50  0001 C CNN
@@
 	4600 2150 4600 2300
 $Comp
-L taobao-d:D_1N4148_T4 D9
+L taobao-d:D_1N4148_T4 D12
 U 1 1 5CECC56E
 P 4450 1950
-F 0 "D9" V 4400 1850 50  0000 R CNN
+F 0 "D12" V 4400 1850 50  0000 R CNN
 F 1 "D_1N4148_T4" V 4450 1850 50  0000 R CNN
 F 2 "Diode_SMD:D_SOD-123" V 4450 1950 50  0001 C CNN
@@
 $EndComp
 $Comp
-L power:GND #PWR063
+L power:GND #PWR0101
 U 1 1 5CECCC65
 P 4600 3000
-F 0 "#PWR063" H 4600 2750 50  0001 C CNN
+F 0 "#PWR0101" H 4600 2750 50  0001 C CNN
 F 1 "GND" H 4650 2800 50  0000 C CNN
 F 2 "" H 4600 3000 50  0001 C CNN
@@
 	2900 2500 3750 2500
 $Comp
-L Connector:Conn_01x02_Female J?
+L Connector:Conn_01x02_Female J24
 U 1 1 5CF28177
 P 2350 1750
-F 0 "J?" H 2200 1950 50  0000 C CNN
+F 0 "J24" H 2200 1950 50  0000 C CNN
 F 1 "Conn_01x02_Female" H 2200 1850 50  0000 C CNN
 F 2 "" H 2350 1750 50  0001 C CNN
@@
 	3400 1750 2550 1750
 $Comp
-L power:GND #PWR?
+L power:GND #PWR0100
 U 1 1 5CF28714
 P 2750 2000
-F 0 "#PWR?" H 2750 1750 50  0001 C CNN
+F 0 "#PWR0100" H 2750 1750 50  0001 C CNN
 F 1 "GND" H 2800 1800 50  0000 C CNN
 F 2 "" H 2750 2000 50  0001 C CNN

Commit message: update footprint,
Parts:
- J24: value Conn_01x02_Female -> BUZZER_HEADER; footprint (none) -> Connector_PinHeader_1.27mm:PinHeader_1x02_P1.27mm_Vertical
Changed lines of the file:
@@
 P 2350 1750
 F 0 "J24" H 2200 1950 50  0000 C CNN
-F 1 "Conn_01x02_Female" H 2200 1850 50  0000 C CNN
-F 2 "" H 2350 1750 50  0001 C CNN
+F 1 "BUZZER_HEADER" H 2200 1850 50  0000 C CNN
+F 2 "Connector_PinHeader_1.27mm:PinHeader_1x02_P1.27mm_Vertical" H 2350 1750 50  0001 C CNN
 F 3 "~" H 2350 1750 50  0001 C CNN
 	1    2350 1750
