File: hardware/test_points.sch (KiCad schematic (older format))
At the start: 6 parts

Commit message: update,
Parts:
- gave numbers to parts that had none: 6
Changed lines of the file:
@@
 EESchema Schematic File Version 4
 LIBS:eval_board-cache
-LIBS:bb-ch340t-cache
 EELAYER 29 0
 EELAYER END
 $Descr A4 11693 8268
 encoding utf-8
-Sheet 22 20
+Sheet 22 22
 Title ""
 Date ""
@@
 $EndDescr
 $Comp
-L Connector:TestPoint TP?
+L Connector:TestPoint TP1
 U 1 1 5CDBAA14
 P 1450 1400
-F 0 "TP?" V 1400 1600 50  0000 L CNN
+F 0 "TP1" V 1400 1600 50  0000 L CNN
 F 1 "TestPoint" V 1450 1600 50  0000 L CNN
 F 2 "TestPoint:TestPoint_Pad_D4.0mm" H 1650 1400 50  0001 C CNN
@@
 $EndComp
 $Comp
-L power:GND #PWR?
+L power:GND #PWR0121
 U 1 1 5CDBACDA
 P 1350 900
-F 0 "#PWR?" H 1350 650 50  0001 C CNN
+F 0 "#PWR0121" H 1350 650 50  0001 C CNN
 F 1 "GND" V 1400 750 50  0000 R CNN
 F 2 "" H 1350 900 50  0001 C CNN
@@
 $EndComp
 $Comp
-L Connector:Conn_01x03_Male J?
+L Connector:Conn_01x03_Male J8
 U 1 1 5CDBBAA7
 P 1650 1150
-F 0 "J?" H 1600 1050 50  0000 R CNN
+F 0 "J8" H 1600 1050 50  0000 R CNN
 F 1 "Conn_01x03_Male" H 1600 1150 50  0000 R CNN
 F 2 "" H 1650 1150 50  0001 C CNN
@@
 Connection ~ 1300 1250
 $Comp
-L Connector:TestPoint TP?
+L Connector:TestPoint TP2
 U 1 1 5CDBDD6C
 P 2750 1400
-F 0 "TP?" V 2700 1600 50  0000 L CNN
+F 0 "TP2" V 2700 1600 50  0000 L CNN
 F 1 "TestPoint" V 2750 1600 50  0000 L CNN
 F 2 "TestPoint:TestPoint_Pad_D4.0mm" H 2950 1400 50  0001 C CNN
@@
 $EndComp
 $Comp
-L Connector:Conn_01x03_Male J?
+L Connector:Conn_01x03_Male J9
 U 1 1 5CDBDD80
 P 2950 1150
-F 0 "J?" H 2900 1050 50  0000 R CNN
+F 0 "J9" H 2900 1050 50  0000 R CNN
 F 1 "Conn_01x03_Male" H 2900 1150 50  0000 R CNN
 F 2 "" H 2950 1150 50  0001 C CNN
@@
 Connection ~ 2600 1250
 $Comp
-L power:+5V #PWR?
+L power:+5V #PWR0122
 U 1 1 5CDBECEF
 P 2650 900
-F 0 "#PWR?" H 2650 750 50  0001 C CNN
+F 0 "#PWR0122" H 2650 750 50  0001 C CNN
 F 1 "+5V" V 2650 1050 50  0000 L CNN
 F 2 "" H 2650 900 50  0001 C CNN
@@
 $EndComp
 $Comp
-L Connector:TestPoint TP?
+L Connector:TestPoint TP3
 U 1 1 5CDBEFA0
 P 3750 1400
-F 0 "TP?" V 3700 1600 50  0000 L CNN
+F 0 "TP3" V 3700 1600 50  0000 L CNN
 F 1 "TestPoint" V 3750 1600 50  0000 L CNN
 F 2 "TestPoint:TestPoint_Pad_D4.0mm" H 3950 1400 50  0001 C CNN
@@
 $EndComp
 $Comp
-L Connector:Conn_01x03_Male J?
+L Connector:Conn_01x03_Male J10
 U 1 1 5CDBEFAA
 P 3950 1150
-F 0 "J?" H 3900 1050 50  0000 R CNN
+F 0 "J10" H 3900 1050 50  0000 R CNN
 F 1 "Conn_01x03_Male" H 3900 1150 50  0000 R CNN
 F 2 "" H 3950 1150 50  0001 C CNN
@@
 Connection ~ 3600 1250
 $Comp
-L power:+3V3 #PWR?
+L power:+3V3 #PWR0123
 U 1 1 5CDBFA1A
 P 3650 900
-F 0 "#PWR?" H 3650 750 50  0001 C CNN
+F 0 "#PWR0123" H 3650 750 50  0001 C CNN
 F 1 "+3V3" V 3650 1050 50  0000 L CNN
 F 2 "" H 3650 900 50  0001 C CNN

Commit message: update,
Parts:
- J10: value Conn_01x03_Male -> 3V3
- J8: value Conn_01x03_Male -> GND
- J9: value Conn_01x03_Male -> 5V
Other:
- moved on the sheet: J10, J8, J9, TP1, TP2, TP3
Changed lines of the file:
@@
 EELAYER 29 0
 EELAYER END
-$Descr A4 11693 8268
+$Descr User 8500 5500
 encoding utf-8
-Sheet 22 22
+Sheet 18 22
 Title ""
 Date ""
@@
 L Connector:TestPoint TP1
 U 1 1 5CDBAA14
-P 1450 1400
-F 0 "TP1" V 1400 1600 50  0000 L CNN
-F 1 "TestPoint" V 1450 1600 50  0000 L CNN
-F 2 "TestPoint:TestPoint_Pad_D4.0mm" H 1650 1400 50  0001 C CNN
-F 3 "~" H 1650 1400 50  0001 C CNN
-	1    1450 1400
+P 2650 2700
+F 0 "TP1" V 2600 2900 50  0000 L CNN
+F 1 "TestPoint" V 2650 2900 50  0000 L CNN
+F 2 "TestPoint:TestPoint_Pad_D4.0mm" H 2850 2700 50  0001 C CNN
+F 3 "~" H 2850 2700 50  0001 C CNN
+	1    2650 2700
 	0    1    1    0
 $EndComp
@@
 L power:GND #PWR0121
 U 1 1 5CDBACDA
-P 1350 900
-F 0 "#PWR0121" H 1350 650 50  0001 C CNN
-F 1 "GND" V 1400 750 50  0000 R CNN
-F 2 "" H 1350 900 50  0001 C CNN
-F 3 "" H 1350 900 50  0001 C CNN
-	1    1350 900
+P 2550 2200
+F 0 "#PWR0121" H 2550 1950 50  0001 C CNN
+F 1 "GND" V 2600 2050 50  0000 R CNN
+F 2 "" H 2550 2200 50  0001 C CNN
+F 3 "" H 2550 2200 50  0001 C CNN
+	1    2550 2200
 	0    -1   -1   0
 $EndComp
@@
 L Connector:Conn_01x03_Male J8
 U 1 1 5CDBBAA7
-P 1650 1150
-F 0 "J8" H 1600 1050 50  0000 R CNN
-F 1 "Conn_01x03_Male" H 1600 1150 50  0000 R CNN
-F 2 "" H 1650 1150 50  0001 C CNN
-F 3 "~" H 1650 1150 50  0001 C CNN
-	1    1650 1150
+P 2850 2450
+F 0 "J8" H 2800 2350 50  0000 R CNN
+F 1 "GND" H 2800 2450 50  0000 R CNN
+F 2 "" H 2850 2450 50  0001 C CNN
+F 3 "~" H 2850 2450 50  0001 C CNN
+	1    2850 2450
 	-1   0    0    1
 $EndComp
 Wire Wire Line
-	1350 900  1300 900
+	2550 2200 2500 2200
 Wire Wire Line
-	1300 900  1300 1050
+	2500 2200 2500 2350
 Wire Wire Line
-	1300 1050 1450 1050
+	2500 2350 2650 2350
 Wire Wire Line
-	1300 1050 1300 1150
+	2500 2350 2500 2450
 Wire Wire Line
-	1300 1150 1450 1150
-Connection ~ 1300 1050
+	2500 2450 2650 2450
+Connection ~ 2500 2350
 Wire Wire Line
-	1300 1150 1300 1250
+	2500 2450 2500 2550
 Wire Wire Line
-	1300 1250 1450 1250
-Connection ~ 1300 1150
+	2500 2550 2650 2550
+Connection ~ 2500 2450
 Wire Wire Line
-	1300 1250 1300 1400
+	2500 2550 2500 2700
 Wire Wire Line
-	1300 1400 1450 1400
-Connection ~ 1300 1250
+	2500 2700 2650 2700
+Connection ~ 2500 2550
 $Comp
 L Connector:TestPoint TP2
 U 1 1 5CDBDD6C
-P 2750 1400
-F 0 "TP2" V 2700 1600 50  0000 L CNN
-F 1 "TestPoint" V 2750 1600 50  0000 L CNN
-F 2 "TestPoint:TestPoint_Pad_D4.0mm" H 2950 1400 50  0001 C CNN
-F 3 "~" H 2950 1400 50  0001 C CNN
-	1    2750 1400
+P 3950 2700
+F 0 "TP2" V 3900 2900 50  0000 L CNN
+F 1 "TestPoint" V 3950 2900 50  0000 L CNN
+F 2 "TestPoint:TestPoint_Pad_D4.0mm" H 4150 2700 50  0001 C CNN
+F 3 "~" H 4150 2700 50  0001 C CNN
+	1    3950 2700
 	0    1    1    0
 $EndComp
@@
 L Connector:Conn_01x03_Male J9
 U 1 1 5CDBDD80
-P 2950 1150
-F 0 "J9" H 2900 1050 50  0000 R CNN
-F 1 "Conn_01x03_Male" H 2900 1150 50  0000 R CNN
-F 2 "" H 2950 1150 50  0001 C CNN
-F 3 "~" H 2950 1150 50  0001 C CNN
-	1    2950 1150
+P 4150 2450
+F 0 "J9" H 4100 2350 50  0000 R CNN
+F 1 "5V" H 4100 2450 50  0000 R CNN
+F 2 "" H 4150 2450 50  0001 C CNN
+F 3 "~" H 4150 2450 50  0001 C CNN
+	1    4150 2450
 	-1   0    0    1
 $EndComp
 Wire Wire Line
-	2650 900  2600 900
+	3850 2200 3800 2200
 Wire Wire Line
-	2600 900  2600 1050
+	3800 2200 3800 2350
 Wire Wire Line
-	2600 1050 2750 1050
+	3800 2350 3950 2350
 Wire Wire Line
-	2600 1050 2600 1150
+	3800 2350 3800 2450
 Wire Wire Line
-	2600 1150 2750 1150
-Connection ~ 2600 1050
+	3800 2450 3950 2450
+Connection ~ 3800 2350
 Wire Wire Line
-	2600 1150 2600 1250
+	3800 2450 3800 2550
 Wire Wire Line
-	2600 1250 2750 1250
-Connection ~ 2600 1150
+	3800 2550 3950 2550
+Connection ~ 3800 2450
 Wire Wire Line
-	2600 1250 2600 1400
+	3800 2550 3800 2700
 Wire Wire Line
-	2600 1400 2750 1400
-Connection ~ 2600 1250
+	3800 2700 3950 2700
+Connection ~ 3800 2550
 $Comp
 L power:+5V #PWR0122
 U 1 1 5CDBECEF
-P 2650 900
-F 0 "#PWR0122" H 2650 750 50  0001 C CNN
-F 1 "+5V" V 2650 1050 50  0000 L CNN
-F 2 "" H 2650 900 50  0001 C CNN
-F 3 "" H 2650 900 50  0001 C CNN
-	1    2650 900
+P 3850 2200
+F 0 "#PWR0122" H 3850 2050 50  0001 C CNN
+F 1 "+5V" V 3850 2350 50  0000 L CNN
+F 2 "" H 3850 2200 50  0001 C CNN
+F 3 "" H 3850 2200 50  0001 C CNN
+	1    3850 2200
 	0    1    1    0
 $EndComp
@@
 L Connector:TestPoint TP3
 U 1 1 5CDBEFA0
-P 3750 1400
-F 0 "TP3" V 3700 1600 50  0000 L CNN
-F 1 "TestPoint" V 3750 1600 50  0000 L CNN
-F 2 "TestPoint:TestPoint_Pad_D4.0mm" H 3950 1400 50  0001 C CNN
-F 3 "~" H 3950 1400 50  0001 C CNN
-	1    3750 1400
+P 4950 2700
+F 0 "TP3" V 4900 2900 50  0000 L CNN
+F 1 "TestPoint" V 4950 2900 50  0000 L CNN
+F 2 "TestPoint:TestPoint_Pad_D4.0mm" H 5150 2700 50  0001 C CNN
+F 3 "~" H 5150 2700 50  0001 C CNN
+	1    4950 2700
 	0    1    1    0
 $EndComp
@@
 L Connector:Conn_01x03_Male J10
 U 1 1 5CDBEFAA
-P 3950 1150
-F 0 "J10" H 3900 1050 50  0000 R CNN
-F 1 "Conn_01x03_Male" H 3900 1150 50  0000 R CNN
-F 2 "" H 3950 1150 50  0001 C CNN
-F 3 "~" H 3950 1150 50  0001 C CNN
-	1    3950 1150
+P 5150 2450
+F 0 "J10" H 5100 2350 50  0000 R CNN
+F 1 "3V3" H 5100 2450 50  0000 R CNN
+F 2 "" H 5150 2450 50  0001 C CNN
+F 3 "~" H 5150 2450 50  0001 C CNN
+	1    5150 2450
 	-1   0    0    1
 $EndComp
 Wire Wire Line
-	3650 900  3600 900
+	4850 2200 4800 2200
 Wire Wire Line
-	3600 900  3600 1050
+	4800 2200 4800 2350
 Wire Wire Line
-	3600 1050 3750 1050
+	4800 2350 4950 2350
 Wire Wire Line
-	3600 1050 3600 1150
+	4800 2350 4800 2450
 Wire Wire Line
-	3600 1150 3750 1150
-Connection ~ 3600 1050
+	4800 2450 4950 2450
+Connection ~ 4800 2350
 Wire Wire Line
-	3600 1150 3600 1250
+	4800 2450 4800 2550
 Wire Wire Line
-	3600 1250 3750 1250
-Connection ~ 3600 1150
+	4800 2550 4950 2550
+Connection ~ 4800 2450
 Wire Wire Line
-	3600 1250 3600 1400
+	4800 2550 4800 2700
 Wire Wire Line
-	3600 1400 3750 1400
-Connection ~ 3600 1250
+	4800 2700 4950 2700
+Connection ~ 4800 2550
 $Comp
 L power:+3V3 #PWR0123
 U 1 1 5CDBFA1A
-P 3650 900
-F 0 "#PWR0123" H 3650 750 50  0001 C CNN
-F 1 "+3V3" V 3650 1050 50  0000 L CNN
-F 2 "" H 3650 900 50  0001 C CNN
-F 3 "" H 3650 900 50  0001 C CNN
-	1    3650 900
+P 4850 2200
+F 0 "#PWR0123" H 4850 2050 50  0001 C CNN
+F 1 "+3V3" V 4850 2350 50  0000 L CNN
+F 2 "" H 4850 2200 50  0001 C CNN
+F 3 "" H 4850 2200 50  0001 C CNN
+	1    4850 2200
 	0    1    1    0
 $EndComp

Commit message: update,
Parts:
- renumbered J8 to J12, J9 to J13, J10 to J14
Changed lines of the file:
@@
 $Descr User 8500 5500
 encoding utf-8
-Sheet 18 27
+Sheet 14 20
 Title ""
 Date ""
@@
 $EndComp
 $Comp
-L power:GND #PWR0121
+L power:GND #PWR062
 U 1 1 5CDBACDA
 P 2550 2200
-F 0 "#PWR0121" H 2550 1950 50  0001 C CNN
+F 0 "#PWR062" H 2550 1950 50  0001 C CNN
 F 1 "GND" V 2600 2050 50  0000 R CNN
 F 2 "" H 2550 2200 50  0001 C CNN
@@
 $EndComp
 $Comp
-L Connector:Conn_01x03_Male J8
+L Connector:Conn_01x03_Male J12
 U 1 1 5CDBBAA7
 P 2850 2450
-F 0 "J8" H 2800 2350 50  0000 R CNN
+F 0 "J12" H 2800 2350 50  0000 R CNN
 F 1 "GND" H 2800 2450 50  0000 R CNN
 F 2 "" H 2850 2450 50  0001 C CNN
@@
 $EndComp
 $Comp
-L Connector:Conn_01x03_Male J9
+L Connector:Conn_01x03_Male J13
 U 1 1 5CDBDD80
 P 4150 2450
-F 0 "J9" H 4100 2350 50  0000 R CNN
+F 0 "J13" H 4100 2350 50  0000 R CNN
 F 1 "5V" H 4100 2450 50  0000 R CNN
 F 2 "" H 4150 2450 50  0001 C CNN
@@
 Connection ~ 3800 2550
 $Comp
-L power:+5V #PWR0122
+L power:+5V #PWR063
 U 1 1 5CDBECEF
 P 3850 2200
-F 0 "#PWR0122" H 3850 2050 50  0001 C CNN
+F 0 "#PWR063" H 3850 2050 50  0001 C CNN
 F 1 "+5V" V 3850 2350 50  0000 L CNN
 F 2 "" H 3850 2200 50  0001 C CNN
@@
 $EndComp
 $Comp
-L Connector:Conn_01x03_Male J10
+L Connector:Conn_01x03_Male J14
 U 1 1 5CDBEFAA
 P 5150 2450
-F 0 "J10" H 5100 2350 50  0000 R CNN
+F 0 "J14" H 5100 2350 50  0000 R CNN
 F 1 "3V3" H 5100 2450 50  0000 R CNN
 F 2 "" H 5150 2450 50  0001 C CNN
@@
 Connection ~ 4800 2550
 $Comp
-L power:+3V3 #PWR0123
+L power:+3V3 #PWR064
 U 1 1 5CDBFA1A
 P 4850 2200
-F 0 "#PWR0123" H 4850 2050 50  0001 C CNN
+F 0 "#PWR064" H 4850 2050 50  0001 C CNN
 F 1 "+3V3" V 4850 2350 50  0000 L CNN
 F 2 "" H 4850 2200 50  0001 C CNN

Commit message: update,
Parts:
- renumbered J12 to J11, J13 to J12, J14 to J13
Changed lines of the file:
@@
 $EndComp
 $Comp
-L power:GND #PWR062
+L power:GND #PWR055
 U 1 1 5CDBACDA
 P 2550 2200
-F 0 "#PWR062" H 2550 1950 50  0001 C CNN
+F 0 "#PWR055" H 2550 1950 50  0001 C CNN
 F 1 "GND" V 2600 2050 50  0000 R CNN
 F 2 "" H 2550 2200 50  0001 C CNN
@@
 $EndComp
 $Comp
-L Connector:Conn_01x03_Male J12
+L Connector:Conn_01x03_Male J11
 U 1 1 5CDBBAA7
 P 2850 2450
-F 0 "J12" H 2800 2350 50  0000 R CNN
+F 0 "J11" H 2800 2350 50  0000 R CNN
 F 1 "GND" H 2800 2450 50  0000 R CNN
 F 2 "" H 2850 2450 50  0001 C CNN
@@
 $EndComp
 $Comp
-L Connector:Conn_01x03_Male J13
+L Connector:Conn_01x03_Male J12
 U 1 1 5CDBDD80
 P 4150 2450
-F 0 "J13" H 4100 2350 50  0000 R CNN
+F 0 "J12" H 4100 2350 50  0000 R CNN
 F 1 "5V" H 4100 2450 50  0000 R CNN
 F 2 "" H 4150 2450 50  0001 C CNN
@@
 Connection ~ 3800 2550
 $Comp
-L power:+5V #PWR063
+L power:+5V #PWR056
 U 1 1 5CDBECEF
 P 3850 2200
-F 0 "#PWR063" H 3850 2050 50  0001 C CNN
+F 0 "#PWR056" H 3850 2050 50  0001 C CNN
 F 1 "+5V" V 3850 2350 50  0000 L CNN
 F 2 "" H 3850 2200 50  0001 C CNN
@@
 $EndComp
 $Comp
-L Connector:Conn_01x03_Male J14
+L Connector:Conn_01x03_Male J13
 U 1 1 5CDBEFAA
 P 5150 2450
-F 0 "J14" H 5100 2350 50  0000 R CNN
+F 0 "J13" H 5100 2350 50  0000 R CNN
 F 1 "3V3" H 5100 2450 50  0000 R CNN
 F 2 "" H 5150 2450 50  0001 C CNN
@@
 Connection ~ 4800 2550
 $Comp
-L power:+3V3 #PWR064
+L power:+3V3 #PWR057
 U 1 1 5CDBFA1A
 P 4850 2200
-F 0 "#PWR064" H 4850 2050 50  0001 C CNN
+F 0 "#PWR057" H 4850 2050 50  0001 C CNN
 F 1 "+3V3" V 4850 2350 50  0000 L CNN
 F 2 "" H 4850 2200 50  0001 C CNN

Commit message: update,
Parts:
- renumbered J11 to J12, J12 to J13, J13 to J14
Changed lines of the file:
@@
 $EndComp
 $Comp
-L power:GND #PWR055
+L power:GND #PWR059
 U 1 1 5CDBACDA
 P 2550 2200
-F 0 "#PWR055" H 2550 1950 50  0001 C CNN
+F 0 "#PWR059" H 2550 1950 50  0001 C CNN
 F 1 "GND" V 2600 2050 50  0000 R CNN
 F 2 "" H 2550 2200 50  0001 C CNN
@@
 $EndComp
 $Comp
-L Connector:Conn_01x03_Male J11
+L Connector:Conn_01x03_Male J12
 U 1 1 5CDBBAA7
 P 2850 2450
-F 0 "J11" H 2800 2350 50  0000 R CNN
+F 0 "J12" H 2800 2350 50  0000 R CNN
 F 1 "GND" H 2800 2450 50  0000 R CNN
 F 2 "" H 2850 2450 50  0001 C CNN
@@
 $EndComp
 $Comp
-L Connector:Conn_01x03_Male J12
+L Connector:Conn_01x03_Male J13
 U 1 1 5CDBDD80
 P 4150 2450
-F 0 "J12" H 4100 2350 50  0000 R CNN
+F 0 "J13" H 4100 2350 50  0000 R CNN
 F 1 "5V" H 4100 2450 50  0000 R CNN
 F 2 "" H 4150 2450 50  0001 C CNN
@@
 Connection ~ 3800 2550
 $Comp
-L power:+5V #PWR056
+L power:+5V #PWR060
 U 1 1 5CDBECEF
 P 3850 2200
-F 0 "#PWR056" H 3850 2050 50  0001 C CNN
+F 0 "#PWR060" H 3850 2050 50  0001 C CNN
 F 1 "+5V" V 3850 2350 50  0000 L CNN
 F 2 "" H 3850 2200 50  0001 C CNN
@@
 $EndComp
 $Comp
-L Connector:Conn_01x03_Male J13
+L Connector:Conn_01x03_Male J14
 U 1 1 5CDBEFAA
 P 5150 2450
-F 0 "J13" H 5100 2350 50  0000 R CNN
+F 0 "J14" H 5100 2350 50  0000 R CNN
 F 1 "3V3" H 5100 2450 50  0000 R CNN
 F 2 "" H 5150 2450 50  0001 C CNN
@@
 Connection ~ 4800 2550
 $Comp
-L power:+3V3 #PWR057
+L power:+3V3 #PWR061
 U 1 1 5CDBFA1A
 P 4850 2200
-F 0 "#PWR057" H 4850 2050 50  0001 C CNN
+F 0 "#PWR061" H 4850 2050 50  0001 C CNN
 F 1 "+3V3" V 4850 2350 50  0000 L CNN
 F 2 "" H 4850 2200 50  0001 C CNN
