File: hardware/arduino_nano.sch (KiCad schematic (older format))
At the start: 4 parts, among them J18 I2C_HEADER, J19 TTL_HEADER, J20 SPI_HEADER, U8 arduino_nano_v3

Commit message: update,
Connections:
- net D3 renamed WS2812_OUT
- net D4 renamed OLED_DC
- net D5 renamed OLED_RST
- net D6 renamed OLED_SS
Changed lines of the file:
@@
 $Descr A4 11693 8268
 encoding utf-8
-Sheet 16 18
+Sheet 14 19
 Title ""
 Date ""
@@
 Text Label 2900 750  2    50   ~ 0
 SCL
+Text HLabel 1200 2650 0    50   Input ~ 0
+PWM
+Text HLabel 1200 2750 0    50   Input ~ 0
+WS2812_OUT
+Wire Wire Line
+	1600 2650 1200 2650
+Text Label 1600 2650 2    50   ~ 0
+D2
+Wire Wire Line
+	1600 2750 1200 2750
+Text Label 1600 2750 2    50   ~ 0
+D3
+Text HLabel 1200 3050 0    50   Input ~ 0
+OLED_DC
+Wire Wire Line
+	1600 3050 1200 3050
+Text Label 1600 3050 2    50   ~ 0
+D4
+Text HLabel 1200 3150 0    50   Input ~ 0
+OLED_RST
+Wire Wire Line
+	1600 3150 1200 3150
+Text Label 1600 3150 2    50   ~ 0
+D5
+Text HLabel 1200 3250 0    50   Input ~ 0
+OLED_SS
+Wire Wire Line
+	1600 3250 1200 3250
+Text Label 1600 3250 2    50   ~ 0
+D6
 $EndSCHEMATC

Commit message: update,
Parts:
- renumbered J18 to J23, J19 to J24, J20 to J25, U8 to U10
Changed lines of the file:
@@
 $Descr A4 11693 8268
 encoding utf-8
-Sheet 14 19
+Sheet 19 19
 Title ""
 Date ""
@@
 $EndDescr
 $Comp
-L taobao-board:Arduino_Nano_V3 U8
+L taobao-board:Arduino_Nano_V3 U10
 U 1 1 5CE64286
 P 3200 2850
-F 0 "U8" H 3200 1800 50  0000 C CNN
+F 0 "U10" H 3200 1800 50  0000 C CNN
 F 1 "arduino_nano_v3" H 3200 1900 50  0000 C CNN
 F 2 "Module:Arduino_Nano" H 3100 1650 50  0001 C CNN
@@
 	2000 3500 2650 3500
 $Comp
-L taobao-components:SPI_HEADER J20
+L taobao-components:SPI_HEADER J25
 U 1 1 5D1622BE
 P 2300 1700
-F 0 "J20" H 2450 2050 50  0000 C CNN
+F 0 "J25" H 2450 2050 50  0000 C CNN
 F 1 "SPI_HEADER" H 2450 1950 50  0000 C CNN
 F 2 "footprint-lib:SPI_DEBUG" H 2300 1300 50  0001 C CNN
@@
 	2500 1750 3200 1750
 $Comp
-L taobao-components:TTL_HEADER J19
+L taobao-components:TTL_HEADER J24
 U 1 1 5D16605D
 P 2500 1200
-F 0 "J19" H 2450 1500 50  0000 C CNN
+F 0 "J24" H 2450 1500 50  0000 C CNN
 F 1 "TTL_HEADER" H 2450 1400 50  0000 C CNN
 F 2 "footprint-lib:TTL_HEADER" H 2500 800 50  0001 C CNN
@@
 $EndComp
 $Comp
-L power:GND #PWR0102
+L power:GND #PWR0101
 U 1 1 5D166AA6
 P 2900 1100
-F 0 "#PWR0102" H 2900 850 50  0001 C CNN
+F 0 "#PWR0101" H 2900 850 50  0001 C CNN
 F 1 "GND" V 2950 950 50  0000 R CNN
 F 2 "" H 2900 1100 50  0001 C CNN
@@
 A1
 $Comp
-L power:+5V #PWR0103
+L power:+5V #PWR0102
 U 1 1 5D18525B
 P 4300 2050
-F 0 "#PWR0103" H 4300 1900 50  0001 C CNN
+F 0 "#PWR0102" H 4300 1900 50  0001 C CNN
 F 1 "+5V" H 4350 2250 50  0000 C CNN
 F 2 "" H 4300 2050 50  0001 C CNN
@@
 Connection ~ 4300 2200
 $Comp
-L power:GND #PWR0104
+L power:GND #PWR0103
 U 1 1 5D188630
 P 4500 2400
-F 0 "#PWR0104" H 4500 2150 50  0001 C CNN
+F 0 "#PWR0103" H 4500 2150 50  0001 C CNN
 F 1 "GND" H 4550 2200 50  0000 C CNN
 F 2 "" H 4500 2400 50  0001 C CNN
@@
 	3800 2300 4500 2300
 $Comp
-L taobao-components:I2C_HEADER J18
+L taobao-components:I2C_HEADER J23
 U 1 1 5D190CE0
 P 2300 700
-F 0 "J18" H 2450 950 50  0000 C CNN
+F 0 "J23" H 2450 950 50  0000 C CNN
 F 1 "I2C_HEADER" H 2450 850 50  0000 C CNN
 F 2 "footprint-lib:I2C_DEBUG" H 2300 300 50  0001 C CNN

Commit message: update,
Parts:
- added J26, J27: Conn_01x15_Female, symbol Connector:Conn_01x15_Female
Connections:
- net +5V: now also J27.1 (Pin_1), J27.4 (Pin_4)
- net 3V3: now also J27.14 (Pin_14)
- net A2: now also J27.10 (Pin_10)
- net A3: now also J27.9 (Pin_9)
- net A6: now also J27.6 (Pin_6)
- net A7: now also J27.5 (Pin_5)
- net AREF: now also J27.13 (Pin_13)
- net D7: now also J26.10 (Pin_10)
- net D8: now also J26.11 (Pin_11)
- net D9: now also J26.12 (Pin_12)
- net GND: now also J26.4 (Pin_4), J27.2 (Pin_2)
- net MISO: now also J26.15 (Pin_15)
- net MOSI: now also J26.14 (Pin_14)
- net OLED_DC: now also J26.7 (Pin_7)
- net OLED_RST: now also J26.8 (Pin_8)
- net OLED_SS: now also J26.9 (Pin_9)
- net RST: now also J26.3 (Pin_3), J27.3 (Pin_3)
- net SCK: now also J27.15 (Pin_15)
- net SCL: now also J27.7 (Pin_7)
- net SDA: now also J27.8 (Pin_8)
- net SS: now also J26.13 (Pin_13)
- net A_IN0 renamed A0
- net A0: now also J27.12 (Pin_12)
- net A_IN1 renamed A1
- net A1: now also J27.11 (Pin_11)
- net PWM renamed D2
- net D2: now also J26.5 (Pin_5)
- net RXD renamed D0
- net D0: now also J26.2 (Pin_2)
- net TXD renamed D1
- net D1: now also J26.1 (Pin_1)
- net WS2812_OUT renamed D3
- net D3: now also J26.6 (Pin_6)
Changed lines of the file:
@@
 	2250 2600 2650 2600
 Wire Wire Line
-	2250 2700 2650 2700
-Wire Wire Line
 	2250 2800 2650 2800
 Wire Wire Line
@@
 Text Label 2250 2500 0    50   ~ 0
 GND
-Text Label 2250 2400 0    50   ~ 0
-RST
 Wire Wire Line
 	2650 2500 2250 2500
@@
 Text Label 4200 2200 2    50   ~ 0
 VIN
-Text HLabel 1200 1200 0    50   Input ~ 0
-TXD
-Text HLabel 1200 1300 0    50   Input ~ 0
-RXD
 $Bitmap
 Pos -950 800
@@
 EndData
 $EndBitmap
-Text HLabel 1200 2050 0    50   Input ~ 0
-PWM
-Wire Wire Line
-	1600 2050 1200 2050
-Text Label 1600 2050 2    50   ~ 0
-D2
 Text HLabel 1200 1550 0    50   Input ~ 0
 SS
@@
 Wire Wire Line
 	2050 2300 2650 2300
-Text Label 1600 1200 2    50   ~ 0
-TX
-Wire Wire Line
-	1600 1200 1200 1200
-Wire Wire Line
-	1600 1300 1200 1300
-Text Label 1600 1300 2    50   ~ 0
-RX
 Text Label 4400 2800 2    50   ~ 0
 SCL
@@
 Wire Wire Line
 	3800 2900 4400 2900
-Text HLabel 1200 2250 0    50   Input ~ 0
-A_IN0
-Text HLabel 1200 2350 0    50   Input ~ 0
-A_IN1
-Wire Wire Line
-	1600 2250 1200 2250
-Text Label 1600 2250 2    50   ~ 0
-A0
-Wire Wire Line
-	1600 2350 1200 2350
-Text Label 1600 2350 2    50   ~ 0
-A1
 $Comp
 L power:+5V #PWR0102
@@
 Text Label 2900 750  2    50   ~ 0
 SCL
-Text HLabel 1200 2650 0    50   Input ~ 0
-PWM
-Text HLabel 1200 2750 0    50   Input ~ 0
-WS2812_OUT
-Wire Wire Line
-	1600 2650 1200 2650
-Text Label 1600 2650 2    50   ~ 0
-D2
+Text Label 1600 3250 2    50   ~ 0
+D6
 Wire Wire Line
-	1600 2750 1200 2750
-Text Label 1600 2750 2    50   ~ 0
-D3
-Text HLabel 1200 3050 0    50   Input ~ 0
-OLED_DC
+	1600 3250 1200 3250
+Text HLabel 1200 3250 0    50   Input ~ 0
+OLED_SS
+Text Label 1600 3150 2    50   ~ 0
+D5
 Wire Wire Line
-	1600 3050 1200 3050
-Text Label 1600 3050 2    50   ~ 0
-D4
+	1600 3150 1200 3150
 Text HLabel 1200 3150 0    50   Input ~ 0
 OLED_RST
+Text Label 1600 3050 2    50   ~ 0
+D4
 Wire Wire Line
-	1600 3150 1200 3150
-Text Label 1600 3150 2    50   ~ 0
+	1600 3050 1200 3050
+Text HLabel 1200 3050 0    50   Input ~ 0
+OLED_DC
+Text Label 2250 2400 0    50   ~ 0
+RST
+$Comp
+L Connector:Conn_01x15_Female J26
+U 1 1 5CEF6157
+P 3050 4900
+F 0 "J26" H 3100 4950 50  0000 L CNN
+F 1 "Conn_01x15_Female" H 3100 4850 50  0000 L CNN
+F 2 "" H 3050 4900 50  0001 C CNN
+F 3 "~" H 3050 4900 50  0001 C CNN
+	1    3050 4900
+	1    0    0    -1
+$EndComp
+$Comp
+L Connector:Conn_01x15_Female J27
+U 1 1 5CEF7253
+P 3400 4900
+F 0 "J27" H 3250 5800 50  0000 C CNN
+F 1 "Conn_01x15_Female" H 3250 5700 50  0000 C CNN
+F 2 "" H 3400 4900 50  0001 C CNN
+F 3 "~" H 3400 4900 50  0001 C CNN
+	1    3400 4900
+	-1   0    0    -1
+$EndComp
+Text Label 2450 4200 0    50   ~ 0
+D1
+Text Label 2450 4300 0    50   ~ 0
+D0
+Text Label 2450 4600 0    50   ~ 0
+D2
+Text Label 2450 4700 0    50   ~ 0
+D3
+Text Label 2450 4800 0    50   ~ 0
+D4
+Text Label 2450 4900 0    50   ~ 0
 D5
-Text HLabel 1200 3250 0    50   Input ~ 0
-OLED_SS
-Wire Wire Line
-	1600 3250 1200 3250
-Text Label 1600 3250 2    50   ~ 0
+Text Label 2450 5000 0    50   ~ 0
 D6
+Text Label 2450 5100 0    50   ~ 0
+D7
+Text Label 2450 5200 0    50   ~ 0
+D8
+Text Label 2450 5300 0    50   ~ 0
+D9
+Text Label 2450 5400 0    50   ~ 0
+D10
+Text Label 2450 5500 0    50   ~ 0
+D11
+Text Label 2450 5600 0    50   ~ 0
+D12
+Wire Wire Line
+	2450 4600 2850 4600
+Wire Wire Line
+	2450 4700 2850 4700
+Wire Wire Line
+	2450 4800 2850 4800
+Wire Wire Line
+	2450 4900 2850 4900
+Wire Wire Line
+	2450 5000 2850 5000
+Wire Wire Line
+	2450 5100 2850 5100
+Wire Wire Line
+	2450 5200 2850 5200
+Wire Wire Line
+	2450 5300 2850 5300
+Text Label 2450 4500 0    50   ~ 0
+GND
+Wire Wire Line
+	2850 4500 2450 4500
+Wire Wire Line
+	2850 4400 2450 4400
+Text Label 2200 5400 0    50   ~ 0
+SS
+Text Label 2200 5500 0    50   ~ 0
+MOSI
+Text Label 2200 5600 0    50   ~ 0
+MISO
+Wire Wire Line
+	2200 5400 2850 5400
+Wire Wire Line
+	2200 5600 2850 5600
+Wire Wire Line
+	2200 5500 2850 5500
+Text Label 2250 4200 0    50   ~ 0
+TX
+Text Label 2250 4300 0    50   ~ 0
+RX
+Wire Wire Line
+	2250 4200 2850 4200
+Wire Wire Line
+	2250 4300 2850 4300
+Text Label 2450 4400 0    50   ~ 0
+RST
+Text Label 4000 4300 2    50   ~ 0
+GND
+Text Label 4000 4400 2    50   ~ 0
+RST
+Text Label 4000 4500 2    50   ~ 0
+5V
+Text Label 4000 4600 2    50   ~ 0
+A7
+Text Label 4000 4700 2    50   ~ 0
+A6
+Text Label 4000 4800 2    50   ~ 0
+A5
+Text Label 4000 4900 2    50   ~ 0
+A4
+Text Label 4000 5000 2    50   ~ 0
+A3
+Text Label 4000 5100 2    50   ~ 0
+A2
+Text Label 4000 5200 2    50   ~ 0
+A1
+Text Label 4000 5300 2    50   ~ 0
+A0
+Text Label 4000 5400 2    50   ~ 0
+AREF
+Text Label 4000 5500 2    50   ~ 0
+3V3
+Text Label 4000 5600 2    50   ~ 0
+D13
+Wire Wire Line
+	3600 4400 4000 4400
+Wire Wire Line
+	3600 4600 4000 4600
+Wire Wire Line
+	3600 4700 4000 4700
+Wire Wire Line
+	3600 5000 4000 5000
+Wire Wire Line
+	3600 5100 4000 5100
+Wire Wire Line
+	3600 5200 4000 5200
+Wire Wire Line
+	3600 5300 4000 5300
+Wire Wire Line
+	3600 5400 4000 5400
+Wire Wire Line
+	3600 5500 4000 5500
+Text Label 4000 4200 2    50   ~ 0
+VIN
+Text Label 4300 5600 2    50   ~ 0
+SCK
+Wire Wire Line
+	3600 5600 4300 5600
+Text Label 4200 4800 2    50   ~ 0
+SCL
+Text Label 4200 4900 2    50   ~ 0
+SDA
+Wire Wire Line
+	3600 4800 4200 4800
+Wire Wire Line
+	3600 4900 4200 4900
+$Comp
+L power:+5V #PWR0104
+U 1 1 5CEFA9B2
+P 4100 4050
+F 0 "#PWR0104" H 4100 3900 50  0001 C CNN
+F 1 "+5V" H 4150 4250 50  0000 C CNN
+F 2 "" H 4100 4050 50  0001 C CNN
+F 3 "" H 4100 4050 50  0001 C CNN
+	1    4100 4050
+	1    0    0    -1
+$EndComp
+Wire Wire Line
+	4100 4050 4100 4200
+Wire Wire Line
+	3600 4200 4100 4200
+Wire Wire Line
+	4100 4200 4100 4500
+Wire Wire Line
+	3600 4500 4100 4500
+Connection ~ 4100 4200
+$Comp
+L power:GND #PWR0105
+U 1 1 5CEFA9C1
+P 4300 4400
+F 0 "#PWR0105" H 4300 4150 50  0001 C CNN
+F 1 "GND" H 4350 4200 50  0000 C CNN
+F 2 "" H 4300 4400 50  0001 C CNN
+F 3 "" H 4300 4400 50  0001 C CNN
+	1    4300 4400
+	1    0    0    -1
+$EndComp
+Wire Wire Line
+	4300 4400 4300 4300
+Wire Wire Line
+	3600 4300 4300 4300
+Wire Wire Line
+	2250 2700 2650 2700
 $EndSCHEMATC

Commit message: update,
Parts:
- J26: value Conn_01x15_Female -> ARDUINO_HEADER1
- J27: value Conn_01x15_Female -> ARDUINO_HEADER2
Changed lines of the file:
@@
 U 1 1 5CEF6157
 P 3050 4900
-F 0 "J26" H 3100 4950 50  0000 L CNN
-F 1 "Conn_01x15_Female" H 3100 4850 50  0000 L CNN
+F 0 "J26" H 2950 4050 50  0000 C CNN
+F 1 "ARDUINO_HEADER1" H 2950 3950 50  0000 C CNN
 F 2 "" H 3050 4900 50  0001 C CNN
 F 3 "~" H 3050 4900 50  0001 C CNN
@@
 P 3400 4900
 F 0 "J27" H 3250 5800 50  0000 C CNN
-F 1 "Conn_01x15_Female" H 3250 5700 50  0000 C CNN
+F 1 "ARDUINO_HEADER2" H 3250 5700 50  0000 C CNN
 F 2 "" H 3400 4900 50  0001 C CNN
 F 3 "~" H 3400 4900 50  0001 C CNN
