File: hardware/nodemcu.sch (KiCad schematic (older format))
At the start: 5 parts, among them U12 nodemcu

Commit message: update,
Connections:
- net SCL: now also U12.29 (D1); no longer U12.30 (D0)
- net SDA: now also U12.30 (D0); no longer U12.29 (D1)
- net A0 renamed A_IN0
- net D2 renamed PWM
Changed lines of the file:
@@
 SCL
 Text Label 1500 1150 2    50   ~ 0
-D1
+SDA
 Text Label 1500 1250 2    50   ~ 0
-D0
+SCL
 Wire Wire Line
 	1050 1150 1500 1150
@@
 Text Label 6550 2200 2    50   ~ 0
 D0
-Wire Wire Line
-	6550 2200 6300 2200
 Text Label 6550 2300 2    50   ~ 0
 D1
@@
 3V3
 Wire Wire Line
-	6300 2300 6550 2300
-Wire Wire Line
 	6300 2400 6550 2400
 Wire Wire Line
@@
 Wire Wire Line
 	2100 1700 2650 1700
+Text HLabel 900  3750 0    50   Input ~ 0
+PWM
+Text HLabel 900  3900 0    50   Input ~ 0
+A_IN0
+Text Label 6950 2200 2    50   ~ 0
+SDA
+Text Label 6950 2300 2    50   ~ 0
+SCL
+Wire Wire Line
+	6300 2200 6950 2200
+Wire Wire Line
+	6300 2300 6950 2300
+Text Label 1500 3900 2    50   ~ 0
+A0
+Wire Wire Line
+	900  3900 1500 3900
+Text Label 1500 3750 2    50   ~ 0
+D2
+Wire Wire Line
+	900  3750 1500 3750
 $EndSCHEMATC

Commit message: update,
Parts:
- gave numbers to parts that had none: 4
Changed lines of the file:
@@
 	1050 900  1500 900
 $Comp
-L power:+3V3 #PWR0144
+L power:+3V3 #PWR0145
 U 1 1 5CF5A3DE
 P 1050 800
-AR Path="/5CECA6C5/5CF5A3DE" Ref="#PWR0144"  Part="1"
+AR Path="/5CECA6C5/5CF5A3DE" Ref="#PWR0145"  Part="1"
 AR Path="/5CF61809/5CF5A3DE" Ref="#PWR?"  Part="1"
 AR Path="/5CF61878/5CF5A3DE" Ref="#PWR?"  Part="1"
-F 0 "#PWR0144" H 1050 650 50  0001 C CNN
+F 0 "#PWR0145" H 1050 650 50  0001 C CNN
 F 1 "+3V3" V 1100 950 50  0000 L CNN
 F 2 "" H 1050 800 50  0001 C CNN
@@
 $EndComp
 $Comp
-L power:GND #PWR0145
+L power:GND #PWR0146
 U 1 1 5CF5AAFF
 P 1050 900
-AR Path="/5CECA6C5/5CF5AAFF" Ref="#PWR0145"  Part="1"
+AR Path="/5CECA6C5/5CF5AAFF" Ref="#PWR0146"  Part="1"
 AR Path="/5CF61809/5CF5AAFF" Ref="#PWR?"  Part="1"
 AR Path="/5CF61878/5CF5AAFF" Ref="#PWR?"  Part="1"
-F 0 "#PWR0145" H 1050 650 50  0001 C CNN
+F 0 "#PWR0146" H 1050 650 50  0001 C CNN
 F 1 "GND" V 1050 750 50  0000 R CNN
 F 2 "" H 1050 900 50  0001 C CNN
@@
 	2150 3550 2450 3550
 $Comp
-L taobao-components:SPI_DEBUG J?
+L taobao-components:SPI_DEBUG J28
 U 1 1 5D0E4A38
 P 1950 3400
-F 0 "J?" H 2100 3750 50  0000 C CNN
+F 0 "J28" H 2100 3750 50  0000 C CNN
 F 1 "SPI_HEADER" H 2100 3650 50  0000 C CNN
 F 2 "footprint-lib:SPI_DEBUG" H 1950 3000 50  0001 C CNN
@@
 	2100 1900 2550 1900
 $Comp
-L power:GND #PWR?
+L power:GND #PWR0147
 U 1 1 5D1036B5
 P 2650 1700
-F 0 "#PWR?" H 2650 1450 50  0001 C CNN
+F 0 "#PWR0147" H 2650 1450 50  0001 C CNN
 F 1 "GND" V 2700 1550 50  0000 R CNN
 F 2 "" H 2650 1700 50  0001 C CNN
@@
 $EndComp
 $Comp
-L taobao-components:SDCARD_HEADER J?
+L taobao-components:SDCARD_HEADER J27
 U 1 1 5D10ADE8
 P 2100 2700
-F 0 "J?" H 2050 3150 50  0000 C CNN
+F 0 "J27" H 2050 3150 50  0000 C CNN
 F 1 "SDCARD_HEADER" H 2050 3050 50  0000 C CNN
 F 2 "footprint-lib:SPI_DEBUG" H 2100 2250 50  0001 C CNN
@@
 	2100 2950 2700 2950
 $Comp
-L taobao-components:TTL_HEADER J?
+L taobao-components:TTL_HEADER J26
 U 1 1 5D1276DB
 P 2100 1800
-F 0 "J?" H 2050 2100 50  0000 C CNN
+F 0 "J26" H 2050 2100 50  0000 C CNN
 F 1 "TTL_HEADER" H 2050 2000 50  0000 C CNN
 F 2 "footprint-lib:TTL_TERMINAL_1.27mm" H 2100 1400 50  0001 C CNN
@@
 $EndComp
 $Comp
-L taobao-components:I2C_DEBUG J?
+L taobao-components:I2C_DEBUG J25
 U 1 1 5D12AEB7
 P 1900 1200
-F 0 "J?" H 2050 1450 50  0000 C CNN
+F 0 "J25" H 2050 1450 50  0000 C CNN
 F 1 "I2C_DEBUG" H 2050 1350 50  0000 C CNN
 F 2 "footprint-lib:I2C_DEBUG" H 1900 800 50  0001 C CNN

Commit message: update,
Parts:
- renumbered J25 to J24, J26 to J25, J27 to J26, J28 to J27, U12 to U11
Changed lines of the file:
@@
 $EndDescr
 $Comp
-L taobao-board:nodemcu_v1 U12
+L taobao-board:nodemcu_v1 U11
 U 1 1 5CECA83D
 P 5800 2850
-AR Path="/5CECA6C5/5CECA83D" Ref="U12"  Part="1"
+AR Path="/5CECA6C5/5CECA83D" Ref="U11"  Part="1"
 AR Path="/5CF61809/5CECA83D" Ref="U?"  Part="1"
 AR Path="/5CF61878/5CECA83D" Ref="U?"  Part="1"
-F 0 "U12" H 5800 3700 50  0000 C CNN
+F 0 "U11" H 5800 3700 50  0000 C CNN
 F 1 "nodemcu" H 5800 1900 50  0001 C CNN
 F 2 "" H 5800 2850 50  0001 C CNN
@@
 	1050 900  1500 900
 $Comp
-L power:+3V3 #PWR0145
+L power:+3V3 #PWR0138
 U 1 1 5CF5A3DE
 P 1050 800
-AR Path="/5CECA6C5/5CF5A3DE" Ref="#PWR0145"  Part="1"
+AR Path="/5CECA6C5/5CF5A3DE" Ref="#PWR0138"  Part="1"
 AR Path="/5CF61809/5CF5A3DE" Ref="#PWR?"  Part="1"
 AR Path="/5CF61878/5CF5A3DE" Ref="#PWR?"  Part="1"
-F 0 "#PWR0145" H 1050 650 50  0001 C CNN
+F 0 "#PWR0138" H 1050 650 50  0001 C CNN
 F 1 "+3V3" V 1100 950 50  0000 L CNN
 F 2 "" H 1050 800 50  0001 C CNN
@@
 $EndComp
 $Comp
-L power:GND #PWR0146
+L power:GND #PWR0139
 U 1 1 5CF5AAFF
 P 1050 900
-AR Path="/5CECA6C5/5CF5AAFF" Ref="#PWR0146"  Part="1"
+AR Path="/5CECA6C5/5CF5AAFF" Ref="#PWR0139"  Part="1"
 AR Path="/5CF61809/5CF5AAFF" Ref="#PWR?"  Part="1"
 AR Path="/5CF61878/5CF5AAFF" Ref="#PWR?"  Part="1"
-F 0 "#PWR0146" H 1050 650 50  0001 C CNN
+F 0 "#PWR0139" H 1050 650 50  0001 C CNN
 F 1 "GND" V 1050 750 50  0000 R CNN
 F 2 "" H 1050 900 50  0001 C CNN
@@
 	2150 3550 2450 3550
 $Comp
-L taobao-components:SPI_DEBUG J28
+L taobao-components:SPI_DEBUG J27
 U 1 1 5D0E4A38
 P 1950 3400
-F 0 "J28" H 2100 3750 50  0000 C CNN
+F 0 "J27" H 2100 3750 50  0000 C CNN
 F 1 "SPI_HEADER" H 2100 3650 50  0000 C CNN
 F 2 "footprint-lib:SPI_DEBUG" H 1950 3000 50  0001 C CNN
@@
 	2100 1900 2550 1900
 $Comp
-L power:GND #PWR0147
+L power:GND #PWR0140
 U 1 1 5D1036B5
 P 2650 1700
-F 0 "#PWR0147" H 2650 1450 50  0001 C CNN
+F 0 "#PWR0140" H 2650 1450 50  0001 C CNN
 F 1 "GND" V 2700 1550 50  0000 R CNN
 F 2 "" H 2650 1700 50  0001 C CNN
@@
 $EndComp
 $Comp
-L taobao-components:SDCARD_HEADER J27
+L taobao-components:SDCARD_HEADER J26
 U 1 1 5D10ADE8
 P 2100 2700
-F 0 "J27" H 2050 3150 50  0000 C CNN
+F 0 "J26" H 2050 3150 50  0000 C CNN
 F 1 "SDCARD_HEADER" H 2050 3050 50  0000 C CNN
 F 2 "footprint-lib:SPI_DEBUG" H 2100 2250 50  0001 C CNN
@@
 	2100 2950 2700 2950
 $Comp
-L taobao-components:TTL_HEADER J26
+L taobao-components:TTL_HEADER J25
 U 1 1 5D1276DB
 P 2100 1800
-F 0 "J26" H 2050 2100 50  0000 C CNN
+F 0 "J25" H 2050 2100 50  0000 C CNN
 F 1 "TTL_HEADER" H 2050 2000 50  0000 C CNN
 F 2 "footprint-lib:TTL_TERMINAL_1.27mm" H 2100 1400 50  0001 C CNN
@@
 $EndComp
 $Comp
-L taobao-components:I2C_DEBUG J25
+L taobao-components:I2C_DEBUG J24
 U 1 1 5D12AEB7
 P 1900 1200
-F 0 "J25" H 2050 1450 50  0000 C CNN
+F 0 "J24" H 2050 1450 50  0000 C CNN
 F 1 "I2C_DEBUG" H 2050 1350 50  0000 C CNN
 F 2 "footprint-lib:I2C_DEBUG" H 1900 800 50  0001 C CNN

Commit message: update,
Parts:
- renumbered J24 to J15, J25 to J16, J26 to J17, J27 to J18, U11 to U7
Changed lines of the file:
@@
 $EndDescr
 $Comp
-L taobao-board:nodemcu_v1 U11
+L taobao-board:nodemcu_v1 U7
 U 1 1 5CECA83D
 P 5800 2850
-AR Path="/5CECA6C5/5CECA83D" Ref="U11"  Part="1"
+AR Path="/5CECA6C5/5CECA83D" Ref="U7"  Part="1"
 AR Path="/5CF61809/5CECA83D" Ref="U?"  Part="1"
 AR Path="/5CF61878/5CECA83D" Ref="U?"  Part="1"
-F 0 "U11" H 5800 3700 50  0000 C CNN
+F 0 "U7" H 5800 3700 50  0000 C CNN
 F 1 "nodemcu" H 5800 1900 50  0001 C CNN
 F 2 "" H 5800 2850 50  0001 C CNN
@@
 	1050 900  1500 900
 $Comp
-L power:+3V3 #PWR0138
+L power:+3V3 #PWR064
 U 1 1 5CF5A3DE
 P 1050 800
-AR Path="/5CECA6C5/5CF5A3DE" Ref="#PWR0138"  Part="1"
+AR Path="/5CECA6C5/5CF5A3DE" Ref="#PWR064"  Part="1"
 AR Path="/5CF61809/5CF5A3DE" Ref="#PWR?"  Part="1"
 AR Path="/5CF61878/5CF5A3DE" Ref="#PWR?"  Part="1"
-F 0 "#PWR0138" H 1050 650 50  0001 C CNN
+F 0 "#PWR064" H 1050 650 50  0001 C CNN
 F 1 "+3V3" V 1100 950 50  0000 L CNN
 F 2 "" H 1050 800 50  0001 C CNN
@@
 $EndComp
 $Comp
-L power:GND #PWR0139
+L power:GND #PWR065
 U 1 1 5CF5AAFF
 P 1050 900
-AR Path="/5CECA6C5/5CF5AAFF" Ref="#PWR0139"  Part="1"
+AR Path="/5CECA6C5/5CF5AAFF" Ref="#PWR065"  Part="1"
 AR Path="/5CF61809/5CF5AAFF" Ref="#PWR?"  Part="1"
 AR Path="/5CF61878/5CF5AAFF" Ref="#PWR?"  Part="1"
-F 0 "#PWR0139" H 1050 650 50  0001 C CNN
+F 0 "#PWR065" H 1050 650 50  0001 C CNN
 F 1 "GND" V 1050 750 50  0000 R CNN
 F 2 "" H 1050 900 50  0001 C CNN
@@
 	2150 3550 2450 3550
 $Comp
-L taobao-components:SPI_DEBUG J27
+L taobao-components:SPI_DEBUG J18
 U 1 1 5D0E4A38
 P 1950 3400
-F 0 "J27" H 2100 3750 50  0000 C CNN
+F 0 "J18" H 2100 3750 50  0000 C CNN
 F 1 "SPI_HEADER" H 2100 3650 50  0000 C CNN
 F 2 "footprint-lib:SPI_DEBUG" H 1950 3000 50  0001 C CNN
@@
 	2100 1900 2550 1900
 $Comp
-L power:GND #PWR0140
+L power:GND #PWR066
 U 1 1 5D1036B5
 P 2650 1700
-F 0 "#PWR0140" H 2650 1450 50  0001 C CNN
+F 0 "#PWR066" H 2650 1450 50  0001 C CNN
 F 1 "GND" V 2700 1550 50  0000 R CNN
 F 2 "" H 2650 1700 50  0001 C CNN
@@
 $EndComp
 $Comp
-L taobao-components:SDCARD_HEADER J26
+L taobao-components:SDCARD_HEADER J17
 U 1 1 5D10ADE8
 P 2100 2700
-F 0 "J26" H 2050 3150 50  0000 C CNN
+F 0 "J17" H 2050 3150 50  0000 C CNN
 F 1 "SDCARD_HEADER" H 2050 3050 50  0000 C CNN
 F 2 "footprint-lib:SPI_DEBUG" H 2100 2250 50  0001 C CNN
@@
 	2100 2950 2700 2950
 $Comp
-L taobao-components:TTL_HEADER J25
+L taobao-components:TTL_HEADER J16
 U 1 1 5D1276DB
 P 2100 1800
-F 0 "J25" H 2050 2100 50  0000 C CNN
+F 0 "J16" H 2050 2100 50  0000 C CNN
 F 1 "TTL_HEADER" H 2050 2000 50  0000 C CNN
 F 2 "footprint-lib:TTL_TERMINAL_1.27mm" H 2100 1400 50  0001 C CNN
@@
 $EndComp
 $Comp
-L taobao-components:I2C_DEBUG J24
+L taobao-components:I2C_DEBUG J15
 U 1 1 5D12AEB7
 P 1900 1200
-F 0 "J24" H 2050 1450 50  0000 C CNN
+F 0 "J15" H 2050 1450 50  0000 C CNN
 F 1 "I2C_DEBUG" H 2050 1350 50  0000 C CNN
 F 2 "footprint-lib:I2C_DEBUG" H 1900 800 50  0001 C CNN

Commit message: update,
Connections:
- net A_IN0 renamed A0
- net PWM renamed D2
- no-connect marks 0 -> 9
Changed lines of the file:
@@
 $Descr A4 11693 8268
 encoding utf-8
-Sheet 18 19
+Sheet 14 19
 Title ""
 Date ""
@@
 	5050 2200 5300 2200
 Wire Wire Line
-	5050 2300 5300 2300
-Wire Wire Line
-	5050 2400 5300 2400
-Wire Wire Line
 	5050 2500 5300 2500
 Wire Wire Line
@@
 Wire Wire Line
 	900  2950 1500 2950
-Text HLabel 1050 1800 0    50   Input ~ 0
-TX
-Text HLabel 1050 1900 0    50   Input ~ 0
-RX
-Text Label 1500 1800 2    50   ~ 0
-TX
-Text Label 1500 1900 2    50   ~ 0
-RX
-Wire Wire Line
-	1050 1800 1500 1800
-Wire Wire Line
-	1050 1900 1500 1900
 Text Label 1500 3250 2    50   ~ 0
 HSCLK
@@
 Wire Wire Line
 	2100 1700 2650 1700
-Text HLabel 900  3750 0    50   Input ~ 0
-PWM
-Text HLabel 900  3900 0    50   Input ~ 0
-A_IN0
 Text Label 6950 2200 2    50   ~ 0
 SDA
@@
 Wire Wire Line
 	6300 2300 6950 2300
-Text Label 1500 3900 2    50   ~ 0
-A0
-Wire Wire Line
-	900  3900 1500 3900
-Text Label 1500 3750 2    50   ~ 0
-D2
-Wire Wire Line
-	900  3750 1500 3750
+NoConn ~ 5300 2300
+NoConn ~ 5300 2400
+NoConn ~ 5050 2200
+NoConn ~ 6550 2400
+NoConn ~ 6550 2500
+NoConn ~ 6550 2600
+NoConn ~ 5050 3300
+NoConn ~ 5050 3400
+NoConn ~ 5050 3600
 $EndSCHEMATC

Commit message: update,
Parts:
- added J?: NODEMCU_HEADER1, symbol Connector:Conn_01x15_Female
- added J?: NODEMCU_HEADER2, symbol Connector:Conn_01x15_Female
Connections:
- wire segments 57 -> 85
- no-connect marks 9 -> 16
Changed lines of the file:
@@
 NoConn ~ 5050 3400
 NoConn ~ 5050 3600
+$Comp
+L Connector:Conn_01x15_Female J?
+U 1 1 5CF023B3
+P 5500 4750
+F 0 "J?" H 5400 3900 50  0000 C CNN
+F 1 "NODEMCU_HEADER1" H 5400 3800 50  0000 C CNN
+F 2 "" H 5500 4750 50  0001 C CNN
+F 3 "~" H 5500 4750 50  0001 C CNN
+	1    5500 4750
+	1    0    0    -1
+$EndComp
+$Comp
+L Connector:Conn_01x15_Female J?
+U 1 1 5CF02B3B
+P 6100 4750
+F 0 "J?" H 5950 5650 50  0000 C CNN
+F 1 "NODEMCU_HEADER2" H 5950 5550 50  0000 C CNN
+F 2 "" H 6100 4750 50  0001 C CNN
+F 3 "~" H 6100 4750 50  0001 C CNN
+	1    6100 4750
+	-1   0    0    -1
+$EndComp
+Text Label 5050 4050 0    50   ~ 0
+A0
+Text Label 5050 4350 0    50   ~ 0
+SDD3
+Text Label 5050 4450 0    50   ~ 0
+SDD2
+Text Label 5050 4550 0    50   ~ 0
+SDD1
+Text Label 5050 4650 0    50   ~ 0
+SDCMD
+Text Label 5050 4750 0    50   ~ 0
+SDD0
+Text Label 5050 4850 0    50   ~ 0
+SDCLK
+Text Label 5050 4950 0    50   ~ 0
+GND
+Text Label 5050 5050 0    50   ~ 0
+3V3
+Text Label 5050 5150 0    50   ~ 0
+EN
+Text Label 5050 5250 0    50   ~ 0
+RST
+Text Label 5050 5350 0    50   ~ 0
+GND
+Text Label 5050 5450 0    50   ~ 0
+VIN
+Wire Wire Line
+	5050 4050 5300 4050
+Wire Wire Line
+	5050 4350 5300 4350
+Wire Wire Line
+	5050 4450 5300 4450
+Wire Wire Line
+	5050 4550 5300 4550
+Wire Wire Line
+	5050 4650 5300 4650
+Wire Wire Line
+	5050 4750 5300 4750
+Wire Wire Line
+	5050 4850 5300 4850
+Wire Wire Line
+	5050 4950 5300 4950
+Wire Wire Line
+	5050 5050 5300 5050
+Wire Wire Line
+	5050 5150 5300 5150
+Wire Wire Line
+	5050 5250 5300 5250
+Wire Wire Line
+	5050 5350 5300 5350
+Wire Wire Line
+	5050 5450 5300 5450
+NoConn ~ 5050 4050
+NoConn ~ 5050 5150
+NoConn ~ 5050 5250
+NoConn ~ 5050 5450
+Text Label 6550 4050 2    50   ~ 0
+D0
+Text Label 6550 4150 2    50   ~ 0
+D1
+Text Label 6550 4250 2    50   ~ 0
+D2
+Text Label 6550 4350 2    50   ~ 0
+D3
+Text Label 6550 4450 2    50   ~ 0
+D4
+Text Label 6550 4550 2    50   ~ 0
+3V3
+Text Label 6550 4650 2    50   ~ 0
+GND
+Text Label 6550 4750 2    50   ~ 0
+D5
+Text Label 6550 4850 2    50   ~ 0
+D6
+Text Label 6550 4950 2    50   ~ 0
+D7
+Text Label 6550 5050 2    50   ~ 0
+D8
+Text Label 6550 5150 2    50   ~ 0
+RX
+Text Label 6550 5250 2    50   ~ 0
+TX
+Text Label 6550 5350 2    50   ~ 0
+GND
+Text Label 6550 5450 2    50   ~ 0
+3V3
+Wire Wire Line
+	6300 4250 6550 4250
+Wire Wire Line
+	6300 4350 6550 4350
+Wire Wire Line
+	6300 4450 6550 4450
+Wire Wire Line
+	6300 4550 6550 4550
+Wire Wire Line
+	6300 4650 6550 4650
+Wire Wire Line
+	6300 5150 6550 5150
+Wire Wire Line
+	6300 5250 6550 5250
+Wire Wire Line
+	6300 5350 6550 5350
+Wire Wire Line
+	6300 5450 6550 5450
+Text Label 6950 4750 2    50   ~ 0
+HSCLK
+Text Label 6950 4850 2    50   ~ 0
+HMISO
+Text Label 6950 4950 2    50   ~ 0
+HMOSI
+Text Label 6950 5050 2    50   ~ 0
+HCS
+Wire Wire Line
+	6300 4750 6950 4750
+Wire Wire Line
+	6300 4850 6950 4850
+Wire Wire Line
+	6300 4950 6950 4950
+Wire Wire Line
+	6300 5050 6950 5050
+Text Label 6950 4050 2    50   ~ 0
+SDA
+Text Label 6950 4150 2    50   ~ 0
+SCL
+Wire Wire Line
+	6300 4050 6950 4050
+Wire Wire Line
+	6300 4150 6950 4150
+NoConn ~ 6550 4250
+NoConn ~ 6550 4350
+NoConn ~ 6550 4450
 $EndSCHEMATC
