File: hardware/ADC.sch (KiCad schematic (older format))
At the start: 6 parts

Commit message: update,
Parts:
- gave numbers to parts that had none: 6
Connections:
- net V_TEMP: now reaches C10.1, R15.2, TH1.1
- net V_VAR: now reaches C9.1, R14.2, R16.1
Changed lines of the file:
@@
 EELAYER 29 0
 EELAYER END
-$Descr A4 11693 8268
+$Descr User 8500 5500
 encoding utf-8
-Sheet 8 27
+Sheet 9 20
 Title ""
 Date ""
@@
 $EndBitmap
 $Comp
-L taobao-components:Thermistor_NTC,0805 TH?
+L taobao-components:Thermistor_NTC,0805 TH1
 U 1 1 5CE530DC
 P 4350 2750
-F 0 "TH?" H 4450 2800 50  0000 L CNN
+F 0 "TH1" H 4450 2800 50  0000 L CNN
 F 1 "Thermistor_NTC,0805" H 4450 2750 50  0000 L CNN
 F 2 "Resistor_SMD:R_0805_2012Metric" H 4350 2800 50  0001 C CNN
@@
 $EndComp
 $Comp
-L taobao-r:R472,0603 R?
+L taobao-r:R472,0603 R15
 U 1 1 5CE54032
 P 3700 2350
-F 0 "R?" H 3800 2400 50  0000 L CNN
+F 0 "R15" H 3800 2400 50  0000 L CNN
 F 1 "R472,0603" H 3800 2350 50  0000 L CNN
 F 2 "Resistor_SMD:R_0603_1608Metric_Pad1.05x0.95mm_HandSolder" H 3700 2350 50  0001 C CNN
@@
 $EndComp
 $Comp
-L taobao-c:C106,0603 C?
+L taobao-c:C106,0603 C10
 U 1 1 5CE54EF6
 P 3700 2750
-F 0 "C?" H 3800 2800 50  0000 L CNN
+F 0 "C10" H 3800 2800 50  0000 L CNN
 F 1 "C106,0603" H 3800 2750 50  0000 L CNN
 F 2 "Capacitor_SMD:C_0603_1608Metric_Pad1.05x0.95mm_HandSolder" H 3700 2750 50  0001 C CNN
@@
 $EndComp
 $Comp
-L power:GND #PWR?
+L power:GND #PWR054
 U 1 1 5CE55D7C
 P 3700 3000
-F 0 "#PWR?" H 3700 2750 50  0001 C CNN
+F 0 "#PWR054" H 3700 2750 50  0001 C CNN
 F 1 "GND" H 3750 2800 50  0000 C CNN
 F 2 "" H 3700 3000 50  0001 C CNN
@@
 $EndComp
 $Comp
-L power:GND #PWR?
+L power:GND #PWR055
 U 1 1 5CE56041
 P 4350 3000
-F 0 "#PWR?" H 4350 2750 50  0001 C CNN
+F 0 "#PWR055" H 4350 2750 50  0001 C CNN
 F 1 "GND" H 4400 2800 50  0000 C CNN
 F 2 "" H 4350 3000 50  0001 C CNN
@@
 	4350 2900 4350 3000
 $Comp
-L power:+3V3 #PWR?
+L power:+3V3 #PWR051
 U 1 1 5CE575B4
 P 3700 2100
-F 0 "#PWR?" H 3700 1950 50  0001 C CNN
+F 0 "#PWR051" H 3700 1950 50  0001 C CNN
 F 1 "+3V3" H 3750 2300 50  0000 C CNN
 F 2 "" H 3700 2100 50  0001 C CNN
@@
 	3700 2550 3700 2650
 $Comp
-L taobao-r:R472,0603 R?
+L taobao-r:R472,0603 R14
 U 1 1 5CE5922D
 P 2300 2350
-F 0 "R?" H 2400 2400 50  0000 L CNN
+F 0 "R14" H 2400 2400 50  0000 L CNN
 F 1 "R472,0603" H 2400 2350 50  0000 L CNN
 F 2 "Resistor_SMD:R_0603_1608Metric_Pad1.05x0.95mm_HandSolder" H 2300 2350 50  0001 C CNN
@@
 $EndComp
 $Comp
-L taobao-c:C106,0603 C?
+L taobao-c:C106,0603 C9
 U 1 1 5CE59237
 P 2300 2750
-F 0 "C?" H 2400 2800 50  0000 L CNN
+F 0 "C9" H 2400 2800 50  0000 L CNN
 F 1 "C106,0603" H 2400 2750 50  0000 L CNN
 F 2 "Capacitor_SMD:C_0603_1608Metric_Pad1.05x0.95mm_HandSolder" H 2300 2750 50  0001 C CNN
@@
 $EndComp
 $Comp
-L power:GND #PWR?
+L power:GND #PWR052
 U 1 1 5CE59241
 P 2300 3000
-F 0 "#PWR?" H 2300 2750 50  0001 C CNN
+F 0 "#PWR052" H 2300 2750 50  0001 C CNN
 F 1 "GND" H 2350 2800 50  0000 C CNN
 F 2 "" H 2300 3000 50  0001 C CNN
@@
 $EndComp
 $Comp
-L power:GND #PWR?
+L power:GND #PWR053
 U 1 1 5CE5924B
 P 2950 3000
-F 0 "#PWR?" H 2950 2750 50  0001 C CNN
+F 0 "#PWR053" H 2950 2750 50  0001 C CNN
 F 1 "GND" H 3000 2800 50  0000 C CNN
 F 2 "" H 2950 3000 50  0001 C CNN
@@
 	2950 2900 2950 3000
 $Comp
-L power:+3V3 #PWR?
+L power:+3V3 #PWR050
 U 1 1 5CE59257
 P 2300 2100
-F 0 "#PWR?" H 2300 1950 50  0001 C CNN
+F 0 "#PWR050" H 2300 1950 50  0001 C CNN
 F 1 "+3V3" H 2350 2300 50  0000 C CNN
 F 2 "" H 2300 2100 50  0001 C CNN
@@
 	2300 2550 2300 2650
 $Comp
-L Device:R_Variable R?
+L Device:R_Variable R16
 U 1 1 5CE5CEF0
 P 2950 2750
-F 0 "R?" H 3100 2800 50  0000 L CNN
+F 0 "R16" H 3100 2800 50  0000 L CNN
 F 1 "R_Variable" H 3100 2750 50  0000 L CNN
 F 2 "" V 2880 2750 50  0001 C CNN
@@
 	1    0    0    -1
 $EndComp
+Text Label 2600 2550 0    50   ~ 0
+V_VAR
+Text Label 3950 2550 0    50   ~ 0
+V_TEMP
+Text HLabel 850  650  0    50   Input ~ 0
+V_VAR
+Text HLabel 850  750  0    50   Input ~ 0
+V_TEMP
+Text Label 1200 650  2    50   ~ 0
+V_VAR
+Text Label 1200 750  2    50   ~ 0
+V_TEMP
+Wire Wire Line
+	850  650  1200 650
+Wire Wire Line
+	850  750  1200 750
 $EndSCHEMATC

Commit message: update,
Parts:
- renumbered C9 to C7, C10 to C8, R15 to R10, R16 to R11, R14 to R9
Changed lines of the file:
@@
 $EndComp
 $Comp
-L taobao-r:R472,0603 R15
+L taobao-r:R472,0603 R10
 U 1 1 5CE54032
 P 3700 2350
-F 0 "R15" H 3800 2400 50  0000 L CNN
+F 0 "R10" H 3800 2400 50  0000 L CNN
 F 1 "R472,0603" H 3800 2350 50  0000 L CNN
 F 2 "Resistor_SMD:R_0603_1608Metric_Pad1.05x0.95mm_HandSolder" H 3700 2350 50  0001 C CNN
@@
 $EndComp
 $Comp
-L taobao-c:C106,0603 C10
+L taobao-c:C106,0603 C8
 U 1 1 5CE54EF6
 P 3700 2750
-F 0 "C10" H 3800 2800 50  0000 L CNN
+F 0 "C8" H 3800 2800 50  0000 L CNN
 F 1 "C106,0603" H 3800 2750 50  0000 L CNN
 F 2 "Capacitor_SMD:C_0603_1608Metric_Pad1.05x0.95mm_HandSolder" H 3700 2750 50  0001 C CNN
@@
 $EndComp
 $Comp
-L power:GND #PWR054
+L power:GND #PWR047
 U 1 1 5CE55D7C
 P 3700 3000
-F 0 "#PWR054" H 3700 2750 50  0001 C CNN
+F 0 "#PWR047" H 3700 2750 50  0001 C CNN
 F 1 "GND" H 3750 2800 50  0000 C CNN
 F 2 "" H 3700 3000 50  0001 C CNN
@@
 $EndComp
 $Comp
-L power:GND #PWR055
+L power:GND #PWR048
 U 1 1 5CE56041
 P 4350 3000
-F 0 "#PWR055" H 4350 2750 50  0001 C CNN
+F 0 "#PWR048" H 4350 2750 50  0001 C CNN
 F 1 "GND" H 4400 2800 50  0000 C CNN
 F 2 "" H 4350 3000 50  0001 C CNN
@@
 	4350 2900 4350 3000
 $Comp
-L power:+3V3 #PWR051
+L power:+3V3 #PWR044
 U 1 1 5CE575B4
 P 3700 2100
-F 0 "#PWR051" H 3700 1950 50  0001 C CNN
+F 0 "#PWR044" H 3700 1950 50  0001 C CNN
 F 1 "+3V3" H 3750 2300 50  0000 C CNN
 F 2 "" H 3700 2100 50  0001 C CNN
@@
 	3700 2550 3700 2650
 $Comp
-L taobao-r:R472,0603 R14
+L taobao-r:R472,0603 R9
 U 1 1 5CE5922D
 P 2300 2350
-F 0 "R14" H 2400 2400 50  0000 L CNN
+F 0 "R9" H 2400 2400 50  0000 L CNN
 F 1 "R472,0603" H 2400 2350 50  0000 L CNN
 F 2 "Resistor_SMD:R_0603_1608Metric_Pad1.05x0.95mm_HandSolder" H 2300 2350 50  0001 C CNN
@@
 $EndComp
 $Comp
-L taobao-c:C106,0603 C9
+L taobao-c:C106,0603 C7
 U 1 1 5CE59237
 P 2300 2750
-F 0 "C9" H 2400 2800 50  0000 L CNN
+F 0 "C7" H 2400 2800 50  0000 L CNN
 F 1 "C106,0603" H 2400 2750 50  0000 L CNN
 F 2 "Capacitor_SMD:C_0603_1608Metric_Pad1.05x0.95mm_HandSolder" H 2300 2750 50  0001 C CNN
@@
 $EndComp
 $Comp
-L power:GND #PWR052
+L power:GND #PWR045
 U 1 1 5CE59241
 P 2300 3000
-F 0 "#PWR052" H 2300 2750 50  0001 C CNN
+F 0 "#PWR045" H 2300 2750 50  0001 C CNN
 F 1 "GND" H 2350 2800 50  0000 C CNN
 F 2 "" H 2300 3000 50  0001 C CNN
@@
 $EndComp
 $Comp
-L power:GND #PWR053
+L power:GND #PWR046
 U 1 1 5CE5924B
 P 2950 3000
-F 0 "#PWR053" H 2950 2750 50  0001 C CNN
+F 0 "#PWR046" H 2950 2750 50  0001 C CNN
 F 1 "GND" H 3000 2800 50  0000 C CNN
 F 2 "" H 2950 3000 50  0001 C CNN
@@
 	2950 2900 2950 3000
 $Comp
-L power:+3V3 #PWR050
+L power:+3V3 #PWR043
 U 1 1 5CE59257
 P 2300 2100
-F 0 "#PWR050" H 2300 1950 50  0001 C CNN
+F 0 "#PWR043" H 2300 1950 50  0001 C CNN
 F 1 "+3V3" H 2350 2300 50  0000 C CNN
 F 2 "" H 2300 2100 50  0001 C CNN
@@
 	2300 2550 2300 2650
 $Comp
-L Device:R_Variable R16
+L Device:R_Variable R11
 U 1 1 5CE5CEF0
 P 2950 2750
-F 0 "R16" H 3100 2800 50  0000 L CNN
+F 0 "R11" H 3100 2800 50  0000 L CNN
 F 1 "R_Variable" H 3100 2750 50  0000 L CNN
 F 2 "" V 2880 2750 50  0001 C CNN
