File: hardware/NEO-6M-0-001.sch (KiCad schematic (older format))
At the start: 1 part

Commit message: update,
Parts:
- U?: footprint (none) -> Connector_PinSocket_2.54mm:PinSocket_1x04_P2.54mm_Vertical
Changed lines of the file:
@@
 F 0 "U?" H 2250 4550 50  0000 L CNN
 F 1 "UBLOX-NEO-6M_DEBUG" H 2250 4500 50  0000 L CNN
-F 2 "" H 2000 4350 50  0001 C CNN
+F 2 "Connector_PinSocket_2.54mm:PinSocket_1x04_P2.54mm_Vertical" H 2000 4350 50  0001 C CNN
 F 3 "" H 2000 4350 50  0001 C CNN
 	1    1850 4500

Commit message: update,
Parts:
- U6: renamed from U?; footprint Connector_PinSocket_2.54mm:PinSocket_1x04_P2.54mm_Vertical -> footprint-lib:UBLOX-NEO-6M_DEBUG
Other:
- moved on the sheet: U6
Changed lines of the file:
@@
 EELAYER 29 0
 EELAYER END
-$Descr A4 11693 8268
+$Descr User 8500 5500
 encoding utf-8
-Sheet 16 27
+Sheet 11 20
 Title ""
 Date ""
@@
 $EndBitmap
 $Comp
-L taobao-board:UBLOX-NEO-6M_DEBUG U?
+L taobao-board:UBLOX-NEO-6M_DEBUG U6
 U 1 1 5CE5E487
-P 1850 4500
-F 0 "U?" H 2250 4550 50  0000 L CNN
-F 1 "UBLOX-NEO-6M_DEBUG" H 2250 4500 50  0000 L CNN
-F 2 "Connector_PinSocket_2.54mm:PinSocket_1x04_P2.54mm_Vertical" H 2000 4350 50  0001 C CNN
-F 3 "" H 2000 4350 50  0001 C CNN
-	1    1850 4500
+P 1950 4150
+F 0 "U6" H 2350 4200 50  0000 L CNN
+F 1 "UBLOX-NEO-6M_DEBUG" H 2350 4150 50  0000 L CNN
+F 2 "footprint-lib:UBLOX-NEO-6M_DEBUG" H 2100 4000 50  0001 C CNN
+F 3 "" H 2100 4000 50  0001 C CNN
+	1    1950 4150
 	1    0    0    -1
 $EndComp
 $Comp
-L power:GND #PWR?
+L power:GND #PWR057
 U 1 1 5CE5EA2C
-P 1550 4800
-F 0 "#PWR?" H 1550 4550 50  0001 C CNN
-F 1 "GND" H 1600 4600 50  0000 C CNN
-F 2 "" H 1550 4800 50  0001 C CNN
-F 3 "" H 1550 4800 50  0001 C CNN
-	1    1550 4800
+P 1650 4450
+F 0 "#PWR057" H 1650 4200 50  0001 C CNN
+F 1 "GND" H 1700 4250 50  0000 C CNN
+F 2 "" H 1650 4450 50  0001 C CNN
+F 3 "" H 1650 4450 50  0001 C CNN
+	1    1650 4450
 	1    0    0    -1
 $EndComp
 Wire Wire Line
-	1650 4650 1550 4650
+	1750 4300 1650 4300
 Wire Wire Line
-	1550 4650 1550 4800
+	1650 4300 1650 4450
 $Comp
-L power:+3V3 #PWR?
+L power:+3V3 #PWR056
 U 1 1 5CE5EF1E
-P 1550 4250
-F 0 "#PWR?" H 1550 4100 50  0001 C CNN
-F 1 "+3V3" H 1600 4450 50  0000 C CNN
-F 2 "" H 1550 4250 50  0001 C CNN
-F 3 "" H 1550 4250 50  0001 C CNN
-	1    1550 4250
+P 1650 3900
+F 0 "#PWR056" H 1650 3750 50  0001 C CNN
+F 1 "+3V3" H 1700 4100 50  0000 C CNN
+F 2 "" H 1650 3900 50  0001 C CNN
+F 3 "" H 1650 3900 50  0001 C CNN
+	1    1650 3900
 	1    0    0    -1
 $EndComp
 Wire Wire Line
-	1550 4250 1550 4350
+	1650 3900 1650 4000
 Wire Wire Line
-	1550 4350 1650 4350
-Text HLabel 1200 4450 0    50   Input ~ 0
+	1650 4000 1750 4000
+Text HLabel 1100 700  0    50   Input ~ 0
 UBLOX_TX
-Text HLabel 1200 4550 0    50   Input ~ 0
+Text HLabel 1100 800  0    50   Input ~ 0
 UBLOX_RX
 Wire Wire Line
-	1200 4450 1650 4450
+	1300 4100 1750 4100
 Wire Wire Line
-	1200 4550 1650 4550
+	1300 4200 1750 4200
+Text Label 1300 4100 0    50   ~ 0
+TX
+Text Label 1300 4200 0    50   ~ 0
+RX
+Text Label 1400 700  2    50   ~ 0
+TX
+Text Label 1400 800  2    50   ~ 0
+RX
+Wire Wire Line
+	1100 700  1400 700
+Wire Wire Line
+	1100 800  1400 800
 $EndSCHEMATC

Commit message: update,
Parts:
- renumbered U6 to U5
Changed lines of the file:
@@
 $EndBitmap
 $Comp
-L taobao-board:UBLOX-NEO-6M_DEBUG U6
+L taobao-board:UBLOX-NEO-6M_DEBUG U5
 U 1 1 5CE5E487
 P 1950 4150
-F 0 "U6" H 2350 4200 50  0000 L CNN
+F 0 "U5" H 2350 4200 50  0000 L CNN
 F 1 "UBLOX-NEO-6M_DEBUG" H 2350 4150 50  0000 L CNN
 F 2 "footprint-lib:UBLOX-NEO-6M_DEBUG" H 2100 4000 50  0001 C CNN
@@
 $EndComp
 $Comp
-L power:GND #PWR057
+L power:GND #PWR050
 U 1 1 5CE5EA2C
 P 1650 4450
-F 0 "#PWR057" H 1650 4200 50  0001 C CNN
+F 0 "#PWR050" H 1650 4200 50  0001 C CNN
 F 1 "GND" H 1700 4250 50  0000 C CNN
 F 2 "" H 1650 4450 50  0001 C CNN
@@
 	1650 4300 1650 4450
 $Comp
-L power:+3V3 #PWR056
+L power:+3V3 #PWR049
 U 1 1 5CE5EF1E
 P 1650 3900
-F 0 "#PWR056" H 1650 3750 50  0001 C CNN
+F 0 "#PWR049" H 1650 3750 50  0001 C CNN
 F 1 "+3V3" H 1700 4100 50  0000 C CNN
 F 2 "" H 1650 3900 50  0001 C CNN
