File: hardware/PWM.sch (KiCad schematic (older format))
At the start: 3 parts

Commit message: update,
Parts:
- J?: footprint (none) -> Connector_PinSocket_2.54mm:PinSocket_1x02_P2.54mm_Vertical
Changed lines of the file:
@@
 F 0 "J?" H 4900 1700 50  0000 L CNN
 F 1 "PWM_OUT" H 4900 1600 50  0000 L CNN
-F 2 "" H 4800 1700 50  0001 C CNN
+F 2 "Connector_PinSocket_2.54mm:PinSocket_1x02_P2.54mm_Vertical" H 4800 1700 50  0001 C CNN
 F 3 "~" H 4800 1700 50  0001 C CNN
 	1    4800 1700

Commit message: update,
Parts:
- gave numbers to parts that had none: 3
Changed lines of the file:
@@
 $Descr A4 11693 8268
 encoding utf-8
-Sheet 14 27
+Sheet 10 20
 Title ""
 Date ""
@@
 $EndBitmap
 $Comp
-L 74xGxx:74AHCT1G125 U?
+L 74xGxx:74AHCT1G125 U5
 U 1 1 5CE46064
 P 3900 1800
-F 0 "U?" H 3900 1550 50  0001 C CNN
+F 0 "U5" H 3900 1550 50  0001 C CNN
 F 1 "74AHCT1G125" H 3900 1600 50  0000 C CNN
 F 2 "Package_TO_SOT_SMD:SOT-23-5_HandSoldering" H 3900 1800 50  0001 C CNN
@@
 $EndComp
 $Comp
-L taobao-r:R223,0603 R?
+L taobao-r:R223,0603 R17
 U 1 1 5CE4623E
 P 3900 1300
-F 0 "R?" V 3650 1300 50  0000 C CNN
+F 0 "R17" V 3650 1300 50  0000 C CNN
 F 1 "R223,0603" V 3750 1300 50  0000 C CNN
 F 2 "Resistor_SMD:R_0603_1608Metric_Pad1.05x0.95mm_HandSolder" H 3900 1300 50  0001 C CNN
@@
 STM32_PWM_OUT
 $Comp
-L Connector_Generic:Conn_01x02 J?
+L Connector_Generic:Conn_01x02 J9
 U 1 1 5CE46D1B
 P 4800 1700
-F 0 "J?" H 4900 1700 50  0000 L CNN
+F 0 "J9" H 4900 1700 50  0000 L CNN
 F 1 "PWM_OUT" H 4900 1600 50  0000 L CNN
 F 2 "Connector_PinSocket_2.54mm:PinSocket_1x02_P2.54mm_Vertical" H 4800 1700 50  0001 C CNN

Commit message: update,
Parts:
- renumbered J9 to J8, R17 to R12, U5 to U4
Connections:
- net GND: now also U4.1
- net VCC renamed +5V
Changed lines of the file:
@@
 $Descr A4 11693 8268
 encoding utf-8
-Sheet 10 20
+Sheet 9 20
 Title ""
 Date ""
@@
 $EndBitmap
 $Comp
-L 74xGxx:74AHCT1G125 U5
+L 74xGxx:74AHCT1G125 U4
 U 1 1 5CE46064
 P 3900 1800
-F 0 "U5" H 3900 1550 50  0001 C CNN
+F 0 "U4" H 3900 1550 50  0001 C CNN
 F 1 "74AHCT1G125" H 3900 1600 50  0000 C CNN
 F 2 "Package_TO_SOT_SMD:SOT-23-5_HandSoldering" H 3900 1800 50  0001 C CNN
@@
 $EndComp
 $Comp
-L taobao-r:R223,0603 R17
+L taobao-r:R223,0603 R12
 U 1 1 5CE4623E
 P 3900 1300
-F 0 "R17" V 3650 1300 50  0000 C CNN
+F 0 "R12" V 3650 1300 50  0000 C CNN
 F 1 "R223,0603" V 3750 1300 50  0000 C CNN
 F 2 "Resistor_SMD:R_0603_1608Metric_Pad1.05x0.95mm_HandSolder" H 3900 1300 50  0001 C CNN
@@
 STM32_PWM_OUT
 $Comp
-L Connector_Generic:Conn_01x02 J9
+L Connector_Generic:Conn_01x02 J8
 U 1 1 5CE46D1B
 P 4800 1700
-F 0 "J9" H 4900 1700 50  0000 L CNN
+F 0 "J8" H 4900 1700 50  0000 L CNN
 F 1 "PWM_OUT" H 4900 1600 50  0000 L CNN
 F 2 "Connector_PinSocket_2.54mm:PinSocket_1x02_P2.54mm_Vertical" H 4800 1700 50  0001 C CNN
@@
 Wire Wire Line
 	3300 1300 3800 1300
+$Comp
+L power:GND #PWR0170
+U 1 1 5CF4DA4F
+P 3650 1600
+F 0 "#PWR0170" H 3650 1350 50  0001 C CNN
+F 1 "GND" H 3700 1400 50  0000 C CNN
+F 2 "" H 3650 1600 50  0001 C CNN
+F 3 "" H 3650 1600 50  0001 C CNN
+	1    3650 1600
+	1    0    0    -1
+$EndComp
+Wire Wire Line
+	3650 1550 3900 1550
+Wire Wire Line
+	3900 1550 3900 1600
+Wire Wire Line
+	3650 1550 3650 1600
+$Comp
+L power:+5V #PWR0171
+U 1 1 5CF4DEC2
+P 3950 1500
+F 0 "#PWR0171" H 3950 1350 50  0001 C CNN
+F 1 "+5V" H 4000 1700 50  0000 C CNN
+F 2 "" H 3950 1500 50  0001 C CNN
+F 3 "" H 3950 1500 50  0001 C CNN
+	1    3950 1500
+	1    0    0    -1
+$EndComp
+$Comp
+L power:GND #PWR0172
+U 1 1 5CF4E2CB
+P 3950 2100
+F 0 "#PWR0172" H 3950 1850 50  0001 C CNN
+F 1 "GND" H 4000 1900 50  0000 C CNN
+F 2 "" H 3950 2100 50  0001 C CNN
+F 3 "" H 3950 2100 50  0001 C CNN
+	1    3950 2100
+	1    0    0    -1
+$EndComp
+Wire Wire Line
+	3950 2100 3950 1850
+Wire Wire Line
+	3950 1500 3950 1750
 $EndSCHEMATC

Commit message: update,
Parts:
- removed R12: R223,0603, Resistor_SMD:R_0603_1608Metric_Pad1.05x0.95mm_HandSolder, symbol taobao-r:R223,0603
Connections:
- net STM32_PWM_OUT is gone; now on net STM32_PWM_IN: U4.2
- net GND: now also J8.2 (Pin_2)
- net at U4.4: now also J8.1 (Pin_1); no longer J8.2 (Pin_2)
Other:
- moved on the sheet: J8
Changed lines of the file:
@@
 $Descr A4 11693 8268
 encoding utf-8
-Sheet 9 20
+Sheet 9 18
 Title ""
 Date ""
@@
 EndData
 $EndBitmap
-$Comp
-L 74xGxx:74AHCT1G125 U4
-U 1 1 5CE46064
-P 3900 1800
-F 0 "U4" H 3900 1550 50  0001 C CNN
-F 1 "74AHCT1G125" H 3900 1600 50  0000 C CNN
-F 2 "Package_TO_SOT_SMD:SOT-23-5_HandSoldering" H 3900 1800 50  0001 C CNN
-F 3 "http://www.ti.com/lit/sg/scyt129e/scyt129e.pdf" H 3900 1800 50  0001 C CNN
-	1    3900 1800
-	1    0    0    -1
-$EndComp
-$Comp
-L taobao-r:R223,0603 R12
-U 1 1 5CE4623E
-P 3900 1300
-F 0 "R12" V 3650 1300 50  0000 C CNN
-F 1 "R223,0603" V 3750 1300 50  0000 C CNN
-F 2 "Resistor_SMD:R_0603_1608Metric_Pad1.05x0.95mm_HandSolder" H 3900 1300 50  0001 C CNN
-F 3 "~" H 3900 1300 50  0001 C CNN
-	1    3900 1300
-	0    1    1    0
-$EndComp
 Wire Wire Line
 	3300 1800 3600 1800
-Text HLabel 3300 1800 0    50   Input ~ 0
-STM32_PWM_OUT
 $Comp
 L Connector_Generic:Conn_01x02 J8
 U 1 1 5CE46D1B
-P 4800 1700
-F 0 "J8" H 4900 1700 50  0000 L CNN
-F 1 "PWM_OUT" H 4900 1600 50  0000 L CNN
-F 2 "Connector_PinSocket_2.54mm:PinSocket_1x02_P2.54mm_Vertical" H 4800 1700 50  0001 C CNN
-F 3 "~" H 4800 1700 50  0001 C CNN
-	1    4800 1700
+P 4800 1800
+F 0 "J8" H 4900 1800 50  0000 L CNN
+F 1 "PWM_OUT" H 4900 1700 50  0000 L CNN
+F 2 "Connector_PinSocket_2.54mm:PinSocket_1x02_P2.54mm_Vertical" H 4800 1800 50  0001 C CNN
+F 3 "~" H 4800 1800 50  0001 C CNN
+	1    4800 1800
 	1    0    0    -1
 $EndComp
 Wire Wire Line
 	4150 1800 4600 1800
-Wire Wire Line
-	4000 1300 4200 1300
-Wire Wire Line
-	4200 1300 4200 1700
-Wire Wire Line
-	4200 1700 4600 1700
-Text HLabel 3300 1300 0    50   Input ~ 0
+Text HLabel 3300 1800 0    50   Input ~ 0
 STM32_PWM_IN
-Wire Wire Line
-	3300 1300 3800 1300
 $Comp
 L power:GND #PWR0170
@@
 Wire Wire Line
 	3950 1500 3950 1750
+$Comp
+L 74xGxx:74AHCT1G125 U4
+U 1 1 5CE46064
+P 3900 1800
+F 0 "U4" H 3900 1550 50  0001 C CNN
+F 1 "74AHCT1G125" H 3900 1600 50  0000 C CNN
+F 2 "Package_TO_SOT_SMD:SOT-23-5_HandSoldering" H 3900 1800 50  0001 C CNN
+F 3 "http://www.ti.com/lit/sg/scyt129e/scyt129e.pdf" H 3900 1800 50  0001 C CNN
+	1    3900 1800
+	1    0    0    -1
+$EndComp
+$Comp
+L power:GND #PWR0173
+U 1 1 5CF7855D
+P 4450 2150
+F 0 "#PWR0173" H 4450 1900 50  0001 C CNN
+F 1 "GND" H 4500 1950 50  0000 C CNN
+F 2 "" H 4450 2150 50  0001 C CNN
+F 3 "" H 4450 2150 50  0001 C CNN
+	1    4450 2150
+	1    0    0    -1
+$EndComp
+Wire Wire Line
+	4450 2150 4450 1900
+Wire Wire Line
+	4450 1900 4600 1900
 $EndSCHEMATC

Commit message: update,
Parts:
- renumbered J8 to J9
Changed lines of the file:
@@
 	3300 1800 3600 1800
 $Comp
-L Connector_Generic:Conn_01x02 J8
+L Connector_Generic:Conn_01x02 J9
 U 1 1 5CE46D1B
 P 4800 1800
-F 0 "J8" H 4900 1800 50  0000 L CNN
+F 0 "J9" H 4900 1800 50  0000 L CNN
 F 1 "PWM_OUT" H 4900 1700 50  0000 L CNN
 F 2 "Connector_PinSocket_2.54mm:PinSocket_1x02_P2.54mm_Vertical" H 4800 1800 50  0001 C CNN
@@
 STM32_PWM_IN
 $Comp
-L power:GND #PWR0170
+L power:GND #PWR050
 U 1 1 5CF4DA4F
 P 3650 1600
-F 0 "#PWR0170" H 3650 1350 50  0001 C CNN
+F 0 "#PWR050" H 3650 1350 50  0001 C CNN
 F 1 "GND" H 3700 1400 50  0000 C CNN
 F 2 "" H 3650 1600 50  0001 C CNN
@@
 	3650 1550 3650 1600
 $Comp
-L power:+5V #PWR0171
+L power:+5V #PWR049
 U 1 1 5CF4DEC2
 P 3950 1500
-F 0 "#PWR0171" H 3950 1350 50  0001 C CNN
+F 0 "#PWR049" H 3950 1350 50  0001 C CNN
 F 1 "+5V" H 4000 1700 50  0000 C CNN
 F 2 "" H 3950 1500 50  0001 C CNN
@@
 $EndComp
 $Comp
-L power:GND #PWR0172
+L power:GND #PWR051
 U 1 1 5CF4E2CB
 P 3950 2100
-F 0 "#PWR0172" H 3950 1850 50  0001 C CNN
+F 0 "#PWR051" H 3950 1850 50  0001 C CNN
 F 1 "GND" H 4000 1900 50  0000 C CNN
 F 2 "" H 3950 2100 50  0001 C CNN
@@
 $EndComp
 $Comp
-L power:GND #PWR0173
+L power:GND #PWR052
 U 1 1 5CF7855D
 P 4450 2150
-F 0 "#PWR0173" H 4450 1900 50  0001 C CNN
+F 0 "#PWR052" H 4450 1900 50  0001 C CNN
 F 1 "GND" H 4500 1950 50  0000 C CNN
 F 2 "" H 4450 2150 50  0001 C CNN
