File: hardware/button.sch (KiCad schematic (older format))
At the start: 4 parts

Commit message: update,
Changed lines of the file:
@@
 U 1 1 5CE61016
 P 4350 3750
-F 0 "SW?" V 4300 3900 50  0000 L CNN
-F 1 "SW_RESET,2_leg,SMD" V 4350 3900 50  0000 L CNN
+F 0 "SW?" V 4300 3700 50  0000 R CNN
+F 1 "SW_RESET,2_leg,SMD" V 4350 3700 50  0000 R CNN
 F 2 "footprint-lib:SW_SPST_CK_RS282G05A3" H 4350 3950 50  0001 C CNN
 F 3 "~" H 4350 3950 50  0001 C CNN
@@
 U 1 1 5CE6161C
 P 5550 3850
-F 0 "R?" H 5650 3900 50  0000 L CNN
-F 1 "R103,0603" H 5650 3850 50  0000 L CNN
+F 0 "R?" H 5450 3800 50  0000 R CNN
+F 1 "R103,0603" H 5450 3850 50  0000 R CNN
 F 2 "Resistor_SMD:R_0603_1608Metric_Pad1.05x0.95mm_HandSolder" H 5550 3850 50  0001 C CNN
 F 3 "~" H 5550 3850 50  0001 C CNN
@@
 U 1 1 5CE61626
 P 5550 3350
-F 0 "SW?" V 5500 3500 50  0000 L CNN
+F 0 "SW?" V 5600 3500 50  0000 L CNN
 F 1 "SW_RESET,2_leg,SMD" V 5550 3500 50  0000 L CNN
 F 2 "footprint-lib:SW_SPST_CK_RS282G05A3" H 5550 3550 50  0001 C CNN

Commit message: update,
Parts:
- gave numbers to parts that had none: 4
Changed lines of the file:
@@
 $Descr A4 11693 8268
 encoding utf-8
-Sheet 11 27
+Sheet 8 20
 Title ""
 Date ""
@@
 $EndBitmap
 $Comp
-L taobao-r:R103,0603 R?
+L taobao-r:R103,0603 R12
 U 1 1 5CE60C34
 P 4350 3250
-F 0 "R?" H 4450 3300 50  0000 L CNN
+F 0 "R12" H 4450 3300 50  0000 L CNN
 F 1 "R103,0603" H 4450 3250 50  0000 L CNN
 F 2 "Resistor_SMD:R_0603_1608Metric_Pad1.05x0.95mm_HandSolder" H 4350 3250 50  0001 C CNN
@@
 $EndComp
 $Comp
-L taobao-button:SW_RESET,2_leg,SMD SW?
+L taobao-button:SW_RESET,2_leg,SMD SW2
 U 1 1 5CE61016
 P 4350 3750
-F 0 "SW?" V 4300 3700 50  0000 R CNN
+F 0 "SW2" V 4300 3700 50  0000 R CNN
 F 1 "SW_RESET,2_leg,SMD" V 4350 3700 50  0000 R CNN
 F 2 "footprint-lib:SW_SPST_CK_RS282G05A3" H 4350 3950 50  0001 C CNN
@@
 $EndComp
 $Comp
-L taobao-r:R103,0603 R?
+L taobao-r:R103,0603 R13
 U 1 1 5CE6161C
 P 5550 3850
-F 0 "R?" H 5450 3800 50  0000 R CNN
+F 0 "R13" H 5450 3800 50  0000 R CNN
 F 1 "R103,0603" H 5450 3850 50  0000 R CNN
 F 2 "Resistor_SMD:R_0603_1608Metric_Pad1.05x0.95mm_HandSolder" H 5550 3850 50  0001 C CNN
@@
 $EndComp
 $Comp
-L taobao-button:SW_RESET,2_leg,SMD SW?
+L taobao-button:SW_RESET,2_leg,SMD SW1
 U 1 1 5CE61626
 P 5550 3350
-F 0 "SW?" V 5600 3500 50  0000 L CNN
+F 0 "SW1" V 5600 3500 50  0000 L CNN
 F 1 "SW_RESET,2_leg,SMD" V 5550 3500 50  0000 L CNN
 F 2 "footprint-lib:SW_SPST_CK_RS282G05A3" H 5550 3550 50  0001 C CNN
@@
 $EndComp
 $Comp
-L power:GND #PWR?
+L power:GND #PWR048
 U 1 1 5CE6251B
 P 4350 4200
-F 0 "#PWR?" H 4350 3950 50  0001 C CNN
+F 0 "#PWR048" H 4350 3950 50  0001 C CNN
 F 1 "GND" H 4400 4000 50  0000 C CNN
 F 2 "" H 4350 4200 50  0001 C CNN
@@
 $EndComp
 $Comp
-L power:GND #PWR?
+L power:GND #PWR049
 U 1 1 5CE6275D
 P 5550 4200
-F 0 "#PWR?" H 5550 3950 50  0001 C CNN
+F 0 "#PWR049" H 5550 3950 50  0001 C CNN
 F 1 "GND" H 5600 4000 50  0000 C CNN
 F 2 "" H 5550 4200 50  0001 C CNN
@@
 Connection ~ 4350 3450
 $Comp
-L power:+3V3 #PWR?
+L power:+3V3 #PWR046
 U 1 1 5CE630C6
 P 4350 3000
-F 0 "#PWR?" H 4350 2850 50  0001 C CNN
+F 0 "#PWR046" H 4350 2850 50  0001 C CNN
 F 1 "+3V3" H 4400 3200 50  0000 C CNN
 F 2 "" H 4350 3000 50  0001 C CNN
@@
 $EndComp
 $Comp
-L power:+3V3 #PWR?
+L power:+3V3 #PWR047
 U 1 1 5CE63769
 P 5550 3000
-F 0 "#PWR?" H 5550 2850 50  0001 C CNN
+F 0 "#PWR047" H 5550 2850 50  0001 C CNN
 F 1 "+3V3" H 5600 3200 50  0000 C CNN
 F 2 "" H 5550 3000 50  0001 C CNN

Commit message: update,
Parts:
- renumbered R12 to R7, R13 to R8
Changed lines of the file:
@@
 $EndBitmap
 $Comp
-L taobao-r:R103,0603 R12
+L taobao-r:R103,0603 R7
 U 1 1 5CE60C34
 P 4350 3250
-F 0 "R12" H 4450 3300 50  0000 L CNN
+F 0 "R7" H 4450 3300 50  0000 L CNN
 F 1 "R103,0603" H 4450 3250 50  0000 L CNN
 F 2 "Resistor_SMD:R_0603_1608Metric_Pad1.05x0.95mm_HandSolder" H 4350 3250 50  0001 C CNN
@@
 $EndComp
 $Comp
-L taobao-r:R103,0603 R13
+L taobao-r:R103,0603 R8
 U 1 1 5CE6161C
 P 5550 3850
-F 0 "R13" H 5450 3800 50  0000 R CNN
+F 0 "R8" H 5450 3800 50  0000 R CNN
 F 1 "R103,0603" H 5450 3850 50  0000 R CNN
 F 2 "Resistor_SMD:R_0603_1608Metric_Pad1.05x0.95mm_HandSolder" H 5550 3850 50  0001 C CNN
@@
 $EndComp
 $Comp
-L power:GND #PWR048
+L power:GND #PWR041
 U 1 1 5CE6251B
 P 4350 4200
-F 0 "#PWR048" H 4350 3950 50  0001 C CNN
+F 0 "#PWR041" H 4350 3950 50  0001 C CNN
 F 1 "GND" H 4400 4000 50  0000 C CNN
 F 2 "" H 4350 4200 50  0001 C CNN
@@
 $EndComp
 $Comp
-L power:GND #PWR049
+L power:GND #PWR042
 U 1 1 5CE6275D
 P 5550 4200
-F 0 "#PWR049" H 5550 3950 50  0001 C CNN
+F 0 "#PWR042" H 5550 3950 50  0001 C CNN
 F 1 "GND" H 5600 4000 50  0000 C CNN
 F 2 "" H 5550 4200 50  0001 C CNN
@@
 Connection ~ 4350 3450
 $Comp
-L power:+3V3 #PWR046
+L power:+3V3 #PWR039
 U 1 1 5CE630C6
 P 4350 3000
-F 0 "#PWR046" H 4350 2850 50  0001 C CNN
+F 0 "#PWR039" H 4350 2850 50  0001 C CNN
 F 1 "+3V3" H 4400 3200 50  0000 C CNN
 F 2 "" H 4350 3000 50  0001 C CNN
@@
 $EndComp
 $Comp
-L power:+3V3 #PWR047
+L power:+3V3 #PWR040
 U 1 1 5CE63769
 P 5550 3000
-F 0 "#PWR047" H 5550 2850 50  0001 C CNN
+F 0 "#PWR040" H 5550 2850 50  0001 C CNN
 F 1 "+3V3" H 5600 3200 50  0000 C CNN
 F 2 "" H 5550 3000 50  0001 C CNN
