File: hardware/spi.sch (KiCad schematic (older format))
At the start: 5 parts, among them J20 I2C_DEBUG, U9 W25Q32JVSSIQ

Commit message: update,
Parts:
- removed U9: W25Q32JVSSIQ, footprint-lib:I2C_DEBUG, symbol taobao-components:W25Q32JVSSIQ
- added U?: W25Q32JVSSIQ, footprint-lib:W25Q32JVSSIQ, symbol taobao-components:W25Q32JVSSIQ
Changed lines of the file:
@@
 $Descr A4 11693 8268
 encoding utf-8
-Sheet 8 27
+Sheet 13 27
 Title ""
 Date ""
@@
 $EndBitmap
 $Comp
-L taobao-components:W25Q32JVSSIQ U9
-U 1 1 5CF2C0C7
-P 4200 3900
-F 0 "U9" H 4200 4350 50  0000 C CNN
-F 1 "W25Q32JVSSIQ" H 4200 4250 50  0000 C CNN
-F 2 "footprint-lib:I2C_DEBUG" H 4100 3700 50  0001 C CNN
-F 3 "" H 4100 3700 50  0001 C CNN
-	1    4200 3900
-	1    0    0    -1
-$EndComp
-$Comp
 L power:GND #PWR0219
 U 1 1 5CF2C6A3
@@
 Wire Wire Line
 	3350 4250 3350 4050
-Wire Wire Line
-	3350 4050 3500 4050
 $Comp
 L taobao-components:I2C_DEBUG J20
@@
 	5450 4800 5450 3950
 Wire Wire Line
-	5450 3950 4900 3950
-Wire Wire Line
 	2150 3950 2300 3950
 Wire Wire Line
@@
 Wire Wire Line
 	5350 4700 5350 4050
-Wire Wire Line
-	5350 4050 4900 4050
 Wire Wire Line
 	2150 3850 2400 3850
@@
 	2800 3750 2800 3400
 Connection ~ 2800 3750
-Wire Wire Line
-	2800 3750 3500 3750
 $Comp
 L power:+3V3 #PWR0220
@@
 	5100 3000 5100 3750
 Wire Wire Line
-	5100 3750 4900 3750
-Wire Wire Line
 	2800 3000 3400 3000
 Connection ~ 2800 3000
@@
 	2800 3000 2800 3200
 Wire Wire Line
-	4900 3850 5100 3850
-Wire Wire Line
 	5100 3850 5100 3750
 Connection ~ 5100 3750
-Wire Wire Line
-	3500 3950 3400 3950
 Wire Wire Line
 	3400 3950 3400 3000
@@
 	2400 3550 2400 3850
 Connection ~ 2400 3850
-Wire Wire Line
-	2400 3850 3500 3850
 Wire Wire Line
 	3050 4700 5350 4700
@@
 Wire Wire Line
 	4400 2700 4550 2700
+$Comp
+L taobao-components:W25Q32JVSSIQ U?
+U 1 1 5CEA6EB7
+P 4200 3900
+F 0 "U?" H 4200 4400 50  0000 C CNN
+F 1 "W25Q32JVSSIQ" H 4200 4300 50  0000 C CNN
+F 2 "footprint-lib:W25Q32JVSSIQ" H 4200 3500 50  0001 C CNN
+F 3 "https://www.google.com/url?sa=t&rct=j&q=&esrc=s&source=web&cd=1&cad=rja&uact=8&ved=2ahUKEwi02JP0prjiAhXaBIgKHRI3AjoQFjAAegQIABAC&url=https%3A%2F%2Fwww.winbond.com%2Fresource-files%2Fw25q32jv%2520spi%2520revc%252008302016.pdf&usg=AOvVaw224j1hLYjMOvdAbYlB56Mn" H 4500 3850 50  0001 C CNN
+	1    4200 3900
+	1    0    0    -1
+$EndComp
+Wire Wire Line
+	4700 3750 5100 3750
+Wire Wire Line
+	4700 3950 5450 3950
+Wire Wire Line
+	4700 4050 5350 4050
+Wire Wire Line
+	2800 3750 3700 3750
+Wire Wire Line
+	4700 3850 5100 3850
+Wire Wire Line
+	3350 4050 3700 4050
+Wire Wire Line
+	3400 3950 3700 3950
+Wire Wire Line
+	2400 3850 3700 3850
 $EndSCHEMATC

Commit message: update,
Parts:
- removed RN4: R_Pack04, Resistor_SMD:R_Array_Concave_4x0603, symbol Device:R_Pack04
- J2: renamed from J20; value I2C_DEBUG -> SPI_DEBUG; symbol taobao-components:I2C_DEBUG -> taobao-components:SPI_DEBUG
- gave numbers to parts that had none: 1
- renumbered C34 to C8, R9 to R6
Connections:
- net labels added: MISO, MOSI, SCK, SS
- wire segments 45 -> 32
Other:
- moved on the sheet: C8, R6, U4

Commit message: update,
Parts:
- renumbered C8 to C6, J2 to J1, R6 to R1, U4 to U3
Changed lines of the file:
@@
 $EndBitmap
 $Comp
-L power:GND #PWR034
+L power:GND #PWR027
 U 1 1 5CF2C6A3
 P 5100 2750
-F 0 "#PWR034" H 5100 2500 50  0001 C CNN
+F 0 "#PWR027" H 5100 2500 50  0001 C CNN
 F 1 "GND" H 5150 2550 50  0000 C CNN
 F 2 "" H 5100 2750 50  0001 C CNN
@@
 	5100 2750 5100 2550
 $Comp
-L taobao-components:SPI_DEBUG J2
+L taobao-components:SPI_DEBUG J1
 U 1 1 5CF3AB80
 P 3700 2400
-F 0 "J2" H 3650 2450 50  0000 R CNN
+F 0 "J1" H 3650 2450 50  0000 R CNN
 F 1 "SPI_DEBUG" H 3650 2350 50  0000 R CNN
 F 2 "footprint-lib:TTL_TERMINAL_2.54mm" H 3700 2000 50  0001 C CNN
@@
 	7100 3200 7100 2550
 $Comp
-L taobao-r:R103,0603 R6
+L taobao-r:R103,0603 R1
 U 1 1 5CF3D550
 P 4550 1800
-F 0 "R6" H 4650 1850 50  0000 L CNN
+F 0 "R1" H 4650 1850 50  0000 L CNN
 F 1 "R103,0603" H 4650 1800 50  0000 L CNN
 F 2 "Resistor_SMD:R_0603_1608Metric_Pad1.05x0.95mm_HandSolder" H 4550 1800 50  0001 C CNN
@@
 Connection ~ 4550 2250
 $Comp
-L power:+3V3 #PWR033
+L power:+3V3 #PWR026
 U 1 1 5CF3F8B4
 P 4550 1400
-F 0 "#PWR033" H 4550 1250 50  0001 C CNN
+F 0 "#PWR026" H 4550 1250 50  0001 C CNN
 F 1 "+3V3" H 4600 1600 50  0000 C CNN
 F 2 "" H 4550 1400 50  0001 C CNN
@@
 	5150 1500 6850 1500
 $Comp
-L power:+3V3 #PWR031
+L power:+3V3 #PWR024
 U 1 1 5CF93293
 P 5800 1200
-F 0 "#PWR031" H 5800 1050 50  0001 C CNN
+F 0 "#PWR024" H 5800 1050 50  0001 C CNN
 F 1 "+3V3" V 5850 1350 50  0000 L CNN
 F 2 "" H 5800 1200 50  0001 C CNN
@@
 $EndComp
 $Comp
-L power:GND #PWR032
+L power:GND #PWR025
 U 1 1 5CF93299
 P 6300 1200
-F 0 "#PWR032" H 6300 950 50  0001 C CNN
+F 0 "#PWR025" H 6300 950 50  0001 C CNN
 F 1 "GND" V 6350 1050 50  0000 R CNN
 F 2 "" H 6300 1200 50  0001 C CNN
@@
 $EndComp
 $Comp
-L taobao-c:C106,0805 C8
+L taobao-c:C106,0805 C6
 U 1 1 5CF9329F
 P 6050 1200
-F 0 "C8" V 5800 1200 50  0000 C CNN
+F 0 "C6" V 5800 1200 50  0000 C CNN
 F 1 "C106,0805" V 5900 1200 50  0000 C CNN
 F 2 "Capacitor_SMD:C_0805_2012Metric_Pad1.15x1.40mm_HandSolder" H 6050 1200 50  0001 C CNN
@@
 	6150 1200 6300 1200
 $Comp
-L taobao-components:W25Q32JVSSIQ U4
+L taobao-components:W25Q32JVSSIQ U3
 U 1 1 5CEA6EB7
 P 5950 2400
-F 0 "U4" H 5950 2900 50  0000 C CNN
+F 0 "U3" H 5950 2900 50  0000 C CNN
 F 1 "W25Q32JVSSIQ" H 5950 2800 50  0000 C CNN
 F 2 "footprint-lib:W25Q32JVSSIQ" H 5950 2000 50  0001 C CNN

Commit message: update,
Parts:
- renumbered J1 to J2
Changed lines of the file:
@@
 $Descr User 8500 5500
 encoding utf-8
-Sheet 5 19
+Sheet 4 19
 Title ""
 Date ""
@@
 	5100 2750 5100 2550
 $Comp
-L taobao-components:SPI_DEBUG J1
+L taobao-components:SPI_DEBUG J2
 U 1 1 5CF3AB80
 P 3700 2400
-F 0 "J1" H 3650 2450 50  0000 R CNN
+F 0 "J2" H 3650 2450 50  0000 R CNN
 F 1 "SPI_DEBUG" H 3650 2350 50  0000 R CNN
 F 2 "footprint-lib:TTL_TERMINAL_2.54mm" H 3700 2000 50  0001 C CNN

Commit message: update,
Parts:
- J2: value SPI_DEBUG -> SPI_HEADER
Changed lines of the file:
@@
 $Descr User 8500 5500
 encoding utf-8
-Sheet 4 19
+Sheet 4 22
 Title ""
 Date ""
@@
 P 3700 2400
 F 0 "J2" H 3650 2450 50  0000 R CNN
-F 1 "SPI_DEBUG" H 3650 2350 50  0000 R CNN
+F 1 "SPI_HEADER" H 3650 2350 50  0000 R CNN
 F 2 "footprint-lib:TTL_TERMINAL_2.54mm" H 3700 2000 50  0001 C CNN
 F 3 "~" H 3700 2450 50  0001 C CNN
