File: hardware/rotatry_encoder.sch (KiCad schematic (older format))
At the start: 7 parts, among them SW3 EC11_VERTICAL

Commit message: update,
Parts:
- added J?: ROT_ENC_HEADER, symbol Connector:Conn_01x03_Female
Connections:
- net A: now also J?.1 (Pin_1)
- net B: now also J?.2 (Pin_2)
- net SW_OUT: now also J?.3 (Pin_3)
Changed lines of the file:
@@
 	2000 3250 2800 3250
 Connection ~ 2800 3250
+$Comp
+L Connector:Conn_01x03_Female J?
+U 1 1 5CF225E9
+P 1100 2200
+F 0 "J?" H 950 2500 50  0000 C CNN
+F 1 "ROT_ENC_HEADER" H 950 2400 50  0000 C CNN
+F 2 "" H 1100 2200 50  0001 C CNN
+F 3 "~" H 1100 2200 50  0001 C CNN
+	1    1100 2200
+	-1   0    0    -1
+$EndComp
+Text Label 1800 2100 2    50   ~ 0
+ROT_ENC_A
+Text Label 1800 2200 2    50   ~ 0
+ROT_ENC_B
+Text Label 1800 2300 2    50   ~ 0
+ROT_ENC_SW
+Wire Wire Line
+	1800 2100 1300 2100
+Wire Wire Line
+	1800 2200 1300 2200
+Wire Wire Line
+	1800 2300 1300 2300
 $EndSCHEMATC

Commit message: update,
Parts:
- gave numbers to parts that had none: 1
- renumbered C14 to C24, C15 to C25, C16 to C26, R13 to R16, R14 to R17, R15 to R18
Changed lines of the file:
@@
 $EndBitmap
 $Comp
-L taobao-r:R273,0603 R13
+L taobao-r:R273,0603 R16
 U 1 1 5CED60AF
 P 3150 2300
-F 0 "R13" V 2900 2300 50  0000 C CNN
+F 0 "R16" V 2900 2300 50  0000 C CNN
 F 1 "R273,0603" V 3000 2300 50  0000 C CNN
 F 2 "Resistor_SMD:R_0603_1608Metric_Pad1.05x0.95mm_HandSolder" H 3150 2300 50  0001 C CNN
@@
 $EndComp
 $Comp
-L taobao-r:R273,0603 R14
+L taobao-r:R273,0603 R17
 U 1 1 5CED6622
 P 3150 2800
-F 0 "R14" V 2900 2800 50  0000 C CNN
+F 0 "R17" V 2900 2800 50  0000 C CNN
 F 1 "R273,0603" V 3000 2800 50  0000 C CNN
 F 2 "Resistor_SMD:R_0603_1608Metric_Pad1.05x0.95mm_HandSolder" H 3150 2800 50  0001 C CNN
@@
 $EndComp
 $Comp
-L taobao-r:R273,0603 R15
+L taobao-r:R273,0603 R18
 U 1 1 5CED67EF
 P 3150 3250
-F 0 "R15" V 2900 3250 50  0000 C CNN
+F 0 "R18" V 2900 3250 50  0000 C CNN
 F 1 "R273,0603" V 3000 3250 50  0000 C CNN
 F 2 "Resistor_SMD:R_0603_1608Metric_Pad1.05x0.95mm_HandSolder" H 3150 3250 50  0001 C CNN
@@
 $EndComp
 $Comp
-L taobao-c:C104,0603 C16
+L taobao-c:C104,0603 C26
 U 1 1 5CED6CD1
 P 2800 3450
-F 0 "C16" H 2900 3500 50  0000 L CNN
+F 0 "C26" H 2900 3500 50  0000 L CNN
 F 1 "C104,0603" H 2900 3450 50  0000 L CNN
 F 2 "Capacitor_SMD:C_0603_1608Metric_Pad1.05x0.95mm_HandSolder" H 2800 3450 50  0001 C CNN
@@
 $EndComp
 $Comp
-L taobao-c:C104,0603 C15
+L taobao-c:C104,0603 C25
 U 1 1 5CED7298
 P 2800 2950
-F 0 "C15" H 2900 3000 50  0000 L CNN
+F 0 "C25" H 2900 3000 50  0000 L CNN
 F 1 "C104,0603" H 2900 2950 50  0000 L CNN
 F 2 "Capacitor_SMD:C_0603_1608Metric_Pad1.05x0.95mm_HandSolder" H 2800 2950 50  0001 C CNN
@@
 $EndComp
 $Comp
-L taobao-c:C104,0603 C14
+L taobao-c:C104,0603 C24
 U 1 1 5CED75A5
 P 2800 2500
-F 0 "C14" H 2900 2550 50  0000 L CNN
+F 0 "C24" H 2900 2550 50  0000 L CNN
 F 1 "C104,0603" H 2900 2500 50  0000 L CNN
 F 2 "Capacitor_SMD:C_0603_1608Metric_Pad1.05x0.95mm_HandSolder" H 2800 2500 50  0001 C CNN
@@
 	2800 3250 2800 3350
 $Comp
-L power:GND #PWR084
+L power:GND #PWR0126
 U 1 1 5CED86F3
 P 2800 2650
-F 0 "#PWR084" H 2800 2400 50  0001 C CNN
+F 0 "#PWR0126" H 2800 2400 50  0001 C CNN
 F 1 "GND" H 2850 2450 50  0000 C CNN
 F 2 "" H 2800 2650 50  0001 C CNN
@@
 	2800 2650 2800 2600
 $Comp
-L power:GND #PWR086
+L power:GND #PWR0128
 U 1 1 5CED8B04
 P 2800 3100
-F 0 "#PWR086" H 2800 2850 50  0001 C CNN
+F 0 "#PWR0128" H 2800 2850 50  0001 C CNN
 F 1 "GND" H 2850 2900 50  0000 C CNN
 F 2 "" H 2800 3100 50  0001 C CNN
@@
 	2800 3100 2800 3050
 $Comp
-L power:GND #PWR087
+L power:GND #PWR0129
 U 1 1 5CED8F95
 P 2800 3600
-F 0 "#PWR087" H 2800 3350 50  0001 C CNN
+F 0 "#PWR0129" H 2800 3350 50  0001 C CNN
 F 1 "GND" H 2850 3400 50  0000 C CNN
 F 2 "" H 2800 3600 50  0001 C CNN
@@
 	2800 3600 2800 3550
 $Comp
-L power:GND #PWR083
+L power:GND #PWR0125
 U 1 1 5CED947F
 P 3350 2600
-F 0 "#PWR083" H 3350 2350 50  0001 C CNN
+F 0 "#PWR0125" H 3350 2350 50  0001 C CNN
 F 1 "GND" H 3400 2400 50  0000 C CNN
 F 2 "" H 3350 2600 50  0001 C CNN
@@
 $EndComp
 $Comp
-L power:GND #PWR085
+L power:GND #PWR0127
 U 1 1 5CED96CA
 P 4400 2900
-F 0 "#PWR085" H 4400 2650 50  0001 C CNN
+F 0 "#PWR0127" H 4400 2650 50  0001 C CNN
 F 1 "GND" H 4450 2700 50  0000 C CNN
 F 2 "" H 4400 2900 50  0001 C CNN
@@
 Connection ~ 2800 3250
 $Comp
-L Connector:Conn_01x03_Female J?
+L Connector:Conn_01x03_Female J35
 U 1 1 5CF225E9
 P 1100 2200
-F 0 "J?" H 950 2500 50  0000 C CNN
+F 0 "J35" H 950 2500 50  0000 C CNN
 F 1 "ROT_ENC_HEADER" H 950 2400 50  0000 C CNN
 F 2 "" H 1100 2200 50  0001 C CNN

Commit message: update,
Parts:
- renumbered J35 to J36
Changed lines of the file:
@@
 Connection ~ 2800 3250
 $Comp
-L Connector:Conn_01x03_Female J35
+L Connector:Conn_01x03_Female J36
 U 1 1 5CF225E9
 P 1100 2200
-F 0 "J35" H 950 2500 50  0000 C CNN
+F 0 "J36" H 950 2500 50  0000 C CNN
 F 1 "ROT_ENC_HEADER" H 950 2400 50  0000 C CNN
 F 2 "" H 1100 2200 50  0001 C CNN

Commit message: update footprint,
Parts:
- J36: footprint (none) -> Connector_PinHeader_1.27mm:PinHeader_1x03_P1.27mm_Vertical
Changed lines of the file:
@@
 F 0 "J36" H 950 2500 50  0000 C CNN
 F 1 "ROT_ENC_HEADER" H 950 2400 50  0000 C CNN
-F 2 "" H 1100 2200 50  0001 C CNN
+F 2 "Connector_PinHeader_1.27mm:PinHeader_1x03_P1.27mm_Vertical" H 1100 2200 50  0001 C CNN
 F 3 "~" H 1100 2200 50  0001 C CNN
 	1    1100 2200
