File: hardware/AMS1117_1.sch (KiCad schematic (older format))
At the start: 9 parts

Commit message: update,
Parts:
- removed C?: C104,0603, Capacitor_SMD:C_0603_1608Metric_Pad1.05x0.95mm_HandSolder, symbol taobao-c:C104,0603
- removed D?: LED_GREEN,0603, LED_SMD:LED_0603_1608Metric_Pad1.05x0.95mm_HandSolder, symbol taobao-led:LED_GREEN,0603
- removed J?: Conn_01x03, Connector_PinHeader_2.54mm:PinHeader_1x03_P2.54mm_Vertical, symbol Connector_Generic:Conn_01x03
- removed JP? (x2): Jumper_NO_Small, symbol Device:Jumper_NO_Small
- removed U?: AMS1117-3.3, Package_TO_SOT_SMD:SOT-223-3_TabPin2, symbol Regulator_Linear:AMS1117-3.3
- added C8: C104,0603, Capacitor_SMD:C_0603_1608Metric_Pad1.05x0.95mm_HandSolder, symbol taobao-c:C104,0603
- added D9: LED_GREEN,0603, LED_SMD:LED_0603_1608Metric_Pad1.05x0.95mm_HandSolder, symbol taobao-led:LED_GREEN,0603
- added J12: Conn_01x03, Connector_PinHeader_2.54mm:PinHeader_1x03_P2.54mm_Vertical, symbol Connector_Generic:Conn_01x03
- added JP3, JP4: Jumper_NO_Small, symbol Device:Jumper_NO_Small
- added U4: AMS1117-3.3, Package_TO_SOT_SMD:SOT-223-3_TabPin2, symbol Regulator_Linear:AMS1117-3.3
- gave numbers to parts that had none: 3
Connections:
- net +3V3: now also D9.2 (A), J12.2 (Pin_2), J12.3 (Pin_3), JP4.1
- net +5V: now also JP3.1
- net GND: now also C8.2, J12.1 (Pin_1), U4.1 (GND)
- net at C10.1, C9.1: now also JP4.2, U4.2 (VO)
- net at R7.1: now also D9.1 (K)
- new net: C8.1, JP3.2, U4.3 (VI)

Commit message: update,
Other:
- moved on the sheet: C10, C8, C9, D9, J12, JP3, JP4, R7, U4

Commit message: update footprint,
Parts:
- JP3: value Jumper_NO_Small -> PWR_SRC; footprint (none) -> Connector_PinHeader_1.27mm:PinHeader_1x02_P1.27mm_Vertical
- JP4: value Jumper_NO_Small -> PWR_OUT; footprint (none) -> Connector_PinHeader_1.27mm:PinHeader_1x02_P1.27mm_Vertical
Changed lines of the file:
@@
 AR Path="/5CF05A5C/5CEC13BC/5CF53028" Ref="JP?"  Part="1"
 F 0 "JP3" V 2200 2150 50  0000 L CNN
-F 1 "Jumper_NO_Small" V 2250 2150 50  0000 L CNN
-F 2 "" H 2250 2100 50  0001 C CNN
+F 1 "PWR_SRC" V 2250 2150 50  0000 L CNN
+F 2 "Connector_PinHeader_1.27mm:PinHeader_1x02_P1.27mm_Vertical" H 2250 2100 50  0001 C CNN
 F 3 "~" H 2250 2100 50  0001 C CNN
 	1    2250 2100
@@
 AR Path="/5CF05A5C/5CEC13BC/5CF5302A" Ref="JP?"  Part="1"
 F 0 "JP4" V 3650 2150 50  0000 L CNN
-F 1 "Jumper_NO_Small" V 3700 2150 50  0000 L CNN
-F 2 "" H 3700 2100 50  0001 C CNN
+F 1 "PWR_OUT" V 3700 2150 50  0000 L CNN
+F 2 "Connector_PinHeader_1.27mm:PinHeader_1x02_P1.27mm_Vertical" H 3700 2100 50  0001 C CNN
 F 3 "~" H 3700 2100 50  0001 C CNN
 	1    3700 2100

Commit message: update footprint,
Parts:
- JP3, JP4: footprint Connector_PinHeader_1.27mm:PinHeader_1x02_P1.27mm_Vertical -> Jumper:SolderJumper-2_P1.3mm_Open_TrianglePad1.0x1.5mm
Changed lines of the file:
@@
 F 0 "JP3" V 2200 2150 50  0000 L CNN
 F 1 "PWR_SRC" V 2250 2150 50  0000 L CNN
-F 2 "Connector_PinHeader_1.27mm:PinHeader_1x02_P1.27mm_Vertical" H 2250 2100 50  0001 C CNN
+F 2 "Jumper:SolderJumper-2_P1.3mm_Open_TrianglePad1.0x1.5mm" H 2250 2100 50  0001 C CNN
 F 3 "~" H 2250 2100 50  0001 C CNN
 	1    2250 2100
@@
 F 0 "JP4" V 3650 2150 50  0000 L CNN
 F 1 "PWR_OUT" V 3700 2150 50  0000 L CNN
-F 2 "Connector_PinHeader_1.27mm:PinHeader_1x02_P1.27mm_Vertical" H 3700 2100 50  0001 C CNN
+F 2 "Jumper:SolderJumper-2_P1.3mm_Open_TrianglePad1.0x1.5mm" H 3700 2100 50  0001 C CNN
 F 3 "~" H 3700 2100 50  0001 C CNN
 	1    3700 2100
