File: hardware/AMS1117_2.sch (KiCad schematic (older format))
At the start: 9 parts

Commit message: update,
Parts:
- removed C?: CP47uf,50V, w_smd_cap:c_elec_6.3x7.7, symbol taobao-cp:CP47uf,50V
- removed C? (x2): C104,0603, Capacitor_SMD:C_0603_1608Metric_Pad1.05x0.95mm_HandSolder, symbol taobao-c:C104,0603
- removed D?: LED_GREEN,0603, LED_SMD:LED_0603_1608Metric_Pad1.05x0.95mm_HandSolder, symbol taobao-led:LED_GREEN,0603
- removed R?: R102,0603, Resistor_SMD:R_0603_1608Metric_Pad1.05x0.95mm_HandSolder, symbol taobao-r:R102,0603
- removed U?: AMS1117-3.3, Package_TO_SOT_SMD:SOT-223-3_TabPin2, symbol Regulator_Linear:AMS1117-3.3
- added C11, C12: C104,0603, Capacitor_SMD:C_0603_1608Metric_Pad1.05x0.95mm_HandSolder, symbol taobao-c:C104,0603
- added C13: CP47uf,50V, w_smd_cap:c_elec_6.3x7.7, symbol taobao-cp:CP47uf,50V
- added D10: LED_GREEN,0603, LED_SMD:LED_0603_1608Metric_Pad1.05x0.95mm_HandSolder, symbol taobao-led:LED_GREEN,0603
- added R8: R102,0603, Resistor_SMD:R_0603_1608Metric_Pad1.05x0.95mm_HandSolder, symbol taobao-r:R102,0603
- added U5: AMS1117-3.3, Package_TO_SOT_SMD:SOT-223-3_TabPin2, symbol Regulator_Linear:AMS1117-3.3
- gave numbers to parts that had none: 3
Connections:
- net +3V3: now also D10.2 (A)
- net GND: now also C11.2, C12.2, C13.2, R8.2, U5.1 (GND)
- net at JP6.2: now also C12.1, C13.1, U5.2 (VO)
- net at JP5.2: now also C11.1, U5.3 (VI)
- new net: D10.1 (K), R8.1

Commit message: update,
Parts:
- JP5, JP6: value Jumper_NO_Small -> NO
Connections:
- net +3V3 renamed Vb
Other:
- moved on the sheet: C11, C12, C13, D10, J13, JP5, JP6, R8, U5

Commit message: update footprint,
Parts:
- JP5: value NO -> PWR_SRC; footprint (none) -> Connector_PinHeader_1.27mm:PinHeader_1x02_P1.27mm_Vertical
- JP6: value NO -> PWR_OUT; footprint (none) -> Connector_PinHeader_1.27mm:PinHeader_1x02_P1.27mm_Vertical
Changed lines of the file:
@@
 AR Path="/5CF05A5C/5CEC1561/5C148323" Ref="JP?"  Part="1"
 F 0 "JP5" V 2100 2050 50  0000 L CNN
-F 1 "NO" V 2150 2050 50  0000 L CNN
-F 2 "" H 2150 2000 50  0001 C CNN
+F 1 "PWR_SRC" V 2150 2050 50  0000 L CNN
+F 2 "Connector_PinHeader_1.27mm:PinHeader_1x02_P1.27mm_Vertical" H 2150 2000 50  0001 C CNN
 F 3 "~" H 2150 2000 50  0001 C CNN
 	1    2150 2000
@@
 AR Path="/5CF05A5C/5CEC1561/5C148F3B" Ref="JP?"  Part="1"
 F 0 "JP6" V 3550 2050 50  0000 L CNN
-F 1 "NO" V 3600 2050 50  0000 L CNN
-F 2 "" H 3600 2000 50  0001 C CNN
+F 1 "PWR_OUT" V 3600 2050 50  0000 L CNN
+F 2 "Connector_PinHeader_1.27mm:PinHeader_1x02_P1.27mm_Vertical" H 3600 2000 50  0001 C CNN
 F 3 "~" H 3600 2000 50  0001 C CNN
 	1    3600 2000

Commit message: update footprint,
Parts:
- JP5, JP6: footprint Connector_PinHeader_1.27mm:PinHeader_1x02_P1.27mm_Vertical -> Jumper:SolderJumper-2_P1.3mm_Open_TrianglePad1.0x1.5mm
Changed lines of the file:
@@
 F 0 "JP5" V 2100 2050 50  0000 L CNN
 F 1 "PWR_SRC" V 2150 2050 50  0000 L CNN
-F 2 "Connector_PinHeader_1.27mm:PinHeader_1x02_P1.27mm_Vertical" H 2150 2000 50  0001 C CNN
+F 2 "Jumper:SolderJumper-2_P1.3mm_Open_TrianglePad1.0x1.5mm" H 2150 2000 50  0001 C CNN
 F 3 "~" H 2150 2000 50  0001 C CNN
 	1    2150 2000
@@
 F 0 "JP6" V 3550 2050 50  0000 L CNN
 F 1 "PWR_OUT" V 3600 2050 50  0000 L CNN
-F 2 "Connector_PinHeader_1.27mm:PinHeader_1x02_P1.27mm_Vertical" H 3600 2000 50  0001 C CNN
+F 2 "Jumper:SolderJumper-2_P1.3mm_Open_TrianglePad1.0x1.5mm" H 3600 2000 50  0001 C CNN
 F 3 "~" H 3600 2000 50  0001 C CNN
 	1    3600 2000
