File: hardware/AMS1117_3.sch (KiCad schematic (older format))
At the start: 9 parts

Commit message: update,
Parts:
- removed C?: CP47uf,50V, w_smd_cap:c_elec_6.3x7.7, symbol taobao-cp:CP47uf,50V
- removed C?: C104,0603, Capacitor_SMD:C_0603_1608Metric_Pad1.05x0.95mm_HandSolder, symbol taobao-c:C104,0603
- removed J?: Conn_01x03, Connector_PinHeader_2.54mm:PinHeader_1x03_P2.54mm_Vertical, symbol Connector_Generic:Conn_01x03
- removed JP? (x2): Jumper_NO_Small, symbol Device:Jumper_NO_Small
- removed R?: R102,0603, Resistor_SMD:R_0603_1608Metric_Pad1.05x0.95mm_HandSolder, symbol taobao-r:R102,0603
- added C15: C104,0603, Capacitor_SMD:C_0603_1608Metric_Pad1.05x0.95mm_HandSolder, symbol taobao-c:C104,0603
- added C16: CP47uf,50V, w_smd_cap:c_elec_6.3x7.7, symbol taobao-cp:CP47uf,50V
- added J14: Conn_01x03, Connector_PinHeader_2.54mm:PinHeader_1x03_P2.54mm_Vertical, symbol Connector_Generic:Conn_01x03
- added JP7, JP8: Jumper_NO_Small, symbol Device:Jumper_NO_Small
- added R9: R102,0603, Resistor_SMD:R_0603_1608Metric_Pad1.05x0.95mm_HandSolder, symbol taobao-r:R102,0603
- gave numbers to parts that had none: 3
Connections:
- net +3V3: now also J14.2 (Pin_2), J14.3 (Pin_3), JP8.1
- net +5V: now also JP7.1
- net GND: now also C15.2, C16.2, J14.1 (Pin_1), R9.2
- net at U6.2 (VO): now also C15.1, C16.1, JP8.2
- net at C14.1, U6.3 (VI): now also JP7.2
- net at D11.1 (K): now also R9.1

Commit message: update,
Parts:
- J14: value Conn_01x03 -> Va_header
- JP7, JP8: value Jumper_NO_Small -> NO
Connections:
- net +3V3 renamed Vc
Other:
- moved on the sheet: C14, C15, C16, D11, J14, JP7, JP8, R9, U6

Commit message: update footprint,
Parts:
- JP7: value NO -> PWR_SRC; footprint (none) -> Connector_PinHeader_1.27mm:PinHeader_1x02_P1.27mm_Vertical
- JP8: value NO -> PWR_OUT; footprint (none) -> Connector_PinHeader_1.27mm:PinHeader_1x02_P1.27mm_Vertical
Changed lines of the file:
@@
 AR Path="/5CF05A5C/5CEC1C2E/5CF53027" Ref="JP?"  Part="1"
 F 0 "JP7" V 2150 1900 50  0000 L CNN
-F 1 "NO" V 2200 1900 50  0000 L CNN
-F 2 "" H 2200 1850 50  0001 C CNN
+F 1 "PWR_SRC" V 2200 1900 50  0000 L CNN
+F 2 "Connector_PinHeader_1.27mm:PinHeader_1x02_P1.27mm_Vertical" H 2200 1850 50  0001 C CNN
 F 3 "~" H 2200 1850 50  0001 C CNN
 	1    2200 1850
@@
 AR Path="/5CF05A5C/5CEC1C2E/5CF53029" Ref="JP?"  Part="1"
 F 0 "JP8" V 3600 1900 50  0000 L CNN
-F 1 "NO" V 3650 1900 50  0000 L CNN
-F 2 "" H 3650 1850 50  0001 C CNN
+F 1 "PWR_OUT" V 3650 1900 50  0000 L CNN
+F 2 "Connector_PinHeader_1.27mm:PinHeader_1x02_P1.27mm_Vertical" H 3650 1850 50  0001 C CNN
 F 3 "~" H 3650 1850 50  0001 C CNN
 	1    3650 1850

Commit message: update footprint,
Parts:
- JP7, JP8: footprint Connector_PinHeader_1.27mm:PinHeader_1x02_P1.27mm_Vertical -> Jumper:SolderJumper-2_P1.3mm_Open_TrianglePad1.0x1.5mm
Changed lines of the file:
@@
 F 0 "JP7" V 2150 1900 50  0000 L CNN
 F 1 "PWR_SRC" V 2200 1900 50  0000 L CNN
-F 2 "Connector_PinHeader_1.27mm:PinHeader_1x02_P1.27mm_Vertical" H 2200 1850 50  0001 C CNN
+F 2 "Jumper:SolderJumper-2_P1.3mm_Open_TrianglePad1.0x1.5mm" H 2200 1850 50  0001 C CNN
 F 3 "~" H 2200 1850 50  0001 C CNN
 	1    2200 1850
@@
 F 0 "JP8" V 3600 1900 50  0000 L CNN
 F 1 "PWR_OUT" V 3650 1900 50  0000 L CNN
-F 2 "Connector_PinHeader_1.27mm:PinHeader_1x02_P1.27mm_Vertical" H 3650 1850 50  0001 C CNN
+F 2 "Jumper:SolderJumper-2_P1.3mm_Open_TrianglePad1.0x1.5mm" H 3650 1850 50  0001 C CNN
 F 3 "~" H 3650 1850 50  0001 C CNN
 	1    3650 1850
