File: hardware/bluepill.kicad_pcb (KiCad board)
At the start: 2 copper layers, 4 parts, among them J28 STM32_2_DEBUG1, J29 STM32_2_DEBUG2, U10 bluepill-stm32f103c8t6

Commit message: update footprint,
Parts:
- RN6: moved to B.Cu
- moved RN6 30.6 mm to (49.6, 62.0)
- moved J44 23.7 mm to (46.5, 55.8), turned to 0 degrees
- moved J43 14.1 mm to (46.9, 46.7)
- renumbered J28 to J43, J29 to J44, U10 to U13
Connections:
- net /PA12 renamed /SS_LORA
- net /PA3 renamed /BTN_PULL_DN
- net /PA8 renamed /LORA_DIO0
- net /PB0 renamed /BTN_PULL_UP
- net /SS_OLED renamed /LORA_RST
- J44 pad 13: /PA11 -> /BUZZER
- J44 pad 8: /BUZZER -> /OLED_RST
- U13 pad 13: /BUZZER -> /OLED_RST
- U13 pad 8: /PA11 -> /BUZZER
