File: hardware/arduino_nano.kicad_pcb (KiCad board)
At the start: 2 copper layers, 6 parts, among them J23 I2C_HEADER, J24 TTL_HEADER, J25 SPI_HEADER, J26 ARDUINO_HEADER1, J27 ARDUINO_HEADER2, U9 arduino_nano_v3

Commit message: update,
Parts:
- moved J26 16.3 mm to (40.0, 19.9)
- moved J23 12.2 mm to (45.0, 50.0)
- moved J27 11.1 mm to (40.0, 42.5)
Changed lines of the file:
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@@
   )
   (module Connector_PinHeader_1.27mm:PinHeader_1x15_P1.27mm_Vertical (layer F.Cu)
-    (at 29 41)
+    (at 40 42.5)
     (descr "Through hole straight pin header, 1x15, 1.27mm pitch, single row")
     (tags "Through hole pin header THT 1x15 1.27mm single row")
@@
   )
   (module Connector_PinHeader_1.27mm:PinHeader_1x15_P1.27mm_Vertical (layer F.Cu)
-    (at 24 23)
+    (at 40 19.9)
     (descr "Through hole straight pin header, 1x15, 1.27mm pitch, single row")
     (tags "Through hole pin header THT 1x15 1.27mm single row")
@@
   )
   (module footprint-lib:I2C_DEBUG (layer F.Cu)
-    (at 38 40 180)
+    (at 45 50 180)
     (descr "Through hole straight pin header, 1x02, 1.27mm pitch, single row")
     (tags "Through hole pin header THT 1x02 1.27mm single row")

Commit message: update footprint,
Parts:
- added J40: OLED_HEADER, Connector_PinHeader_1.27mm:PinHeader_1x05_P1.27mm_Vertical, F.Cu at (44.6, 24.8)
- renumbered J23 to J37, J24 to J38, J25 to J39, J26 to J41, J27 to J42, U9 to U12
Changed lines of the file:
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@@
     (tracks 0)
     (zones 0)
-    (modules 6)
+    (modules 7)
     (nets 28)
   )
@@
     (add_net GND)
   )
+  (module Connector_PinHeader_1.27mm:PinHeader_1x05_P1.27mm_Vertical (layer F.Cu)
+    (at 44.577 24.765)
+    (descr "Through hole straight pin header, 1x05, 1.27mm pitch, single row")
+    (tags "Through hole pin header THT 1x05 1.27mm single row")
+    (fp_text reference J40 (at 0 -1.695) (layer F.SilkS)
+      (effects (font (size 1 1) (thickness 0.15)))
+    )
+    (fp_text value OLED_HEADER (at 0 6.775) (layer F.Fab)
+      (effects (font (size 1 1) (thickness 0.15)))
+    )
+    (fp_text user %R (at 0 2.54 90) (layer F.Fab)
+      (effects (font (size 1 1) (thickness 0.15)))
+    )
+    (fp_line (start 1.55 -1.15) (end -1.55 -1.15) (layer F.CrtYd) (width 0.05))
+    (fp_line (start 1.55 6.25) (end 1.55 -1.15) (layer F.CrtYd) (width 0.05))
+    (fp_line (start -1.55 6.25) (end 1.55 6.25) (layer F.CrtYd) (width 0.05))
+    (fp_line (start -1.55 -1.15) (end -1.55 6.25) (layer F.CrtYd) (width 0.05))
+    (fp_line (start -1.11 -0.76) (end 0 -0.76) (layer F.SilkS) (width 0.12))
+    (fp_line (start -1.11 0) (end -1.11 -0.76) (layer F.SilkS) (width 0.12))
+    (fp_line (start 0.563471 0.76) (end 1.11 0.76) (layer F.SilkS) (width 0.12))
+    (fp_line (start -1.11 0.76) (end -0.563471 0.76) (layer F.SilkS) (width 0.12))
+    (fp_line (start 1.11 0.76) (end 1.11 5.775) (layer F.SilkS) (width 0.12))
+    (fp_line (start -1.11 0.76) (end -1.11 5.775) (layer F.SilkS) (width 0.12))
+    (fp_line (start 0.30753 5.775) (end 1.11 5.775) (layer F.SilkS) (width 0.12))
+    (fp_line (start -1.11 5.775) (end -0.30753 5.775) (layer F.SilkS) (width 0.12))
+    (fp_line (start -1.05 -0.11) (end -0.525 -0.635) (layer F.Fab) (width 0.1))
+    (fp_line (start -1.05 5.715) (end -1.05 -0.11) (layer F.Fab) (width 0.1))
+    (fp_line (start 1.05 5.715) (end -1.05 5.715) (layer F.Fab) (width 0.1))
+    (fp_line (start 1.05 -0.635) (end 1.05 5.715) (layer F.Fab) (width 0.1))
+    (fp_line (start -0.525 -0.635) (end 1.05 -0.635) (layer F.Fab) (width 0.1))
+    (pad 5 thru_hole oval (at 0 5.08) (size 1 1) (drill 0.65) (layers *.Cu *.Mask)
+      (net 13 /OLED_SS))
+    (pad 4 thru_hole oval (at 0 3.81) (size 1 1) (drill 0.65) (layers *.Cu *.Mask)
+      (net 14 /OLED_RST))
+    (pad 3 thru_hole oval (at 0 2.54) (size 1 1) (drill 0.65) (layers *.Cu *.Mask)
+      (net 15 /OLED_DC))
+    (pad 2 thru_hole oval (at 0 1.27) (size 1 1) (drill 0.65) (layers *.Cu *.Mask)
+      (net 9 /SCK))
+    (pad 1 thru_hole rect (at 0 0) (size 1 1) (drill 0.65) (layers *.Cu *.Mask)
+      (net 8 /MOSI))
+    (model ${KISYS3DMOD}/Connector_PinHeader_1.27mm.3dshapes/PinHeader_1x05_P1.27mm_Vertical.wrl
+      (at (xyz 0 0 0))
+      (scale (xyz 1 1 1))
+      (rotate (xyz 0 0 0))
+    )
+  )
   (module Module:Arduino_Nano (layer F.Cu)
     (at 19.05 22.91)
     (descr "Arduino Nano, http://www.mouser.com/pdfdocs/Gravitech_Arduino_Nano3_0.pdf")
     (tags "Arduino Nano")
-    (fp_text reference U9 (at 7.62 -5.08) (layer F.SilkS)
+    (fp_text reference U12 (at 7.62 -5.08) (layer F.SilkS)
       (effects (font (size 1 1) (thickness 0.15)))
     )
@@
     (descr "Through hole straight pin header, 1x15, 1.27mm pitch, single row")
     (tags "Through hole pin header THT 1x15 1.27mm single row")
-    (fp_text reference J27 (at 0 -1.695) (layer F.SilkS)
+    (fp_text reference J42 (at 0 -1.695) (layer F.SilkS)
       (effects (font (size 1 1) (thickness 0.15)))
     )
@@
     (descr "Through hole straight pin header, 1x15, 1.27mm pitch, single row")
     (tags "Through hole pin header THT 1x15 1.27mm single row")
-    (fp_text reference J26 (at 0 -1.695) (layer F.SilkS)
+    (fp_text reference J41 (at 0 -1.695) (layer F.SilkS)
       (effects (font (size 1 1) (thickness 0.15)))
     )
@@
     (descr "Through hole straight pin header, 1x04, 1.27mm pitch, single row")
     (tags "SPI DEBUG")
-    (fp_text reference J25 (at 0 -1.695) (layer F.SilkS)
+    (fp_text reference J39 (at 0 -1.695) (layer F.SilkS)
       (effects (font (size 1 1) (thickness 0.15)))
     )
@@
     (descr "Through hole straight pin header, 1x03, 1.27mm pitch, single row")
     (tags "Through hole pin header THT 1x03 1.27mm single row")
-    (fp_text reference J24 (at 0 -1.695) (layer F.SilkS)
+    (fp_text reference J38 (at 0 -1.695) (layer F.SilkS)
       (effects (font (size 1 1) (thickness 0.15)))
     )
@@
     (descr "Through hole straight pin header, 1x02, 1.27mm pitch, single row")
     (tags "Through hole pin header THT 1x02 1.27mm single row")
-    (fp_text reference J23 (at 0 -1.695) (layer F.SilkS)
-      (effects (font (size 1 1) (thickness 0.15)))
-    )
+    (fp_text reference J37 (at 0 -1.695) (layer F.SilkS)
+      (effects (font (size 1 1) (thickness 0.15)))
+    )
