File: hardware/nodemcu.kicad_pcb (KiCad board)
At the start: 2 copper layers, 7 parts, among them J15 I2C_DEBUG, J16 TTL_HEADER, J17 SDCARD_HEADER, J18 SPI_HEADER, J19 NODEMCU_HEADER1, J20 NODEMCU_HEADER2, U7 nodemcu

Commit message: update,
Parts:
- moved J19 46.3 mm to (70.0, 70.0), turned to 180 degrees
- moved J20 18.7 mm to (70.0, 30.9)
- moved J16 12.9 mm to (75.0, 47.1)
- moved J18 12.7 mm to (75.0, 41.3)
- moved J15 5.10 mm to (75.0, 30.0)
Changed lines of the file:
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@@
   )
   (module footprint-lib:TTL_TERMINAL_1.27mm (layer F.Cu)
-    (at 70 59 180)
+    (at 75 47.1 180)
     (descr "TTL DEBUG TERMINAL")
     (tags "TTL DEBUG")
@@
   )
   (module Connector_PinHeader_1.27mm:PinHeader_1x15_P1.27mm_Vertical (layer F.Cu)
-    (at 59 46)
+    (at 70 30.9)
     (descr "Through hole straight pin header, 1x15, 1.27mm pitch, single row")
     (tags "Through hole pin header THT 1x15 1.27mm single row")
@@
   )
   (module Connector_PinHeader_1.27mm:PinHeader_1x15_P1.27mm_Vertical (layer F.Cu)
-    (at 45 31)
+    (at 70 70 180)
     (descr "Through hole straight pin header, 1x15, 1.27mm pitch, single row")
     (tags "Through hole pin header THT 1x15 1.27mm single row")
@@
     (fp_line (start 1.05 -0.635) (end 1.05 18.415) (layer F.Fab) (width 0.1))
     (fp_line (start -0.525 -0.635) (end 1.05 -0.635) (layer F.Fab) (width 0.1))
-    (pad 15 thru_hole oval (at 0 17.78) (size 1 1) (drill 0.65) (layers *.Cu *.Mask)
+    (pad 15 thru_hole oval (at 0 17.78 180) (size 1 1) (drill 0.65) (layers *.Cu *.Mask)
       (net 7 /VIN))
-    (pad 14 thru_hole oval (at 0 16.51) (size 1 1) (drill 0.65) (layers *.Cu *.Mask)
-      (net 8 GND))
-    (pad 13 thru_hole oval (at 0 15.24) (size 1 1) (drill 0.65) (layers *.Cu *.Mask)
+    (pad 14 thru_hole oval (at 0 16.51 180) (size 1 1) (drill 0.65) (layers *.Cu *.Mask)
+      (net 8 GND))
+    (pad 13 thru_hole oval (at 0 15.24 180) (size 1 1) (drill 0.65) (layers *.Cu *.Mask)
       (net 9 /RST))
-    (pad 12 thru_hole oval (at 0 13.97) (size 1 1) (drill 0.65) (layers *.Cu *.Mask)
+    (pad 12 thru_hole oval (at 0 13.97 180) (size 1 1) (drill 0.65) (layers *.Cu *.Mask)
       (net 10 /EN))
-    (pad 11 thru_hole oval (at 0 12.7) (size 1 1) (drill 0.65) (layers *.Cu *.Mask)
-      (net 11 +3V3))
-    (pad 10 thru_hole oval (at 0 11.43) (size 1 1) (drill 0.65) (layers *.Cu *.Mask)
-      (net 8 GND))
-    (pad 9 thru_hole oval (at 0 10.16) (size 1 1) (drill 0.65) (layers *.Cu *.Mask)
+    (pad 11 thru_hole oval (at 0 12.7 180) (size 1 1) (drill 0.65) (layers *.Cu *.Mask)
+      (net 11 +3V3))
+    (pad 10 thru_hole oval (at 0 11.43 180) (size 1 1) (drill 0.65) (layers *.Cu *.Mask)
+      (net 8 GND))
+    (pad 9 thru_hole oval (at 0 10.16 180) (size 1 1) (drill 0.65) (layers *.Cu *.Mask)
       (net 12 /SDDCLK))
-    (pad 8 thru_hole oval (at 0 8.89) (size 1 1) (drill 0.65) (layers *.Cu *.Mask)
+    (pad 8 thru_hole oval (at 0 8.89 180) (size 1 1) (drill 0.65) (layers *.Cu *.Mask)
       (net 13 /SDD0))
-    (pad 7 thru_hole oval (at 0 7.62) (size 1 1) (drill 0.65) (layers *.Cu *.Mask)
+    (pad 7 thru_hole oval (at 0 7.62 180) (size 1 1) (drill 0.65) (layers *.Cu *.Mask)
       (net 14 /SDDCMD))
-    (pad 6 thru_hole oval (at 0 6.35) (size 1 1) (drill 0.65) (layers *.Cu *.Mask)
+    (pad 6 thru_hole oval (at 0 6.35 180) (size 1 1) (drill 0.65) (layers *.Cu *.Mask)
       (net 15 /SDD1))
-    (pad 5 thru_hole oval (at 0 5.08) (size 1 1) (drill 0.65) (layers *.Cu *.Mask)
+    (pad 5 thru_hole oval (at 0 5.08 180) (size 1 1) (drill 0.65) (layers *.Cu *.Mask)
       (net 16 /SDD2))
-    (pad 4 thru_hole oval (at 0 3.81) (size 1 1) (drill 0.65) (layers *.Cu *.Mask)
+    (pad 4 thru_hole oval (at 0 3.81 180) (size 1 1) (drill 0.65) (layers *.Cu *.Mask)
       (net 17 /SDD3))
-    (pad 3 thru_hole oval (at 0 2.54) (size 1 1) (drill 0.65) (layers *.Cu *.Mask)
+    (pad 3 thru_hole oval (at 0 2.54 180) (size 1 1) (drill 0.65) (layers *.Cu *.Mask)
       (net 18 /RSV_3))
-    (pad 2 thru_hole oval (at 0 1.27) (size 1 1) (drill 0.65) (layers *.Cu *.Mask)
+    (pad 2 thru_hole oval (at 0 1.27 180) (size 1 1) (drill 0.65) (layers *.Cu *.Mask)
       (net 19 /RSV_2))
-    (pad 1 thru_hole rect (at 0 0) (size 1 1) (drill 0.65) (layers *.Cu *.Mask)
+    (pad 1 thru_hole rect (at 0 0 180) (size 1 1) (drill 0.65) (layers *.Cu *.Mask)
       (net 20 /A0))
     (model ${KISYS3DMOD}/Connector_PinHeader_1.27mm.3dshapes/PinHeader_1x15_P1.27mm_Vertical.wrl
@@
   )
   (module footprint-lib:SPI_DEBUG (layer F.Cu)
-    (at 70 53 180)
+    (at 75 41.3 180)
     (descr "Through hole straight pin header, 1x04, 1.27mm pitch, single row")
     (tags "SPI DEBUG")
@@
   )
   (module footprint-lib:I2C_DEBUG (layer F.Cu)
-    (at 70 31)
+    (at 75 30)
     (descr "Through hole straight pin header, 1x02, 1.27mm pitch, single row")
     (tags "Through hole pin header THT 1x02 1.27mm single row")

Commit message: update footprint,
Parts:
- added J29: OLED_HEADER, Connector_PinHeader_1.27mm:PinHeader_1x05_P1.27mm_Vertical, F.Cu at (79.1, 29.6)
- moved J30 6.07 mm to (76.1, 70.1)
- renumbered J15 to J25, J16 to J26, J17 to J27, J18 to J28, J19 to J30, J20 to J31, U7 to U10
Connections:
- net /D2 renamed /OLED_DC
- net /D3 renamed /OLED_RST
- net /D4 renamed /OLED_SS
Changed lines of the file:
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@@
     (tracks 0)
     (zones 0)
-    (modules 7)
+    (modules 8)
     (nets 26)
   )
@@
   (net 21 /TX)
   (net 22 /RX)
-  (net 23 /D4)
-  (net 24 /D3)
-  (net 25 /D2)
+  (net 23 /OLED_SS)
+  (net 24 /OLED_RST)
+  (net 25 /OLED_DC)
   (net_class Default "This is the default net class."
     (clearance 0.2)
@@
     (add_net +3V3)
     (add_net /A0)
-    (add_net /D2)
-    (add_net /D3)
-    (add_net /D4)
     (add_net /EN)
     (add_net /HCS)
@@
     (add_net /HMOSI)
     (add_net /HSCLK)
+    (add_net /OLED_DC)
+    (add_net /OLED_RST)
+    (add_net /OLED_SS)
     (add_net /RST)
     (add_net /RSV_2)
@@
     (add_net GND)
   )
+  (module Connector_PinHeader_1.27mm:PinHeader_1x05_P1.27mm_Vertical (layer F.Cu)
+    (at 79.0575 29.591)
+    (descr "Through hole straight pin header, 1x05, 1.27mm pitch, single row")
+    (tags "Through hole pin header THT 1x05 1.27mm single row")
+    (fp_text reference J29 (at 0 -1.695) (layer F.SilkS)
+      (effects (font (size 1 1) (thickness 0.15)))
+    )
+    (fp_text value OLED_HEADER (at 0 6.775) (layer F.Fab)
+      (effects (font (size 1 1) (thickness 0.15)))
+    )
+    (fp_text user %R (at 0 2.54 90) (layer F.Fab)
+      (effects (font (size 1 1) (thickness 0.15)))
+    )
+    (fp_line (start 1.55 -1.15) (end -1.55 -1.15) (layer F.CrtYd) (width 0.05))
+    (fp_line (start 1.55 6.25) (end 1.55 -1.15) (layer F.CrtYd) (width 0.05))
+    (fp_line (start -1.55 6.25) (end 1.55 6.25) (layer F.CrtYd) (width 0.05))
+    (fp_line (start -1.55 -1.15) (end -1.55 6.25) (layer F.CrtYd) (width 0.05))
+    (fp_line (start -1.11 -0.76) (end 0 -0.76) (layer F.SilkS) (width 0.12))
+    (fp_line (start -1.11 0) (end -1.11 -0.76) (layer F.SilkS) (width 0.12))
+    (fp_line (start 0.563471 0.76) (end 1.11 0.76) (layer F.SilkS) (width 0.12))
+    (fp_line (start -1.11 0.76) (end -0.563471 0.76) (layer F.SilkS) (width 0.12))
+    (fp_line (start 1.11 0.76) (end 1.11 5.775) (layer F.SilkS) (width 0.12))
+    (fp_line (start -1.11 0.76) (end -1.11 5.775) (layer F.SilkS) (width 0.12))
+    (fp_line (start 0.30753 5.775) (end 1.11 5.775) (layer F.SilkS) (width 0.12))
+    (fp_line (start -1.11 5.775) (end -0.30753 5.775) (layer F.SilkS) (width 0.12))
+    (fp_line (start -1.05 -0.11) (end -0.525 -0.635) (layer F.Fab) (width 0.1))
+    (fp_line (start -1.05 5.715) (end -1.05 -0.11) (layer F.Fab) (width 0.1))
+    (fp_line (start 1.05 5.715) (end -1.05 5.715) (layer F.Fab) (width 0.1))
+    (fp_line (start 1.05 -0.635) (end 1.05 5.715) (layer F.Fab) (width 0.1))
+    (fp_line (start -0.525 -0.635) (end 1.05 -0.635) (layer F.Fab) (width 0.1))
+    (pad 5 thru_hole oval (at 0 5.08) (size 1 1) (drill 0.65) (layers *.Cu *.Mask)
+      (net 23 /OLED_SS))
+    (pad 4 thru_hole oval (at 0 3.81) (size 1 1) (drill 0.65) (layers *.Cu *.Mask)
+      (net 24 /OLED_RST))
+    (pad 3 thru_hole oval (at 0 2.54) (size 1 1) (drill 0.65) (layers *.Cu *.Mask)
+      (net 25 /OLED_DC))
+    (pad 2 thru_hole oval (at 0 1.27) (size 1 1) (drill 0.65) (layers *.Cu *.Mask)
+      (net 6 /HSCLK))
+    (pad 1 thru_hole rect (at 0 0) (size 1 1) (drill 0.65) (layers *.Cu *.Mask)
+      (net 5 /HMOSI))
+    (model ${KISYS3DMOD}/Connector_PinHeader_1.27mm.3dshapes/PinHeader_1x05_P1.27mm_Vertical.wrl
+      (at (xyz 0 0 0))
+      (scale (xyz 1 1 1))
+      (rotate (xyz 0 0 0))
+    )
+  )
   (module footprint-lib:SDCARD_HEADER (layer F.Cu)
     (at 34 45 180)
     (descr "Through hole straight pin header, 1x06, 1.27mm pitch, single row")
     (tags "SDCARD HEADER")
-    (fp_text reference J17 (at 0 -1.695) (layer F.SilkS)
+    (fp_text reference J27 (at 0 -1.695) (layer F.SilkS)
       (effects (font (size 1 1) (thickness 0.15)))
     )
@@
     (descr "TTL DEBUG TERMINAL")
     (tags "TTL DEBUG")
-    (fp_text reference J16 (at 0 -1.695) (layer F.SilkS)
+    (fp_text reference J26 (at 0 -1.695) (layer F.SilkS)
       (effects (font (size 1 1) (thickness 0.15)))
     )
@@
   (module "footprint-lib:NodeMCU1.0(12-E)" (layer F.Cu)
     (at 51.81 47.88)
-    (fp_text reference U7 (at 0 0) (layer F.SilkS)
+    (fp_text reference U10 (at 0 0) (layer F.SilkS)
       (effects (font (size 1 1) (thickness 0.15)))
     )
@@
       (net 11 +3V3))
     (pad 26 thru_hole circle (at 13.97 -7.62) (size 1.524 1.524) (drill 0.762) (layers *.Cu *.Mask F.SilkS)
-      (net 23 /D4))
+      (net 23 /OLED_SS))
     (pad 27 thru_hole circle (at 13.97 -10.16) (size 1.524 1.524) (drill 0.762) (layers *.Cu *.Mask F.SilkS)
-      (net 24 /D3))
+      (net 24 /OLED_RST))
     (pad 28 thru_hole circle (at 13.97 -12.7) (size 1.524 1.524) (drill 0.762) (layers *.Cu *.Mask F.SilkS)
-      (net 25 /D2))
+      (net 25 /OLED_DC))
     (pad 29 thru_hole circle (at 13.97 -15.24) (size 1.524 1.524) (drill 0.762) (layers *.Cu *.Mask F.SilkS)
       (net 2 /SCL))
@@
     (descr "Through hole straight pin header, 1x15, 1.27mm pitch, single row")
     (tags "Through hole pin header THT 1x15 1.27mm single row")
-    (fp_text reference J20 (at 0 -1.695) (layer F.SilkS)
+    (fp_text reference J31 (at 0 -1.695) (layer F.SilkS)
       (effects (font (size 1 1) (thickness 0.15)))
     )
@@
       (net 11 +3V3))
     (pad 5 thru_hole oval (at 0 5.08) (size 1 1) (drill 0.65) (layers *.Cu *.Mask)
-      (net 23 /D4))
+      (net 23 /OLED_SS))
     (pad 4 thru_hole oval (at 0 3.81) (size 1 1) (drill 0.65) (layers *.Cu *.Mask)
-      (net 24 /D3))
+      (net 24 /OLED_RST))
     (pad 3 thru_hole oval (at 0 2.54) (size 1 1) (drill 0.65) (layers *.Cu *.Mask)
-      (net 25 /D2))
+      (net 25 /OLED_DC))
     (pad 2 thru_hole oval (at 0 1.27) (size 1 1) (drill 0.65) (layers *.Cu *.Mask)
       (net 2 /SCL))
@@
   )
   (module Connector_PinHeader_1.27mm:PinHeader_1x15_P1.27mm_Vertical (layer F.Cu)
-    (at 70 70 180)
+    (at 76.073 70.104 180)
     (descr "Through hole straight pin header, 1x15, 1.27mm pitch, single row")
     (tags "Through hole pin header THT 1x15 1.27mm single row")
-    (fp_text reference J19 (at 0 -1.695) (layer F.SilkS)
+    (fp_text reference J30 (at 0 -1.695) (layer F.SilkS)
       (effects (font (size 1 1) (thickness 0.15)))
     )
@@
     (descr "Through hole straight pin header, 1x04, 1.27mm pitch, single row")
     (tags "SPI DEBUG")
-    (fp_text reference J18 (at 0 -1.695) (layer F.SilkS)
+    (fp_text reference J28 (at 0 -1.695) (layer F.SilkS)
       (effects (font (size 1 1) (thickness 0.15)))
     )
@@
     (descr "Through hole straight pin header, 1x02, 1.27mm pitch, single row")
     (tags "Through hole pin header THT 1x02 1.27mm single row")
-    (fp_text reference J15 (at 0 -1.695) (layer F.SilkS)
-      (effects (font (size 1 1) (thickness 0.15)))
-    )
+    (fp_text reference J25 (at 0 -1.695) (layer F.SilkS)
+      (effects (font (size 1 1) (thickness 0.15)))
+    )
