File: hardware/LM75_i2c.sch (KiCad schematic (older format))
At the start: 5 parts, among them J1 A0_SEL, U2 LM75

Commit message: update,
Parts:
- added C?: C106,0603, Capacitor_SMD:C_0603_1608Metric_Pad1.05x0.95mm_HandSolder, symbol taobao-c:C106,0603
- added J?: OLED_I2C_HEADER, symbol Connector:Conn_01x04_Female
Connections:
- wire segments 44 -> 52
Changed lines of the file:
@@
 	850  750  1350 750
 NoConn ~ 3700 2200
+$Comp
+L power:+3V3 #PWR?
+U 1 1 5CF1B420
+P 2350 2050
+F 0 "#PWR?" H 2350 1900 50  0001 C CNN
+F 1 "+3V3" H 2400 2250 50  0000 C CNN
+F 2 "" H 2350 2050 50  0001 C CNN
+F 3 "" H 2350 2050 50  0001 C CNN
+	1    2350 2050
+	1    0    0    -1
+$EndComp
+Wire Wire Line
+	2800 2350 2800 2600
+Wire Wire Line
+	2050 2350 2800 2350
+Wire Wire Line
+	2650 2550 2050 2550
+Wire Wire Line
+	2650 2450 2050 2450
+Text Label 2650 2550 2    50   ~ 0
+LM75_SDA
+Text Label 2650 2450 2    50   ~ 0
+LM75_SCL
+$Comp
+L power:GND #PWR?
+U 1 1 5CF1B42C
+P 2800 2600
+F 0 "#PWR?" H 2800 2350 50  0001 C CNN
+F 1 "GND" H 2850 2400 50  0000 C CNN
+F 2 "" H 2800 2600 50  0001 C CNN
+F 3 "" H 2800 2600 50  0001 C CNN
+	1    2800 2600
+	1    0    0    -1
+$EndComp
+Wire Wire Line
+	2350 2250 2050 2250
+Wire Wire Line
+	2350 2050 2350 2250
+$Comp
+L Connector:Conn_01x04_Female J?
+U 1 1 5CF1B434
+P 1850 2350
+F 0 "J?" H 1700 2650 50  0000 C CNN
+F 1 "OLED_I2C_HEADER" H 1700 2550 50  0000 C CNN
+F 2 "" H 1850 2350 50  0001 C CNN
+F 3 "~" H 1850 2350 50  0001 C CNN
+	1    1850 2350
+	-1   0    0    -1
+$EndComp
+$Comp
+L power:+3V3 #PWR?
+U 1 1 5CF1DEFA
+P 4700 1850
+F 0 "#PWR?" H 4700 1700 50  0001 C CNN
+F 1 "+3V3" H 4750 2050 50  0000 C CNN
+F 2 "" H 4700 1850 50  0001 C CNN
+F 3 "" H 4700 1850 50  0001 C CNN
+	1    4700 1850
+	0    -1   -1   0
+$EndComp
+$Comp
+L power:GND #PWR?
+U 1 1 5CF1E2B6
+P 5050 1850
+F 0 "#PWR?" H 5050 1600 50  0001 C CNN
+F 1 "GND" H 5100 1650 50  0000 C CNN
+F 2 "" H 5050 1850 50  0001 C CNN
+F 3 "" H 5050 1850 50  0001 C CNN
+	1    5050 1850
+	0    -1   -1   0
+$EndComp
+$Comp
+L taobao-c:C106,0603 C?
+U 1 1 5CF1EAE0
+P 4850 1850
+F 0 "C?" V 4600 1850 50  0000 C CNN
+F 1 "C106,0603" V 4700 1850 50  0000 C CNN
+F 2 "Capacitor_SMD:C_0603_1608Metric_Pad1.05x0.95mm_HandSolder" H 4850 1850 50  0001 C CNN
+F 3 "~" H 4850 1850 50  0001 C CNN
+	1    4850 1850
+	0    1    1    0
+$EndComp
+Wire Wire Line
+	4700 1850 4750 1850
+Wire Wire Line
+	4950 1850 5050 1850
 $EndSCHEMATC

Commit message: update,
Parts:
- gave numbers to parts that had none: 2
- renumbered J1 to J3
Changed lines of the file:
@@
 $EndBitmap
 $Comp
-L power:+3V3 #PWR021
+L power:+3V3 #PWR025
 U 1 1 5CFA024B
 P 5450 2150
-F 0 "#PWR021" H 5450 2000 50  0001 C CNN
+F 0 "#PWR025" H 5450 2000 50  0001 C CNN
 F 1 "+3V3" H 5500 2350 50  0000 C CNN
 F 2 "" H 5450 2150 50  0001 C CNN
@@
 $EndComp
 $Comp
-L power:GND #PWR022
+L power:GND #PWR027
 U 1 1 5CFA0A82
 P 4350 2850
-F 0 "#PWR022" H 4350 2600 50  0001 C CNN
+F 0 "#PWR027" H 4350 2600 50  0001 C CNN
 F 1 "GND" H 4400 2650 50  0000 C CNN
 F 2 "" H 4350 2850 50  0001 C CNN
@@
 	5450 2300 5300 2300
 $Comp
-L power:GND #PWR023
+L power:GND #PWR028
 U 1 1 5CFA112C
 P 6100 3000
-F 0 "#PWR023" H 6100 2750 50  0001 C CNN
+F 0 "#PWR028" H 6100 2750 50  0001 C CNN
 F 1 "GND" H 6150 2800 50  0000 C CNN
 F 2 "" H 6100 3000 50  0001 C CNN
@@
 $EndComp
 $Comp
-L power:+3V3 #PWR020
+L power:+3V3 #PWR024
 U 1 1 5CFA13EE
 P 6100 2050
-F 0 "#PWR020" H 6100 1900 50  0001 C CNN
+F 0 "#PWR024" H 6100 1900 50  0001 C CNN
 F 1 "+3V3" H 6150 2250 50  0000 C CNN
 F 2 "" H 6100 2050 50  0001 C CNN
@@
 $EndComp
 $Comp
-L Jumper:SolderJumper_3_Open J1
+L Jumper:SolderJumper_3_Open J3
 U 1 1 5CFA2233
 P 6400 2400
-F 0 "J1" V 6350 2500 50  0000 L CNN
+F 0 "J3" V 6350 2500 50  0000 L CNN
 F 1 "A0_SEL" V 6400 2500 50  0000 L CNN
 F 2 "" H 6400 2400 50  0001 C CNN
@@
 	6100 2900 6100 2950
 $Comp
-L power:+3V3 #PWR019
+L power:+3V3 #PWR020
 U 1 1 5CFA5F7E
 P 3750 1650
-F 0 "#PWR019" H 3750 1500 50  0001 C CNN
+F 0 "#PWR020" H 3750 1500 50  0001 C CNN
 F 1 "+3V3" H 3800 1850 50  0000 C CNN
 F 2 "" H 3750 1650 50  0001 C CNN
@@
 U 1 1 5CF1B420
 P 2350 2050
-F 0 "#PWR?" H 2350 1900 50  0001 C CNN
+AR Path="/5CDAB790/5CF1B420" Ref="#PWR?"  Part="1"
+AR Path="/5CDAB838/5CF1B420" Ref="#PWR023"  Part="1"
+F 0 "#PWR023" H 2350 1900 50  0001 C CNN
 F 1 "+3V3" H 2400 2250 50  0000 C CNN
 F 2 "" H 2350 2050 50  0001 C CNN
@@
 U 1 1 5CF1B42C
 P 2800 2600
-F 0 "#PWR?" H 2800 2350 50  0001 C CNN
+AR Path="/5CDAB790/5CF1B42C" Ref="#PWR?"  Part="1"
+AR Path="/5CDAB838/5CF1B42C" Ref="#PWR026"  Part="1"
+F 0 "#PWR026" H 2800 2350 50  0001 C CNN
 F 1 "GND" H 2850 2400 50  0000 C CNN
 F 2 "" H 2800 2600 50  0001 C CNN
@@
 U 1 1 5CF1B434
 P 1850 2350
-F 0 "J?" H 1700 2650 50  0000 C CNN
+AR Path="/5CDAB790/5CF1B434" Ref="J?"  Part="1"
+AR Path="/5CDAB838/5CF1B434" Ref="J2"  Part="1"
+F 0 "J2" H 1700 2650 50  0000 C CNN
 F 1 "OLED_I2C_HEADER" H 1700 2550 50  0000 C CNN
 F 2 "" H 1850 2350 50  0001 C CNN
@@
 $EndComp
 $Comp
-L power:+3V3 #PWR?
+L power:+3V3 #PWR021
 U 1 1 5CF1DEFA
 P 4700 1850
-F 0 "#PWR?" H 4700 1700 50  0001 C CNN
+F 0 "#PWR021" H 4700 1700 50  0001 C CNN
 F 1 "+3V3" H 4750 2050 50  0000 C CNN
 F 2 "" H 4700 1850 50  0001 C CNN
@@
 $EndComp
 $Comp
-L power:GND #PWR?
+L power:GND #PWR022
 U 1 1 5CF1E2B6
 P 5050 1850
-F 0 "#PWR?" H 5050 1600 50  0001 C CNN
+F 0 "#PWR022" H 5050 1600 50  0001 C CNN
 F 1 "GND" H 5100 1650 50  0000 C CNN
 F 2 "" H 5050 1850 50  0001 C CNN
@@
 $EndComp
 $Comp
-L taobao-c:C106,0603 C?
+L taobao-c:C106,0603 C6
 U 1 1 5CF1EAE0
 P 4850 1850
-F 0 "C?" V 4600 1850 50  0000 C CNN
+F 0 "C6" V 4600 1850 50  0000 C CNN
 F 1 "C106,0603" V 4700 1850 50  0000 C CNN
 F 2 "Capacitor_SMD:C_0603_1608Metric_Pad1.05x0.95mm_HandSolder" H 4850 1850 50  0001 C CNN

Commit message: update footprint,
Parts:
- RN1: footprint (none) -> Resistor_SMD:R_Array_Concave_4x0603
Changed lines of the file:
@@
 F 0 "RN1" H 4100 2050 50  0000 L CNN
 F 1 "R_Pack04" H 4100 2000 50  0000 L CNN
-F 2 "" V 4175 2000 50  0001 C CNN
+F 2 "Resistor_SMD:R_Array_Concave_4x0603" V 4175 2000 50  0001 C CNN
 F 3 "~" H 3900 2000 50  0001 C CNN
 	1    3900 2000

Commit message: update footprint,
Parts:
- J2: footprint (none) -> Connector_PinHeader_1.27mm:PinHeader_1x04_P1.27mm_Vertical
Changed lines of the file:
@@
 F 0 "J2" H 1700 2650 50  0000 C CNN
 F 1 "OLED_I2C_HEADER" H 1700 2550 50  0000 C CNN
-F 2 "" H 1850 2350 50  0001 C CNN
+F 2 "Connector_PinHeader_1.27mm:PinHeader_1x04_P1.27mm_Vertical" H 1850 2350 50  0001 C CNN
 F 3 "~" H 1850 2350 50  0001 C CNN
 	1    1850 2350

Commit message: update footprint,
Parts:
- J3, JP1, JP2: footprint (none) -> Jumper:SolderJumper-2_P1.3mm_Open_TrianglePad1.0x1.5mm
Changed lines of the file:
@@
 F 0 "J3" V 6350 2500 50  0000 L CNN
 F 1 "A0_SEL" V 6400 2500 50  0000 L CNN
-F 2 "" H 6400 2400 50  0001 C CNN
+F 2 "Jumper:SolderJumper-2_P1.3mm_Open_TrianglePad1.0x1.5mm" H 6400 2400 50  0001 C CNN
 F 3 "~" H 6400 2400 50  0001 C CNN
 	1    6400 2400
@@
 F 0 "JP1" V 6050 2600 50  0000 L CNN
 F 1 "A1_SEL" V 6100 2600 50  0000 L CNN
-F 2 "" H 6100 2500 50  0001 C CNN
+F 2 "Jumper:SolderJumper-2_P1.3mm_Open_TrianglePad1.0x1.5mm" H 6100 2500 50  0001 C CNN
 F 3 "~" H 6100 2500 50  0001 C CNN
 	1    6100 2500
@@
 F 0 "JP2" V 5650 2700 50  0000 L CNN
 F 1 "A2_SEL" V 5700 2700 50  0000 L CNN
-F 2 "" H 5700 2600 50  0001 C CNN
+F 2 "Jumper:SolderJumper-2_P1.3mm_Open_TrianglePad1.0x1.5mm" H 5700 2600 50  0001 C CNN
 F 3 "~" H 5700 2600 50  0001 C CNN
 	1    5700 2600

Commit message: update footprint,
Parts:
- J3, JP1, JP2: footprint Jumper:SolderJumper-2_P1.3mm_Open_TrianglePad1.0x1.5mm -> Jumper:SolderJumper-3_P2.0mm_Open_TrianglePad1.0x1.5mm_NumberLabels
Changed lines of the file:
@@
 F 0 "J3" V 6350 2500 50  0000 L CNN
 F 1 "A0_SEL" V 6400 2500 50  0000 L CNN
-F 2 "Jumper:SolderJumper-2_P1.3mm_Open_TrianglePad1.0x1.5mm" H 6400 2400 50  0001 C CNN
+F 2 "Jumper:SolderJumper-3_P2.0mm_Open_TrianglePad1.0x1.5mm_NumberLabels" H 6400 2400 50  0001 C CNN
 F 3 "~" H 6400 2400 50  0001 C CNN
 	1    6400 2400
@@
 F 0 "JP1" V 6050 2600 50  0000 L CNN
 F 1 "A1_SEL" V 6100 2600 50  0000 L CNN
-F 2 "Jumper:SolderJumper-2_P1.3mm_Open_TrianglePad1.0x1.5mm" H 6100 2500 50  0001 C CNN
+F 2 "Jumper:SolderJumper-3_P2.0mm_Open_TrianglePad1.0x1.5mm_NumberLabels" H 6100 2500 50  0001 C CNN
 F 3 "~" H 6100 2500 50  0001 C CNN
 	1    6100 2500
@@
 F 0 "JP2" V 5650 2700 50  0000 L CNN
 F 1 "A2_SEL" V 5700 2700 50  0000 L CNN
-F 2 "Jumper:SolderJumper-2_P1.3mm_Open_TrianglePad1.0x1.5mm" H 5700 2600 50  0001 C CNN
+F 2 "Jumper:SolderJumper-3_P2.0mm_Open_TrianglePad1.0x1.5mm_NumberLabels" H 5700 2600 50  0001 C CNN
 F 3 "~" H 5700 2600 50  0001 C CNN
 	1    5700 2600
