File: hardware/rotatry_encoder.kicad_pcb (KiCad board)
At the start: 2 copper layers, 7 parts, among them SW3 EC11_VERTICAL

Commit message: update footprint,
Parts:
- removed C16: C104,0603, Capacitor_SMD:C_0603_1608Metric_Pad1.05x0.95mm_HandSolder
- added C26: C104,0603, Capacitor_SMD:C_0603_1608Metric_Pad1.05x0.95mm_HandSolder, F.Cu at (33.0, 39.0)
- added J36: ROT_ENC_HEADER, Connector_PinHeader_1.27mm:PinHeader_1x03_P1.27mm_Vertical, F.Cu at (39.0, 28.0)
- renumbered C14 to C24, C15 to C25, R13 to R16, R14 to R17, R15 to R18
Routing:
- net Net-(R16-Pad1): track 0.00 -> 45.3 mm
- net GND: track 0.00 -> 31.1 mm
- net Net-(R17-Pad1): track 0.00 -> 20.7 mm
- net /SW_OUT: track 0.00 -> 10.6 mm
- net /B: track 0.00 -> 8.67 mm
- net Net-(R18-Pad1): track 0.00 -> 7.96 mm
- net /A: track 0.00 -> 7.18 mm
Changed lines of the file:
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@@
     (thickness 1.6)
     (drawings 0)
-    (tracks 0)
+    (tracks 37)
     (zones 0)
-    (modules 7)
+    (modules 8)
     (nets 8)
   )
@@
   (net 3 /B)
   (net 4 /SW_OUT)
-  (net 5 "Net-(R13-Pad1)")
-  (net 6 "Net-(R14-Pad1)")
-  (net 7 "Net-(R15-Pad1)")
+  (net 5 "Net-(R16-Pad1)")
+  (net 6 "Net-(R17-Pad1)")
+  (net 7 "Net-(R18-Pad1)")
   (net_class Default "This is the default net class."
     (clearance 0.2)
@@
     (add_net /SW_OUT)
     (add_net GND)
-    (add_net "Net-(R13-Pad1)")
-    (add_net "Net-(R14-Pad1)")
-    (add_net "Net-(R15-Pad1)")
+    (add_net "Net-(R16-Pad1)")
+    (add_net "Net-(R17-Pad1)")
+    (add_net "Net-(R18-Pad1)")
+  )
+  (module Connector_PinHeader_1.27mm:PinHeader_1x03_P1.27mm_Vertical (layer F.Cu)
+    (at 39 28)
+    (descr "Through hole straight pin header, 1x03, 1.27mm pitch, single row")
+    (tags "Through hole pin header THT 1x03 1.27mm single row")
+    (fp_text reference J36 (at 0 -1.695) (layer F.SilkS)
+      (effects (font (size 1 1) (thickness 0.15)))
+    )
+    (fp_text value ROT_ENC_HEADER (at 0 4.235) (layer F.Fab)
+      (effects (font (size 1 1) (thickness 0.15)))
+    )
+    (fp_text user %R (at 0 1.27 90) (layer F.Fab)
+      (effects (font (size 1 1) (thickness 0.15)))
+    )
+    (fp_line (start 1.55 -1.15) (end -1.55 -1.15) (layer F.CrtYd) (width 0.05))
+    (fp_line (start 1.55 3.7) (end 1.55 -1.15) (layer F.CrtYd) (width 0.05))
+    (fp_line (start -1.55 3.7) (end 1.55 3.7) (layer F.CrtYd) (width 0.05))
+    (fp_line (start -1.55 -1.15) (end -1.55 3.7) (layer F.CrtYd) (width 0.05))
+    (fp_line (start -1.11 -0.76) (end 0 -0.76) (layer F.SilkS) (width 0.12))
+    (fp_line (start -1.11 0) (end -1.11 -0.76) (layer F.SilkS) (width 0.12))
+    (fp_line (start 0.563471 0.76) (end 1.11 0.76) (layer F.SilkS) (width 0.12))
+    (fp_line (start -1.11 0.76) (end -0.563471 0.76) (layer F.SilkS) (width 0.12))
+    (fp_line (start 1.11 0.76) (end 1.11 3.235) (layer F.SilkS) (width 0.12))
+    (fp_line (start -1.11 0.76) (end -1.11 3.235) (layer F.SilkS) (width 0.12))
+    (fp_line (start 0.30753 3.235) (end 1.11 3.235) (layer F.SilkS) (width 0.12))
+    (fp_line (start -1.11 3.235) (end -0.30753 3.235) (layer F.SilkS) (width 0.12))
+    (fp_line (start -1.05 -0.11) (end -0.525 -0.635) (layer F.Fab) (width 0.1))
+    (fp_line (start -1.05 3.175) (end -1.05 -0.11) (layer F.Fab) (width 0.1))
+    (fp_line (start 1.05 3.175) (end -1.05 3.175) (layer F.Fab) (width 0.1))
+    (fp_line (start 1.05 -0.635) (end 1.05 3.175) (layer F.Fab) (width 0.1))
+    (fp_line (start -0.525 -0.635) (end 1.05 -0.635) (layer F.Fab) (width 0.1))
+    (pad 3 thru_hole oval (at 0 2.54) (size 1 1) (drill 0.65) (layers *.Cu *.Mask)
+      (net 4 /SW_OUT))
+    (pad 2 thru_hole oval (at 0 1.27) (size 1 1) (drill 0.65) (layers *.Cu *.Mask)
+      (net 3 /B))
+    (pad 1 thru_hole rect (at 0 0) (size 1 1) (drill 0.65) (layers *.Cu *.Mask)
+      (net 2 /A))
+    (model ${KISYS3DMOD}/Connector_PinHeader_1.27mm.3dshapes/PinHeader_1x03_P1.27mm_Vertical.wrl
+      (at (xyz 0 0 0))
+      (scale (xyz 1 1 1))
+      (rotate (xyz 0 0 0))
+    )
   )
   (module footprint-lib:RotaryEncoder_Alps_EC11E_Vertical_H20mm (layer F.Cu)
@@
     )
     (pad A thru_hole rect (at 0 0) (size 2 2) (drill 1.2) (layers *.Cu *.Mask)
-      (net 6 "Net-(R14-Pad1)"))
+      (net 6 "Net-(R17-Pad1)"))
     (pad C thru_hole circle (at 0 2.5) (size 2 2) (drill 1.2) (layers *.Cu *.Mask)
       (net 1 GND))
     (pad B thru_hole circle (at 0 5) (size 2 2) (drill 1.2) (layers *.Cu *.Mask)
-      (net 5 "Net-(R13-Pad1)"))
+      (net 5 "Net-(R16-Pad1)"))
     (pad MP thru_hole rect (at 7.5 -3.1) (size 3.5 2.5) (drill oval 2.8 1.5) (layers *.Cu *.Mask))
     (pad MP thru_hole rect (at 7.5 8.1) (size 3.5 2.5) (drill oval 2.8 1.5) (layers *.Cu *.Mask))
     (pad D thru_hole circle (at 14.5 0) (size 2 2) (drill 1.2) (layers *.Cu *.Mask)
-      (net 7 "Net-(R15-Pad1)"))
+      (net 7 "Net-(R18-Pad1)"))
     (pad E thru_hole circle (at 14.5 5) (size 2 2) (drill 1.2) (layers *.Cu *.Mask)
       (net 1 GND))
@@
     (tags "resistor handsolder")
     (attr smd)
-    (fp_text reference R15 (at 0 -1.43) (layer F.SilkS)
+    (fp_text reference R18 (at 0 -1.43) (layer F.SilkS)
       (effects (font (size 1 1) (thickness 0.15)))
     )
@@
       (net 4 /SW_OUT))
     (pad 1 smd roundrect (at -0.875 0) (size 1.05 0.95) (layers F.Cu F.Paste F.Mask) (roundrect_rratio 0.25)
-      (net 7 "Net-(R15-Pad1)"))
+      (net 7 "Net-(R18-Pad1)"))
     (model ${KISYS3DMOD}/Resistor_SMD.3dshapes/R_0603_1608Metric.wrl
       (at (xyz 0 0 0))
@@
     (tags "resistor handsolder")
     (attr smd)
-    (fp_text reference R14 (at 0 -1.43) (layer F.SilkS)
+    (fp_text reference R17 (at 0 -1.43) (layer F.SilkS)
       (effects (font (size 1 1) (thickness 0.15)))
     )
@@
       (net 3 /B))
     (pad 1 smd roundrect (at -0.875 0) (size 1.05 0.95) (layers F.Cu F.Paste F.Mask) (roundrect_rratio 0.25)
-      (net 6 "Net-(R14-Pad1)"))
+      (net 6 "Net-(R17-Pad1)"))
     (model ${KISYS3DMOD}/Resistor_SMD.3dshapes/R_0603_1608Metric.wrl
       (at (xyz 0 0 0))
@@
     (tags "resistor handsolder")
     (attr smd)
-    (fp_text reference R13 (at 0 -1.43) (layer F.SilkS)
+    (fp_text reference R16 (at 0 -1.43) (layer F.SilkS)
       (effects (font (size 1 1) (thickness 0.15)))
     )
@@
       (net 2 /A))
     (pad 1 smd roundrect (at -0.875 0) (size 1.05 0.95) (layers F.Cu F.Paste F.Mask) (roundrect_rratio 0.25)
-      (net 5 "Net-(R13-Pad1)"))
+      (net 5 "Net-(R16-Pad1)"))
     (model ${KISYS3DMOD}/Resistor_SMD.3dshapes/R_0603_1608Metric.wrl
       (at (xyz 0 0 0))
@@
     (tags "capacitor handsolder")
     (attr smd)
-    (fp_text reference C16 (at 0 -1.43) (layer F.SilkS)
+    (fp_text reference C26 (at 0 -1.43) (layer F.SilkS)
       (effects (font (size 1 1) (thickness 0.15)))
     )
@@
     (tags "capacitor handsolder")
     (attr smd)
-    (fp_text reference C15 (at 0 -1.43) (layer F.SilkS)
+    (fp_text reference C25 (at 0 -1.43) (layer F.SilkS)
       (effects (font (size 1 1) (thickness 0.15)))
     )
@@
   )
   (module Capacitor_SMD:C_0603_1608Metric_Pad1.05x0.95mm_HandSolder (layer F.Cu)
-    (at 32.874999 30 180)
+    (at 32.875 30 180)
     (descr "Capacitor SMD 0603 (1608 Metric), square (rectangular) end terminal, IPC_7351 nominal with elongated pad for handsoldering. (Body size source: http://www.tortai-tech.com/upload/download/2011102023233369053.pdf), generated with kicad-footprint-generator")
     (tags "capacitor handsolder")
     (attr smd)
-    (fp_text reference C14 (at 0 -1.43) (layer F.SilkS)
+    (fp_text reference C24 (at 0 -1.43) (layer F.SilkS)
       (effects (font (size 1 1) (thickness 0.15)))
     )
@@
     )
   )
+  (segment (start 31.7901 38.6651) (end 28.745 35.62) (width 0.25) (layer F.Cu) (net 1))
+  (segment (start 28.745 35.62) (end 28.3 35.62) (width 0.25) (layer F.Cu) (net 1))
+  (segment (start 32.125 39) (end 31.7901 38.6651) (width 0.25) (layer F.Cu) (net 1))
+  (segment (start 32.125 35) (end 33 35.875) (width 0.25) (layer F.Cu) (net 1))
+  (segment (start 33 35.875) (end 33 37.4552) (width 0.25) (layer F.Cu) (net 1))
+  (segment (start 33 37.4552) (end 31.7901 38.6651) (width 0.25) (layer F.Cu) (net 1))
+  (segment (start 32 30) (end 33 31) (width 0.25) (layer F.Cu) (net 1))
+  (segment (start 33 31) (end 33 34.125) (width 0.25) (layer F.Cu) (net 1))
+  (segment (start 33 34.125) (end 32.125 35) (width 0.25) (layer F.Cu) (net 1))
+  (segment (start 28.3 35.62) (end 16.3 35.62) (width 0.25) (layer B.Cu) (net 1))
+  (segment (start 16.3 35.62) (end 13.8 33.12) (width 0.25) (layer B.Cu) (net 1))
+  (segment (start 33.875 28) (end 38.1747 28) (width 0.25) (layer F.Cu) (net 2))
+  (segment (start 39 28) (end 38.1747 28) (width 0.25) (layer F.Cu) (net 2))
+  (segment (start 33.75 30) (end 33.875 29.875) (width 0.25) (layer F.Cu) (net 2))
+  (segment (start 33.875 29.875) (end 33.875 28) (width 0.25) (layer F.Cu) (net 2))
+  (segment (start 33.875 33) (end 34.4447 33) (width 0.25) (layer F.Cu) (net 3))
+  (segment (start 34.4447 33) (end 38.1747 29.27) (width 0.25) (layer F.Cu) (net 3))
+  (segment (start 39 29.27) (end 38.1747 29.27) (width 0.25) (layer F.Cu) (net 3))
+  (segment (start 33.875 35) (end 33.875 33) (width 0.25) (layer F.Cu) (net 3))
+  (segment (start 33.875 37) (end 39 31.875) (width 0.25) (layer F.Cu) (net 4))
+  (segment (start 39 31.875) (end 39 30.54) (width 0.25) (layer F.Cu) (net 4))
+  (segment (start 33.875 39) (end 33.875 37) (width 0.25) (layer F.Cu) (net 4))
+  (segment (start 32.125 28) (end 32.9504 27.1746) (width 0.25) (layer F.Cu) (net 5))
+  (segment (start 32.9504 27.1746) (end 39.7102 27.1746) (width 0.25) (layer F.Cu) (net 5))
+  (segment (start 39.7102 27.1746) (end 39.8744 27.3388) (width 0.25) (layer F.Cu) (net 5))
+  (segment (start 39.8744 27.3388) (end 39.8744 34.3922) (width 0.25) (layer F.Cu) (net 5))
+  (segment (start 39.8744 34.3922) (end 34.4218 39.8448) (width 0.25) (layer F.Cu) (net 5))
+  (segment (start 34.4218 39.8448) (end 29.6748 39.8448) (width 0.25) (layer F.Cu) (net 5))
+  (segment (start 29.6748 39.8448) (end 25.45 35.62) (width 0.25) (layer F.Cu) (net 5))
+  (segment (start 25.45 35.62) (end 13.8 35.62) (width 0.25) (layer F.Cu) (net 5))
+  (segment (start 13.8 30.62) (end 15.1253 30.62) (width 0.25) (layer F.Cu) (net 6))
+  (segment (start 32.125 33) (end 32.125 32.528) (width 0.25) (layer F.Cu) (net 6))
+  (segment (start 32.125 32.528) (end 28.8917 29.2947) (width 0.25) (layer F.Cu) (net 6))
+  (segment (start 28.8917 29.2947) (end 16.4506 29.2947) (width 0.25) (layer F.Cu) (net 6))
+  (segment (start 16.4506 29.2947) (end 15.1253 30.62) (width 0.25) (layer F.Cu) (net 6))
+  (segment (start 32.125 37) (end 28.3 33.175) (width 0.25) (layer F.Cu) (net 7))
+  (segment (start 28.3 33.175) (end 28.3 30.62) (width 0.25) (layer F.Cu) (net 7))
 )
