File: hardware/eval_board.kicad_pcb (KiCad board)
At the start: 2 copper layers, 86 parts, among them J1 SSD1306-OLED-SPI, J11 Conn_01x12, J12 Conn_01x14, J13 Conn_01x12, J14 STM32_USB_DEBUG, J15 STM32_GTR, J16 SPI_DEBUG, J17 SWD, SW1 SW_Push, SW2 RST, U1 ESP12, U3 CH340H_T, U4 STM32F103C8T6, U5 AMS1117-3.3, U6 STM32F407VET6, Y1 O_12M/OPTIONAL, Y2 O_12M,3225, Y3 O_8M

Commit message: update,
Parts:
- moved U5 43.0 mm to (151.5, 94.3)
- moved BOOT1 43.0 mm to (141.8, 100.5)
- moved J11 43.0 mm to (144.5, 80.5)
- moved C15 43.0 mm to (140.5, 107.0)
- moved C18 43.0 mm to (156.6, 99.7)
- moved C22 43.0 mm to (209.0, 100.8)
- moved C25 43.0 mm to (213.5, 93.7)
- moved C28 43.0 mm to (213.4, 99.8)
- moved C7 43.0 mm to (144.8, 107.0)
- moved D1 43.0 mm to (240.9, 96.2)
- moved JP3 43.0 mm to (213.5, 96.7)
- moved R14 43.0 mm to (217.7, 101.2)
- moved R15 43.0 mm to (217.9, 93.7)
- moved BOOT2 43.0 mm to (161.4, 85.8)
- moved C1 43.0 mm to (243.2, 88.0)
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Other:
- board outline added: 100 x 100 mm

Commit message: update,
Parts:
- moved D2 175.1 mm to (111.1, 30.5)
- moved D3 175.1 mm to (111.1, 27.9)
- moved C1 175.1 mm to (68.2, 93.0)
- moved C2 175.1 mm to (72.5, 92.5)
- moved C3 175.1 mm to (74.5, 90.0)
- moved C4 175.1 mm to (76.9, 92.5)
- moved C5 175.1 mm to (63.9, 93.0)
- moved J1 175.1 mm to (60.9, 58.5)
- moved R1 175.1 mm to (70.1, 90.0)
- moved R2 175.1 mm to (115.4, 30.4)
- moved R3 175.1 mm to (115.4, 27.8)
- moved TP1 175.1 mm to (113.2, 59.2)
- moved TP2 175.1 mm to (107.1, 59.2)
- moved TP3 175.1 mm to (101.1, 59.2)
- moved U1 175.1 mm to (75.7, 40.1)
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
Commit message: update,
Parts:
- removed the R9 at (53.0, 94.1)
- removed USTM32F1_1: bluepill-stm32f103c8t6, Package_DIP:DIP-40_W15.24mm_LongPads
- removed the Y1 at (65.8, 83.0)
- added BZ1: BUZZER,MLT-8530, footprint-lib:MLT-8530, F.Cu at (50.0, 100.0)
- added C10: C106,0603, Capacitor_SMD:C_0603_1608Metric_Pad1.05x0.95mm_HandSolder, F.Cu at (117.5, 99.2)
- added C11: CP22uf,16V, Capacitor_SMD:CP_Elec_4x5.3, F.Cu at (79.3, 41.7)
- added C6: C106,0805, Capacitor_SMD:C_0805_2012Metric_Pad1.15x1.40mm_HandSolder, F.Cu at (80.9, 51.7)
- added C7: C106,0805, Capacitor_SMD:C_0805_2012Metric_Pad1.15x1.40mm_HandSolder, F.Cu at (75.1, 56.3)
- added C8: C106,0805, Capacitor_SMD:C_0805_2012Metric_Pad1.15x1.40mm_HandSolder, F.Cu at (73.5, 77.6)
- added C9: C106,0603, Capacitor_SMD:C_0603_1608Metric_Pad1.05x0.95mm_HandSolder, F.Cu at (113.1, 102.2)
- added D10: D_1N4148_T4, Diode_SMD:D_SOD-123, F.Cu at (58.4, 96.2)
- added D2: WS2812, LED_SMD:LED_WS2812_PLCC6_5.0x5.0mm_P1.6mm, F.Cu at (68.5, 60.1)
- added D3: WS2812, LED_SMD:LED_WS2812_PLCC6_5.0x5.0mm_P1.6mm, F.Cu at (60.1, 60.1)
- added D4: WS2812, LED_SMD:LED_WS2812_PLCC6_5.0x5.0mm_P1.6mm, F.Cu at (68.5, 53.5)
- added D5: WS2812, LED_SMD:LED_WS2812_PLCC6_5.0x5.0mm_P1.6mm, F.Cu at (60.1, 53.5)
- added J10: LORA_DEBUG1, footprint-lib:LORA_DEBUG1, F.Cu at (81.7, 28.2)
- added J11: LORA_DEBUG2, footprint-lib:LORA_DEBUG2, F.Cu at (77.5, 28.2)
- added J2: SPI_DEBUG, footprint-lib:TTL_TERMINAL_2.54mm, F.Cu at (83.8, 71.5)
- added J22: STM32_2_DEBUG1, Connector_PinHeader_1.00mm:PinHeader_1x20_P1.00mm_Vertical, F.Cu at (66.5, 79.7)
- added J23: STM32_2_DEBUG2, Connector_PinHeader_1.00mm:PinHeader_1x20_P1.00mm_Vertical, F.Cu at (63.1, 79.7)
- added J9: PWM_OUT, Connector_PinSocket_2.54mm:PinSocket_1x02_P2.54mm_Vertical, F.Cu at (98.0, 28.8)
- added Q1: SS9013_J3, footprint-lib:9013,J3,SOT23, F.Cu at (63.3, 96.5)
- added R11: VAR_3V3,0805, footprint-lib:VAR_0805, F.Cu at (62.5, 70.6)
- added R12: R103,0603, Resistor_SMD:R_0603_1608Metric_Pad1.05x0.95mm_HandSolder, F.Cu at (84.1, 86.8)
- added R13: R103,0603, Resistor_SMD:R_0603_1608Metric_Pad1.05x0.95mm_HandSolder, F.Cu at (84.1, 84.2)
- added R14: R472,0603, Resistor_SMD:R_0603_1608Metric_Pad1.05x0.95mm_HandSolder, F.Cu at (108.8, 102.2)
- added R15: R472,0603, Resistor_SMD:R_0603_1608Metric_Pad1.05x0.95mm_HandSolder, F.Cu at (113.2, 99.2)
- added R17: R223,0603, Resistor_SMD:R_0603_1608Metric_Pad1.05x0.95mm_HandSolder, F.Cu at (102.5, 32.4)
- added R2: R151,0603, Resistor_SMD:R_0603_1608Metric_Pad1.05x0.95mm_HandSolder, F.Cu at (79.7, 59.0)
- added R28: R471,0603, Resistor_SMD:R_0603_1608Metric_Pad1.05x0.95mm_HandSolder, F.Cu at (57.7, 99.1)
- added R3: R151,0603, Resistor_SMD:R_0603_1608Metric_Pad1.05x0.95mm_HandSolder, F.Cu at (58.1, 64.7)
- added R4: R151,0603, Resistor_SMD:R_0603_1608Metric_Pad1.05x0.95mm_HandSolder, F.Cu at (66.8, 64.7)
- added R5: R151,0603, Resistor_SMD:R_0603_1608Metric_Pad1.05x0.95mm_HandSolder, F.Cu at (62.4, 64.7)
- added R6: R103,0603, Resistor_SMD:R_0603_1608Metric_Pad1.05x0.95mm_HandSolder, F.Cu at (78.0, 77.4)
- added R7: R471,0603, Resistor_SMD:R_0603_1608Metric_Pad1.05x0.95mm_HandSolder, F.Cu at (97.9, 38.4)
- added R8: VAR_5V6,0805, footprint-lib:VAR_0805, F.Cu at (58.1, 70.6)
- added RN1: R_Pack04, Resistor_SMD:R_Array_Concave_4x0603, F.Cu at (98.1, 52.6)
- added RN2: R_Pack04, Resistor_SMD:R_Array_Concave_4x0603, F.Cu at (94.0, 52.6)
- added SW1: SW_RESET,2_leg,SMD, footprint-lib:SW_SPST_CK_RS282G05A3, F.Cu at (76.5, 90.7)
- added SW2: SW_RESET,2_leg,SMD, footprint-lib:SW_SPST_CK_RS282G05A3, F.Cu at (76.5, 85.6)
- added TH1: Thermistor_NTC,0805, Resistor_SMD:R_0805_2012Metric, F.Cu at (108.8, 99.5)
- added U10: STM32F103C8T6, footprint-lib:STM32F103C8T6, F.Cu at (128.4, 83.9)
- added U2: 74AHCT1G125, Package_TO_SOT_SMD:SOT-23-5_HandSoldering, F.Cu at (75.7, 52.5)
- added U5: 74AHCT1G125, Package_TO_SOT_SMD:SOT-23-5_HandSoldering, F.Cu at (103.2, 28.8)
- added U6: UBLOX-NEO-6M_DEBUG, footprint-lib:UBLOX-NEO-6M_DEBUG, F.Cu at (46.8, 80.5)
- added U7: Ai-Thinker-Ra-02, footprint-lib:Ai-Thinker-Ra-02-LoRa, F.Cu at (65.7, 36.0)
- added U9: arduino_nano_v3, Module:Arduino_Nano, F.Cu at (63.5, 31.1)
- C1, C2: value C225,0603 -> C106,0805; footprint Capacitor_SMD:C_0603_1608Metric_Pad1.05x0.95mm_HandSolder -> Capacitor_SMD:C_0805_2012Metric_Pad1.15x1.40mm_HandSolder
- C3: value C103,0603 -> C106,0805; footprint Capacitor_SMD:C_0603_1608Metric_Pad1.05x0.95mm_HandSolder -> Capacitor_SMD:C_0805_2012Metric_Pad1.15x1.40mm_HandSolder
- C4, C5: value C22pf,0603 -> C106,0805; footprint Capacitor_SMD:C_0603_1608Metric_Pad1.05x0.95mm_HandSolder -> Capacitor_SMD:C_0805_2012Metric_Pad1.15x1.40mm_HandSolder
- D11: renamed from D4; footprint LED_SMD:LED_0805_2012Metric_Pad1.15x1.40mm_HandSolder -> footprint-lib:LED_0603_1608Metric
- D12: renamed from D5; footprint LED_SMD:LED_0805_2012Metric_Pad1.15x1.40mm_HandSolder -> footprint-lib:LED_0603_1608Metric
- D6: value LED_ORANGE -> LED_GREEN,0603; footprint LED_SMD:LED_0805_2012Metric_Pad1.15x1.40mm_HandSolder -> footprint-lib:LED_0603_1608Metric
- D7: renamed from D2; footprint LED_SMD:LED_0603_1608Metric_Pad1.05x0.95mm_HandSolder -> footprint-lib:LED_0603_1608Metric
- D8: renamed from D3; footprint LED_SMD:LED_0603_1608Metric_Pad1.05x0.95mm_HandSolder -> footprint-lib:LED_0603_1608Metric
- D9: renamed from D7; footprint LED_SMD:LED_0603_1608Metric_Pad1.05x0.95mm_HandSolder -> footprint-lib:LED_0603_1608Metric
- L1: value L_Small -> L_2R2,1210; footprint w_smd_inductors:inductor_smd_0603 -> Inductor_SMD:L_1210_3225Metric_Pad1.42x2.65mm_HandSolder
- R1: value R103,0603 -> R151,0603
- U1: value ESP12 -> SSD1306-OLED-I2C; footprint footprint-lib:ESP-12 -> footprint-lib:CONN_I2C_SSD1306
- U3: value CH340H_T -> LM75; footprint Package_SO:SSOP-20_5.3x7.2mm_P0.65mm -> Package_SO:SOP-8_3.76x4.96mm_P1.27mm
- U4: value STM32F103C8T6 -> W25Q32JVSSIQ; footprint Package_QFP:LQFP-48_7x7mm_P0.5mm -> footprint-lib:W25Q32JVSSIQ
- Y2: value O_12M,3225 -> O8M; footprint footprint-lib:OSC_3225 -> w_crystal:hc-49_smd
- moved D6 87.7 mm to (97.7, 41.0)
- moved Y2 50.4 mm to (114.6, 81.3)
- moved U3 50.2 mm to (127.3, 101.2)
- moved C1 44.9 mm to (94.3, 56.5)
- moved C2 39.6 mm to (94.3, 59.4)
- moved C4 36.3 mm to (79.9, 56.3)
- moved C5 35.6 mm to (75.1, 59.3)
- moved R1 30.0 mm to (79.7, 61.6)
- moved C3 27.8 mm to (75.1, 62.2)
- moved U4 19.1 mm to (76.3, 72.6)
- moved U1 18.6 mm to (89.6, 52.5)
- renumbered C19 to C13, C20 to C14, C21 to C15, C22 to C16, C23 to C17, C24 to C18, C25 to C19, C26 to C20, C27 to C21, C28 to C22, C29 to C23, C30 to C24, C31 to C25, C6 to C26, C7 to C27, C8 to C28, C9 to C29, C10 to C30, C11 to C31, C12 to C32, C13 to C33, C14 to C34, C15 to C35, C16 to C36, C17 to C37, C18 to C38, J14 to J15, J15 to J16, J16 to J17, J17 to J18, J11 to J19, J12 to J20, J13 to J21, JP2 to JP4, JP3 to JP5, JP1 to JP6, R3 to R10, R10 to R18, R11 to R19, R12 to R20, R13 to R21, R14 to R22, R15 to R23, R16 to R24, R17 to R25, R18 to R26, R19 to R27, R4 to R29, R5 to R30, R6 to R31, R7 to R32, R8 to R33, R2 to R9, SW2 to SW3, SW1 to SW4, U5 to U11, STM32F1_1 to U13, U6 to U8, Y3 to Y1
Connections:
- C1 pad 1: Net-(C1-Pad1) -> GND
- C1 pad 2: Net-(C1-Pad2) -> +3V3
- C2 pad 1: Net-(C1-Pad1) -> GND
- C2 pad 2: Net-(C1-Pad2) -> +3V3
- C3 pad 1: Net-(C3-Pad1) -> GND
- C3 pad 2: Net-(C1-Pad2) -> Net-(C3-Pad2)
- C4 pad 1: Net-(C4-Pad1) -> GND
- C5 pad 1: Net-(C5-Pad1) -> GND
- C5 pad 2: Net-(C4-Pad2) -> Net-(C5-Pad2)
- D1 pad 1: (no net) -> Net-(D1-Pad1)
- D1 pad 2: (no net) -> Net-(D1-Pad2)
- D1 pad 3: (no net) -> Net-(C3-Pad2)
- D1 pad 5: (no net) -> +5V
- D1 pad 6: (no net) -> GND
- D6 pad 1: Net-(D6-Pad1) -> (no net)
- D6 pad 2: +3V3 -> Net-(D6-Pad2)
- R1 pad 1: (no net) -> +5V
- R1 pad 2: (no net) -> Net-(C3-Pad2)
- U1 pad 1: (no net) -> +3V3
- U1 pad 2: (no net) -> GND
- U1 pad 3: (no net) -> /SCL
- U1 pad 4: (no net) -> /SDA
- U3 pad 1: (no net) -> /SDA
- U3 pad 2: (no net) -> /SCL
- U3 pad 4: (no net) -> GND
- U3 pad 5: Net-(C3-Pad1) -> (no net)
- U3 pad 8: Net-(C1-Pad2) -> +3V3
- U4 pad 1: +3V3 -> /spi.sch/SS
- U4 pad 2: /stm32f103c8t6/PC13 -> (no net)
- U4 pad 3: /stm32f103c8t6/PC14 -> +3V3
- U4 pad 4: /stm32f103c8t6/PC15 -> GND
- U4 pad 5: /stm32f103c8t6/OSCIN -> (no net)
- U4 pad 6: /stm32f103c8t6/OSCOUT -> (no net)
- U4 pad 7: /stm32f103c8t6/RESET -> +3V3
- U4 pad 8: GND -> +3V3
- Y2 pad 1: Net-(C4-Pad1) -> /stm32f103c8t6/OSCOUT
- Y2 pad 2: Net-(C4-Pad2) -> GND

Commit message: update footprint,
Parts:
- removed BOOT1, BOOT2: SolderJumper_3_Open, Jumper:SolderJumper-3_P2.0mm_Open_TrianglePad1.0x1.5mm
- removed BZ1: BUZZER,MLT-8530, footprint-lib:MLT-8530
- removed C1, C2, C3, C4, C5, C6, C7, C8: C106,0805, Capacitor_SMD:C_0805_2012Metric_Pad1.15x1.40mm_HandSolder
- removed C10, C9: C106,0603, Capacitor_SMD:C_0603_1608Metric_Pad1.05x0.95mm_HandSolder
- removed C11: CP22uf,16V, Capacitor_SMD:CP_Elec_4x5.3
- removed C13, C16, C17, C18, C19, C20, C21, C22, C23: C104,0603, Capacitor_SMD:C_0603_1608Metric_Pad1.05x0.95mm_HandSolder
- removed C14, C15: C10pf,0603, Capacitor_SMD:C_0603_1608Metric_Pad1.05x0.95mm_HandSolder
- removed C24, C25: C105,0603, Capacitor_SMD:C_0603_1608Metric_Pad1.05x0.95mm_HandSolder
- removed C26, C31, C32, C33, C34: C104, Capacitor_SMD:C_0603_1608Metric_Pad1.05x0.95mm_HandSolder
- removed C27, C30: C105, Capacitor_SMD:C_0603_1608Metric_Pad1.05x0.95mm_HandSolder
- removed C28, C29: TC106,10V, Capacitor_Tantalum_SMD:CP_EIA-3216-12_Kemet-S_Pad1.58x1.35mm_HandSolder
- removed C35, C36, C37, C38: C20pf, Capacitor_SMD:C_0603_1608Metric_Pad1.05x0.95mm_HandSolder
- removed D1, D2, D3, D4, D5: WS2812, LED_SMD:LED_WS2812_PLCC6_5.0x5.0mm_P1.6mm
- removed D10: D_1N4148_T4, Diode_SMD:D_SOD-123
- removed D11, D12: LED_GREEN, footprint-lib:LED_0603_1608Metric
- removed D6: LED_GREEN,0603, footprint-lib:LED_0603_1608Metric
- removed D7: 5V_STATUS, footprint-lib:LED_0603_1608Metric
- removed D8: 3V3_STATUS, footprint-lib:LED_0603_1608Metric
- removed D9: PB9, footprint-lib:LED_0603_1608Metric
- removed J1: SSD1306-OLED-SPI, footprint-lib:CONN_SPI_SSD1306
- removed J10: LORA_DEBUG1, footprint-lib:LORA_DEBUG1
- removed J11: LORA_DEBUG2, footprint-lib:LORA_DEBUG2
- removed J15: STM32_USB_DEBUG, Connector_PinHeader_1.27mm:PinHeader_1x05_P1.27mm_Vertical
- removed J16: STM32_GTR, Connector_PinHeader_1.27mm:PinHeader_1x03_P1.27mm_Vertical
- removed J17: SPI_DEBUG, Connector_PinHeader_1.27mm:PinHeader_1x04_P1.27mm_Vertical
- removed J18: SWD, Connector_PinHeader_2.54mm:PinHeader_1x04_P2.54mm_Vertical
- removed J19: Conn_01x12, Connector_PinHeader_1.27mm:PinHeader_1x12_P1.27mm_Vertical
- removed J2: SPI_DEBUG, footprint-lib:TTL_TERMINAL_2.54mm
- removed J20: Conn_01x14, Connector_PinHeader_1.27mm:PinHeader_1x14_P1.27mm_Vertical
- removed J21: Conn_01x12, Connector_PinHeader_1.27mm:PinHeader_1x20_P1.27mm_Vertical
- removed J22: STM32_2_DEBUG1, Connector_PinHeader_1.00mm:PinHeader_1x20_P1.00mm_Vertical
- removed J23: STM32_2_DEBUG2, Connector_PinHeader_1.00mm:PinHeader_1x20_P1.00mm_Vertical
- removed J9: PWM_OUT, Connector_PinSocket_2.54mm:PinSocket_1x02_P2.54mm_Vertical
- removed JP4: BOOT0, Jumper:SolderJumper-2_P1.3mm_Open_TrianglePad1.0x1.5mm
- removed JP5: BOOT1, Jumper:SolderJumper-2_P1.3mm_Open_TrianglePad1.0x1.5mm
- removed JP6: Jumper_NO_Small, Jumper:SolderJumper-2_P1.3mm_Open_TrianglePad1.0x1.5mm
- removed L1: L_2R2,1210, Inductor_SMD:L_1210_3225Metric_Pad1.42x2.65mm_HandSolder
- removed Q1: SS9013_J3, footprint-lib:9013,J3,SOT23
- removed R1, R2, R3, R4, R5: R151,0603, Resistor_SMD:R_0603_1608Metric_Pad1.05x0.95mm_HandSolder
- removed R10, R12, R13, R26, R27, R6, R9: R103,0603, Resistor_SMD:R_0603_1608Metric_Pad1.05x0.95mm_HandSolder
- removed R11: VAR_3V3,0805, footprint-lib:VAR_0805
- removed R14, R15, R24, R25: R472,0603, Resistor_SMD:R_0603_1608Metric_Pad1.05x0.95mm_HandSolder
- removed R17: R223,0603, Resistor_SMD:R_0603_1608Metric_Pad1.05x0.95mm_HandSolder
- removed R18, R19: R220,0603, Resistor_SMD:R_0603_1608Metric_Pad1.05x0.95mm_HandSolder
- removed R20: R152,0603, Resistor_SMD:R_0603_1608Metric_Pad1.05x0.95mm_HandSolder
- removed R21: R102,0603, Resistor_SMD:R_0805_2012Metric_Pad1.15x1.40mm_HandSolder
- removed R22: R0,0603, Capacitor_SMD:C_0603_1608Metric_Pad1.05x0.95mm_HandSolder
- removed R23: R0,0603, Resistor_SMD:R_0603_1608Metric_Pad1.05x0.95mm_HandSolder
- removed R28, R7: R471,0603, Resistor_SMD:R_0603_1608Metric_Pad1.05x0.95mm_HandSolder
- removed R29: R103, Resistor_SMD:R_0603_1608Metric_Pad1.05x0.95mm_HandSolder
- removed R30, R31: R104, Resistor_SMD:R_0603_1608Metric_Pad1.05x0.95mm_HandSolder
- removed R32, R33: R511, Resistor_SMD:R_0603_1608Metric_Pad1.05x0.95mm_HandSolder
- removed R8: VAR_5V6,0805, footprint-lib:VAR_0805
- removed RN1, RN2: R_Pack04, Resistor_SMD:R_Array_Concave_4x0603
- removed SW1, SW2: SW_RESET,2_leg,SMD, footprint-lib:SW_SPST_CK_RS282G05A3
- removed SW3: RST, Button_Switch_SMD:SW_SPST_CK_RS282G05A3
- removed SW4: SW_Push, Button_Switch_SMD:SW_SPST_CK_RS282G05A3
- removed TH1: Thermistor_NTC,0805, Resistor_SMD:R_0805_2012Metric
- removed TP1, TP2, TP3: TestPoint, TestPoint:TestPoint_Pad_D4.0mm
- removed U1: SSD1306-OLED-I2C, footprint-lib:CONN_I2C_SSD1306
- removed U10: STM32F103C8T6, footprint-lib:STM32F103C8T6
- removed U11: AMS1117-3.3, Package_TO_SOT_SMD:SOT-223-3_TabPin2
- removed U13: bluepill-stm32f103c8t6, Package_DIP:DIP-40_W15.24mm_LongPads
- removed U2, U5: 74AHCT1G125, Package_TO_SOT_SMD:SOT-23-5_HandSoldering
- removed U3: LM75, Package_SO:SOP-8_3.76x4.96mm_P1.27mm
- removed U4: W25Q32JVSSIQ, footprint-lib:W25Q32JVSSIQ
- removed U6: UBLOX-NEO-6M_DEBUG, footprint-lib:UBLOX-NEO-6M_DEBUG
- removed U7: Ai-Thinker-Ra-02, footprint-lib:Ai-Thinker-Ra-02-LoRa
- removed U8: STM32F407VET6, w_smd_lqfp:TQFP-100
- removed U9: arduino_nano_v3, Module:Arduino_Nano
- removed Y1: O_8M, Crystal:Crystal_HC49-4H_Vertical
- removed Y2: O8M, w_crystal:hc-49_smd
Other:
- outline, holes or cut-outs redrawn

Commit message: update,
Parts:
- added BZ1: BUZZER,MLT-8530, footprint-lib:MLT-8530, F.Cu at (371.0, 116.5)
- added C1: C106,0805, Capacitor_SMD:C_0805_2012Metric_Pad1.15x1.40mm_HandSolder, F.Cu at (358.9, 106.3)
- added C10: CP47uf,50V, w_smd_cap:c_elec_6.3x7.7, F.Cu at (340.5, 125.5)
- added C11: C104,0603, Capacitor_SMD:C_0603_1608Metric_Pad1.05x0.95mm_HandSolder, F.Cu at (304.9, 181.3)
- added C12: C104,0603, Capacitor_SMD:C_0603_1608Metric_Pad1.05x0.95mm_HandSolder, F.Cu at (300.5, 182.8)
- added C13: CP47uf,50V, w_smd_cap:c_elec_6.3x7.7, F.Cu at (294.6, 175.7)
- added C14: C104,0603, Capacitor_SMD:C_0603_1608Metric_Pad1.05x0.95mm_HandSolder, F.Cu at (266.1, 184.9)
- added C15: C104,0603, Capacitor_SMD:C_0603_1608Metric_Pad1.05x0.95mm_HandSolder, F.Cu at (274.9, 181.3)
- added C16: CP47uf,50V, w_smd_cap:c_elec_6.3x7.7, F.Cu at (264.7, 175.7)
- added C17: C106,0603, Capacitor_SMD:C_0603_1608Metric_Pad1.05x0.95mm_HandSolder, F.Cu at (245.2, 188.8)
- added C18: C106,0603, Capacitor_SMD:C_0603_1608Metric_Pad1.05x0.95mm_HandSolder, F.Cu at (249.5, 186.3)
- added C19: CP22uf,16V, Capacitor_SMD:CP_Elec_4x5.3, F.Cu at (283.0, 141.3)
- added C2: C106,0805, Capacitor_SMD:C_0805_2012Metric_Pad1.15x1.40mm_HandSolder, F.Cu at (363.7, 106.3)
- added C20: C104,0603, Capacitor_SMD:C_0603_1608Metric_Pad1.05x0.95mm_HandSolder, F.Cu at (289.6, 127.4)
- added C21: C475,0805, Capacitor_SMD:C_0603_1608Metric_Pad1.05x0.95mm_HandSolder, B.Cu at (24.1, 114.8)
- added C22: C106,0805, Capacitor_SMD:C_0805_2012Metric_Pad1.15x1.40mm_HandSolder, F.Cu at (368.1, 80.4)
- added C23: C106,0805, Capacitor_SMD:C_0805_2012Metric_Pad1.15x1.40mm_HandSolder, F.Cu at (372.3, 76.6)
- added C24: C104,0603, Capacitor_SMD:C_0603_1608Metric_Pad1.05x0.95mm_HandSolder, F.Cu at (319.8, 150.2)
- added C25: C104,0603, Capacitor_SMD:C_0603_1608Metric_Pad1.05x0.95mm_HandSolder, F.Cu at (323.9, 144.2)
- added C26: C104,0603, Capacitor_SMD:C_0603_1608Metric_Pad1.05x0.95mm_HandSolder, F.Cu at (319.8, 155.2)
- added C27: C1pf,0603, Capacitor_SMD:C_0603_1608Metric_Pad1.05x0.95mm_HandSolder, F.Cu at (306.1, 130.0)
- added C28: C1pf,0603, Capacitor_SMD:C_0603_1608Metric_Pad1.05x0.95mm_HandSolder, F.Cu at (306.1, 132.5)
- added C29: C1pf,0603, Capacitor_SMD:C_0603_1608Metric_Pad1.05x0.95mm_HandSolder, F.Cu at (310.4, 130.0)
- added C3: C106,0805, Capacitor_SMD:C_0805_2012Metric_Pad1.15x1.40mm_HandSolder, F.Cu at (375.8, 104.3)
- added C30: C1pf,0603, Capacitor_SMD:C_0603_1608Metric_Pad1.05x0.95mm_HandSolder, F.Cu at (310.4, 132.5)
- added C31: C1pf,0603, Capacitor_SMD:C_0603_1608Metric_Pad1.05x0.95mm_HandSolder, F.Cu at (306.3, 135.0)
- added C32: C1pf,0603, Capacitor_SMD:C_0603_1608Metric_Pad1.05x0.95mm_HandSolder, F.Cu at (301.9, 137.1)
- added C33: C1pf,0603, Capacitor_SMD:C_0603_1608Metric_Pad1.05x0.95mm_HandSolder, F.Cu at (318.6, 122.8)
- added C34: C1pf,0603, Capacitor_SMD:C_0603_1608Metric_Pad1.05x0.95mm_HandSolder, F.Cu at (314.8, 130.0)
- added C35: C1pf,0603, Capacitor_SMD:C_0603_1608Metric_Pad1.05x0.95mm_HandSolder, F.Cu at (318.6, 125.3)
- added C36: C1pf,0603, Capacitor_SMD:C_0603_1608Metric_Pad1.05x0.95mm_HandSolder, F.Cu at (306.3, 137.5)
- added C37: C1pf,0603, Capacitor_SMD:C_0603_1608Metric_Pad1.05x0.95mm_HandSolder, F.Cu at (314.8, 132.5)
- added C38: C1pf,0603, Capacitor_SMD:C_0603_1608Metric_Pad1.05x0.95mm_HandSolder, F.Cu at (322.9, 122.8)
- added C39: C1pf,0603, Capacitor_SMD:C_0603_1608Metric_Pad1.05x0.95mm_HandSolder, F.Cu at (310.6, 135.0)
- added C4: C106,0805, Capacitor_SMD:C_0805_2012Metric_Pad1.15x1.40mm_HandSolder, F.Cu at (381.6, 99.7)
- added C40: C1pf,0603, Capacitor_SMD:C_0603_1608Metric_Pad1.05x0.95mm_HandSolder, F.Cu at (319.1, 127.9)
- added C41: C1pf,0603, Capacitor_SMD:C_0603_1608Metric_Pad1.05x0.95mm_HandSolder, F.Cu at (322.9, 125.3)
- added C42: C1pf,0603, Capacitor_SMD:C_0603_1608Metric_Pad1.05x0.95mm_HandSolder, F.Cu at (323.5, 127.9)
- added C5: C106,0805, Capacitor_SMD:C_0805_2012Metric_Pad1.15x1.40mm_HandSolder, F.Cu at (368.4, 106.3)
- added C6: C106,0603, Capacitor_SMD:C_0603_1608Metric_Pad1.05x0.95mm_HandSolder, F.Cu at (350.4, 144.6)
- added C7: C106,0805, Capacitor_SMD:C_0805_2012Metric_Pad1.15x1.40mm_HandSolder, F.Cu at (361.5, 148.2)
- added C8: C104,0603, Capacitor_SMD:C_0603_1608Metric_Pad1.05x0.95mm_HandSolder, F.Cu at (350.8, 131.1)
- added C9: C104,0603, Capacitor_SMD:C_0603_1608Metric_Pad1.05x0.95mm_HandSolder, F.Cu at (342.1, 131.1)
- added D1: WS2812B, LED_SMD:LED_WS2812B_PLCC4_5.0x5.0mm_P3.2mm, F.Cu at (377.6, 94.9)
- added D10: LED_GREEN,0603, LED_SMD:LED_0603_1608Metric_Pad1.05x0.95mm_HandSolder, F.Cu at (291.8, 180.9)
- added D11: LED_GREEN,0603, LED_SMD:LED_0603_1608Metric_Pad1.05x0.95mm_HandSolder, F.Cu at (261.8, 180.9)
- added D12: D_1N4148_T4, Diode_SMD:D_SOD-123, F.Cu at (379.4, 112.7)
- added D2: WS2812B, LED_SMD:LED_WS2812B_PLCC4_5.0x5.0mm_P3.2mm, F.Cu at (369.2, 101.5)
- added D3: WS2812B, LED_SMD:LED_WS2812B_PLCC4_5.0x5.0mm_P3.2mm, F.Cu at (369.2, 94.9)
- added D4: WS2812B, LED_SMD:LED_WS2812B_PLCC4_5.0x5.0mm_P3.2mm, F.Cu at (360.8, 101.5)
- added D5: WS2812B, LED_SMD:LED_WS2812B_PLCC4_5.0x5.0mm_P3.2mm, F.Cu at (360.8, 94.9)
- added D6: LED_GREEN,0603, footprint-lib:LED_0603_1608Metric, F.Cu at (262.6, 193.8)
- added D7: 5V_STATUS, footprint-lib:LED_0603_1608Metric, F.Cu at (177.3, 191.0)
- added D8: 3V3_STATUS, footprint-lib:LED_0603_1608Metric, F.Cu at (172.9, 193.9)
- added D9: LED_GREEN,0603, LED_SMD:LED_0603_1608Metric_Pad1.05x0.95mm_HandSolder, F.Cu at (337.7, 130.6)
- added H1: MountingHole, footprint-lib:MountingHole_2.7mm_M2.5,rpi_like, F.Cu at (117.0, 112.0)
- added H2: MountingHole, footprint-lib:MountingHole_2.7mm_M2.5,rpi_like, F.Cu at (23.0, 112.0)
- added H3: MountingHole, footprint-lib:MountingHole_2.7mm_M2.5,rpi_like, F.Cu at (23.0, 18.0)
- added H4: MountingHole, footprint-lib:MountingHole_2.7mm_M2.5,rpi_like, F.Cu at (117.0, 18.0)
- added J1: WS2812_HEADER, Connector_PinHeader_1.27mm:PinHeader_1x02_P1.27mm_Vertical, F.Cu at (380.2, 104.5)
- added J10: A_MEAS, Connector_PinHeader_1.27mm:PinHeader_1x02_P1.27mm_Vertical, F.Cu at (168.7, 191.0)
- added J11: 3V3_IN, Connector_PinHeader_2.54mm:PinHeader_1x02_P2.54mm_Vertical, F.Cu at (164.8, 184.4)
- added J12: Conn_01x03, Connector_PinHeader_2.54mm:PinHeader_1x03_P2.54mm_Vertical, F.Cu at (357.8, 123.9)
- added J13: Conn_01x03, Connector_PinHeader_2.54mm:PinHeader_1x03_P2.54mm_Vertical, F.Cu at (311.9, 174.2)
- added J14: Va_header, Connector_PinHeader_2.54mm:PinHeader_1x03_P2.54mm_Vertical, F.Cu at (281.9, 174.2)
- added J15: BTN_HEADER, Connector_PinHeader_1.27mm:PinHeader_1x03_P1.27mm_Vertical, F.Cu at (332.5, 163.2)
- added J16: ADC_HEADER, Connector_PinHeader_1.27mm:PinHeader_1x03_P1.27mm_Vertical, F.Cu at (240.9, 183.8)
- added J17: PWM_OUT, Connector_PinHeader_2.54mm:PinHeader_1x02_P2.54mm_Vertical, F.Cu at (367.8, 127.6)
- added J18: UBLOX_HEADER, Connector_PinHeader_1.27mm:PinHeader_1x04_P1.27mm_Vertical, F.Cu at (195.7, 183.8)
- added J19: LORA_HEADER_LOW, footprint-lib:LORA_DEBUG1, F.Cu at (281.2, 127.8)
- added J2: OLED_I2C_HEADER, Connector_PinHeader_1.27mm:PinHeader_1x04_P1.27mm_Vertical, F.Cu at (346.2, 141.4)
- added J20: LORA_HEADER_HIGH, footprint-lib:LORA_DEBUG2, F.Cu at (285.4, 127.8)
- added J21: GND, Connector_PinHeader_1.27mm:PinHeader_1x03_P1.27mm_Vertical, F.Cu at (222.1, 189.8)
- added J22: 5V, Connector_PinHeader_1.27mm:PinHeader_1x03_P1.27mm_Vertical, F.Cu at (228.2, 183.8)
- added J23: 3V3, Connector_PinHeader_1.27mm:PinHeader_1x03_P1.27mm_Vertical, F.Cu at (232.3, 183.8)
- added J24: BUZZER_HEADER, Connector_PinHeader_1.27mm:PinHeader_1x02_P1.27mm_Vertical, F.Cu at (378.6, 116.0)
- added J25: I2C_DEBUG, footprint-lib:I2C_DEBUG, F.Cu at (114.0, 69.0)
- added J26: TTL_HEADER, footprint-lib:TTL_TERMINAL_1.27mm, F.Cu at (96.0, 69.0)
- added J27: SDCARD_HEADER, footprint-lib:SDCARD_HEADER, F.Cu at (91.0, 69.0)
- added J28: SPI_HEADER, footprint-lib:SPI_DEBUG, F.Cu at (106.8, 68.8)
- added J29: OLED_HEADER, Connector_PinHeader_1.27mm:PinHeader_1x05_P1.27mm_Vertical, F.Cu at (101.0, 68.8)
- added J3: A0_SEL, Jumper:SolderJumper-2_P1.3mm_Open_TrianglePad1.0x1.5mm, F.Cu at (350.4, 141.5)
- added J30: NODEMCU_HEADER1, Connector_PinHeader_1.27mm:PinHeader_1x15_P1.27mm_Vertical, F.Cu at (79.0, 47.0)
- added J31: NODEMCU_HEADER2, Connector_PinHeader_1.27mm:PinHeader_1x15_P1.27mm_Vertical, F.Cu at (83.0, 47.0)
- added J32: sdcard_header, footprint-lib:SDCARD_HEADER, B.Cu at (37.0, 90.0)
- added J33: SSD1306-OLED-SPI, footprint-lib:CONN_SPI_SSD1306, F.Cu at (358.9, 70.3)
- added J34: OLED_SPI_HEADER, Connector_PinHeader_1.27mm:PinHeader_1x07_P1.27mm_Vertical, F.Cu at (367.8, 69.6)
- added J35: OLED_I2C_HEADER, Connector_PinHeader_1.27mm:PinHeader_1x04_P1.27mm_Vertical, F.Cu at (372.0, 69.6)
- added J36: ROT_ENC_HEADER, Connector_PinHeader_1.27mm:PinHeader_1x03_P1.27mm_Vertical, F.Cu at (319.6, 144.7)
- added J37: I2C_HEADER, footprint-lib:I2C_DEBUG, F.Cu at (79.0, 40.0)
- added J38: TTL_HEADER, footprint-lib:TTL_HEADER, F.Cu at (79.0, 34.0)
- added J39: SPI_HEADER, footprint-lib:SPI_DEBUG, F.Cu at (79.0, 27.0)
- added J4: SPI_HEADER, footprint-lib:TTL_TERMINAL_2.54mm, F.Cu at (371.8, 142.1)
- added J40: OLED_HEADER, Connector_PinHeader_1.27mm:PinHeader_1x05_P1.27mm_Vertical, F.Cu at (78.4, 18.8)
- added J41: ARDUINO_HEADER1, Connector_PinHeader_1.27mm:PinHeader_1x15_P1.27mm_Vertical, F.Cu at (74.0, 18.0)
- added J42: ARDUINO_HEADER2, Connector_PinHeader_1.27mm:PinHeader_1x15_P1.27mm_Vertical, F.Cu at (74.0, 41.6)
- added J43: STM32_2_DEBUG1, Connector_PinHeader_1.00mm:PinHeader_1x20_P1.00mm_Vertical, F.Cu at (45.0, 37.0)
- added J44: STM32_2_DEBUG2, Connector_PinHeader_1.00mm:PinHeader_1x20_P1.00mm_Vertical, F.Cu at (45.0, 47.0)
- added J45: HEADER_DEBUG1, Connector_PinHeader_1.27mm:PinHeader_1x04_P1.27mm_Vertical, F.Cu at (310.1, 123.3)
- added J46: HEADER_DEBUG2, Connector_PinHeader_1.27mm:PinHeader_1x04_P1.27mm_Vertical, F.Cu at (301.9, 123.3)
- added J47: HEADER_DEBUG3, Connector_PinHeader_1.27mm:PinHeader_1x04_P1.27mm_Vertical, F.Cu at (301.9, 130.4)
- added J48: HEADER_DEBUG4, Connector_PinHeader_1.27mm:PinHeader_1x04_P1.27mm_Vertical, F.Cu at (306.0, 123.3)
- added J49: HEADER_DEBUG5, Connector_PinHeader_1.27mm:PinHeader_1x04_P1.27mm_Vertical, F.Cu at (314.3, 123.3)
- added J5: BLINK_HEADER, Connector_PinHeader_1.27mm:PinHeader_1x02_P1.27mm_Vertical, F.Cu at (258.5, 191.7)
- added J6: V_MEAS, Connector_PinHeader_1.27mm:PinHeader_1x02_P1.27mm_Vertical, F.Cu at (164.6, 191.0)
- added J7: A_MEAS, Connector_PinHeader_1.27mm:PinHeader_1x02_P1.27mm_Vertical, F.Cu at (178.0, 183.8)
- added J8: 5V_IN, Connector_PinHeader_2.54mm:PinHeader_1x02_P2.54mm_Vertical, F.Cu at (169.5, 184.4)
- added J9: V_MEAS, Connector_PinHeader_1.27mm:PinHeader_1x02_P1.27mm_Vertical, F.Cu at (173.9, 183.8)
- added JP1: A1_SEL, Jumper:SolderJumper-2_P1.3mm_Open_TrianglePad1.0x1.5mm, F.Cu at (346.2, 148.7)
- added JP2: A2_SEL, Jumper:SolderJumper-2_P1.3mm_Open_TrianglePad1.0x1.5mm, F.Cu at (341.8, 148.7)
- added JP3: PWR_SRC, Jumper:SolderJumper-2_P1.3mm_Open_TrianglePad1.0x1.5mm, F.Cu at (342.0, 134.1)
- added JP4: PWR_OUT, Jumper:SolderJumper-2_P1.3mm_Open_TrianglePad1.0x1.5mm, F.Cu at (346.4, 133.1)
- added JP5: PWR_SRC, Jumper:SolderJumper-2_P1.3mm_Open_TrianglePad1.0x1.5mm, F.Cu at (296.2, 181.9)
- added JP6: PWR_OUT, Jumper:SolderJumper-2_P1.3mm_Open_TrianglePad1.0x1.5mm, F.Cu at (291.8, 183.9)
- added JP7: PWR_SRC, Jumper:SolderJumper-2_P1.3mm_Open_TrianglePad1.0x1.5mm, F.Cu at (261.8, 183.9)
- added JP8: PWR_OUT, Jumper:SolderJumper-2_P1.3mm_Open_TrianglePad1.0x1.5mm, F.Cu at (266.2, 181.9)
- added Q1: SS9013_J3, footprint-lib:9013,J3,SOT23, F.Cu at (382.7, 116.4)
- added R1: R103,0603, Resistor_SMD:R_0603_1608Metric_Pad1.05x0.95mm_HandSolder, F.Cu at (366.0, 148.0)
- added R10: R103,0603, Resistor_SMD:R_0603_1608Metric_Pad1.05x0.95mm_HandSolder, F.Cu at (332.6, 168.6)
- added R11: R103,0603, Resistor_SMD:R_0603_1608Metric_Pad1.05x0.95mm_HandSolder, F.Cu at (336.8, 162.7)
- added R12: R472,0603, Resistor_SMD:R_0603_1608Metric_Pad1.05x0.95mm_HandSolder, F.Cu at (249.6, 183.3)
- added R13: R472,0603, Resistor_SMD:R_0603_1608Metric_Pad1.05x0.95mm_HandSolder, F.Cu at (245.2, 186.3)
- added R15: R471,0603, Resistor_SMD:R_0603_1608Metric_Pad1.05x0.95mm_HandSolder, F.Cu at (378.7, 120.2)
- added R16: R273,0603, Resistor_SMD:R_0603_1608Metric_Pad1.05x0.95mm_HandSolder, F.Cu at (319.8, 152.7)
- added R17: R273,0603, Resistor_SMD:R_0603_1608Metric_Pad1.05x0.95mm_HandSolder, F.Cu at (323.9, 146.8)
- added R18: R273,0603, Resistor_SMD:R_0603_1608Metric_Pad1.05x0.95mm_HandSolder, F.Cu at (324.1, 149.3)
- added R19: R0,0603, Resistor_SMD:R_0603_1608Metric_Pad1.05x0.95mm_HandSolder, F.Cu at (315.0, 135.0)
- added R2: R471,0603, Resistor_SMD:R_0603_1608Metric_Pad1.05x0.95mm_HandSolder, F.Cu at (262.7, 191.3)
- added R20: R0,0603, Resistor_SMD:R_0603_1608Metric_Pad1.05x0.95mm_HandSolder, F.Cu at (327.2, 122.8)
- added R21: R0,0603, Resistor_SMD:R_0603_1608Metric_Pad1.05x0.95mm_HandSolder, F.Cu at (315.0, 137.5)
- added R22: R0,0603, Resistor_SMD:R_0603_1608Metric_Pad1.05x0.95mm_HandSolder, F.Cu at (327.2, 125.3)
- added R23: R0,0603, Resistor_SMD:R_0603_1608Metric_Pad1.05x0.95mm_HandSolder, F.Cu at (327.9, 127.9)
- added R24: R0,0603, Resistor_SMD:R_0603_1608Metric_Pad1.05x0.95mm_HandSolder, F.Cu at (323.5, 130.4)
- added R25: R0,0603, Resistor_SMD:R_0603_1608Metric_Pad1.05x0.95mm_HandSolder, F.Cu at (310.6, 137.5)
- added R26: R0,0603, Resistor_SMD:R_0603_1608Metric_Pad1.05x0.95mm_HandSolder, F.Cu at (319.4, 132.9)
- added R27: R0,0603, Resistor_SMD:R_0603_1608Metric_Pad1.05x0.95mm_HandSolder, F.Cu at (319.4, 135.4)
- added R28: R0,0603, Resistor_SMD:R_0603_1608Metric_Pad1.05x0.95mm_HandSolder, F.Cu at (327.9, 130.4)
- added R29: R0,0603, Resistor_SMD:R_0603_1608Metric_Pad1.05x0.95mm_HandSolder, F.Cu at (319.4, 137.9)
- added R3: VAR_5V6,0805, footprint-lib:VAR_0805, F.Cu at (174.0, 188.2)
- added R30: R0,0603, Resistor_SMD:R_0603_1608Metric_Pad1.05x0.95mm_HandSolder, F.Cu at (323.7, 135.4)
- added R31: R0,0603, Resistor_SMD:R_0603_1608Metric_Pad1.05x0.95mm_HandSolder, F.Cu at (328.1, 132.9)
- added R32: R0,0603, Resistor_SMD:R_0603_1608Metric_Pad1.05x0.95mm_HandSolder, F.Cu at (323.7, 137.9)
- added R33: R0,0603, Resistor_SMD:R_0603_1608Metric_Pad1.05x0.95mm_HandSolder, F.Cu at (323.7, 132.9)
- added R34: R0,0603, Resistor_SMD:R_0603_1608Metric_Pad1.05x0.95mm_HandSolder, F.Cu at (319.1, 130.4)
- added R4: R103,0603, Resistor_SMD:R_0603_1608Metric_Pad1.05x0.95mm_HandSolder, F.Cu at (182.3, 183.3)
- added R5: R103,0603, Resistor_SMD:R_0603_1608Metric_Pad1.05x0.95mm_HandSolder, F.Cu at (178.4, 188.0)
- added R6: VAR_3V3,0805, footprint-lib:VAR_0805, F.Cu at (173.0, 191.2)
- added R7: R102,0603, Resistor_SMD:R_0603_1608Metric_Pad1.05x0.95mm_HandSolder, F.Cu at (337.7, 133.2)
- added R8: R102,0603, Resistor_SMD:R_0603_1608Metric_Pad1.05x0.95mm_HandSolder, F.Cu at (296.1, 184.9)
- added R9: R102,0603, Resistor_SMD:R_0603_1608Metric_Pad1.05x0.95mm_HandSolder, F.Cu at (270.5, 182.8)
- added RN1: R_Pack04, Resistor_SMD:R_Array_Concave_4x0603, F.Cu at (337.6, 148.7)
- added RN2: R_Pack04, Resistor_SMD:R_Array_Concave_4x0603, B.Cu at (20.0, 101.5)
- added RN3: R_Pack04, Resistor_SMD:R_Array_Concave_4x0603, B.Cu at (24.2, 111.2)
- added RN4: R_Pack04, Resistor_SMD:R_Array_Concave_4x0603, F.Cu at (376.1, 70.4)
- added RN5: R_Pack04, Resistor_SMD:R_Array_Concave_4x0603, F.Cu at (363.2, 82.6)
- added RN6: R_Pack04, Resistor_SMD:R_Array_Concave_4x0603, B.Cu at (45.0, 42.0)
- added SDC1: TF_CARD_SOCKET,SELF_EJECT, footprint-lib:SUNTECH_ST-TF-003A, B.Cu at (37.1, 106.1)
- added SW1: SW_RESET,2_leg,SMD, footprint-lib:SW_SPST_CK_RS282G05A3, F.Cu at (325.0, 164.1)
- added SW2: SW_RESET,2_leg,SMD, footprint-lib:SW_SPST_CK_RS282G05A3, F.Cu at (325.0, 169.2)
- added SW3: EC11_VERTICAL, footprint-lib:RotaryEncoder_Alps_EC11E_Vertical_H20mm, F.Cu at (301.6, 147.9)
- added TH1: Thermistor_NTC,0805, Resistor_SMD:R_0805_2012Metric, F.Cu at (245.2, 183.6)
- added TP1: TestPoint, TestPoint:TestPoint_Pad_D4.0mm, F.Cu at (217.0, 185.1)
- added TP2: TestPoint, TestPoint:TestPoint_Pad_D4.0mm, F.Cu at (217.0, 191.2)
- added TP3: TestPoint, TestPoint:TestPoint_Pad_D4.0mm, F.Cu at (223.1, 185.1)
- added U1: 74AHCT1G125, Package_TO_SOT_SMD:SOT-23-5_HandSoldering, F.Cu at (376.3, 100.5)
- added U10: nodemcu, footprint-lib:NodeMCU1.0(12-E), F.Cu at (101.3, 40.9)
- added U11: SSD1306-OLED-I2C, footprint-lib:CONN_I2C_SSD1306, F.Cu at (363.5, 70.3)
- added U12: arduino_nano_v3, Module:Arduino_Nano, F.Cu at (53.0, 21.0)
- added U13: bluepill-stm32f103c8t6, Package_DIP:DIP-40_W15.24mm_LongPads, F.Cu at (25.0, 19.0)
- added U2: LM75, Package_SO:SOP-8_3.76x4.96mm_P1.27mm, F.Cu at (339.8, 143.0)
- added U3: W25Q32JVSSIQ, footprint-lib:W25Q32JVSSIQ, F.Cu at (364.3, 143.2)
- added U4: AMS1117-3.3, Package_TO_SOT_SMD:SOT-223-3_TabPin2, F.Cu at (350.5, 125.7)
- added U5: AMS1117-3.3, Package_TO_SOT_SMD:SOT-223-3_TabPin2, F.Cu at (304.6, 176.0)
- added U6: AMS1117-3.3, Package_TO_SOT_SMD:SOT-223-3_TabPin2, F.Cu at (274.6, 176.0)
- added U7: 74AHCT1G125, Package_TO_SOT_SMD:SOT-23-5_HandSoldering, F.Cu at (373.0, 127.6)
- added U8: UBLOX-NEO-6M_DEBUG, footprint-lib:UBLOX-NEO-6M_DEBUG, F.Cu at (191.4, 184.4)
- added U9: Ai-Thinker-Ra-02, footprint-lib:Ai-Thinker-Ra-02-LoRa, F.Cu at (269.4, 135.7)
Other:
- outline, holes or cut-outs redrawn
- rule pad_to_mask_clearance: 0.051 -> 0

Commit message: update sdcard header,
Parts:
- C21, RN2, RN3: moved to F.Cu
- J32: footprint footprint-lib:SDCARD_HEADER -> footprint-lib:SDCARD_HEADER_10PIN
- moved U11 340.5 mm to (24.0, 97.0)
- moved RN5 335.7 mm to (27.9, 96.4), turned to 180 degrees
- moved J33 334.9 mm to (24.0, 74.3)
- moved C22 333.0 mm to (35.1, 84.4)
- moved C23 333.0 mm to (39.3, 80.6)
- moved J34 333.0 mm to (34.8, 73.6)
- moved J35 333.0 mm to (39.0, 73.6)
- moved RN4 333.0 mm to (43.1, 74.4)
- moved C21 18.2 mm to (38.0, 103.0), turned to 0 degrees
- moved RN2 17.6 mm to (37.0, 106.0), turned to 270 degrees
- moved RN3 9.36 mm to (32.0, 106.0), turned to 270 degrees
- moved J32 8.94 mm to (33.0, 98.0)
Connections:
- SDC1 pad 9: (no net) -> Net-(J32-PadCD)

Commit message: update footprint,
Parts:
- J3, JP1, JP2: footprint Jumper:SolderJumper-2_P1.3mm_Open_TrianglePad1.0x1.5mm -> Jumper:SolderJumper-3_P2.0mm_Open_TrianglePad1.0x1.5mm_NumberLabels
- moved R17 260.1 mm to (67.0, 106.0)
- moved R18 260.1 mm to (67.0, 110.0)
- moved C25 259.4 mm to (67.0, 108.0), turned to 180 degrees
- moved R16 258.0 mm to (67.0, 101.0)
- moved SW3 257.6 mm to (47.8, 103.6)
- moved C24 257.2 mm to (66.9, 103.0), turned to 180 degrees
- moved C26 256.4 mm to (67.0, 112.0), turned to 180 degrees
- moved J36 250.5 mm to (73.0, 101.0)
Routing:
- net Net-(R16-Pad1): track 0.00 -> 45.3 mm
- net GND: track 0.00 -> 31.1 mm
- net Net-(R17-Pad1): track 0.00 -> 20.7 mm
- net /ROT_ENC_SW: track 0.00 -> 10.6 mm
- net /ROT_ENC_B: track 0.00 -> 8.67 mm
- net Net-(R18-Pad1): track 0.00 -> 7.96 mm
- net /ROT_ENC_A: track 0.00 -> 7.18 mm

Commit message: update footprint,
Parts:
- moved J33 1.00 mm to (25.0, 74.3)
Connections:
- SDC1 pad G: (no net) -> GND
