File: hardware/eval_board.kicad_pcb (KiCad board)
At the start: 2 copper layers, 100 x 100 mm, 177 parts, among them J1 WS2812_HEADER, J10 A_MEAS, J11 3V3_IN, J12 Conn_01x03, J13 Conn_01x03, J14 Va_header, J15 BTN_HEADER, J16 ADC_HEADER, J17 PWM_OUT, J18 UBLOX_HEADER, J19 LORA_HEADER_LOW, J2 OLED_I2C_HEADER, J20 LORA_HEADER_HIGH, J21 GND, J22 5V, J23 3V3, J24 BUZZER_HEADER, J25 I2C_DEBUG, J26 TTL_HEADER, J27 SDCARD_HEADER, J28 SPI_HEADER, J29 OLED_HEADER, J3 A0_SEL, J30 NODEMCU_HEADER1, J31 NODEMCU_HEADER2, J32 sdcard_header, J33 SSD1306-OLED-SPI, J34 OLED_SPI_HEADER, J35 OLED_I2C_HEADER, J36 ROT_ENC_HEADER, J37 I2C_HEADER, J38 TTL_HEADER, J39 SPI_HEADER, J4 SPI_HEADER, J40 OLED_HEADER, J41 ARDUINO_HEADER1, J42 ARDUINO_HEADER2, J43 STM32_2_DEBUG1, J44 STM32_2_DEBUG2, J45 HEADER_DEBUG1, J46 HEADER_DEBUG2, J47 HEADER_DEBUG3, J48 HEADER_DEBUG4, J49 HEADER_DEBUG5, J5 BLINK_HEADER, J6 V_MEAS, J7 A_MEAS, J8 5V_IN, J9 V_MEAS, Q1 SS9013_J3, SW1 SW_RESET,2_leg,SMD, SW2 SW_RESET,2_leg,SMD, SW3 EC11_VERTICAL, U1 74AHCT1G125, U10 nodemcu, U11 SSD1306-OLED-I2C, U12 arduino_nano_v3, U13 bluepill-stm32f103c8t6, U2 LM75, U3 W25Q32JVSSIQ, U4 AMS1117-3.3, U5 AMS1117-3.3, U6 AMS1117-3.3, U7 74AHCT1G125, U8 UBLOX-NEO-6M_DEBUG, U9 Ai-Thinker-Ra-02

Commit message: update,
Parts:
- removed C11, C12, C14, C15, C20: C104,0603, Capacitor_SMD:C_0603_1608Metric_Pad1.05x0.95mm_HandSolder
- removed C13, C16: CP47uf,50V, w_smd_cap:c_elec_6.3x7.7
- removed C19: CP22uf,16V, Capacitor_SMD:CP_Elec_4x5.3
- removed C27, C28, C29, C30, C31, C32, C33, C34, C35, C36, C37, C38, C39, C40, C41, C42: C1pf,0603, Capacitor_SMD:C_0603_1608Metric_Pad1.05x0.95mm_HandSolder
- removed C4, C5: C106,0805, Capacitor_SMD:C_0805_2012Metric_Pad1.15x1.40mm_HandSolder
- removed D10, D11: LED_GREEN,0603, LED_SMD:LED_0603_1608Metric_Pad1.05x0.95mm_HandSolder
- removed D4, D5: WS2812B, LED_SMD:LED_WS2812B_PLCC4_5.0x5.0mm_P3.2mm
- removed D7: 5V_STATUS, footprint-lib:LED_0603_1608Metric
- removed D8: 3V3_STATUS, footprint-lib:LED_0603_1608Metric
- removed J10, J7: A_MEAS, Connector_PinHeader_1.27mm:PinHeader_1x02_P1.27mm_Vertical
- removed J11: 3V3_IN, Connector_PinHeader_2.54mm:PinHeader_1x02_P2.54mm_Vertical
- removed J13: Conn_01x03, Connector_PinHeader_2.54mm:PinHeader_1x03_P2.54mm_Vertical
- removed J14: Va_header, Connector_PinHeader_2.54mm:PinHeader_1x03_P2.54mm_Vertical
- removed J17: PWM_OUT, Connector_PinHeader_2.54mm:PinHeader_1x02_P2.54mm_Vertical
- removed J18: UBLOX_HEADER, Connector_PinHeader_1.27mm:PinHeader_1x04_P1.27mm_Vertical
- removed J19: LORA_HEADER_LOW, footprint-lib:LORA_DEBUG1
- removed J20: LORA_HEADER_HIGH, footprint-lib:LORA_DEBUG2
- removed J45: HEADER_DEBUG1, Connector_PinHeader_1.27mm:PinHeader_1x04_P1.27mm_Vertical
- removed J46: HEADER_DEBUG2, Connector_PinHeader_1.27mm:PinHeader_1x04_P1.27mm_Vertical
- removed J47: HEADER_DEBUG3, Connector_PinHeader_1.27mm:PinHeader_1x04_P1.27mm_Vertical
- removed J48: HEADER_DEBUG4, Connector_PinHeader_1.27mm:PinHeader_1x04_P1.27mm_Vertical
- removed J49: HEADER_DEBUG5, Connector_PinHeader_1.27mm:PinHeader_1x04_P1.27mm_Vertical
- removed J6, J9: V_MEAS, Connector_PinHeader_1.27mm:PinHeader_1x02_P1.27mm_Vertical
- removed J8: 5V_IN, Connector_PinHeader_2.54mm:PinHeader_1x02_P2.54mm_Vertical
- removed JP5, JP7: PWR_SRC, Jumper:SolderJumper-2_P1.3mm_Open_TrianglePad1.0x1.5mm
- removed JP6, JP8: PWR_OUT, Jumper:SolderJumper-2_P1.3mm_Open_TrianglePad1.0x1.5mm
- removed R19, R20, R21, R22, R23, R24, R25, R26, R27, R28, R29, R30, R31, R32, R33, R34: R0,0603, Resistor_SMD:R_0603_1608Metric_Pad1.05x0.95mm_HandSolder
- removed R3: VAR_5V6,0805, footprint-lib:VAR_0805
- removed R4, R5: R103,0603, Resistor_SMD:R_0603_1608Metric_Pad1.05x0.95mm_HandSolder
- removed R6: VAR_3V3,0805, footprint-lib:VAR_0805
- removed R8, R9: R102,0603, Resistor_SMD:R_0603_1608Metric_Pad1.05x0.95mm_HandSolder
- removed U5, U6: AMS1117-3.3, Package_TO_SOT_SMD:SOT-223-3_TabPin2
- removed U7: 74AHCT1G125, Package_TO_SOT_SMD:SOT-23-5_HandSoldering
- removed U8: UBLOX-NEO-6M_DEBUG, footprint-lib:UBLOX-NEO-6M_DEBUG
- removed U9: Ai-Thinker-Ra-02, footprint-lib:Ai-Thinker-Ra-02-LoRa
- C1, C2, C3, C7, C8, C9, R1, R10, R11, R7: moved to B.Cu
- J4: footprint footprint-lib:TTL_TERMINAL_2.54mm -> footprint-lib:SPI_DEBUG
- RN6: moved to F.Cu
- U4: footprint Package_TO_SOT_SMD:SOT-223-3_TabPin2 -> footprint-lib:AMS1117_SOT-223
- moved J4 324.0 mm to (55.5, 71.5), turned to 90 degrees
- moved R1 316.1 mm to (58.5, 75.0), turned to 90 degrees
- moved U3 314.2 mm to (57.3, 76.2)
- moved C7 313.7 mm to (56.0, 77.0), turned to 90 degrees
- moved Q1 310.0 mm to (73.5, 95.0), turned to 270 degrees
- moved D12 307.2 mm to (73.0, 90.5), turned to 90 degrees
- moved R15 306.0 mm to (73.5, 97.5)
- moved BZ1 305.4 mm to (66.5, 93.0)
- moved J24 302.3 mm to (77.0, 96.0)
- moved J1 283.7 mm to (96.5, 100.5), turned to 90 degrees
- moved C6 282.1 mm to (70.1, 113.0)
- moved U1 279.3 mm to (97.0, 96.5), turned to 90 degrees
- moved J2 276.7 mm to (72.0, 104.0), turned to 270 degrees
- moved RN1 276.6 mm to (64.0, 108.0), turned to 180 degrees
- moved J3 276.4 mm to (76.0, 109.0), turned to 270 degrees
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Connections:
- J33 pad DI: (no net) -> /MOSI
- J33 pad DO: (no net) -> /SCK
- JP3 pad 1: +5V -> (no net)
Routing:
- net GND: track 31.1 -> 118.2 mm, vias 0 -> 2
- net +3V3: track 0.00 -> 70.8 mm, vias 0 -> 3
- net Net-(JP1-Pad2): track 0.00 -> 30.2 mm
- net Net-(C10-Pad1): track 0.00 -> 22.7 mm, vias 0 -> 1
- net /A_IN1: track 0.00 -> 16.8 mm, vias 0 -> 2
- net Net-(JP2-Pad2): track 0.00 -> 14.7 mm
- net Net-(D9-Pad1): track 0.00 -> 8.81 mm, vias 0 -> 1
- net /SCL: track 0.00 -> 8.39 mm
- net /A_IN0: track 0.00 -> 8.23 mm
- net +5V: track 0.00 -> 8.03 mm
- net Net-(C8-Pad1): track 0.00 -> 7.65 mm, vias 0 -> 1
- net /SDA: track 0.00 -> 6.01 mm
- net Net-(J3-Pad2): track 0.00 -> 3.73 mm
- net Net-(RN1-Pad2): track 0.00 -> 3.12 mm
